File: ethernet.sch (KiCad schematic (older format))
At the start: 29 parts, among them IC1 RTL8211EG-VB-CG, J8 HR911130A, Y2 Crystal

Commit message: Wired the RTL8211EG more.
Parts:
- R47: footprint Resistor_SMD:R_0201_0603Metric -> Resistor_SMD:R_0603_1608Metric
Connections:
- wire segments 46 -> 45
Changed lines of the file:
@@
 EESchema Schematic File Version 4
-LIBS:test1-cache
 EELAYER 30 0
 EELAYER END
@@
 U 1 1 5DE60B81
 P 7500 4400
-F 0 "R47" V 7293 4400 50  0000 C CNN
-F 1 "100" V 7384 4400 50  0000 C CNN
-F 2 "Resistor_SMD:R_0201_0603Metric" V 7430 4400 50  0001 C CNN
+F 0 "R47" V 7400 4400 50  0000 C CNN
+F 1 "100" V 7500 4400 50  0000 C CNN
+F 2 "Resistor_SMD:R_0603_1608Metric" V 7430 4400 50  0001 C CNN
 F 3 "~" H 7500 4400 50  0001 C CNN
 	1    7500 4400
@@
 Text GLabel 1150 6900 0    50   Input ~ 0
 ETH_LED1
-Connection ~ 1450 6750
-Wire Wire Line
-	1450 6750 1650 6750
 Text GLabel 2500 6800 0    50   Input ~ 0
 ETH_MDI_3-

Commit message: Fixed wiring ad7511 and wired the rtl8211EG IC
Connections:
- net labels added: ETH_COL_MODE, ETH_CRS, ETH_INTB, ETH_MDC, ETH_MDIO, ETH_RXC, ETH_RXD0, ETH_RXD1, ETH_RXD2, ETH_RXD3, ETH_RXD4, ETH_RXD5, ETH_RXD6, ETH_RXD7, ETH_RXDV, ETH_RXER, ETH_TXER

Commit message: First step to implement floppy interface. ESP32 check wireing in.
Parts:
- removed C42, C45: 4.7uF, Capacitor_SMD:C_0805_2012Metric, symbol Device:C
- removed C43, C44, C46: 100nF, Capacitor_SMD:C_0603_1608Metric, symbol Device:C
- removed C47, C48: 22pF, Capacitor_SMD:C_0603_1608Metric, symbol Device:C
- removed IC1: RTL8211EG-VB-CG, QFN50P900X900X100-65N-D, symbol RTL8211EG-VB-CG:RTL8211EG-VB-CG
- removed J8: HR911130A, HR911130A, symbol HR911130A:HR911130A
- removed L5: L, Inductor_SMD:L_0805_2012Metric, symbol Device:L
- removed R30, R33, R34, R36, R37, R38, R39, R40, R41, R42, R43, R44, R45, R46: 4.7K, Resistor_SMD:R_0603_1608Metric, symbol Device:R
- removed R31, R32: 530, Resistor_SMD:R_0603_1608Metric, symbol Device:R
- removed R35: 2.49K, Resistor_SMD:R_0603_1608Metric, symbol Device:R
- removed R47: 100, Resistor_SMD:R_0603_1608Metric, symbol Device:R
- removed Y2: Crystal, Crystal:Crystal_SMD_HC49-SD, symbol Device:Crystal
Connections:
- net labels removed: 3V3, ETH_CKXTAL1, ETH_CKXTAL2, ETH_COL_MODE, ETH_CRS, ETH_GTX_CLK, ETH_INTB, ETH_LED0, ETH_LED1, ETH_MDC, ETH_MDIO, ETH_MDI_0+, ETH_MDI_0-, ETH_MDI_1+, ETH_MDI_1-, ETH_MDI_2+, ETH_MDI_2-, ETH_MDI_3+, ETH_MDI_3-, ETH_PHYRSTB, ETH_REG_OUT, ETH_REG_OUT_OUT, ETH_RXC, ETH_RXD0, ETH_RXD1, ETH_RXD2, ETH_RXD3, ETH_RXD4, ETH_RXD5, ETH_RXD6, ETH_RXD7, ETH_RXDV, ETH_RXER, ETH_TXD0, ETH_TXD1, ETH_TXD2, ETH_TXD3, ETH_TXD4, ETH_TXD5, ETH_TXD6, ETH_TXD7, ETH_TXDCLK, ETH_TXEN, ETH_TXER, GND
- wire segments 45 -> 0
