File: MCU.sch (KiCad schematic (older format))
At the start: 42 parts, among them J4 ARM_JTAG, SW1 SW_Push, U1 MCU-STM32F407VET6(LQFP100), Y1 Crystal

Commit message: Fixed wiring ad7511 and wired the rtl8211EG IC
Connections:
- net labels removed: VDD3V3
Changed lines of the file:
@@
 $EndComp
 Text GLabel 4500 1000 0    50   Input ~ 0
-VDD3V3
+3V3
 Text GLabel 8800 3600 2    50   Input ~ 0
 GND

Commit message: Added protection diodes to the joystick ports.
Connections:
- net labels added: STM_SPI1_CS, STM_SPI1_MISO, STM_SPI1_MOSI, STM_SPI1_NSS, STM_SPI1_SCK, STM_USART1_CK, STM_USART1_CTS, STM_USART1_RTS, STM_USART1_RX, STM_USART1_TX
Changed lines of the file:
@@
 Text GLabel 5800 5500 3    50   Input ~ 0
 SD_SPI2_CS
+Text GLabel 6900 2350 1    50   Input ~ 0
+STM_SPI1_NSS
+Text GLabel 6800 2350 1    50   Input ~ 0
+STM_SPI1_SCK
+Text GLabel 6700 2350 1    50   Input ~ 0
+STM_SPI1_MISO
+Text GLabel 6600 2350 1    50   Input ~ 0
+STM_SPI1_MOSI
+Text GLabel 7000 2350 1    50   Input ~ 0
+STM_SPI1_CS
+Text GLabel 6500 2350 1    50   Input ~ 0
+STM_USART1_CK
+Text GLabel 6400 2350 1    50   Input ~ 0
+STM_USART1_TX
+Text GLabel 6300 2350 1    50   Input ~ 0
+STM_USART1_RX
+Text GLabel 6200 2350 1    50   Input ~ 0
+STM_USART1_CTS
+Text GLabel 6100 2350 1    50   Input ~ 0
+STM_USART1_RTS
 $EndSCHEMATC

Commit message: Fixed connections for the adv7511. Fixed some minor footprint issues with the fpga board footprint.
Parts:
- U1: footprint LQFP100-0.5-13.8X13.8MM -> stm32-f407:LQFP100-0.5-13.8X13.8MM
Connections:
- net labels added: STM_IO_33, STM_IO_34
Changed lines of the file:
@@
 F 0 "U1" V 5654 1906 50  0000 R CNN
 F 1 "MCU-STM32F407VET6(LQFP100)" V 5750 4350 50  0000 R CNN
-F 2 "LQFP100-0.5-13.8X13.8MM" H 5700 3800 50  0001 L BNN
+F 2 "stm32-f407:LQFP100-0.5-13.8X13.8MM" H 5700 3800 50  0001 L BNN
 F 3 "LQFP-100 STMicroelectronics" H 5700 3800 50  0001 L BNN
 F 4 "STMicroelectronics" H 5700 3800 50  0001 L BNN "Field4"
@@
 Text GLabel 6100 2350 1    50   Input ~ 0
 STM_USART1_RTS
+Text GLabel 3850 3500 0    50   Input ~ 0
+STM_IO_33
+Text GLabel 3850 3600 0    50   Input ~ 0
+STM_IO_34
 $EndSCHEMATC

Commit message: Connected adv7511 unused inputs to ground. Added high voltage protection on PS2 port. Added indicators for the rubber glue on feet.
Parts:
- removed C1, C10, C11, C12, C13, C17, C2, C3, C4, C5, C6, C7, C8, C9: 100nF, Capacitor_SMD:C_0603_1608Metric, symbol Device:C
Connections:
- net labels removed: VDD
- wire segments 163 -> 135

Commit message: First step to implement floppy interface. ESP32 check wireing in.
Parts:
- removed C14, C16, C24: 100nF, Capacitor_SMD:C_0603_1608Metric, symbol Device:C
- removed C15, C18: 2.2uF, Capacitor_SMD:C_0603_1608Metric, symbol Device:C
- removed C19: 1uF, Capacitor_SMD:C_0603_1608Metric, symbol Device:C
- removed C20: 4.7uF, Capacitor_SMD:C_0603_1608Metric, symbol Device:C
- removed C25, C26: 22pF, Capacitor_SMD:C_0603_1608Metric, symbol Device:C
- removed D3, D4: LED, LED_SMD:LED_0603_1608Metric, symbol Device:LED
- removed J4: ARM_JTAG, Connector_PinHeader_2.54mm:PinHeader_2x10_P2.54mm_Vertical, symbol Connector_Generic:Conn_02x10_Odd_Even
- removed R18, R19, R20, R21: 10K, Resistor_SMD:R_0603_1608Metric, symbol Device:R
- removed R22, R23: 1k, Resistor_SMD:R_0603_1608Metric, symbol Device:R
- removed U1: MCU-STM32F407VET6(LQFP100), stm32-f407:LQFP100-0.5-13.8X13.8MM, symbol STM32F407VET6:MCU-STM32F407VET6(LQFP100)
- removed Y1: Crystal, Crystal:Crystal_SMD_HC49-SD, symbol Device:Crystal
- added C10, C2, C3, C7, C8: 100nF, Capacitor_SMD:C_0603_1608Metric, symbol Device:C
- added C4: 1uF, Capacitor_SMD:C_0603_1608Metric, symbol Device:C
- added C9: 4.7uF, Capacitor_SMD:C_0603_1608Metric, symbol Device:C
- added J4: 10118193-0001LF, 10118193-001:FCI_10118193-0001LF, symbol 10118193-0001LF:10118193-0001LF
- added Q1, Q2: MMBT2222A, Package_TO_SOT_SMD:SOT-23, symbol MMBT2222A:MMBT2222A
- added R30, R31: 10k, Resistor_SMD:R_0603_1608Metric, symbol Device:R
- added TP1, TP2: TestPoint, TestPoint:TestPoint_Pad_1.0x1.0mm, symbol Connector:TestPoint
- added U1: ESP32-WROOM, ESP32:ESP32-WROOM, symbol ESP32:ESP32-WROOM
- added U4: INTERFACE-CP2102-GMR(QFN28), Package_DFN_QFN:QFN-28-1EP_5x5mm_P0.5mm_EP3.35x3.35mm, symbol CP2102:INTERFACE-CP2102-GMR(QFN28)
- D1, D2: value LED -> GREEN
- R24: value 1k -> 10k
- R26: value 10k -> 1k
- R27: value 1M -> 10k
Connections:
- net labels added: ADV_SCL, ADV_SDA, ESP_FLASH, ESP_RST, ESP_SD_CLK, ESP_SD_CMD, ESP_SD_DATA0, ESP_SD_DATA1, ESP_SD_DATA2, ESP_SD_DATA3, ESP_SD_SW, ESP_SD_VCC_EN, ESP_UART0_RX, ESP_UART0_TX, ESP_UART1_RX, ESP_UART1_TX, USB_DTR, USB_RTS, VIN5V
- net labels removed: JTAG_TCK, JTAG_TDI, JTAG_TDO, JTAG_TMS, JTAG_TRST, LED0, LED1, LED2, LED3, NRST, SD_SPI2_CS, SD_SPI2_MISO, SD_SPI2_MOSI, SD_SPI2_NSS, SD_SPI2_SCK, SD_SW, STM_IO_33, STM_IO_34, STM_SPI1_CS, STM_SPI1_MISO, STM_SPI1_MOSI, STM_SPI1_NSS, STM_SPI1_SCK, STM_USART1_CK, STM_USART1_CTS, STM_USART1_RTS, STM_USART1_RX, STM_USART1_TX
- wire segments 135 -> 53
- no-connect marks 0 -> 34
Other:
- note removed: "Decoupling capacitors MCU"
- note removed: "JTAG interface"
- note removed: "LED indicators"

Commit message: Integrated the Rover V2 into the board, added level shifters for the floppy interface.
Parts:
- removed U1: ESP32-WROOM, ESP32:ESP32-WROOM, symbol ESP32:ESP32-WROOM
- added C42: 4.7uF, Capacitor_SMD:C_0805_2012Metric, symbol Device:C
- added D11: LED4, LED_SMD:LED_0603_1608Metric, symbol Device:LED
- added D4: LED5, LED_SMD:LED_0603_1608Metric, symbol Device:LED
- added IC1: ESP32-WROVER-B_(16MB), ESP32WROVERIB16MB, symbol ESP32-WROVER-B_(16MB):ESP32-WROVER-B_(16MB)
- added R38, R39: 1k, Resistor_SMD:R_0603_1608Metric, symbol Device:R
- C9: footprint Capacitor_SMD:C_0603_1608Metric -> Capacitor_SMD:C_0805_2012Metric
- J4: symbol 10118193-0001LF:10118193-0001LF -> qmtech-minimig-rescue:10118193-0001LF-10118193-0001LF
Connections:
- net labels added: D+, D-, LED0, LED1
- wire segments 53 -> 63
- no-connect marks 34 -> 32
