File: MCU.sch (KiCad schematic (older format))
At the start: 29 parts, among them IC1 ESP32-WROVER-B_(16MB), J4 10118193-0001LF, Q1 MMBT2222A, Q2 MMBT2222A, SW1 SW_Push, U4 INTERFACE-CP2102-GMR(QFN28)

Commit message: Add the External floppy interface. Routed the HDMI tracks + match impendence.
Connections:
- net labels added: ADV_INT, VUSB5V
- net labels removed: VIN5V
- no-connect marks 32 -> 31
Changed lines of the file:
@@
 GND
 Text GLabel 3400 2950 2    50   Input ~ 0
-VIN5V
+VUSB5V
 Text GLabel 5425 3550 3    50   Input ~ 0
-VIN5V
+VUSB5V
 Text GLabel 4925 2650 0    50   Input ~ 0
 GND
@@
 GND
 Text GLabel 4925 3050 0    50   Input ~ 0
-VIN5V
+VUSB5V
 Wire Wire Line
 	3400 2950 3150 2950
@@
 	1    0    0    -1
 $EndComp
-Text GLabel 2375 4675 3    50   Input ~ 0
-3V3
 Text GLabel 5325 1950 1    50   Input ~ 0
 GND
@@
 NoConn ~ 5100 5900
 NoConn ~ 5100 6000
-NoConn ~ 5100 6100
 NoConn ~ 5100 6400
 NoConn ~ 3600 7200
@@
 Text GLabel 4375 3325 3    50   Input ~ 0
 GND
+Text GLabel 5100 6100 2    50   Input ~ 0
+ADV_INT
 $EndSCHEMATC

Commit message: Fixed HDMI Impedance to 50Ohm, 100Ohm differential, for 0.1mm bord. Add pullups to HDMI I2C, connected DE pin to FPGA.
Connections:
- net labels added: ESP_VSPI_CLK, ESP_VSPI_CS, ESP_VSPI_MISO, ESP_VSPI_MOSI
- net labels removed: ESP_UART1_RX, ESP_UART1_TX
- no-connect marks 31 -> 29
Changed lines of the file:
@@
 	-1   0    0    1
 $EndComp
-Text GLabel 5100 6200 2    50   Input ~ 0
-ESP_SD_VCC_EN
 Text GLabel 5100 5800 2    50   Input ~ 0
 ESP_SD_DATA1
@@
 Text GLabel 1900 7000 2    50   Input ~ 0
 ESP_RST
-Text GLabel 3600 6100 0    50   Input ~ 0
-ESP_UART1_TX
-Text GLabel 3600 6200 0    50   Input ~ 0
-ESP_UART1_RX
 Text GLabel 3600 5800 0    50   Input ~ 0
 ESP_SD_SW
@@
 NoConn ~ 5100 5900
 NoConn ~ 5100 6000
-NoConn ~ 5100 6400
 NoConn ~ 3600 7200
 NoConn ~ 3600 7100
 NoConn ~ 3600 7000
 NoConn ~ 3600 6900
-NoConn ~ 3600 6000
-NoConn ~ 3600 5900
 Wire Wire Line
 	2325 2350 2400 2350
@@
 Text Label 7500 5650 3    50   ~ 0
 LED1
-Text Label 5100 6300 0    50   ~ 0
+Text Label 5100 6800 0    50   ~ 0
 LED1
 Text Label 5100 6500 0    50   ~ 0
 LED0
-NoConn ~ 5100 6800
-NoConn ~ 5100 6900
 Text Label 2600 2750 0    50   ~ 0
 D+
@@
 Text GLabel 4375 3325 3    50   Input ~ 0
 GND
-Text GLabel 5100 6100 2    50   Input ~ 0
+Text GLabel 3600 5900 0    50   Input ~ 0
 ADV_INT
+NoConn ~ 5100 6100
+Text GLabel 3600 6000 0    50   Input ~ 0
+ESP_SD_VCC_EN
+Text GLabel 5100 6900 2    50   Input ~ 0
+ESP_VSPI_MOSI
+Text GLabel 5100 6300 2    50   Input ~ 0
+ESP_VSPI_MISO
+Text GLabel 5100 6200 2    50   Input ~ 0
+ESP_VSPI_CLK
+Text GLabel 3600 6100 0    50   Input ~ 0
+ESP_VSPI_CS
+NoConn ~ 3600 6200
+NoConn ~ 5100 6400
 $EndSCHEMATC

Commit message: Fixed some issues with the 50 Ohm impedance of the SPI lines. Added pinout .odt.
Parts:
- added C43, C44, C45: 10nF, Capacitor_SMD:C_0603_1608Metric, symbol Device:C
- added R44, R45: 20, Resistor_SMD:R_0603_1608Metric, symbol Device:R
Connections:
- wire segments 63 -> 77
Other:
- note added: "RF decoupling SPI"
Changed lines of the file:
@@
 Text GLabel 3600 6000 0    50   Input ~ 0
 ESP_SD_VCC_EN
-Text GLabel 5100 6900 2    50   Input ~ 0
+Text GLabel 6000 6900 2    50   Input ~ 0
 ESP_VSPI_MOSI
 Text GLabel 5100 6300 2    50   Input ~ 0
 ESP_VSPI_MISO
-Text GLabel 5100 6200 2    50   Input ~ 0
+Text GLabel 6000 6200 2    50   Input ~ 0
 ESP_VSPI_CLK
 Text GLabel 3600 6100 0    50   Input ~ 0
@@
 NoConn ~ 3600 6200
 NoConn ~ 5100 6400
+$Comp
+L Device:C C43
+U 1 1 5DAD7FFC
+P 10000 5250
+F 0 "C43" V 9950 5075 50  0000 C CNN
+F 1 "10nF" V 9950 5400 50  0000 C CNN
+F 2 "Capacitor_SMD:C_0603_1608Metric" H 10038 5100 50  0001 C CNN
+F 3 "~" H 10000 5250 50  0001 C CNN
+	1    10000 5250
+	0    1    1    0
+$EndComp
+Wire Wire Line
+	9850 5250 9750 5250
+Wire Wire Line
+	9750 5750 9850 5750
+Wire Wire Line
+	9750 5000 9750 5250
+Connection ~ 9750 5250
+Wire Wire Line
+	9750 5250 9750 5500
+Wire Wire Line
+	9850 5500 9750 5500
+Connection ~ 9750 5500
+Wire Wire Line
+	9750 5500 9750 5750
+Wire Wire Line
+	10250 5000 10250 5250
+Wire Wire Line
+	10250 5750 10150 5750
+Wire Wire Line
+	10150 5500 10250 5500
+Connection ~ 10250 5500
+Wire Wire Line
+	10250 5500 10250 5750
+Wire Wire Line
+	10250 5250 10150 5250
+Connection ~ 10250 5250
+Wire Wire Line
+	10250 5250 10250 5500
+Text GLabel 9750 5000 1    50   Input ~ 0
+3V3
+Text GLabel 10250 5000 1    50   Input ~ 0
+GND
+$Comp
+L Device:C C44
+U 1 1 5DAE087E
+P 10000 5500
+F 0 "C44" V 9950 5325 50  0000 C CNN
+F 1 "10nF" V 9950 5650 50  0000 C CNN
+F 2 "Capacitor_SMD:C_0603_1608Metric" H 10038 5350 50  0001 C CNN
+F 3 "~" H 10000 5500 50  0001 C CNN
+	1    10000 5500
+	0    1    1    0
+$EndComp
+$Comp
+L Device:C C45
+U 1 1 5DAE0A60
+P 10000 5750
+F 0 "C45" V 9950 5575 50  0000 C CNN
+F 1 "10nF" V 9950 5900 50  0000 C CNN
+F 2 "Capacitor_SMD:C_0603_1608Metric" H 10038 5600 50  0001 C CNN
+F 3 "~" H 10000 5750 50  0001 C CNN
+	1    10000 5750
+	0    1    1    0
+$EndComp
+Text Notes 9650 4750 0    50   ~ 0
+RF decoupling SPI
+$Comp
+L Device:R R45
+U 1 1 5DAEDCB1
+P 5850 6900
+F 0 "R45" V 5643 6900 50  0000 C CNN
+F 1 "20" V 5734 6900 50  0000 C CNN
+F 2 "Resistor_SMD:R_0603_1608Metric" V 5780 6900 50  0001 C CNN
+F 3 "~" H 5850 6900 50  0001 C CNN
+	1    5850 6900
+	0    1    1    0
+$EndComp
+Wire Wire Line
+	5700 6900 5100 6900
+$Comp
+L Device:R R44
+U 1 1 5DAF128C
+P 5850 6200
+F 0 "R44" V 5643 6200 50  0000 C CNN
+F 1 "20" V 5734 6200 50  0000 C CNN
+F 2 "Resistor_SMD:R_0603_1608Metric" V 5780 6200 50  0001 C CNN
+F 3 "~" H 5850 6200 50  0001 C CNN
+	1    5850 6200
+	0    1    1    0
+$EndComp
+Wire Wire Line
+	5700 6200 5100 6200
 $EndSCHEMATC

Commit message: Added ESD protection, and removed the curved lines around the adv7511.
Parts:
- added C47: 10n, Capacitor_SMD:C_0603_1608Metric, symbol Device:C
Other:
- note added: "Decouple the USB signal"
Changed lines of the file:
@@
 Wire Wire Line
 	5700 6200 5100 6200
+$Comp
+L Device:C C47
+U 1 1 5DA58F16
+P 2100 1500
+F 0 "C47" V 1848 1500 50  0000 C CNN
+F 1 "10n" V 1939 1500 50  0000 C CNN
+F 2 "Capacitor_SMD:C_0603_1608Metric" H 2138 1350 50  0001 C CNN
+F 3 "~" H 2100 1500 50  0001 C CNN
+	1    2100 1500
+	0    1    1    0
+$EndComp
+Text GLabel 1950 1500 0    50   Input ~ 0
+GND
+Text GLabel 2250 1500 2    50   Input ~ 0
+3V3
+Text Notes 1700 1175 0    50   ~ 0
+Decouple the USB signal
 $EndSCHEMATC

Commit message: Changed zener diode footprint for easy soldering. Fixed pins, U861/2 and U761/2 they now connect correctly to ground.
Parts:
- C47: value 10n -> 10nF
- IC1: footprint ESP32WROVERIB16MB -> ESP32-WROVER-B_(16MB):ESP32WROVERIB16MB
Changed lines of the file:
@@
 EESchema Schematic File Version 4
-LIBS:qmtech-minimig-cache
 EELAYER 30 0
 EELAYER END
@@
 F 0 "IC1" H 4350 5565 50  0000 C CNN
 F 1 "ESP32-WROVER-B_(16MB)" H 4350 5474 50  0000 C CNN
-F 2 "ESP32WROVERIB16MB" H 4950 5400 50  0001 L CNN
+F 2 "ESP32-WROVER-B_(16MB):ESP32WROVERIB16MB" H 4950 5400 50  0001 L CNN
 F 3 "https://www.mouser.es/datasheet/2/891/esp32-wrover-b_datasheet_en-1384674.pdf" H 4950 5300 50  0001 L CNN
 F 4 "WiFi Modules (802.11) SMD Module, ESP32-D0WD, 64Mbits PSRAM, 128Mbits SPI flash, PCB Antenna" H 4950 5200 50  0001 L CNN "Description"
@@
 P 2100 1500
 F 0 "C47" V 1848 1500 50  0000 C CNN
-F 1 "10n" V 1939 1500 50  0000 C CNN
+F 1 "10nF" V 1939 1500 50  0000 C CNN
 F 2 "Capacitor_SMD:C_0603_1608Metric" H 2138 1350 50  0001 C CNN
 F 3 "~" H 2100 1500 50  0001 C CNN

Commit message: Fixed reversed labeling of the QMTECH FPGA board pins.
Changed lines of the file:
@@
 L Device:R R25
 U 1 1 5D83EA5A
-P 6500 1150
-F 0 "R25" V 6425 1150 50  0000 C CNN
-F 1 "1k" V 6500 1150 50  0000 C CNN
-F 2 "Resistor_SMD:R_0603_1608Metric" V 6430 1150 50  0001 C CNN
-F 3 "~" H 6500 1150 50  0001 C CNN
-	1    6500 1150
+P 6125 1150
+F 0 "R25" V 6050 1150 50  0000 C CNN
+F 1 "1k" V 6125 1150 50  0000 C CNN
+F 2 "Resistor_SMD:R_0603_1608Metric" V 6055 1150 50  0001 C CNN
+F 3 "~" H 6125 1150 50  0001 C CNN
+	1    6125 1150
 	0    1    1    0
 $EndComp
 Text GLabel 6650 1150 2    50   Input ~ 0
-GND
+3V3
 Wire Wire Line
 	6350 1150 6275 1150
@@
 L Device:R R26
 U 1 1 5D840D1C
-P 6500 1375
-F 0 "R26" V 6425 1375 50  0000 C CNN
-F 1 "1k" V 6500 1375 50  0000 C CNN
-F 2 "Resistor_SMD:R_0603_1608Metric" V 6430 1375 50  0001 C CNN
-F 3 "~" H 6500 1375 50  0001 C CNN
-	1    6500 1375
+P 6125 1375
+F 0 "R26" V 6050 1375 50  0000 C CNN
+F 1 "1k" V 6125 1375 50  0000 C CNN
+F 2 "Resistor_SMD:R_0603_1608Metric" V 6055 1375 50  0001 C CNN
+F 3 "~" H 6125 1375 50  0001 C CNN
+	1    6125 1375
 	0    1    1    0
 $EndComp
 Text GLabel 6650 1375 2    50   Input ~ 0
-GND
+3V3
 Wire Wire Line
 	6350 1375 6275 1375
@@
 L Device:LED D1
 U 1 1 5D8F4A33
-P 6125 1150
-F 0 "D1" H 6118 895 50  0000 C CNN
-F 1 "GREEN" H 6118 986 50  0000 C CNN
-F 2 "LED_SMD:LED_0603_1608Metric" H 6125 1150 50  0001 C CNN
-F 3 "~" H 6125 1150 50  0001 C CNN
-	1    6125 1150
-	-1   0    0    1
+P 6500 1150
+F 0 "D1" H 6500 800 50  0000 C CNN
+F 1 "GREEN" H 6500 725 50  0000 C CNN
+F 2 "LED_SMD:LED_0603_1608Metric" H 6500 1150 50  0001 C CNN
+F 3 "~" H 6500 1150 50  0001 C CNN
+	1    6500 1150
+	1    0    0    -1
 $EndComp
 $Comp
 L Device:LED D2
 U 1 1 5D8F4D93
-P 6125 1375
-F 0 "D2" H 6125 1575 50  0000 C CNN
-F 1 "GREEN" H 6125 1475 50  0000 C CNN
-F 2 "LED_SMD:LED_0603_1608Metric" H 6125 1375 50  0001 C CNN
-F 3 "~" H 6125 1375 50  0001 C CNN
-	1    6125 1375
-	-1   0    0    1
+P 6500 1375
+F 0 "D2" H 6500 1700 50  0000 C CNN
+F 1 "GREEN" H 6500 1775 50  0000 C CNN
+F 2 "LED_SMD:LED_0603_1608Metric" H 6500 1375 50  0001 C CNN
+F 3 "~" H 6500 1375 50  0001 C CNN
+	1    6500 1375
+	1    0    0    -1
 $EndComp
 Text GLabel 5100 5800 2    50   Input ~ 0

Commit message: Change order of the VSPI to FPGA to make sure the clock pin connects to an FPGA clock capable pin.
Parts:
- removed R44, R45: 20, Resistor_SMD:R_0603_1608Metric, symbol Device:R
- TP1: value TestPoint -> GND; footprint TestPoint:TestPoint_Pad_1.0x1.0mm -> TestPoint:TestPoint_THTPad_1.0x1.0mm_Drill0.5mm
- TP2: value TestPoint -> USB5V; footprint TestPoint:TestPoint_Pad_1.0x1.0mm -> TestPoint:TestPoint_THTPad_1.0x1.0mm_Drill0.5mm
Connections:
- wire segments 77 -> 75
Changed lines of the file:
@@
 P 3150 2950
 F 0 "TP2" H 3092 2976 50  0000 R CNN
-F 1 "TestPoint" H 3092 3067 50  0000 R CNN
-F 2 "TestPoint:TestPoint_Pad_1.0x1.0mm" H 3350 2950 50  0001 C CNN
+F 1 "USB5V" H 3092 3067 50  0000 R CNN
+F 2 "TestPoint:TestPoint_THTPad_1.0x1.0mm_Drill0.5mm" H 3350 2950 50  0001 C CNN
 F 3 "~" H 3350 2950 50  0001 C CNN
 	1    3150 2950
@@
 P 2400 2350
 F 0 "TP1" H 2458 2468 50  0000 L CNN
-F 1 "TestPoint" H 2458 2377 50  0000 L CNN
-F 2 "TestPoint:TestPoint_Pad_1.0x1.0mm" H 2600 2350 50  0001 C CNN
+F 1 "GND" H 2458 2377 50  0000 L CNN
+F 2 "TestPoint:TestPoint_THTPad_1.0x1.0mm_Drill0.5mm" H 2600 2350 50  0001 C CNN
 F 3 "~" H 2600 2350 50  0001 C CNN
 	1    2400 2350
@@
 Text GLabel 3600 6000 0    50   Input ~ 0
 ESP_SD_VCC_EN
-Text GLabel 6000 6900 2    50   Input ~ 0
+Text GLabel 5100 6900 2    50   Input ~ 0
 ESP_VSPI_MOSI
 Text GLabel 5100 6300 2    50   Input ~ 0
 ESP_VSPI_MISO
-Text GLabel 6000 6200 2    50   Input ~ 0
+Text GLabel 5100 6200 2    50   Input ~ 0
 ESP_VSPI_CLK
 Text GLabel 3600 6100 0    50   Input ~ 0
@@
 	9850 5250 9750 5250
 Wire Wire Line
-	9750 5750 9850 5750
-Wire Wire Line
 	9750 5000 9750 5250
 Connection ~ 9750 5250
@@
 Wire Wire Line
 	9850 5500 9750 5500
-Connection ~ 9750 5500
-Wire Wire Line
-	9750 5500 9750 5750
 Wire Wire Line
 	10250 5000 10250 5250
 Wire Wire Line
-	10250 5750 10150 5750
-Wire Wire Line
 	10150 5500 10250 5500
-Connection ~ 10250 5500
-Wire Wire Line
-	10250 5500 10250 5750
 Wire Wire Line
 	10250 5250 10150 5250
@@
 	0    1    1    0
 $EndComp
-$Comp
-L Device:C C45
-U 1 1 5DAE0A60
-P 10000 5750
-F 0 "C45" V 9950 5575 50  0000 C CNN
-F 1 "10nF" V 9950 5900 50  0000 C CNN
-F 2 "Capacitor_SMD:C_0603_1608Metric" H 10038 5600 50  0001 C CNN
-F 3 "~" H 10000 5750 50  0001 C CNN
-	1    10000 5750
-	0    1    1    0
-$EndComp
 Text Notes 9650 4750 0    50   ~ 0
 RF decoupling SPI
-$Comp
-L Device:R R45
-U 1 1 5DAEDCB1
-P 5850 6900
-F 0 "R45" V 5643 6900 50  0000 C CNN
-F 1 "20" V 5734 6900 50  0000 C CNN
-F 2 "Resistor_SMD:R_0603_1608Metric" V 5780 6900 50  0001 C CNN
-F 3 "~" H 5850 6900 50  0001 C CNN
-	1    5850 6900
-	0    1    1    0
-$EndComp
-Wire Wire Line
-	5700 6900 5100 6900
-$Comp
-L Device:R R44
-U 1 1 5DAF128C
-P 5850 6200
-F 0 "R44" V 5643 6200 50  0000 C CNN
-F 1 "20" V 5734 6200 50  0000 C CNN
-F 2 "Resistor_SMD:R_0603_1608Metric" V 5780 6200 50  0001 C CNN
-F 3 "~" H 5850 6200 50  0001 C CNN
-	1    5850 6200
-	0    1    1    0
-$EndComp
-Wire Wire Line
-	5700 6200 5100 6200
 $Comp
 L Device:C C47
@@
 Text Notes 1700 1175 0    50   ~ 0
 Decouple the USB signal
+Wire Wire Line
+	9750 5500 9750 5750
+Wire Wire Line
+	9850 5750 9750 5750
+Wire Wire Line
+	10150 5750 10250 5750
+Wire Wire Line
+	10250 5500 10250 5750
+$Comp
+L Device:C C45
+U 1 1 5E248164
+P 10000 5750
+F 0 "C45" V 9950 5575 50  0000 C CNN
+F 1 "10nF" V 9950 5900 50  0000 C CNN
+F 2 "Capacitor_SMD:C_0603_1608Metric" H 10038 5600 50  0001 C CNN
+F 3 "~" H 10000 5750 50  0001 C CNN
+	1    10000 5750
+	0    1    1    0
+$EndComp
 $EndSCHEMATC

Commit message: Add PS/2 Mouse connector to the board, USB has too much overhead.
Parts:
- removed C43, C45: 10nF, Capacitor_SMD:C_0603_1608Metric, symbol Device:C
- added R3: 47K, Resistor_SMD:R_0603_1608Metric, symbol Device:R
- renumbered TP2 to U5V1, TP1 to UG1
Connections:
- net labels added: ESP_INT
- wire segments 75 -> 73
- no-connect marks 29 -> 28
Changed lines of the file:
@@
 Text GLabel 2325 2550 2    50   Input ~ 0
 GND
-Text GLabel 3400 2950 2    50   Input ~ 0
+Text GLabel 2500 4225 3    50   Input ~ 0
 VUSB5V
 Text GLabel 5425 3550 3    50   Input ~ 0
@@
 Text GLabel 4925 2650 0    50   Input ~ 0
 GND
-Text GLabel 4125 2950 0    50   Input ~ 0
-3V3
 $Comp
 L Device:C C10
 U 1 1 5D81A5D8
-P 4125 3175
-F 0 "C10" V 4325 3175 50  0000 C CNN
-F 1 "100nF" V 4250 3175 50  0000 C CNN
-F 2 "Capacitor_SMD:C_0603_1608Metric" H 4163 3025 50  0001 C CNN
-F 3 "~" H 4125 3175 50  0001 C CNN
-	1    4125 3175
+P 3275 3175
+F 0 "C10" V 3475 3175 50  0000 C CNN
+F 1 "100nF" V 3400 3175 50  0000 C CNN
+F 2 "Capacitor_SMD:C_0603_1608Metric" H 3313 3025 50  0001 C CNN
+F 3 "~" H 3275 3175 50  0001 C CNN
+	1    3275 3175
 	-1   0    0    1
 $EndComp
-Text GLabel 4125 3325 3    50   Input ~ 0
-GND
-Text GLabel 4925 3050 0    50   Input ~ 0
-VUSB5V
-Wire Wire Line
-	3400 2950 3150 2950
+Text GLabel 3275 3325 3    50   Input ~ 0
+GND
+Wire Wire Line
+	2500 4225 2500 3975
 Wire Wire Line
 	2325 2850 4925 2850
@@
 L Device:C C8
 U 1 1 5D81FF64
-P 2350 3100
-F 0 "C8" H 2465 3146 50  0000 L CNN
-F 1 "100nF" H 2465 3055 50  0000 L CNN
-F 2 "Capacitor_SMD:C_0603_1608Metric" H 2388 2950 50  0001 C CNN
-F 3 "~" H 2350 3100 50  0001 C CNN
-	1    2350 3100
-	1    0    0    -1
-$EndComp
-Connection ~ 2350 2950
-Wire Wire Line
-	2350 2950 2325 2950
+P 2350 3175
+F 0 "C8" H 2465 3221 50  0000 L CNN
+F 1 "100nF" H 2465 3130 50  0000 L CNN
+F 2 "Capacitor_SMD:C_0603_1608Metric" H 2388 3025 50  0001 C CNN
+F 3 "~" H 2350 3175 50  0001 C CNN
+	1    2350 3175
+	0    1    1    0
+$EndComp
+Connection ~ 2500 3175
 $Comp
 L Device:C C9
 U 1 1 5D821065
-P 2850 3100
-F 0 "C9" H 2965 3146 50  0000 L CNN
-F 1 "4.7uF" H 2965 3055 50  0000 L CNN
-F 2 "Capacitor_SMD:C_0805_2012Metric" H 2888 2950 50  0001 C CNN
-F 3 "~" H 2850 3100 50  0001 C CNN
-	1    2850 3100
-	1    0    0    -1
-$EndComp
-Connection ~ 2850 2950
-Wire Wire Line
-	2850 2950 2350 2950
-Text GLabel 2350 3250 3    50   Input ~ 0
-GND
-Text GLabel 2850 3250 3    50   Input ~ 0
+P 2350 3675
+F 0 "C9" H 2465 3721 50  0000 L CNN
+F 1 "4.7uF" H 2465 3630 50  0000 L CNN
+F 2 "Capacitor_SMD:C_0805_2012Metric" H 2388 3525 50  0001 C CNN
+F 3 "~" H 2350 3675 50  0001 C CNN
+	1    2350 3675
+	0    1    1    0
+$EndComp
+Connection ~ 2500 3675
+Wire Wire Line
+	2500 3675 2500 3175
+Text GLabel 2200 3175 0    50   Input ~ 0
+GND
+Text GLabel 2200 3675 0    50   Input ~ 0
 GND
 Text GLabel 2850 2350 2    50   Input ~ 0
@@
 GND
 $Comp
-L Connector:TestPoint TP2
+L Connector:TestPoint U5V1
 U 1 1 5D8A1A13
-P 3150 2950
-F 0 "TP2" H 3092 2976 50  0000 R CNN
-F 1 "USB5V" H 3092 3067 50  0000 R CNN
-F 2 "TestPoint:TestPoint_THTPad_1.0x1.0mm_Drill0.5mm" H 3350 2950 50  0001 C CNN
-F 3 "~" H 3350 2950 50  0001 C CNN
-	1    3150 2950
-	-1   0    0    1
-$EndComp
-Connection ~ 3150 2950
-Wire Wire Line
-	3150 2950 2850 2950
-$Comp
-L Connector:TestPoint TP1
+P 2500 3975
+F 0 "U5V1" H 2442 4001 50  0000 R CNN
+F 1 "USB5V" H 2442 4092 50  0000 R CNN
+F 2 "TestPoint:TestPoint_THTPad_1.0x1.0mm_Drill0.5mm" H 2700 3975 50  0001 C CNN
+F 3 "~" H 2700 3975 50  0001 C CNN
+	1    2500 3975
+	0    -1   -1   0
+$EndComp
+Connection ~ 2500 3975
+Wire Wire Line
+	2500 3975 2500 3675
+$Comp
+L Connector:TestPoint UG1
 U 1 1 5D8AC051
 P 2400 2350
-F 0 "TP1" H 2458 2468 50  0000 L CNN
+F 0 "UG1" H 2458 2468 50  0000 L CNN
 F 1 "GND" H 2458 2377 50  0000 L CNN
 F 2 "TestPoint:TestPoint_THTPad_1.0x1.0mm_Drill0.5mm" H 2600 2350 50  0001 C CNN
@@
 D-
 Wire Wire Line
-	4125 3025 4125 2950
-Wire Wire Line
-	4125 2950 4375 2950
+	3275 3025 3275 2950
+Wire Wire Line
+	3275 2950 3525 2950
 $Comp
 L Device:C C42
 U 1 1 5DB2BACA
-P 4375 3175
-F 0 "C42" H 4490 3221 50  0000 L CNN
-F 1 "4.7uF" H 4490 3130 50  0000 L CNN
-F 2 "Capacitor_SMD:C_0805_2012Metric" H 4413 3025 50  0001 C CNN
-F 3 "~" H 4375 3175 50  0001 C CNN
-	1    4375 3175
-	1    0    0    -1
-$EndComp
-Wire Wire Line
-	4375 2950 4375 3025
-Connection ~ 4375 2950
-Wire Wire Line
-	4375 2950 4925 2950
-Text GLabel 4375 3325 3    50   Input ~ 0
+P 3525 3175
+F 0 "C42" H 3640 3221 50  0000 L CNN
+F 1 "4.7uF" H 3640 3130 50  0000 L CNN
+F 2 "Capacitor_SMD:C_0805_2012Metric" H 3563 3025 50  0001 C CNN
+F 3 "~" H 3525 3175 50  0001 C CNN
+	1    3525 3175
+	1    0    0    -1
+$EndComp
+Wire Wire Line
+	3525 2950 3525 3025
+Connection ~ 3525 2950
+Wire Wire Line
+	3525 2950 4800 2950
+Text GLabel 3525 3325 3    50   Input ~ 0
 GND
 Text GLabel 3600 5900 0    50   Input ~ 0
@@
 Text GLabel 3600 6100 0    50   Input ~ 0
 ESP_VSPI_CS
-NoConn ~ 3600 6200
 NoConn ~ 5100 6400
-$Comp
-L Device:C C43
-U 1 1 5DAD7FFC
-P 10000 5250
-F 0 "C43" V 9950 5075 50  0000 C CNN
-F 1 "10nF" V 9950 5400 50  0000 C CNN
-F 2 "Capacitor_SMD:C_0603_1608Metric" H 10038 5100 50  0001 C CNN
-F 3 "~" H 10000 5250 50  0001 C CNN
-	1    10000 5250
-	0    1    1    0
-$EndComp
-Wire Wire Line
-	9850 5250 9750 5250
-Wire Wire Line
-	9750 5000 9750 5250
-Connection ~ 9750 5250
-Wire Wire Line
-	9750 5250 9750 5500
 Wire Wire Line
 	9850 5500 9750 5500
 Wire Wire Line
-	10250 5000 10250 5250
-Wire Wire Line
 	10150 5500 10250 5500
-Wire Wire Line
-	10250 5250 10150 5250
-Connection ~ 10250 5250
-Wire Wire Line
-	10250 5250 10250 5500
-Text GLabel 9750 5000 1    50   Input ~ 0
-3V3
-Text GLabel 10250 5000 1    50   Input ~ 0
+Text GLabel 9750 5250 1    50   Input ~ 0
+3V3
+Text GLabel 10250 5250 1    50   Input ~ 0
 GND
 $Comp
@@
 	0    1    1    0
 $EndComp
-Text Notes 9650 4750 0    50   ~ 0
+Text Notes 9650 5000 0    50   ~ 0
 RF decoupling SPI
 $Comp
@@
 Decouple the USB signal
 Wire Wire Line
-	9750 5500 9750 5750
-Wire Wire Line
-	9850 5750 9750 5750
-Wire Wire Line
-	10150 5750 10250 5750
-Wire Wire Line
-	10250 5500 10250 5750
-$Comp
-L Device:C C45
-U 1 1 5E248164
-P 10000 5750
-F 0 "C45" V 9950 5575 50  0000 C CNN
-F 1 "10nF" V 9950 5900 50  0000 C CNN
-F 2 "Capacitor_SMD:C_0603_1608Metric" H 10038 5600 50  0001 C CNN
-F 3 "~" H 10000 5750 50  0001 C CNN
-	1    10000 5750
-	0    1    1    0
-$EndComp
+	2500 2950 2325 2950
+Wire Wire Line
+	2500 2950 2500 3175
+Text GLabel 3275 2950 0    50   Input ~ 0
+3V3
+Wire Wire Line
+	4925 3050 4800 3050
+Wire Wire Line
+	4800 3050 4800 2950
+Connection ~ 4800 2950
+Wire Wire Line
+	4800 2950 4925 2950
+Text GLabel 2600 6200 0    50   Input ~ 0
+ESP_INT
+$Comp
+L Device:R R?
+U 1 1 5E2C81AE
+P 2825 6350
+AR Path="/5DE41876/5E2C81AE" Ref="R?"  Part="1"
+AR Path="/5D5D9AB7/5E2C81AE" Ref="R3"  Part="1"
+F 0 "R3" H 2895 6396 50  0000 L CNN
+F 1 "47K" H 2895 6305 50  0000 L CNN
+F 2 "Resistor_SMD:R_0603_1608Metric" V 2755 6350 50  0001 C CNN
+F 3 "~" H 2825 6350 50  0001 C CNN
+	1    2825 6350
+	-1   0    0    1
+$EndComp
+Text GLabel 2825 6500 3    50   Input ~ 0
+3V3
+Wire Wire Line
+	3600 6200 2825 6200
+Connection ~ 2825 6200
+Wire Wire Line
+	2600 6200 2825 6200
+Wire Wire Line
+	9750 5250 9750 5500
+Wire Wire Line
+	10250 5250 10250 5500
 $EndSCHEMATC
