File: MCU.sch (KiCad schematic (older format))
At the start: 32 parts, among them IC1 ESP32-WROVER-B_(16MB), J4 10118193-0001LF, Q1 MMBT2222A, Q2 MMBT2222A, SW1 SW_Push, U4 INTERFACE-CP2102-GMR(QFN28), U5V1 USB5V

Commit message: Minimig V2
Connections:
- net labels added: RST_n
- wire segments 73 -> 70
- no-connect marks 28 -> 27
Changed lines of the file:
@@
 Text Notes 1000 6500 0    100  ~ 0
 Reset button\n
-Text GLabel 4300 4300 2    50   Input ~ 0
-3V3
 $Comp
 L Device:C C?
@@
 	1    0    0    1
 $EndComp
-$Comp
-L CP2102:INTERFACE-CP2102-GMR(QFN28) U4
-U 1 1 5D810043
-P 5725 2750
-F 0 "U4" H 6569 2796 50  0000 L CNN
-F 1 "INTERFACE-CP2102-GMR(QFN28)" H 5125 3150 50  0000 L CNN
-F 2 "Package_DFN_QFN:QFN-28-1EP_5x5mm_P0.5mm_EP3.35x3.35mm" H 5725 2750 50  0001 L BNN
-F 3 "" H 5725 2750 50  0001 L BNN
-F 4 "Unavailable" H 5725 2750 50  0001 L BNN "Field4"
-F 5 "Silicon" H 5725 2750 50  0001 L BNN "Field5"
-F 6 "None" H 5725 2750 50  0001 L BNN "Field6"
-F 7 "CP2102-GMR" H 5725 2750 50  0001 L BNN "Field7"
-F 8 "VFQFN-28 Vishay Siliconix" H 5725 2750 50  0001 L BNN "Field8"
-	1    5725 2750
-	1    0    0    -1
-$EndComp
 Text GLabel 5425 1950 1    50   Input ~ 0
 USB_DTR
@@
 NoConn ~ 4925 2450
 NoConn ~ 4925 2550
-NoConn ~ 5725 3550
 NoConn ~ 5825 3550
 NoConn ~ 2325 2650
@@
 Connection ~ 3600 4300
 Wire Wire Line
-	4100 4300 4300 4300
-Connection ~ 4100 4300
-Wire Wire Line
 	3600 5500 2300 5500
 Wire Wire Line
@@
 	3525 2950 3525 3025
 Connection ~ 3525 2950
-Wire Wire Line
-	3525 2950 4800 2950
 Text GLabel 3525 3325 3    50   Input ~ 0
 GND
@@
 Wire Wire Line
 	2500 2950 2500 3175
-Text GLabel 3275 2950 0    50   Input ~ 0
-3V3
-Wire Wire Line
-	4925 3050 4800 3050
-Wire Wire Line
-	4800 3050 4800 2950
-Connection ~ 4800 2950
-Wire Wire Line
-	4800 2950 4925 2950
 Text GLabel 2600 6200 0    50   Input ~ 0
 ESP_INT
@@
 Wire Wire Line
 	10250 5250 10250 5500
+Text Label 5525 3750 0    50   ~ 0
+RST_n
+$Comp
+L CP2102:INTERFACE-CP2102-GMR(QFN28) U4
+U 1 1 5D810043
+P 5725 2750
+F 0 "U4" H 6569 2796 50  0000 L CNN
+F 1 "INTERFACE-CP2102-GMR(QFN28)" H 5125 3150 50  0000 L CNN
+F 2 "Package_DFN_QFN:QFN-28-1EP_5x5mm_P0.5mm_EP3.35x3.35mm" H 5725 2750 50  0001 L BNN
+F 3 "" H 5725 2750 50  0001 L BNN
+F 4 "Unavailable" H 5725 2750 50  0001 L BNN "Field4"
+F 5 "Silicon" H 5725 2750 50  0001 L BNN "Field5"
+F 6 "None" H 5725 2750 50  0001 L BNN "Field6"
+F 7 "CP2102-GMR" H 5725 2750 50  0001 L BNN "Field7"
+F 8 "VFQFN-28 Vishay Siliconix" H 5725 2750 50  0001 L BNN "Field8"
+	1    5725 2750
+	1    0    0    -1
+$EndComp
+Wire Wire Line
+	3525 2950 4925 2950
+Text GLabel 4925 3050 0    50   Input ~ 0
+VUSB5V
+Connection ~ 4100 4300
+Wire Wire Line
+	4100 4300 4300 4300
+Text GLabel 4300 4300 2    50   Input ~ 0
+3V3
 $EndSCHEMATC

Commit message: Did some placement to make the PCB smaller.
Parts:
- U4: symbol CP2102:INTERFACE-CP2102-GMR(QFN28) -> INTERFACE-CP2102-GMR_QFN28_:INTERFACE-CP2102-GMR(QFN28)
Changed lines of the file:
@@
 RST_n
 $Comp
-L CP2102:INTERFACE-CP2102-GMR(QFN28) U4
+L INTERFACE-CP2102-GMR_QFN28_:INTERFACE-CP2102-GMR(QFN28) U4
 U 1 1 5D810043
 P 5725 2750

Commit message: First rough version of the Open AARS V4
Parts:
- removed U5V1: USB5V, TestPoint:TestPoint_THTPad_1.0x1.0mm_Drill0.5mm, symbol Connector:TestPoint
- removed UG1: GND, TestPoint:TestPoint_THTPad_1.0x1.0mm_Drill0.5mm, symbol Connector:TestPoint
Connections:
- wire segments 70 -> 67
Changed lines of the file:
@@
 	-1   0    0    1
 $EndComp
-Text GLabel 2325 2550 2    50   Input ~ 0
+Text GLabel 2325 2350 2    50   Input ~ 0
 GND
 Text GLabel 2500 4225 3    50   Input ~ 0
@@
 GND
 Wire Wire Line
-	2500 4225 2500 3975
-Wire Wire Line
 	2325 2850 4925 2850
 Wire Wire Line
@@
 GND
 Text GLabel 2200 3675 0    50   Input ~ 0
-GND
-Text GLabel 2850 2350 2    50   Input ~ 0
 GND
 $Comp
@@
 Text GLabel 2150 5700 0    50   Input ~ 0
 GND
-$Comp
-L Connector:TestPoint U5V1
-U 1 1 5D8A1A13
-P 2500 3975
-F 0 "U5V1" H 2442 4001 50  0000 R CNN
-F 1 "USB5V" H 2442 4092 50  0000 R CNN
-F 2 "TestPoint:TestPoint_THTPad_1.0x1.0mm_Drill0.5mm" H 2700 3975 50  0001 C CNN
-F 3 "~" H 2700 3975 50  0001 C CNN
-	1    2500 3975
-	0    -1   -1   0
-$EndComp
-Connection ~ 2500 3975
-Wire Wire Line
-	2500 3975 2500 3675
-$Comp
-L Connector:TestPoint UG1
-U 1 1 5D8AC051
-P 2400 2350
-F 0 "UG1" H 2458 2468 50  0000 L CNN
-F 1 "GND" H 2458 2377 50  0000 L CNN
-F 2 "TestPoint:TestPoint_THTPad_1.0x1.0mm_Drill0.5mm" H 2600 2350 50  0001 C CNN
-F 3 "~" H 2600 2350 50  0001 C CNN
-	1    2400 2350
-	1    0    0    -1
-$EndComp
-Wire Wire Line
-	2850 2350 2400 2350
 $Comp
 L Device:LED D1
@@
 NoConn ~ 3600 7000
 NoConn ~ 3600 6900
-Wire Wire Line
-	2325 2350 2400 2350
-Connection ~ 2400 2350
 $Comp
 L Device:LED D11
@@
 Text GLabel 4300 4300 2    50   Input ~ 0
 3V3
+Wire Wire Line
+	2500 3675 2500 4225
+Text GLabel 2325 2550 2    50   Input ~ 0
+GND
 $EndSCHEMATC

Commit message: Brought compenents back to the front for easy soldering.
Parts:
- removed U4: INTERFACE-CP2102-GMR(QFN28), Package_DFN_QFN:QFN-28-1EP_5x5mm_P0.5mm_EP3.35x3.35mm, symbol INTERFACE-CP2102-GMR_QFN28_:INTERFACE-CP2102-GMR(QFN28)
- added D14, D15: GREEN, LED_SMD:LED_0603_1608Metric, symbol Device:LED
- added J11: Conn_01x02_Male, Connector_PinHeader_2.54mm:PinHeader_1x02_P2.54mm_Vertical, symbol Connector:Conn_01x02_Male
- added R1, R11: 1k, Resistor_SMD:R_0603_1608Metric, symbol Device:R
- added U10: CP2105-F01-GM, qmtech-minimig-new:Silicon_Labs-CP2105-F01-GM-Level_A, symbol eec:CP2105-F01-GM
Connections:
- net labels added: FGPA_UART0_TX, FPGA_UART0_RX
- wire segments 67 -> 86
- no-connect marks 27 -> 22

Commit message: Removed ESP32, as it's no longer needed, we have soft cores.
Parts:
- removed C2, C3, C7: 100nF, Capacitor_SMD:C_0603_1608Metric, symbol Device:C
- removed C4: 1uF, Capacitor_SMD:C_0603_1608Metric, symbol Device:C
- removed C44: 10nF, Capacitor_SMD:C_0603_1608Metric, symbol Device:C
- removed D1, D2: GREEN, LED_SMD:LED_0603_1608Metric, symbol Device:LED
- removed D11: LED4, LED_SMD:LED_0603_1608Metric, symbol Device:LED
- removed D4: LED5, LED_SMD:LED_0603_1608Metric, symbol Device:LED
- removed IC1: ESP32-WROVER-B_(16MB), ESP32-WROVER-B_(16MB):ESP32WROVERIB16MB, symbol ESP32-WROVER-B_(16MB):ESP32-WROVER-B_(16MB)
- removed J11: Conn_01x02_Male, Connector_PinHeader_2.54mm:PinHeader_1x02_P2.54mm_Vertical, symbol Connector:Conn_01x02_Male
- removed Q1, Q2: MMBT2222A, Package_TO_SOT_SMD:SOT-23, symbol MMBT2222A:MMBT2222A
- removed R17: 10K, Resistor_SMD:R_0603_1608Metric, symbol Device:R
- removed R25, R26, R38, R39: 1k, Resistor_SMD:R_0603_1608Metric, symbol Device:R
- removed R27, R30, R31: 10k, Resistor_SMD:R_0603_1608Metric, symbol Device:R
- removed R3: 47K, Resistor_SMD:R_0603_1608Metric, symbol Device:R
- removed SW1: SW_Push, Button_Switch_SMD:SW_SPST_EVQQ2, symbol Switch:SW_Push
- removed U10: CP2105-F01-GM, qmtech-minimig-new:Silicon_Labs-CP2105-F01-GM-Level_A, symbol eec:CP2105-F01-GM
- added U1: CP2102N-A01-GQFN28, Package_DFN_QFN:QFN-28-1EP_5x5mm_P0.5mm_EP3.35x3.35mm, symbol Interface_USB:CP2102N-A01-GQFN28
- renumbered C47 to C1, C8 to C2, C9 to C3, C10 to C4, C42 to C5, D14 to D1, D15 to D2, J4 to J1, R24 to R1, R1 to R2, R11 to R3
Connections:
- net labels added: FPGA_UART0_TX
- net labels removed: ADV_INT, ADV_SCL, ADV_SDA, ESP_FLASH, ESP_INT, ESP_RST, ESP_SD_CLK, ESP_SD_CMD, ESP_SD_DATA0, ESP_SD_DATA1, ESP_SD_DATA2, ESP_SD_DATA3, ESP_SD_SW, ESP_SD_VCC_EN, ESP_UART0_RX, ESP_UART0_TX, ESP_VSPI_CLK, ESP_VSPI_CS, ESP_VSPI_MISO, ESP_VSPI_MOSI, FGPA_UART0_TX, LED0, LED1, RST_n, USB_DTR, USB_RTS
- wire segments 86 -> 18
- no-connect marks 22 -> 3
Other:
- note removed: "RF decoupling SPI"
- note removed: "Reset button\n"
- moved on the sheet: J1
