File: hdmi_transmitter.sch (KiCad schematic (older format))
At the start: 20 parts, among them U3 LT1963AxST-1.8

Commit message: Fixed wiring ad7511 and wired the rtl8211EG IC
Parts:
- added C40, C41: 100nF, Capacitor_SMD:C_0603_1608Metric, symbol Device:C
- added J7: HDMI_D_1.4, Connector_HDMI:HDMI_Micro-D_Molex_46765-0x01, symbol Connector:HDMI_D_1.4
Connections:
- net labels added: ADV_HEAC+, ADV_HEAC-, ADV_TX0+, ADV_TX0-, ADV_TX1+, ADV_TX1-, ADV_TX2+, ADV_TX2-, ADV_TXC+, ADV_TXC-
- wire segments 58 -> 62
Changed lines of the file:
@@
 	5950 6150 5000 6150
 Wire Wire Line
-	8800 7200 8800 7700
+	8800 7200 8800 8000
 Wire Wire Line
 	8900 3800 8900 3500
@@
 Text GLabel 8900 3150 1    50   Input ~ 0
 ADV_DVDD
-Text GLabel 8800 8000 3    50   Input ~ 0
+Text GLabel 8800 8300 3    50   Input ~ 0
 ADV_DVDD
 Text GLabel 5300 4350 0    50   Input ~ 0
@@
 GND
 Wire Wire Line
-	8000 8000 8000 7700
-Text GLabel 8000 8000 3    50   Input ~ 0
+	8000 8300 8000 8000
+Text GLabel 8000 8300 3    50   Input ~ 0
 ADV_AVDD
 Wire Wire Line
@@
 L Device:C C37
 U 1 1 5DD51D08
-P 7850 7700
-F 0 "C37" V 7598 7700 50  0000 C CNN
-F 1 "100nF" V 7689 7700 50  0000 C CNN
-F 2 "Capacitor_SMD:C_0603_1608Metric" H 7888 7550 50  0001 C CNN
-F 3 "~" H 7850 7700 50  0001 C CNN
-	1    7850 7700
-	0    1    1    0
-$EndComp
-Connection ~ 8000 7700
-Wire Wire Line
-	8000 7700 8000 7200
+P 7850 8000
+F 0 "C37" V 7598 8000 50  0000 C CNN
+F 1 "100nF" V 7689 8000 50  0000 C CNN
+F 2 "Capacitor_SMD:C_0603_1608Metric" H 7888 7850 50  0001 C CNN
+F 3 "~" H 7850 8000 50  0001 C CNN
+	1    7850 8000
+	0    1    1    0
+$EndComp
+Connection ~ 8000 8000
+Wire Wire Line
+	8000 8000 8000 7200
 $Comp
 L Device:C C38
 U 1 1 5DD5829D
-P 8650 7700
-F 0 "C38" V 8398 7700 50  0000 C CNN
-F 1 "100nF" V 8489 7700 50  0000 C CNN
-F 2 "Capacitor_SMD:C_0603_1608Metric" H 8688 7550 50  0001 C CNN
-F 3 "~" H 8650 7700 50  0001 C CNN
-	1    8650 7700
-	0    1    1    0
-$EndComp
-Connection ~ 8800 7700
-Wire Wire Line
-	8800 7700 8800 8000
-Text GLabel 7700 7700 0    50   Input ~ 0
-GND
-Text GLabel 8500 7700 0    50   Input ~ 0
+P 8650 8000
+F 0 "C38" V 8398 8000 50  0000 C CNN
+F 1 "100nF" V 8489 8000 50  0000 C CNN
+F 2 "Capacitor_SMD:C_0603_1608Metric" H 8688 7850 50  0001 C CNN
+F 3 "~" H 8650 8000 50  0001 C CNN
+	1    8650 8000
+	0    1    1    0
+$EndComp
+Connection ~ 8800 8000
+Wire Wire Line
+	8800 8000 8800 8300
+Text GLabel 7700 8000 0    50   Input ~ 0
+GND
+Text GLabel 8500 8000 0    50   Input ~ 0
 GND
 $Comp
@@
 Text GLabel 8600 3800 1    50   Input ~ 0
 ADV_CLK
+Text GLabel 7100 7200 3    50   Input ~ 0
+ADV_TXC-
+Text GLabel 7200 7200 3    50   Input ~ 0
+ADV_TXC+
+Wire Wire Line
+	6800 8300 6800 8000
+Text GLabel 6800 8300 3    50   Input ~ 0
+ADV_AVDD
+$Comp
+L Device:C C40
+U 1 1 5D78372C
+P 6950 8000
+F 0 "C40" V 6698 8000 50  0000 C CNN
+F 1 "100nF" V 6789 8000 50  0000 C CNN
+F 2 "Capacitor_SMD:C_0603_1608Metric" H 6988 7850 50  0001 C CNN
+F 3 "~" H 6950 8000 50  0001 C CNN
+	1    6950 8000
+	0    1    1    0
+$EndComp
+Connection ~ 6800 8000
+Wire Wire Line
+	6800 8000 6800 7200
+Text GLabel 7100 8000 2    50   Input ~ 0
+GND
+Text GLabel 7400 7200 3    50   Input ~ 0
+ADV_TX0-
+Text GLabel 7500 7200 3    50   Input ~ 0
+ADV_TX0+
+Text GLabel 7800 7200 3    50   Input ~ 0
+ADV_TX1-
+Text GLabel 7900 7200 3    50   Input ~ 0
+ADV_TX1+
+Text GLabel 8100 7200 3    50   Input ~ 0
+ADV_TX2-
+Text GLabel 8200 7200 3    50   Input ~ 0
+ADV_TX2+
+Wire Wire Line
+	7300 7200 7300 8250
+Text GLabel 7300 8350 3    50   Input ~ 0
+ADV_AVDD
+$Comp
+L Device:C C41
+U 1 1 5D79F1F0
+P 7450 8250
+F 0 "C41" V 7198 8250 50  0000 C CNN
+F 1 "100nF" V 7289 8250 50  0000 C CNN
+F 2 "Capacitor_SMD:C_0603_1608Metric" H 7488 8100 50  0001 C CNN
+F 3 "~" H 7450 8250 50  0001 C CNN
+	1    7450 8250
+	0    1    1    0
+$EndComp
+Connection ~ 7300 8250
+Wire Wire Line
+	7300 8250 7300 8350
+Text GLabel 7600 8250 2    50   Input ~ 0
+GND
+$Comp
+L Connector:HDMI_D_1.4 J7
+U 1 1 5D7CFF38
+P 13300 2000
+F 0 "J7" H 13730 2046 50  0000 L CNN
+F 1 "HDMI_D_1.4" H 13730 1955 50  0000 L CNN
+F 2 "Connector_HDMI:HDMI_Micro-D_Molex_46765-0x01" H 13325 2000 50  0001 C CNN
+F 3 "http://pinoutguide.com/PortableDevices/micro_hdmi_type_d_pinout.shtml" H 13325 2000 50  0001 C CNN
+	1    13300 2000
+	1    0    0    -1
+$EndComp
+Text GLabel 12900 2700 0    50   Input ~ 0
+ADV_HEAC-
+Text GLabel 12900 2600 0    50   Input ~ 0
+ADV_HEAC+
+Text GLabel 12900 1900 0    50   Input ~ 0
+ADV_TXC-
+Text GLabel 12900 1800 0    50   Input ~ 0
+ADV_TXC+
+Text GLabel 12900 1700 0    50   Input ~ 0
+ADV_TX0-
+Text GLabel 12900 1600 0    50   Input ~ 0
+ADV_TX0+
+Text GLabel 12900 1500 0    50   Input ~ 0
+ADV_TX1-
+Text GLabel 12900 1400 0    50   Input ~ 0
+ADV_TX1+
+Text GLabel 12900 1300 0    50   Input ~ 0
+ADV_TX2-
+Text GLabel 12900 1200 0    50   Input ~ 0
+ADV_TX2+
+Text GLabel 13600 3100 3    50   Input ~ 0
+GND
+Text GLabel 13500 3100 3    50   Input ~ 0
+GND
 $EndSCHEMATC

Commit message: Moved to full size HDMI.
Parts:
- removed J7: HDMI_D_1.4, Connector_HDMI:HDMI_Micro-D_Molex_46765-0x01, symbol Connector:HDMI_D_1.4
- added J9: 47151-0001, 47151-0001-HDMI:47151-0001, symbol 47151-0001:47151-0001
Connections:
- net labels added: ADV_5V, ADV_CEC, ADV_CEC_CLK, ADV_DDCSCL, ADV_DDCSDA, ADV_HOTPLUG, ADV_SCL, ADV_SDA
Changed lines of the file:
@@
 EESchema Schematic File Version 4
+LIBS:qmtech-minimig-cache
 EELAYER 30 0
 EELAYER END
@@
 Text GLabel 7600 8250 2    50   Input ~ 0
 GND
-$Comp
-L Connector:HDMI_D_1.4 J7
-U 1 1 5D7CFF38
-P 13300 2000
-F 0 "J7" H 13730 2046 50  0000 L CNN
-F 1 "HDMI_D_1.4" H 13730 1955 50  0000 L CNN
-F 2 "Connector_HDMI:HDMI_Micro-D_Molex_46765-0x01" H 13325 2000 50  0001 C CNN
-F 3 "http://pinoutguide.com/PortableDevices/micro_hdmi_type_d_pinout.shtml" H 13325 2000 50  0001 C CNN
-	1    13300 2000
-	1    0    0    -1
-$EndComp
-Text GLabel 12900 2700 0    50   Input ~ 0
+Text GLabel 9500 6650 2    50   Input ~ 0
+ADV_HEAC+
+Text GLabel 9500 6750 2    50   Input ~ 0
 ADV_HEAC-
-Text GLabel 12900 2600 0    50   Input ~ 0
-ADV_HEAC+
-Text GLabel 12900 1900 0    50   Input ~ 0
+$Comp
+L 47151-0001:47151-0001 J9
+U 1 1 5D70E8AE
+P 12800 4100
+F 0 "J9" H 13250 4367 50  0000 C CNN
+F 1 "47151-0001" H 13250 4276 50  0000 C CNN
+F 2 "47151-0001-HDMI:47151-0001" H 12800 4100 50  0001 L BNN
+F 3 "None" H 12800 4100 50  0001 L BNN
+F 4 "47151-0001" H 12800 4100 50  0001 L BNN "Field4"
+F 5 "Molex" H 12800 4100 50  0001 L BNN "Field5"
+F 6 "Conn.; Data; HDMI; Recept.; 19 Cir.; RtAngle, w/o Back Cover; Black Housing" H 12800 4100 50  0001 L BNN "Field6"
+F 7 "None" H 12800 4100 50  0001 L BNN "Field7"
+F 8 "Unavailable" H 12800 4100 50  0001 L BNN "Field8"
+	1    12800 4100
+	1    0    0    -1
+$EndComp
+Text GLabel 12800 4100 0    50   Input ~ 0
+ADV_TX2+
+Text GLabel 12800 4200 0    50   Input ~ 0
+ADV_TX2-
+Text GLabel 13700 4200 2    50   Input ~ 0
+ADV_TX1+
+Text GLabel 13700 4300 2    50   Input ~ 0
+ADV_TX1-
+Text GLabel 12800 4400 0    50   Input ~ 0
+ADV_TX0+
+Text GLabel 12800 4500 0    50   Input ~ 0
+ADV_TX0-
+Text GLabel 13700 4500 2    50   Input ~ 0
+ADV_TXC+
+Text GLabel 13700 4600 2    50   Input ~ 0
 ADV_TXC-
-Text GLabel 12900 1800 0    50   Input ~ 0
-ADV_TXC+
-Text GLabel 12900 1700 0    50   Input ~ 0
-ADV_TX0-
-Text GLabel 12900 1600 0    50   Input ~ 0
-ADV_TX0+
-Text GLabel 12900 1500 0    50   Input ~ 0
-ADV_TX1-
-Text GLabel 12900 1400 0    50   Input ~ 0
-ADV_TX1+
-Text GLabel 12900 1300 0    50   Input ~ 0
-ADV_TX2-
-Text GLabel 12900 1200 0    50   Input ~ 0
-ADV_TX2+
-Text GLabel 13600 3100 3    50   Input ~ 0
-GND
-Text GLabel 13500 3100 3    50   Input ~ 0
+Text GLabel 8900 7200 3    50   Input ~ 0
+ADV_CEC_CLK
+Text GLabel 8700 7200 3    50   Input ~ 0
+ADV_CEC
+Text GLabel 12800 4700 0    50   Input ~ 0
+ADV_CEC
+Text GLabel 12800 5000 0    50   Input ~ 0
+ADV_HOTPLUG
+Text GLabel 13700 4900 2    50   Input ~ 0
+ADV_5V
+Text GLabel 9500 6450 2    50   Input ~ 0
+ADV_DDCSDA
+Text GLabel 9500 6550 2    50   Input ~ 0
+ADV_DDCSCL
+Text GLabel 9500 6250 2    50   Input ~ 0
+ADV_SDA
+Text GLabel 9500 6350 2    50   Input ~ 0
+ADV_SCL
+Text GLabel 12800 4800 0    50   Input ~ 0
+ADV_DDCSCL
+Text GLabel 13700 4800 2    50   Input ~ 0
+ADV_DDCSDA
+Text GLabel 12800 4900 0    50   Input ~ 0
 GND
 $EndSCHEMATC

Commit message: Added protection diodes to the joystick ports.
Parts:
- added D11: D, Diode_SMD:D_SOD-523, symbol Device:D
- added R54: 27K, Resistor_SMD:R_0603_1608Metric, symbol Device:R
Connections:
- net labels added: ADV_I2S0, ADV_I2S1, ADV_I2S2, ADV_I2S3, ADV_LRCLK, ADV_SCLK
- wire segments 62 -> 65
Changed lines of the file:
@@
 Text GLabel 12800 4900 0    50   Input ~ 0
 GND
+Wire Wire Line
+	2000 9700 2000 10000
+Wire Wire Line
+	2000 10000 2500 10000
+Connection ~ 2000 10000
+Wire Wire Line
+	1500 10000 2000 10000
+$Comp
+L Device:D D11
+U 1 1 5D7E9F98
+P 2000 9550
+F 0 "D11" V 2046 9471 50  0000 R CNN
+F 1 "D" V 1955 9471 50  0000 R CNN
+F 2 "Diode_SMD:D_SOD-523" H 2000 9550 50  0001 C CNN
+F 3 "~" H 2000 9550 50  0001 C CNN
+	1    2000 9550
+	0    -1   -1   0
+$EndComp
+$Comp
+L Device:R R54
+U 1 1 5D7EAB6A
+P 2000 9250
+F 0 "R54" H 2070 9296 50  0000 L CNN
+F 1 "27K" H 2070 9205 50  0000 L CNN
+F 2 "Resistor_SMD:R_0603_1608Metric" H 2070 9159 50  0001 L CNN
+F 3 "~" H 2000 9250 50  0001 C CNN
+	1    2000 9250
+	1    0    0    -1
+$EndComp
+Text GLabel 2000 9100 1    50   Input ~ 0
+3V3
+Text GLabel 1500 10000 0    50   Input ~ 0
+ADV_CEC
+Text GLabel 2500 10000 2    50   Input ~ 0
+ADV_CEC
+Text GLabel 5950 5450 0    50   Input ~ 0
+ADV_I2S0
+Text GLabel 5950 5550 0    50   Input ~ 0
+ADV_I2S1
+Text GLabel 5950 5650 0    50   Input ~ 0
+ADV_I2S2
+Text GLabel 5950 5750 0    50   Input ~ 0
+ADV_I2S3
+Text GLabel 5950 5850 0    50   Input ~ 0
+ADV_SCLK
+Text GLabel 5950 5950 0    50   Input ~ 0
+ADV_LRCLK
 $EndSCHEMATC

Commit message: Fixed connections for the adv7511. Fixed some minor footprint issues with the fpga board footprint.
Parts:
- added R55: 2K, Resistor_SMD:R_0603_1608Metric, symbol Device:R
Connections:
- net labels added: ADV_INT
- wire segments 65 -> 66
Changed lines of the file:
@@
 	5950 6150 5000 6150
-Wire Wire Line
-	8800 7200 8800 8000
 Wire Wire Line
 	8900 3800 8900 3500
@@
 ADV_DVDD
 Text GLabel 8900 3150 1    50   Input ~ 0
-ADV_DVDD
-Text GLabel 8800 8300 3    50   Input ~ 0
 ADV_DVDD
 Text GLabel 5300 4350 0    50   Input ~ 0
@@
 Wire Wire Line
 	8000 8000 8000 7200
-$Comp
-L Device:C C38
-U 1 1 5DD5829D
-P 8650 8000
-F 0 "C38" V 8398 8000 50  0000 C CNN
-F 1 "100nF" V 8489 8000 50  0000 C CNN
-F 2 "Capacitor_SMD:C_0603_1608Metric" H 8688 7850 50  0001 C CNN
-F 3 "~" H 8650 8000 50  0001 C CNN
-	1    8650 8000
-	0    1    1    0
-$EndComp
-Connection ~ 8800 8000
-Wire Wire Line
-	8800 8000 8800 8300
 Text GLabel 7700 8000 0    50   Input ~ 0
-GND
-Text GLabel 8500 8000 0    50   Input ~ 0
 GND
 $Comp
@@
 Text GLabel 13700 4600 2    50   Input ~ 0
 ADV_TXC-
-Text GLabel 8900 7200 3    50   Input ~ 0
-ADV_CEC_CLK
 Text GLabel 8700 7200 3    50   Input ~ 0
 ADV_CEC
@@
 Text GLabel 5950 5950 0    50   Input ~ 0
 ADV_LRCLK
+Text GLabel 8900 7200 3    50   Input ~ 0
+ADV_CEC_CLK
+Text GLabel 8500 8000 0    50   Input ~ 0
+GND
+Wire Wire Line
+	8800 8000 8800 8300
+Connection ~ 8800 8000
+$Comp
+L Device:C C38
+U 1 1 5DD5829D
+P 8650 8000
+F 0 "C38" V 8398 8000 50  0000 C CNN
+F 1 "100nF" V 8489 8000 50  0000 C CNN
+F 2 "Capacitor_SMD:C_0603_1608Metric" H 8688 7850 50  0001 C CNN
+F 3 "~" H 8650 8000 50  0001 C CNN
+	1    8650 8000
+	0    1    1    0
+$EndComp
+Text GLabel 8800 8300 3    50   Input ~ 0
+ADV_DVDD
+Wire Wire Line
+	8800 7200 8800 8000
+$Comp
+L Device:R R55
+U 1 1 5D748417
+P 7700 7500
+F 0 "R55" V 7700 7600 50  0000 L CNN
+F 1 "2K" V 7700 7450 50  0000 L CNN
+F 2 "Resistor_SMD:R_0603_1608Metric" V 7630 7500 50  0001 C CNN
+F 3 "~" H 7700 7500 50  0001 C CNN
+	1    7700 7500
+	1    0    0    -1
+$EndComp
+Text GLabel 7700 7650 3    50   Input ~ 0
+GND
+Wire Wire Line
+	7700 7200 7700 7350
+Text GLabel 8400 7200 3    50   Input ~ 0
+ADV_INT
 $EndSCHEMATC

Commit message: Connected adv7511 unused inputs to ground. Added high voltage protection on PS2 port. Added indicators for the rubber glue on feet.
Parts:
- removed D11: D, Diode_SMD:D_SOD-523, symbol Device:D
- removed R54: 27K, Resistor_SMD:R_0603_1608Metric, symbol Device:R
- added C1: 100nF, Capacitor_SMD:C_0603_1608Metric, symbol Device:C
- added R56: 10k, Resistor_SMD:R_0603_1608Metric, symbol Device:R
- added R57: 887, Resistor_SMD:R_0603_1608Metric, symbol Device:R
Connections:
- net labels added: ADV_HPD, VIN5V
- net labels removed: ADV_5V, ADV_CEC_CLK, ADV_HEAC+, ADV_HEAC-, ADV_HOTPLUG
- wire segments 66 -> 68
Changed lines of the file:
@@
 Title ""
 Date ""
-Rev ""
-Comp ""
+Rev "0.1"
+Comp "deFEEST"
 Comment1 ""
 Comment2 ""
@@
 GND
 Text GLabel 9500 6650 2    50   Input ~ 0
-ADV_HEAC+
+GND
 Text GLabel 9500 6750 2    50   Input ~ 0
-ADV_HEAC-
+GND
 $Comp
 L 47151-0001:47151-0001 J9
@@
 ADV_TXC-
 Text GLabel 8700 7200 3    50   Input ~ 0
-ADV_CEC
+GND
 Text GLabel 12800 4700 0    50   Input ~ 0
 ADV_CEC
-Text GLabel 12800 5000 0    50   Input ~ 0
-ADV_HOTPLUG
+Text GLabel 12300 5000 0    50   Input ~ 0
+ADV_HPD
 Text GLabel 13700 4900 2    50   Input ~ 0
-ADV_5V
+VIN5V
 Text GLabel 9500 6450 2    50   Input ~ 0
 ADV_DDCSDA
@@
 Text GLabel 12800 4900 0    50   Input ~ 0
 GND
-Wire Wire Line
-	2000 9700 2000 10000
-Wire Wire Line
-	2000 10000 2500 10000
-Connection ~ 2000 10000
-Wire Wire Line
-	1500 10000 2000 10000
-$Comp
-L Device:D D11
-U 1 1 5D7E9F98
-P 2000 9550
-F 0 "D11" V 2046 9471 50  0000 R CNN
-F 1 "D" V 1955 9471 50  0000 R CNN
-F 2 "Diode_SMD:D_SOD-523" H 2000 9550 50  0001 C CNN
-F 3 "~" H 2000 9550 50  0001 C CNN
-	1    2000 9550
-	0    -1   -1   0
-$EndComp
-$Comp
-L Device:R R54
-U 1 1 5D7EAB6A
-P 2000 9250
-F 0 "R54" H 2070 9296 50  0000 L CNN
-F 1 "27K" H 2070 9205 50  0000 L CNN
-F 2 "Resistor_SMD:R_0603_1608Metric" H 2070 9159 50  0001 L CNN
-F 3 "~" H 2000 9250 50  0001 C CNN
-	1    2000 9250
-	1    0    0    -1
-$EndComp
-Text GLabel 2000 9100 1    50   Input ~ 0
-3V3
-Text GLabel 1500 10000 0    50   Input ~ 0
-ADV_CEC
-Text GLabel 2500 10000 2    50   Input ~ 0
-ADV_CEC
 Text GLabel 5950 5450 0    50   Input ~ 0
 ADV_I2S0
@@
 ADV_LRCLK
 Text GLabel 8900 7200 3    50   Input ~ 0
-ADV_CEC_CLK
-Text GLabel 8500 8000 0    50   Input ~ 0
+GND
+Text GLabel 9100 8000 2    50   Input ~ 0
 GND
 Wire Wire Line
@@
 L Device:C C38
 U 1 1 5DD5829D
-P 8650 8000
-F 0 "C38" V 8398 8000 50  0000 C CNN
-F 1 "100nF" V 8489 8000 50  0000 C CNN
-F 2 "Capacitor_SMD:C_0603_1608Metric" H 8688 7850 50  0001 C CNN
-F 3 "~" H 8650 8000 50  0001 C CNN
-	1    8650 8000
+P 8950 8000
+F 0 "C38" V 8698 8000 50  0000 C CNN
+F 1 "100nF" V 8789 8000 50  0000 C CNN
+F 2 "Capacitor_SMD:C_0603_1608Metric" H 8988 7850 50  0001 C CNN
+F 3 "~" H 8950 8000 50  0001 C CNN
+	1    8950 8000
 	0    1    1    0
 $EndComp
@@
 Text GLabel 8400 7200 3    50   Input ~ 0
 ADV_INT
+Text GLabel 6900 7200 3    50   Input ~ 0
+ADV_HPD
+$Comp
+L Device:R R56
+U 1 1 5D83D42F
+P 12550 5150
+F 0 "R56" V 12650 5150 50  0000 C CNN
+F 1 "10k" V 12550 5150 50  0000 C CNN
+F 2 "Resistor_SMD:R_0603_1608Metric" V 12480 5150 50  0001 C CNN
+F 3 "~" H 12550 5150 50  0001 C CNN
+	1    12550 5150
+	-1   0    0    1
+$EndComp
+Wire Wire Line
+	12800 5000 12550 5000
+Connection ~ 12550 5000
+Wire Wire Line
+	12550 5000 12300 5000
+Text GLabel 12550 5300 3    50   Input ~ 0
+GND
+Text GLabel 5950 4550 0    50   Input ~ 0
+GND
+Text GLabel 5950 4650 0    50   Input ~ 0
+GND
+Text GLabel 5950 4750 0    50   Input ~ 0
+GND
+Text GLabel 5950 4850 0    50   Input ~ 0
+GND
+Text GLabel 5950 4950 0    50   Input ~ 0
+GND
+Text GLabel 5950 5050 0    50   Input ~ 0
+GND
+Text GLabel 5950 5150 0    50   Input ~ 0
+GND
+Text GLabel 5950 5250 0    50   Input ~ 0
+GND
+Text GLabel 5950 5350 0    50   Input ~ 0
+GND
+$Comp
+L Device:R R57
+U 1 1 5D84D6DF
+P 6700 7450
+F 0 "R57" V 6800 7400 50  0000 L CNN
+F 1 "887" V 6700 7350 50  0000 L CNN
+F 2 "Resistor_SMD:R_0603_1608Metric" V 6630 7450 50  0001 C CNN
+F 3 "~" H 6700 7450 50  0001 C CNN
+	1    6700 7450
+	1    0    0    -1
+$EndComp
+Text GLabel 6700 7600 3    50   Input ~ 0
+GND
+Wire Wire Line
+	6700 7200 6700 7300
+Wire Wire Line
+	8600 7200 8600 9000
+Text GLabel 8600 9250 3    50   Input ~ 0
+3V3
+$Comp
+L Device:C C1
+U 1 1 5D85D4AB
+P 8750 9000
+F 0 "C1" V 8498 9000 50  0000 C CNN
+F 1 "100nF" V 8589 9000 50  0000 C CNN
+F 2 "Capacitor_SMD:C_0603_1608Metric" H 8788 8850 50  0001 C CNN
+F 3 "~" H 8750 9000 50  0001 C CNN
+	1    8750 9000
+	0    1    1    0
+$EndComp
+Connection ~ 8600 9000
+Wire Wire Line
+	8600 9000 8600 9250
+Text GLabel 8900 9000 2    50   Input ~ 0
+GND
+Text GLabel 6800 3800 1    50   Input ~ 0
+GND
+Text GLabel 6900 3800 1    50   Input ~ 0
+GND
+Text GLabel 7000 3800 1    50   Input ~ 0
+GND
+Text GLabel 7100 3800 1    50   Input ~ 0
+GND
+Text GLabel 7200 3800 1    50   Input ~ 0
+GND
+Text GLabel 8100 3800 1    50   Input ~ 0
+GND
+Text GLabel 8200 3800 1    50   Input ~ 0
+GND
+Text GLabel 8300 3800 1    50   Input ~ 0
+GND
+Text GLabel 8400 3800 1    50   Input ~ 0
+GND
+Text GLabel 9500 5050 2    50   Input ~ 0
+GND
+Text GLabel 9500 5150 2    50   Input ~ 0
+GND
+Text GLabel 9500 5250 2    50   Input ~ 0
+GND
+Text GLabel 9500 5350 2    50   Input ~ 0
+GND
 $EndSCHEMATC

Commit message: First step to implement floppy interface. ESP32 check wireing in.
Parts:
- added R18, R19: 4.7k, Resistor_SMD:R_0603_1608Metric, symbol Device:R
- added R34: 10k, Resistor_SMD:R_0603_1608Metric, symbol Device:R
Connections:
- net labels removed: ADV_CEC
- wire segments 68 -> 72
- no-connect marks 0 -> 7
Other:
- note added: "I2C bus resistors\n"
Changed lines of the file:
@@
 	7600 7200 7600 7350
-Wire Wire Line
-	8300 7200 8300 7350
 Wire Wire Line
 	9500 4350 9650 4350
@@
 Text GLabel 7600 7350 3    50   Input ~ 0
 GND
-Text GLabel 8300 7350 3    50   Input ~ 0
+Text GLabel 8300 7200 3    50   Input ~ 0
 GND
 Text GLabel 9650 4350 2    50   Input ~ 0
@@
 Text GLabel 8700 7200 3    50   Input ~ 0
 GND
-Text GLabel 12800 4700 0    50   Input ~ 0
-ADV_CEC
 Text GLabel 12300 5000 0    50   Input ~ 0
 ADV_HPD
-Text GLabel 13700 4900 2    50   Input ~ 0
+Text GLabel 14475 4900 2    50   Input ~ 0
 VIN5V
 Text GLabel 9500 6450 2    50   Input ~ 0
@@
 Text GLabel 9500 5350 2    50   Input ~ 0
 GND
+Text Notes 13500 7000 0    89   ~ 0
+I2C bus resistors\n
+Wire Wire Line
+	13700 7650 14100 7650
+Text GLabel 13700 7650 0    50   Input ~ 0
+ADV_SCL
+Text GLabel 13700 8250 0    50   Input ~ 0
+ADV_SDA
+$Comp
+L Device:R R18
+U 1 1 5D7A6E2F
+P 14100 7500
+F 0 "R18" H 14170 7546 50  0000 L CNN
+F 1 "4.7k" H 14170 7455 50  0000 L CNN
+F 2 "Resistor_SMD:R_0603_1608Metric" V 14030 7500 50  0001 C CNN
+F 3 "~" H 14100 7500 50  0001 C CNN
+	1    14100 7500
+	1    0    0    -1
+$EndComp
+Connection ~ 14100 7650
+Wire Wire Line
+	14100 7650 14700 7650
+Text GLabel 14100 7350 1    50   Input ~ 0
+3V3
+$Comp
+L Device:R R19
+U 1 1 5D7AA6C2
+P 14100 8100
+F 0 "R19" H 14170 8146 50  0000 L CNN
+F 1 "4.7k" H 14170 8055 50  0000 L CNN
+F 2 "Resistor_SMD:R_0603_1608Metric" V 14030 8100 50  0001 C CNN
+F 3 "~" H 14100 8100 50  0001 C CNN
+	1    14100 8100
+	1    0    0    -1
+$EndComp
+Text GLabel 14100 7950 1    50   Input ~ 0
+3V3
+Wire Wire Line
+	13700 8250 14100 8250
+Connection ~ 14100 8250
+Wire Wire Line
+	14100 8250 14700 8250
+NoConn ~ 8500 7200
+NoConn ~ 12800 4600
+NoConn ~ 12800 4300
+NoConn ~ 13700 4100
+NoConn ~ 13700 4400
+NoConn ~ 13700 4700
+NoConn ~ 12800 4700
+$Comp
+L Device:R R34
+U 1 1 5DA28805
+P 14325 4900
+F 0 "R34" V 14118 4900 50  0000 C CNN
+F 1 "10k" V 14209 4900 50  0000 C CNN
+F 2 "Resistor_SMD:R_0603_1608Metric" V 14255 4900 50  0001 C CNN
+F 3 "~" H 14325 4900 50  0001 C CNN
+	1    14325 4900
+	0    1    1    0
+$EndComp
+Wire Wire Line
+	14175 4900 13700 4900
 $EndSCHEMATC
