File: hdmi_transmitter.sch (KiCad schematic (older format))
At the start: 36 parts, among them J9 47151-0001, U3 LT1963AxST-1.8

Commit message: Fixed some issues with the 50 Ohm impedance of the SPI lines. Added pinout .odt.
Parts:
- gave numbers to parts that had none: 2
Changed lines of the file:
@@
 	14900 4800 14825 4800
 $Comp
-L Device:R R?
+L Device:R R43
 U 1 1 5DAC4C64
 P 14825 4950
-F 0 "R?" V 14618 4950 50  0000 C CNN
+F 0 "R43" V 14618 4950 50  0000 C CNN
 F 1 "2k" V 14709 4950 50  0000 C CNN
 F 2 "Resistor_SMD:R_0603_1608Metric" V 14755 4950 50  0001 C CNN
@@
 	11675 4800 11775 4800
 $Comp
-L Device:R R?
+L Device:R R42
 U 1 1 5DAC8AED
 P 11775 4950
-F 0 "R?" V 11875 4950 50  0000 C CNN
+F 0 "R42" V 11875 4950 50  0000 C CNN
 F 1 "2k" V 11775 4950 50  0000 C CNN
 F 2 "Resistor_SMD:R_0603_1608Metric" V 11705 4950 50  0001 C CNN

Commit message: Added ESD protection, and removed the curved lines around the adv7511.
Parts:
- added C48: 100nF, Resistor_SMD:R_0603_1608Metric, symbol Device:C
- added U1: TPD12S520DBT, Package_SO:TSSOP-38_4.4x9.7mm_P0.5mm, symbol Interface_HDMI:TPD12S520DBT
Connections:
- net labels added: ADV_CEC, ADV_CECCLK, ADV_CEC_C, ADV_DDCSCL_C, ADV_DDCSDA_C, ADV_HPD_C, HDMI5V
- wire segments 77 -> 80
- no-connect marks 7 -> 6

Commit message: Add an oscillator for the CEC functionality.
Parts:
- added C49: 100nF, Capacitor_SMD:C_0603_1608Metric, symbol Device:C
- added D30: 1N4148, Diode_SMD:D_SOD-323, symbol Device:D
- added R54, R58: 2K, Resistor_SMD:R_0603_1608Metric, symbol Device:R
- added R59: 27k, Resistor_SMD:R_0603_1608Metric, symbol Device:R
- added R60, R?: 10k, Resistor_SMD:R_0603_1608Metric, symbol Device:R
- added R61: 27, Resistor_SMD:R_0603_1608Metric, symbol Device:R
- added X1: MCSJK-3N-16.00-3.3-50-B, Oscillator:Oscillator_SMD_Abracon_ASE-4Pin_3.2x2.5mm, symbol Oscillator:ASE-xxxMHz
Connections:
- wire segments 80 -> 101
Other:
- note added: "1V8 linear regulator"
- note added: "CEC Clock Generator"
- note added: "ESD protection IC"
- note added: "HDMI Plug"
Changed lines of the file:
@@
 	8625 7550 8625 7725
 Connection ~ 8625 7550
-Text GLabel 8325 7550 0    50   Input ~ 0
-3V3
 $Comp
 L Device:R R41
@@
 Text GLabel 9725 4875 2    50   Input ~ 0
 ADV_SDA
-Text GLabel 9725 5175 2    50   Input ~ 0
+Text GLabel 10500 5175 2    50   Input ~ 0
 ADV_DDCSCL
-Text GLabel 9725 5075 2    50   Input ~ 0
+Text GLabel 10500 5075 2    50   Input ~ 0
 ADV_DDCSDA
 Text GLabel 9725 5375 2    50   Input ~ 0
@@
 Text GLabel 3575 9625 0    50   Input ~ 0
 ADV_DDCSDA
-Text GLabel 3575 9825 0    50   Input ~ 0
+Text GLabel 2900 9825 0    50   Input ~ 0
 ADV_HPD
 Text GLabel 5175 9825 2    50   Input ~ 0
@@
 Text GLabel 8925 5825 3    50   Input ~ 0
 ADV_CEC
-Text GLabel 3575 9325 0    50   Input ~ 0
+Text GLabel 2250 9325 0    50   Input ~ 0
 ADV_CEC
 Text GLabel 5175 9325 2    50   Input ~ 0
@@
 Text GLabel 12800 4700 0    50   Input ~ 0
 ADV_CEC_C
+Text GLabel 8325 7550 0    50   Input ~ 0
+3V3
+Wire Wire Line
+	10500 5175 10375 5175
+$Comp
+L Device:R R58
+U 1 1 5DB8B5F8
+P 10375 5325
+F 0 "R58" H 10445 5371 50  0000 L CNN
+F 1 "2K" H 10445 5280 50  0000 L CNN
+F 2 "Resistor_SMD:R_0603_1608Metric" V 10305 5325 50  0001 C CNN
+F 3 "~" H 10375 5325 50  0001 C CNN
+	1    10375 5325
+	1    0    0    -1
+$EndComp
+Connection ~ 10375 5175
+Wire Wire Line
+	10375 5175 9725 5175
+Text Label 10375 5475 3    50   ~ 0
+HDMI5V
+Wire Wire Line
+	10375 5475 10375 5800
+Connection ~ 10375 5075
+Wire Wire Line
+	10375 5075 10500 5075
+Wire Wire Line
+	9725 5075 10375 5075
+Wire Wire Line
+	10375 4775 10375 4500
+$Comp
+L Device:R R54
+U 1 1 5DB8AF05
+P 10375 4925
+F 0 "R54" H 10445 4971 50  0000 L CNN
+F 1 "2K" H 10445 4880 50  0000 L CNN
+F 2 "Resistor_SMD:R_0603_1608Metric" V 10305 4925 50  0001 C CNN
+F 3 "~" H 10375 4925 50  0001 C CNN
+	1    10375 4925
+	1    0    0    -1
+$EndComp
+Text Label 10375 4775 1    50   ~ 0
+HDMI5V
+Wire Wire Line
+	2250 9325 2500 9325
+$Comp
+L Device:R R59
+U 1 1 5DBB8413
+P 2500 8875
+F 0 "R59" H 2570 8921 50  0000 L CNN
+F 1 "27k" H 2570 8830 50  0000 L CNN
+F 2 "Resistor_SMD:R_0603_1608Metric" V 2430 8875 50  0001 C CNN
+F 3 "~" H 2500 8875 50  0001 C CNN
+	1    2500 8875
+	1    0    0    -1
+$EndComp
+Connection ~ 2500 9325
+Wire Wire Line
+	2500 9325 3575 9325
+$Comp
+L Device:D D30
+U 1 1 5DBBA4B5
+P 2500 9175
+F 0 "D30" V 2546 9096 50  0000 R CNN
+F 1 "1N4148" V 2455 9096 50  0000 R CNN
+F 2 "Diode_SMD:D_SOD-323" H 2500 9175 50  0001 C CNN
+F 3 "~" H 2500 9175 50  0001 C CNN
+	1    2500 9175
+	0    -1   -1   0
+$EndComp
+Text GLabel 2500 8725 1    50   Input ~ 0
+3V3
+$Comp
+L Oscillator:ASE-xxxMHz X1
+U 1 1 5DC2E9FD
+P 9200 10400
+F 0 "X1" H 9544 10446 50  0000 L CNN
+F 1 "MCSJK-3N-16.00-3.3-50-B" H 8775 10750 50  0000 L CNN
+F 2 "Oscillator:Oscillator_SMD_Abracon_ASE-4Pin_3.2x2.5mm" H 9900 10050 50  0001 C CNN
+F 3 "http://www.farnell.com/datasheets/2864171.pdf" H 9100 10400 50  0001 C CNN
+	1    9200 10400
+	1    0    0    -1
+$EndComp
+$Comp
+L Device:R R60
+U 1 1 5DC3073E
+P 8675 10250
+F 0 "R60" H 8745 10296 50  0000 L CNN
+F 1 "10k" H 8745 10205 50  0000 L CNN
+F 2 "Resistor_SMD:R_0603_1608Metric" V 8605 10250 50  0001 C CNN
+F 3 "~" H 8675 10250 50  0001 C CNN
+	1    8675 10250
+	1    0    0    -1
+$EndComp
+Wire Wire Line
+	8900 10400 8675 10400
+Wire Wire Line
+	8675 10100 8675 9900
+Wire Wire Line
+	8675 9900 9200 9900
+Wire Wire Line
+	9200 9900 9200 10100
+Text GLabel 9200 9900 1    50   Input ~ 0
+3V3
+Text GLabel 9200 10700 3    50   Input ~ 0
+GND
+$Comp
+L Device:C C49
+U 1 1 5DC368A8
+P 8300 10250
+F 0 "C49" H 8415 10296 50  0000 L CNN
+F 1 "100nF" H 8415 10205 50  0000 L CNN
+F 2 "Capacitor_SMD:C_0603_1608Metric" H 8338 10100 50  0001 C CNN
+F 3 "~" H 8300 10250 50  0001 C CNN
+	1    8300 10250
+	1    0    0    -1
+$EndComp
+Wire Wire Line
+	8675 9900 8300 9900
+Wire Wire Line
+	8300 9900 8300 10100
+Connection ~ 8675 9900
+Wire Wire Line
+	8300 10400 8300 10700
+Wire Wire Line
+	8300 10700 9200 10700
+$Comp
+L Device:R R61
+U 1 1 5DC3C581
+P 9825 10400
+F 0 "R61" V 9618 10400 50  0000 C CNN
+F 1 "27" V 9709 10400 50  0000 C CNN
+F 2 "Resistor_SMD:R_0603_1608Metric" V 9755 10400 50  0001 C CNN
+F 3 "~" H 9825 10400 50  0001 C CNN
+	1    9825 10400
+	0    1    1    0
+$EndComp
+Wire Wire Line
+	9500 10400 9675 10400
+Text GLabel 10175 10400 2    50   Input ~ 0
+ADV_CECCLK
+Wire Wire Line
+	9975 10400 10175 10400
+Text Notes 8925 9625 0    50   ~ 0
+CEC Clock Generator
+Text Notes 4050 7675 0    50   ~ 0
+ESD protection IC
+Text Notes 1475 1575 0    50   ~ 0
+1V8 linear regulator
+Text Notes 13050 3700 0    50   ~ 0
+HDMI Plug
+$Comp
+L Device:R R?
+U 1 1 5DC70DAC
+P 3250 10075
+F 0 "R?" H 3320 10121 50  0000 L CNN
+F 1 "10k" H 3320 10030 50  0000 L CNN
+F 2 "Resistor_SMD:R_0603_1608Metric" V 3180 10075 50  0001 C CNN
+F 3 "~" H 3250 10075 50  0001 C CNN
+	1    3250 10075
+	1    0    0    -1
+$EndComp
+Wire Wire Line
+	3575 9825 3250 9825
+Wire Wire Line
+	3250 9925 3250 9825
+Connection ~ 3250 9825
+Wire Wire Line
+	3250 9825 2900 9825
+Text GLabel 3250 10225 3    50   Input ~ 0
+GND
 $EndSCHEMATC

Commit message: Added mounting holes.
Parts:
- gave numbers to parts that had none: 1
Changed lines of the file:
@@
 HDMI Plug
 $Comp
-L Device:R R?
+L Device:R R62
 U 1 1 5DC70DAC
 P 3250 10075
-F 0 "R?" H 3320 10121 50  0000 L CNN
+F 0 "R62" H 3320 10121 50  0000 L CNN
 F 1 "10k" H 3320 10030 50  0000 L CNN
 F 2 "Resistor_SMD:R_0603_1608Metric" V 3180 10075 50  0001 C CNN

Commit message: Changed zener diode footprint for easy soldering. Fixed pins, U861/2 and U761/2 they now connect correctly to ground.
Parts:
- C48: footprint Resistor_SMD:R_0603_1608Metric -> Capacitor_SMD:C_0603_1608Metric
Changed lines of the file:
@@
 EESchema Schematic File Version 4
-LIBS:qmtech-minimig-cache
 EELAYER 30 0
 EELAYER END
@@
 F 0 "C48" V 5173 8425 50  0000 C CNN
 F 1 "100nF" V 5264 8425 50  0000 C CNN
-F 2 "Resistor_SMD:R_0603_1608Metric" H 5463 8275 50  0001 C CNN
+F 2 "Capacitor_SMD:C_0603_1608Metric" H 5463 8275 50  0001 C CNN
 F 3 "~" H 5425 8425 50  0001 C CNN
 	1    5425 8425

Commit message: Fixed reversed labeling of the QMTECH FPGA board pins.
Connections:
- net labels removed: ADV_I2S2, ADV_I2S3
Changed lines of the file:
@@
 ADV_SCLK
 Text GLabel 6175 4375 0    50   Input ~ 0
-ADV_I2S3
+GND
 Text GLabel 6175 4275 0    50   Input ~ 0
-ADV_I2S2
+GND
 Text GLabel 6175 4175 0    50   Input ~ 0
 ADV_I2S1

Commit message: Change order of the VSPI to FPGA to make sure the clock pin connects to an FPGA clock capable pin.
Parts:
- 1V8: renamed from TP7; footprint TestPoint:TestPoint_Keystone_5019_Minature -> TestPoint:TestPoint_THTPad_1.0x1.0mm_Drill0.5mm
- 3V3: renamed from TP6; footprint TestPoint:TestPoint_Keystone_5019_Minature -> TestPoint:TestPoint_THTPad_1.0x1.0mm_Drill0.5mm
- GND2: renamed from TP5; value TestPoint -> GND; footprint TestPoint:TestPoint_Keystone_5019_Minature -> TestPoint:TestPoint_THTPad_1.0x1.0mm_Drill0.5mm
Changed lines of the file:
@@
 Connection ~ 1050 2725
 $Comp
-L Connector:TestPoint TP5
+L Connector:TestPoint GND2
 U 1 1 5DA4EE17
 P 1050 2725
-F 0 "TP5" H 1108 2843 50  0000 L CNN
-F 1 "TestPoint" H 1108 2752 50  0000 L CNN
-F 2 "TestPoint:TestPoint_Keystone_5019_Minature" H 1250 2725 50  0001 C CNN
+F 0 "GND2" H 1108 2843 50  0001 L CNN
+F 1 "GND" H 1108 2752 50  0000 L CNN
+F 2 "TestPoint:TestPoint_THTPad_1.0x1.0mm_Drill0.5mm" H 1250 2725 50  0001 C CNN
 F 3 "~" H 1250 2725 50  0001 C CNN
 	1    1050 2725
@@
 Connection ~ 1825 3875
 $Comp
-L Connector:TestPoint TP7
+L Connector:TestPoint 1V8
 U 1 1 5DA49C5B
 P 1825 3875
-F 0 "TP7" V 2020 3947 50  0000 C CNN
+F 0 "1V8" V 2020 3947 50  0000 C CNN
 F 1 "TestPoint" V 1929 3947 50  0000 C CNN
-F 2 "TestPoint:TestPoint_Keystone_5019_Minature" H 2025 3875 50  0001 C CNN
+F 2 "TestPoint:TestPoint_THTPad_1.0x1.0mm_Drill0.5mm" H 2025 3875 50  0001 C CNN
 F 3 "~" H 2025 3875 50  0001 C CNN
 	1    1825 3875
@@
 Connection ~ 1825 2000
 $Comp
-L Connector:TestPoint TP6
+L Connector:TestPoint 3V3
 U 1 1 5DA49761
 P 1825 2000
-F 0 "TP6" V 1779 2188 50  0000 L CNN
+F 0 "3V3" V 1779 2188 50  0000 L CNN
 F 1 "TestPoint" V 1870 2188 50  0000 L CNN
-F 2 "TestPoint:TestPoint_Keystone_5019_Minature" H 2025 2000 50  0001 C CNN
+F 2 "TestPoint:TestPoint_THTPad_1.0x1.0mm_Drill0.5mm" H 2025 2000 50  0001 C CNN
 F 3 "~" H 2025 2000 50  0001 C CNN
 	1    1825 2000

Commit message: Add 3d models to most components, Add decoupling of the Line ins of the max9850. Add new defeest Logos.
Parts:
- added TP1: TP_SCL, TestPoint:TestPoint_Pad_D1.0mm, symbol Connector:TestPoint
- added TP2: TP_SDA, TestPoint:TestPoint_Pad_D1.0mm, symbol Connector:TestPoint
- added TP3: TP_GND, TestPoint:TestPoint_Pad_D1.0mm, symbol Connector:TestPoint
Connections:
- wire segments 101 -> 103
Other:
- note added: "I2C Test points\n"
Changed lines of the file:
@@
 $EndComp
 Connection ~ 14100 7650
-Wire Wire Line
-	14100 7650 14700 7650
 Text GLabel 14100 7350 1    50   Input ~ 0
 3V3
@@
 	13700 8250 14100 8250
 Connection ~ 14100 8250
-Wire Wire Line
-	14100 8250 14700 8250
 NoConn ~ 12800 4600
 NoConn ~ 12800 4300
@@
 Text GLabel 3250 10225 3    50   Input ~ 0
 GND
+Text GLabel 14825 8475 0    50   Input ~ 0
+GND
+$Comp
+L Connector:TestPoint TP1
+U 1 1 5E5CEE84
+P 14825 8025
+F 0 "TP1" V 14779 8213 50  0000 L CNN
+F 1 "TP_SCL" V 14870 8213 50  0000 L CNN
+F 2 "TestPoint:TestPoint_Pad_D1.0mm" H 15025 8025 50  0001 C CNN
+F 3 "~" H 15025 8025 50  0001 C CNN
+	1    14825 8025
+	0    1    1    0
+$EndComp
+$Comp
+L Connector:TestPoint TP2
+U 1 1 5E5CF65D
+P 14825 8250
+F 0 "TP2" V 14779 8438 50  0000 L CNN
+F 1 "TP_SDA" V 14870 8438 50  0000 L CNN
+F 2 "TestPoint:TestPoint_Pad_D1.0mm" H 15025 8250 50  0001 C CNN
+F 3 "~" H 15025 8250 50  0001 C CNN
+	1    14825 8250
+	0    1    1    0
+$EndComp
+$Comp
+L Connector:TestPoint TP3
+U 1 1 5E5D2A3A
+P 14825 8475
+F 0 "TP3" V 14779 8663 50  0000 L CNN
+F 1 "TP_GND" V 14870 8663 50  0000 L CNN
+F 2 "TestPoint:TestPoint_Pad_D1.0mm" H 15025 8475 50  0001 C CNN
+F 3 "~" H 15025 8475 50  0001 C CNN
+	1    14825 8475
+	0    1    1    0
+$EndComp
+Wire Wire Line
+	14100 8250 14825 8250
+Wire Wire Line
+	14100 7650 14550 7650
+Text Notes 14800 7875 0    50   ~ 0
+I2C Test points\n
+Wire Wire Line
+	14825 8025 14550 8025
+Wire Wire Line
+	14550 8025 14550 7650
 $EndSCHEMATC
