File: hdmi_transmitter.sch (KiCad schematic (older format))
At the start: 50 parts, among them J9 47151-0001, U1 TPD12S520DBT, U3 LT1963AxST-1.8, X1 MCSJK-3N-16.00-3.3-50-B

Commit message: Did some placement to make the PCB smaller.
Parts:
- removed 1V8, 3V3: TestPoint, TestPoint:TestPoint_THTPad_1.0x1.0mm_Drill0.5mm, symbol Connector:TestPoint
- removed GND2: GND, TestPoint:TestPoint_THTPad_1.0x1.0mm_Drill0.5mm, symbol Connector:TestPoint
Connections:
- wire segments 103 -> 100
Changed lines of the file:
@@
-	0    1    1    0
-$EndComp
-Wire Wire Line
-	1050 2725 1425 2725
-Connection ~ 1050 2725
-$Comp
-L Connector:TestPoint GND2
-U 1 1 5DA4EE17
-P 1050 2725
-F 0 "GND2" H 1108 2843 50  0001 L CNN
-F 1 "GND" H 1108 2752 50  0000 L CNN
-F 2 "TestPoint:TestPoint_THTPad_1.0x1.0mm_Drill0.5mm" H 1250 2725 50  0001 C CNN
-F 3 "~" H 1250 2725 50  0001 C CNN
-	1    1050 2725
-	1    0    0    -1
-$EndComp
-Wire Wire Line
-	1000 2725 1050 2725
-Wire Wire Line
-	1825 3875 1825 3625
-Connection ~ 1825 3875
-$Comp
-L Connector:TestPoint 1V8
-U 1 1 5DA49C5B
-P 1825 3875
-F 0 "1V8" V 2020 3947 50  0000 C CNN
-F 1 "TestPoint" V 1929 3947 50  0000 C CNN
-F 2 "TestPoint:TestPoint_THTPad_1.0x1.0mm_Drill0.5mm" H 2025 3875 50  0001 C CNN
-F 3 "~" H 2025 3875 50  0001 C CNN
-	1    1825 3875
-	0    -1   -1   0
-$EndComp
-Wire Wire Line
-	1825 2000 1825 1825
-Connection ~ 1825 2000
-$Comp
-L Connector:TestPoint 3V3
-U 1 1 5DA49761
-P 1825 2000
-F 0 "3V3" V 1779 2188 50  0000 L CNN
-F 1 "TestPoint" V 1870 2188 50  0000 L CNN
-F 2 "TestPoint:TestPoint_THTPad_1.0x1.0mm_Drill0.5mm" H 2025 2000 50  0001 C CNN
-F 3 "~" H 2025 2000 50  0001 C CNN
-	1    1825 2000
 	0    1    1    0
 $EndComp
@@
 	2725 6925 2725 7025
 $Comp
-L Power:GND #PWR0102
+L power:GND #PWR0102
 U 1 1 5DD3B1BA
 P 2725 7025
@@
 	0    1    1    0
 $EndComp
-Wire Wire Line
-	1825 2125 1825 2000
 Connection ~ 1825 2125
 $Comp
@@
 Wire Wire Line
 	2725 3625 3725 3625
-Wire Wire Line
-	1825 4625 1825 3875
 Connection ~ 1825 4625
 Wire Wire Line
@@
 	2725 3925 2725 4025
 $Comp
-L Power:GND #PWR0109
+L power:GND #PWR0109
 U 1 1 5D6D859E
 P 2725 6025
@@
 $EndComp
 $Comp
-L Power:GND #PWR0108
+L power:GND #PWR0108
 U 1 1 5D6D8141
 P 2725 5025
@@
 $EndComp
 $Comp
-L Power:GND #PWR0107
+L power:GND #PWR0107
 U 1 1 5D6D7DC5
 P 2725 4025
@@
 Wire Wire Line
 	14550 8025 14550 7650
+Wire Wire Line
+	1825 3625 1825 4625
+Wire Wire Line
+	1000 2725 1425 2725
+Wire Wire Line
+	1825 1825 1825 2125
 $EndSCHEMATC

Commit message: First rough version of the Open AARS V4
Connections:
- net labels added: ADV_D0, ADV_D1, ADV_D10, ADV_D11, ADV_D2, ADV_D3, ADV_D4, ADV_D5, ADV_D6, ADV_D7, ADV_D8, ADV_D9
- net labels removed: ADV_B_0, ADV_B_1, ADV_B_2, ADV_B_3, ADV_B_4, ADV_B_5, ADV_B_6, ADV_B_7, ADV_CLK, ADV_G_0, ADV_G_1, ADV_G_2, ADV_G_3, ADV_G_4, ADV_G_5, ADV_G_6, ADV_G_7, ADV_R_0, ADV_R_1, ADV_R_2, ADV_R_3, ADV_R_4, ADV_R_5, ADV_R_6, ADV_R_7
Other:
- note added: "Input ID = 5, left aligned (R0x48[5] = 1) \n\n"
Changed lines of the file:
@@
 $EndComp
 NoConn ~ 8725 5825
-Text GLabel 9725 3975 2    50   Input ~ 0
-GND
-Text GLabel 9725 3875 2    50   Input ~ 0
-GND
-Text GLabel 9725 3775 2    50   Input ~ 0
-GND
-Text GLabel 9725 3675 2    50   Input ~ 0
+Text GLabel 9725 3575 2    50   Input ~ 0
+GND
+Text GLabel 9725 3475 2    50   Input ~ 0
+GND
+Text GLabel 9725 3375 2    50   Input ~ 0
+GND
+Text GLabel 9725 3275 2    50   Input ~ 0
 GND
 Text GLabel 8625 2425 1    50   Input ~ 0
@@
 Text GLabel 7325 5825 3    50   Input ~ 0
 ADV_TXC-
-Text GLabel 8825 2425 1    50   Input ~ 0
-ADV_CLK
-Text GLabel 7525 2425 1    50   Input ~ 0
-ADV_B_0
-Text GLabel 7625 2425 1    50   Input ~ 0
-ADV_B_1
-Text GLabel 7725 2425 1    50   Input ~ 0
-ADV_B_2
-Text GLabel 7825 2425 1    50   Input ~ 0
-ADV_B_3
-Text GLabel 7925 2425 1    50   Input ~ 0
-ADV_B_4
-Text GLabel 8025 2425 1    50   Input ~ 0
-ADV_B_5
-Text GLabel 8125 2425 1    50   Input ~ 0
-ADV_B_6
-Text GLabel 8225 2425 1    50   Input ~ 0
-ADV_B_7
-Text GLabel 8725 2425 1    50   Input ~ 0
-ADV_G_0
-Text GLabel 8925 2425 1    50   Input ~ 0
-ADV_G_1
-Text GLabel 9725 3075 2    50   Input ~ 0
-ADV_G_2
-Text GLabel 9725 3175 2    50   Input ~ 0
-ADV_G_3
-Text GLabel 9725 3275 2    50   Input ~ 0
-ADV_G_4
-Text GLabel 9725 3375 2    50   Input ~ 0
-ADV_G_5
-Text GLabel 9725 3475 2    50   Input ~ 0
-ADV_G_6
-Text GLabel 9725 3575 2    50   Input ~ 0
-ADV_G_7
-Text GLabel 9725 4075 2    50   Input ~ 0
-ADV_R_0
 Text GLabel 9725 4175 2    50   Input ~ 0
-ADV_R_1
+ADV_D5
 Text GLabel 9725 4275 2    50   Input ~ 0
-ADV_R_2
+ADV_D6
 Text GLabel 9725 4375 2    50   Input ~ 0
-ADV_R_3
+ADV_D7
 Text GLabel 9725 4475 2    50   Input ~ 0
-ADV_R_4
+ADV_D8
 Text GLabel 9725 4575 2    50   Input ~ 0
-ADV_R_5
+ADV_D9
 Text GLabel 9725 4675 2    50   Input ~ 0
-ADV_R_6
+ADV_D10
 Text GLabel 9725 4775 2    50   Input ~ 0
-ADV_R_7
+ADV_D11
 Text GLabel 1000 2725 0    50   Input ~ 0
 GND
@@
 Wire Wire Line
 	1825 1825 1825 2125
+Text GLabel 9725 3175 2    50   Input ~ 0
+GND
+Text GLabel 9725 3075 2    50   Input ~ 0
+GND
+Text GLabel 8025 2425 1    50   Input ~ 0
+GND
+Text GLabel 7925 2425 1    50   Input ~ 0
+GND
+Text GLabel 7825 2425 1    50   Input ~ 0
+GND
+Text GLabel 7725 2425 1    50   Input ~ 0
+GND
+Text GLabel 7625 2425 1    50   Input ~ 0
+GND
+Text GLabel 7525 2425 1    50   Input ~ 0
+GND
+Text GLabel 8925 2425 1    50   Input ~ 0
+GND
+Text GLabel 8825 2425 1    50   Input ~ 0
+GND
+Text GLabel 8725 2425 1    50   Input ~ 0
+GND
+Text GLabel 8225 2425 1    50   Input ~ 0
+GND
+Text GLabel 8125 2425 1    50   Input ~ 0
+GND
+Text GLabel 9725 3675 2    50   Input ~ 0
+ADV_D0
+Text GLabel 9725 3775 2    50   Input ~ 0
+ADV_D1
+Text GLabel 9725 3975 2    50   Input ~ 0
+ADV_D3
+Text GLabel 9725 4075 2    50   Input ~ 0
+ADV_D4
+Text Notes 7300 4350 0    50   ~ 0
+Input ID = 5, left aligned (R0x48[5] = 1) \n\n
+Text GLabel 9725 3875 2    50   Input ~ 0
+ADV_D2
 $EndSCHEMATC

Commit message: Fixed issues with V4 board, length matching, region matching, footprints, symbols.
Connections:
- net labels added: ADV_CLK
Changed lines of the file:
@@
 Text GLabel 8925 2425 1    50   Input ~ 0
-GND
-Text GLabel 8825 2425 1    50   Input ~ 0
 GND
 Text GLabel 8725 2425 1    50   Input ~ 0
@@
 Text GLabel 9725 3875 2    50   Input ~ 0
 ADV_D2
+Text GLabel 8825 2425 1    50   Input ~ 0
+ADV_CLK
 $EndSCHEMATC

Commit message: Brought compenents back to the front for easy soldering.
Parts:
- removed C49: 100nF, Capacitor_SMD:C_0603_1608Metric, symbol Device:C
- removed R60: 10k, Resistor_SMD:R_0603_1608Metric, symbol Device:R
- removed R61: 27, Resistor_SMD:R_0603_1608Metric, symbol Device:R
- removed X1: MCSJK-3N-16.00-3.3-50-B, Oscillator:Oscillator_SMD_Abracon_ASE-4Pin_3.2x2.5mm, symbol Oscillator:ASE-xxxMHz
Connections:
- wire segments 100 -> 90
Other:
- note removed: "CEC Clock Generator"
Changed lines of the file:
@@
 Wire Wire Line
 	1825 5625 1825 6625
-Text GLabel 3725 6625 2    50   Input ~ 0
-ADV_BGVDD
 Connection ~ 2725 6625
 Wire Wire Line
@@
 Text GLabel 2500 8725 1    50   Input ~ 0
 3V3
-$Comp
-L Oscillator:ASE-xxxMHz X1
-U 1 1 5DC2E9FD
-P 9200 10400
-F 0 "X1" H 9544 10446 50  0000 L CNN
-F 1 "MCSJK-3N-16.00-3.3-50-B" H 8775 10750 50  0000 L CNN
-F 2 "Oscillator:Oscillator_SMD_Abracon_ASE-4Pin_3.2x2.5mm" H 9900 10050 50  0001 C CNN
-F 3 "http://www.farnell.com/datasheets/2864171.pdf" H 9100 10400 50  0001 C CNN
-	1    9200 10400
-	1    0    0    -1
-$EndComp
-$Comp
-L Device:R R60
-U 1 1 5DC3073E
-P 8675 10250
-F 0 "R60" H 8745 10296 50  0000 L CNN
-F 1 "10k" H 8745 10205 50  0000 L CNN
-F 2 "Resistor_SMD:R_0603_1608Metric" V 8605 10250 50  0001 C CNN
-F 3 "~" H 8675 10250 50  0001 C CNN
-	1    8675 10250
-	1    0    0    -1
-$EndComp
-Wire Wire Line
-	8900 10400 8675 10400
-Wire Wire Line
-	8675 10100 8675 9900
-Wire Wire Line
-	8675 9900 9200 9900
-Wire Wire Line
-	9200 9900 9200 10100
-Text GLabel 9200 9900 1    50   Input ~ 0
-3V3
-Text GLabel 9200 10700 3    50   Input ~ 0
-GND
-$Comp
-L Device:C C49
-U 1 1 5DC368A8
-P 8300 10250
-F 0 "C49" H 8415 10296 50  0000 L CNN
-F 1 "100nF" H 8415 10205 50  0000 L CNN
-F 2 "Capacitor_SMD:C_0603_1608Metric" H 8338 10100 50  0001 C CNN
-F 3 "~" H 8300 10250 50  0001 C CNN
-	1    8300 10250
-	1    0    0    -1
-$EndComp
-Wire Wire Line
-	8675 9900 8300 9900
-Wire Wire Line
-	8300 9900 8300 10100
-Connection ~ 8675 9900
-Wire Wire Line
-	8300 10400 8300 10700
-Wire Wire Line
-	8300 10700 9200 10700
-$Comp
-L Device:R R61
-U 1 1 5DC3C581
-P 9825 10400
-F 0 "R61" V 9618 10400 50  0000 C CNN
-F 1 "27" V 9709 10400 50  0000 C CNN
-F 2 "Resistor_SMD:R_0603_1608Metric" V 9755 10400 50  0001 C CNN
-F 3 "~" H 9825 10400 50  0001 C CNN
-	1    9825 10400
-	0    1    1    0
-$EndComp
-Wire Wire Line
-	9500 10400 9675 10400
-Text GLabel 10175 10400 2    50   Input ~ 0
-ADV_CECCLK
-Wire Wire Line
-	9975 10400 10175 10400
-Text Notes 8925 9625 0    50   ~ 0
-CEC Clock Generator
 Text Notes 4050 7675 0    50   ~ 0
 ESD protection IC
@@
 Text GLabel 8825 2425 1    50   Input ~ 0
 ADV_CLK
+Text GLabel 3725 6625 2    50   Input ~ 0
+ADV_BGVDD
 $EndSCHEMATC

Commit message: Removed ESP32, as it's no longer needed, we have soft cores.
Parts:
- renumbered C23 to C10, C31 to C11, C32 to C12, C33 to C13, C48 to C14, C34 to C15, C35 to C16, C36 to C17, C40 to C18, C41 to C19, C37 to C20, C1 to C21, C38 to C22, C39 to C23, C29 to C6, C30 to C7, C21 to C8, C22 to C9, D30 to D3, J9 to J2, R58 to R10, R42 to R11, R56 to R12, R18 to R13, R19 to R14, R34 to R15, R43 to R16, R59 to R4, R62 to R5, R57 to R6, R55 to R7, R41 to R8, R54 to R9, U3 to U2, U1 to U3

Commit message: open changes.
Parts:
- removed TP1: TP_SCL, TestPoint:TestPoint_Pad_D1.0mm, symbol Connector:TestPoint
- removed TP2: TP_SDA, TestPoint:TestPoint_Pad_D1.0mm, symbol Connector:TestPoint
- removed TP3: TP_GND, TestPoint:TestPoint_Pad_D1.0mm, symbol Connector:TestPoint
- added J10: Conn_01x03, Connector_PinHeader_2.54mm:PinHeader_1x03_P2.54mm_Vertical, symbol Connector_Generic:Conn_01x03
Changed lines of the file:
@@
 Text GLabel 3250 10225 3    50   Input ~ 0
 GND
-Text GLabel 14825 8475 0    50   Input ~ 0
+Text GLabel 14825 8050 0    50   Input ~ 0
 GND
-$Comp
-L Connector:TestPoint TP1
-U 1 1 5E5CEE84
-P 14825 8025
-F 0 "TP1" V 14779 8213 50  0000 L CNN
-F 1 "TP_SCL" V 14870 8213 50  0000 L CNN
-F 2 "TestPoint:TestPoint_Pad_D1.0mm" H 15025 8025 50  0001 C CNN
-F 3 "~" H 15025 8025 50  0001 C CNN
-	1    14825 8025
-	0    1    1    0
-$EndComp
-$Comp
-L Connector:TestPoint TP2
-U 1 1 5E5CF65D
-P 14825 8250
-F 0 "TP2" V 14779 8438 50  0000 L CNN
-F 1 "TP_SDA" V 14870 8438 50  0000 L CNN
-F 2 "TestPoint:TestPoint_Pad_D1.0mm" H 15025 8250 50  0001 C CNN
-F 3 "~" H 15025 8250 50  0001 C CNN
-	1    14825 8250
-	0    1    1    0
-$EndComp
-$Comp
-L Connector:TestPoint TP3
-U 1 1 5E5D2A3A
-P 14825 8475
-F 0 "TP3" V 14779 8663 50  0000 L CNN
-F 1 "TP_GND" V 14870 8663 50  0000 L CNN
-F 2 "TestPoint:TestPoint_Pad_D1.0mm" H 15025 8475 50  0001 C CNN
-F 3 "~" H 15025 8475 50  0001 C CNN
-	1    14825 8475
-	0    1    1    0
-$EndComp
 Wire Wire Line
 	14100 8250 14825 8250
@@
 I2C Test points\n
 Wire Wire Line
-	14825 8025 14550 8025
+	14825 8150 14550 8150
 Wire Wire Line
-	14550 8025 14550 7650
+	14550 8150 14550 7650
 Wire Wire Line
 	1825 3625 1825 4625
@@
 Text GLabel 3725 6625 2    50   Input ~ 0
 ADV_BGVDD
+$Comp
+L Connector_Generic:Conn_01x03 J10
+U 1 1 5FA8F41B
+P 15025 8150
+F 0 "J10" H 15105 8192 50  0000 L CNN
+F 1 "Conn_01x03" H 15105 8101 50  0000 L CNN
+F 2 "Connector_PinHeader_2.54mm:PinHeader_1x03_P2.54mm_Vertical" H 15025 8150 50  0001 C CNN
+F 3 "~" H 15025 8150 50  0001 C CNN
+	1    15025 8150
+	1    0    0    -1
+$EndComp
 $EndSCHEMATC

Commit message: Connect I2S to both Max9850 and ADV7511.
Connections:
- net labels added: MAX_I2S0, MAX_LRCLK, MAX_SCLK
- net labels removed: ADV_I2S0, ADV_I2S1, ADV_LRCLK, ADV_SCLK
Changed lines of the file:
@@
 ADV_CECCLK
 Text GLabel 6175 4575 0    50   Input ~ 0
-ADV_LRCLK
+MAX_LRCLK
 Text GLabel 6175 4475 0    50   Input ~ 0
-ADV_SCLK
+MAX_SCLK
 Text GLabel 6175 4375 0    50   Input ~ 0
 GND
 Text GLabel 6175 4275 0    50   Input ~ 0
 GND
-Text GLabel 6175 4175 0    50   Input ~ 0
-ADV_I2S1
 Text GLabel 6175 4075 0    50   Input ~ 0
-ADV_I2S0
+MAX_I2S0
 Text GLabel 9725 4975 2    50   Input ~ 0
 ADV_SCL
@@
 	1    0    0    -1
 $EndComp
+Text GLabel 6175 4175 0    50   Input ~ 0
+GND
 $EndSCHEMATC

Commit message: Fixed issue with missing PS2 pullups, add line to adv interrupt.
Connections:
- no-connect marks 6 -> 2
Changed lines of the file:
@@
 	13700 8250 14100 8250
 Connection ~ 14100 8250
-NoConn ~ 12800 4600
-NoConn ~ 12800 4300
-NoConn ~ 13700 4100
-NoConn ~ 13700 4400
 NoConn ~ 13700 4700
 $Comp
@@
 Text GLabel 6175 4175 0    50   Input ~ 0
 GND
+Text GLabel 12800 4300 0    50   Input ~ 0
+GND
+Text GLabel 13700 4400 2    50   Input ~ 0
+GND
+Text GLabel 13700 4100 2    50   Input ~ 0
+GND
+Text GLabel 12800 4600 0    50   Input ~ 0
+GND
 $EndSCHEMATC
