File: qmtech-minimig.kicad_pcb (KiCad board)
At the start: 4 copper layers, 142.2 x 105.7 mm, 189 parts, among them IC1 ESP32-WROVER-B_(16MB), J1 DB9_Male, J10 DB23_Female_MountingHoles, J11 Conn_01x03_Male, J2 DB9_Male, J3 SCHA5B0200, J4 10118193-0001LF, J5 AUDIO-CONNECTOR-6P-SMD-344003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, J6 Mini-DIN-6, J7 Conn_02x13_Odd_Even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

Commit message: Renamed some values for consistency
Parts:
- C12: value 100n -> 100nF
- C27, C28: value 4700pF -> 4.7uF
- C47: value 10n -> 10nF
- D28, D29: value 3.6V -> D_Zener 3.6V BZT52C395
- R1, R10, R11, R12, R13, R14, R15, R16, R2, R3, R4, R5, R6, R7, R8, R9: value 47K -> 47k
- R17, R33: value 10K -> 10k
- R28, R29: value 3.3K -> 3.3k
- R41, R54, R55, R58: value 2K -> 2k
Changed lines of the file:
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@@
       (effects (font (size 1 1) (thickness 0.15)))
     )
-    (fp_text value 47K (at 0 1.43) (layer F.Fab)
+    (fp_text value 47k (at 0 1.43) (layer F.Fab)
       (effects (font (size 1 1) (thickness 0.15)))
     )
@@
       (effects (font (size 1 1) (thickness 0.15)))
     )
-    (fp_text value 47K (at 0 1.43) (layer F.Fab)
+    (fp_text value 47k (at 0 1.43) (layer F.Fab)
       (effects (font (size 1 1) (thickness 0.15)))
     )
@@
       (effects (font (size 1 1) (thickness 0.15)))
     )
-    (fp_text value 47K (at 0 1.43) (layer F.Fab)
+    (fp_text value 47k (at 0 1.43) (layer F.Fab)
       (effects (font (size 1 1) (thickness 0.15)))
     )
@@
       (effects (font (size 1 1) (thickness 0.15)))
     )
-    (fp_text value 47K (at 0 1.43) (layer F.Fab)
+    (fp_text value 47k (at 0 1.43) (layer F.Fab)
       (effects (font (size 1 1) (thickness 0.15)))
     )
@@
       (effects (font (size 1 1) (thickness 0.15)))
     )
-    (fp_text value 47K (at 0 1.43) (layer F.Fab)
+    (fp_text value 47k (at 0 1.43) (layer F.Fab)
       (effects (font (size 1 1) (thickness 0.15)))
     )
@@
       (effects (font (size 1 1) (thickness 0.15)))
     )
-    (fp_text value 47K (at 0 1.43) (layer F.Fab)
+    (fp_text value 47k (at 0 1.43) (layer F.Fab)
       (effects (font (size 1 1) (thickness 0.15)))
     )
@@
       (effects (font (size 1 1) (thickness 0.15)))
     )
-    (fp_text value 47K (at 0 1.43) (layer F.Fab)
+    (fp_text value 47k (at 0 1.43) (layer F.Fab)
       (effects (font (size 1 1) (thickness 0.15)))
     )
@@
       (effects (font (size 1 1) (thickness 0.15)))
     )
-    (fp_text value 47K (at 0 1.43) (layer F.Fab)
+    (fp_text value 47k (at 0 1.43) (layer F.Fab)
       (effects (font (size 1 1) (thickness 0.15)))
     )
@@
       (effects (font (size 1 1) (thickness 0.15)))
     )
-    (fp_text value 47K (at 0 1.43) (layer F.Fab)
+    (fp_text value 47k (at 0 1.43) (layer F.Fab)
       (effects (font (size 1 1) (thickness 0.15)))
     )
@@
       (effects (font (size 1 1) (thickness 0.15)))
     )
-    (fp_text value 47K (at 0 1.43) (layer F.Fab)
+    (fp_text value 47k (at 0 1.43) (layer F.Fab)
       (effects (font (size 1 1) (thickness 0.15)))
     )
@@
       (effects (font (size 1 1) (thickness 0.15)))
     )
-    (fp_text value 47K (at 0 1.43) (layer F.Fab)
+    (fp_text value 47k (at 0 1.43) (layer F.Fab)
       (effects (font (size 1 1) (thickness 0.15)))
     )
@@
       (effects (font (size 1 1) (thickness 0.15)))
     )
-    (fp_text value 47K (at 0 1.43) (layer F.Fab)
+    (fp_text value 47k (at 0 1.43) (layer F.Fab)
       (effects (font (size 1 1) (thickness 0.15)))
     )
@@
       (effects (font (size 1 1) (thickness 0.15)))
     )
-    (fp_text value 47K (at 0 1.43) (layer F.Fab)
+    (fp_text value 47k (at 0 1.43) (layer F.Fab)
       (effects (font (size 1 1) (thickness 0.15)))
     )
@@
       (effects (font (size 1 1) (thickness 0.15)))
     )
-    (fp_text value 47K (at 0 1.43) (layer F.Fab)
+    (fp_text value 47k (at 0 1.43) (layer F.Fab)
       (effects (font (size 1 1) (thickness 0.15)))
     )
@@
       (effects (font (size 1 1) (thickness 0.15)))
     )
-    (fp_text value 47K (at 0 1.43) (layer F.Fab)
+    (fp_text value 47k (at 0 1.43) (layer F.Fab)
       (effects (font (size 1 1) (thickness 0.15)))
     )
@@
       (effects (font (size 1 1) (thickness 0.15)))
     )
-    (fp_text value 47K (at 0 1.43) (layer F.Fab)
+    (fp_text value 47k (at 0 1.43) (layer F.Fab)
       (effects (font (size 1 1) (thickness 0.15)))
     )
@@
       (effects (font (size 1 1) (thickness 0.15)))
     )
-    (fp_text value 2K (at 0 1.43) (layer F.Fab)
+    (fp_text value 2k (at 0 1.43) (layer F.Fab)
       (effects (font (size 1 1) (thickness 0.15)))
     )
@@
       (effects (font (size 1 1) (thickness 0.15)))
     )
-    (fp_text value 2K (at 0 1.43) (layer F.Fab)
+    (fp_text value 2k (at 0 1.43) (layer F.Fab)
       (effects (font (size 1 1) (thickness 0.15)))
     )
@@
       (effects (font (size 1 1) (thickness 0.15)))
     )
-    (fp_text value 10n (at 0 1.43) (layer F.Fab)
+    (fp_text value 10nF (at 0 1.43) (layer F.Fab)
       (effects (font (size 1 1) (thickness 0.15)))
     )
@@
       (effects (font (size 1 1) (thickness 0.15)))
     )
-    (fp_text value 2K (at 0 1.43 45) (layer F.Fab)
+    (fp_text value 2k (at 0 1.43 45) (layer F.Fab)
       (effects (font (size 1 1) (thickness 0.15)))
     )
@@
       (effects (font (size 1 1) (thickness 0.15)))
     )
-    (fp_text value 4700pF (at 0 1.65) (layer F.Fab)
+    (fp_text value 4.7uF (at 0 1.65) (layer F.Fab)
       (effects (font (size 1 1) (thickness 0.15)))
     )
@@
       (effects (font (size 1 1) (thickness 0.15)))
     )
-    (fp_text value 4700pF (at 5.292499 -0.0812) (layer F.Fab)
+    (fp_text value 4.7uF (at 5.292499 -0.0812) (layer F.Fab)
       (effects (font (size 1 1) (thickness 0.15)))
     )
@@
       (effects (font (size 1 1) (thickness 0.15)))
     )
-    (fp_text value 10K (at 0 1.43 90) (layer F.Fab)
+    (fp_text value 10k (at 0 1.43 90) (layer F.Fab)
       (effects (font (size 1 1) (thickness 0.15)))
     )
@@
       (effects (font (size 1 1) (thickness 0.15)))
     )
-    (fp_text value 100n (at 0 1.43 90) (layer F.Fab)
+    (fp_text value 100nF (at 0 1.43 90) (layer F.Fab)
       (effects (font (size 1 1) (thickness 0.15)))
     )
@@
       (effects (font (size 1 1) (thickness 0.15)))
     )
-    (fp_text value 10K (at 0 1.43 90) (layer F.Fab)
+    (fp_text value 10k (at 0 1.43 90) (layer F.Fab)
       (effects (font (size 1 1) (thickness 0.15)))
     )
@@
       (effects (font (size 1 1) (thickness 0.15)))
     )
-    (fp_text value 3.6V (at 0.1 1.9) (layer F.Fab)
+    (fp_text value "D_Zener 3.6V BZT52C395" (at 0.1 1.9) (layer F.Fab)
       (effects (font (size 1 1) (thickness 0.15)))
     )
@@
       (effects (font (size 1 1) (thickness 0.15)))
     )
-    (fp_text value 3.6V (at 0.1 1.9) (layer F.Fab)
+    (fp_text value "D_Zener 3.6V BZT52C395" (at 0.1 1.9) (layer F.Fab)
       (effects (font (size 1 1) (thickness 0.15)))
     )
@@
       (effects (font (size 1 1) (thickness 0.15)) (justify mirror))
     )
-    (fp_text value 2K (at 2.500546 -1.732412 135) (layer B.Fab)
+    (fp_text value 2k (at 2.500546 -1.732412 135) (layer B.Fab)
       (effects (font (size 1 1) (thickness 0.15)) (justify mirror))
     )
@@
       (effects (font (size 1 1) (thickness 0.15)))
     )
-    (fp_text value 3.3K (at 3.2765 0) (layer F.Fab)
+    (fp_text value 3.3k (at 3.2765 0) (layer F.Fab)
       (effects (font (size 1 1) (thickness 0.15)))
     )
@@
       (effects (font (size 1 1) (thickness 0.15)))
     )
-    (fp_text value 3.3K (at 3.0225 0) (layer F.Fab)
+    (fp_text value 3.3k (at 3.0225 0) (layer F.Fab)
       (effects (font (size 1 1) (thickness 0.15)))
     )

Commit message: LEDs
Parts:
- D1, D2: value GREEN -> LED
- D10: value LED0 -> LED
- D11, D6: value LED4 -> LED
- D4, D5: value LED5 -> LED
- D7: value LED3 -> LED
- D8: value LED2 -> LED
- D9: value LED1 -> LED
Changed lines of the file:
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@@
       (effects (font (size 1 1) (thickness 0.15)))
     )
-    (fp_text value LED4 (at 0 1.43 90) (layer F.Fab)
+    (fp_text value LED (at 0 1.43 90) (layer F.Fab)
       (effects (font (size 1 1) (thickness 0.15)))
     )
@@
       (effects (font (size 1 1) (thickness 0.15)))
     )
-    (fp_text value LED5 (at 0 1.43 90) (layer F.Fab)
+    (fp_text value LED (at 0 1.43 90) (layer F.Fab)
       (effects (font (size 1 1) (thickness 0.15)))
     )
@@
       (effects (font (size 1 1) (thickness 0.15)))
     )
-    (fp_text value GREEN (at 0 1.43 90) (layer F.Fab) hide
+    (fp_text value LED (at 0 1.43 90) (layer F.Fab) hide
       (effects (font (size 1 1) (thickness 0.15)))
     )
@@
       (effects (font (size 1 1) (thickness 0.15)))
     )
-    (fp_text value GREEN (at 0 1.43 90) (layer F.Fab) hide
+    (fp_text value LED (at 0 1.43 90) (layer F.Fab) hide
       (effects (font (size 1 1) (thickness 0.15)))
     )
@@
       (effects (font (size 1 1) (thickness 0.15)))
     )
-    (fp_text value LED0 (at 3.3 0.1) (layer F.SilkS)
+    (fp_text value LED (at 3.3 0.1) (layer F.SilkS)
       (effects (font (size 1 1) (thickness 0.15)))
     )
@@
       (effects (font (size 1 1) (thickness 0.15)))
     )
-    (fp_text value LED1 (at 3.3 0.1) (layer F.SilkS)
+    (fp_text value LED (at 3.3 0.1) (layer F.SilkS)
       (effects (font (size 1 1) (thickness 0.15)))
     )
@@
       (effects (font (size 1 1) (thickness 0.15)))
     )
-    (fp_text value LED2 (at 3.3125 0.1) (layer F.SilkS)
+    (fp_text value LED (at 3.3125 0.1) (layer F.SilkS)
       (effects (font (size 1 1) (thickness 0.15)))
     )
@@
       (effects (font (size 1 1) (thickness 0.15)))
     )
-    (fp_text value LED3 (at 3.404999 0.104999) (layer F.SilkS)
+    (fp_text value LED (at 3.404999 0.104999) (layer F.SilkS)
       (effects (font (size 1 1) (thickness 0.15)))
     )
@@
       (effects (font (size 1 1) (thickness 0.15)))
     )
-    (fp_text value LED4 (at 3.4 0) (layer F.SilkS)
+    (fp_text value LED (at 3.4 0) (layer F.SilkS)
       (effects (font (size 1 1) (thickness 0.15)))
     )
@@
       (effects (font (size 1 1) (thickness 0.15)))
     )
-    (fp_text value LED5 (at 3.5 0) (layer F.SilkS)
+    (fp_text value LED (at 3.5 0) (layer F.SilkS)
       (effects (font (size 1 1) (thickness 0.15)))
     )
