File: main_board.sch (KiCad schematic (older format))
At the start: 13 parts, among them U2 QM_XC7A35T_DDR3

Commit message: Integrated the Rover V2 into the board, added level shifters for the floppy interface.
Connections:
- net labels removed: EXP_06, EXP_14
Changed lines of the file:
@@
 Text GLabel 3450 4250 2    50   Input ~ 0
 EXP_04
-Text GLabel 3450 4350 2    50   Input ~ 0
+Text GLabel 1850 4350 0    50   Input ~ 0
 EXP_08
-Text GLabel 1850 4350 0    50   Input ~ 0
-EXP_06
 Text GLabel 1850 4450 0    50   Input ~ 0
-EXP_10
+EXP_12
 Text GLabel 3450 4450 2    50   Input ~ 0
-EXP_12
-Text GLabel 1850 4550 0    50   Input ~ 0
-EXP_14
+EXP_16
 Text GLabel 3450 4550 2    50   Input ~ 0
-EXP_16
-Text GLabel 1850 4650 0    50   Input ~ 0
-EXP_18
+EXP_20
 Text GLabel 3450 4650 2    50   Input ~ 0
-EXP_20
-Text GLabel 1850 4750 0    50   Input ~ 0
-EXP_22
-Text GLabel 3450 4750 2    50   Input ~ 0
 EXP_24
 $Comp
@@
 	1    0    0    -1
 $EndComp
+Text GLabel 3450 4750 2    50   Input ~ 0
+EXP_28
+Text GLabel 3450 4850 2    50   Input ~ 0
+EXP_32
 Text GLabel 1850 4850 0    50   Input ~ 0
+EXP_30
+Text GLabel 1850 4950 0    50   Input ~ 0
+EXP_34
+Text GLabel 1850 4750 0    50   Input ~ 0
 EXP_26
-Text GLabel 3450 4850 2    50   Input ~ 0
-EXP_28
-Text GLabel 3450 4950 2    50   Input ~ 0
-EXP_32
-Text GLabel 1850 4950 0    50   Input ~ 0
-EXP_30
-Text GLabel 1850 5050 0    50   Input ~ 0
-EXP_34
+Text GLabel 1850 4650 0    50   Input ~ 0
+EXP_22
+Text GLabel 1850 4550 0    50   Input ~ 0
+EXP_18
+Text GLabel 3450 4350 2    50   Input ~ 0
+EXP_10
 $EndSCHEMATC

Commit message: Add the External floppy interface. Routed the HDMI tracks + match impendence.
Connections:
- net labels added: EXP_35
Changed lines of the file:
@@
 Text GLabel 3450 4350 2    50   Input ~ 0
 EXP_10
+Text GLabel 3450 4950 2    50   Input ~ 0
+EXP_35
 $EndSCHEMATC

Commit message: Fixed HDMI Impedance to 50Ohm, 100Ohm differential, for 0.1mm bord. Add pullups to HDMI I2C, connected DE pin to FPGA.
Connections:
- net labels added: ADV_DE, ESP_VSPI_CLK, ESP_VSPI_CS, ESP_VSPI_MISO, ESP_VSPI_MOSI
- net labels removed: ESP_UART1_RX, ESP_UART1_TX, STM_IO_33, STM_IO_34, STM_SPI1_CS, STM_SPI1_MISO, STM_SPI1_MOSI, STM_SPI1_NSS, STM_SPI1_SCK, STM_USART1_CK, STM_USART1_CTS, STM_USART1_RTS, STM_USART1_RX, STM_USART1_TX
Changed lines of the file:
@@
 Text GLabel 8350 5350 0    50   Input ~ 0
 VIN5V
-Text GLabel 8350 2750 0    50   Input ~ 0
+Text GLabel 8350 2850 0    50   Input ~ 0
 ADV_B_0
-Text GLabel 8350 2850 0    50   Input ~ 0
+Text GLabel 8350 2950 0    50   Input ~ 0
 ADV_B_1
-Text GLabel 8350 2950 0    50   Input ~ 0
+Text GLabel 8350 3050 0    50   Input ~ 0
 ADV_B_2
-Text GLabel 8350 3050 0    50   Input ~ 0
+Text GLabel 8350 3150 0    50   Input ~ 0
 ADV_B_3
-Text GLabel 8350 3150 0    50   Input ~ 0
+Text GLabel 8350 3250 0    50   Input ~ 0
 ADV_B_4
-Text GLabel 8350 3250 0    50   Input ~ 0
+Text GLabel 8350 3350 0    50   Input ~ 0
 ADV_B_5
-Text GLabel 8350 3350 0    50   Input ~ 0
+Text GLabel 8350 3450 0    50   Input ~ 0
 ADV_B_6
-Text GLabel 8350 3450 0    50   Input ~ 0
+Text GLabel 8350 3550 0    50   Input ~ 0
 ADV_B_7
 Text GLabel 8350 2550 0    50   Input ~ 0
@@
 Text GLabel 3450 2550 2    50   Input ~ 0
 ADV_R_7
-Text GLabel 8350 3550 0    50   Input ~ 0
+Text GLabel 8350 3650 0    50   Input ~ 0
 ADV_G_0
-Text GLabel 8350 3650 0    50   Input ~ 0
+Text GLabel 8350 3750 0    50   Input ~ 0
 ADV_CLK
-Text GLabel 8350 3750 0    50   Input ~ 0
+Text GLabel 8350 3850 0    50   Input ~ 0
 ADV_G_1
 Text GLabel 9950 2550 2    50   Input ~ 0
@@
 Text GLabel 9950 4350 2    50   Input ~ 0
 JS2_1
-Text GLabel 1850 3650 0    50   Input ~ 0
-STM_SPI1_CS
-Text GLabel 1850 3550 0    50   Input ~ 0
-STM_SPI1_NSS
-Text GLabel 1850 3450 0    50   Input ~ 0
-STM_SPI1_SCK
-Text GLabel 1850 3350 0    50   Input ~ 0
-STM_SPI1_MISO
-Text GLabel 1850 3250 0    50   Input ~ 0
-STM_SPI1_MOSI
-Text GLabel 1850 2550 0    50   Input ~ 0
-STM_USART1_RTS
-Text GLabel 1850 2650 0    50   Input ~ 0
-STM_USART1_CTS
-Text GLabel 1850 2750 0    50   Input ~ 0
-STM_USART1_RX
-Text GLabel 1850 2850 0    50   Input ~ 0
-STM_USART1_TX
-Text GLabel 1850 2950 0    50   Input ~ 0
-STM_USART1_CK
 $Comp
 L Device:LED D?
@@
 Wire Wire Line
 	3350 6000 3350 6200
-Text GLabel 8350 3850 0    50   Input ~ 0
+Text GLabel 8350 3950 0    50   Input ~ 0
 ADV_I2S0
-Text GLabel 8350 3950 0    50   Input ~ 0
+Text GLabel 8350 4050 0    50   Input ~ 0
 ADV_I2S1
-Text GLabel 8350 4050 0    50   Input ~ 0
+Text GLabel 8350 4150 0    50   Input ~ 0
 ADV_I2S2
-Text GLabel 8350 4150 0    50   Input ~ 0
+Text GLabel 8350 4250 0    50   Input ~ 0
 ADV_I2S3
 Text GLabel 3450 3950 2    50   Input ~ 0
@@
 Text GLabel 3450 4050 2    50   Input ~ 0
 ADV_SDA
-Text GLabel 8350 4250 0    50   Input ~ 0
+Text GLabel 8350 4350 0    50   Input ~ 0
 ADV_SCLK
-Text GLabel 8350 4350 0    50   Input ~ 0
+Text GLabel 8350 4450 0    50   Input ~ 0
 ADV_LRCLK
-Text GLabel 8350 4450 0    50   Input ~ 0
+Text GLabel 8350 4550 0    50   Input ~ 0
 ADV_INT
-Text GLabel 1850 3150 0    50   Input ~ 0
-STM_IO_33
-Text GLabel 1850 3050 0    50   Input ~ 0
-STM_IO_34
-Text GLabel 1850 4150 0    50   Input ~ 0
-ESP_UART1_RX
-Text GLabel 1850 4250 0    50   Input ~ 0
-ESP_UART1_TX
 NoConn ~ 9950 3350
 NoConn ~ 9950 3450
@@
 Text GLabel 3450 4950 2    50   Input ~ 0
 EXP_35
+Text GLabel 1850 2850 0    50   Input ~ 0
+ESP_VSPI_CLK
+Text GLabel 1850 2950 0    50   Input ~ 0
+ESP_VSPI_MISO
+Text GLabel 1850 3050 0    50   Input ~ 0
+ESP_VSPI_MOSI
+Text GLabel 1850 3150 0    50   Input ~ 0
+ESP_VSPI_CS
+Text GLabel 8350 2750 0    50   Input ~ 0
+ADV_DE
 $EndSCHEMATC

Commit message: Fixed some issues with the 50 Ohm impedance of the SPI lines. Added pinout .odt.
Connections:
- no-connect marks 18 -> 32
Changed lines of the file:
@@
 Text GLabel 8350 2750 0    50   Input ~ 0
 ADV_DE
+NoConn ~ 1850 4150
+NoConn ~ 1850 4250
+NoConn ~ 1850 3650
+NoConn ~ 1850 3550
+NoConn ~ 1850 3450
+NoConn ~ 1850 3350
+NoConn ~ 1850 3250
+NoConn ~ 1850 5050
+NoConn ~ 1850 5150
+NoConn ~ 1850 2750
+NoConn ~ 1850 2650
+NoConn ~ 1850 2550
+NoConn ~ 3450 5050
+NoConn ~ 3450 5150
 $EndSCHEMATC

Commit message: Added ESD protection, and removed the curved lines around the adv7511.
Connections:
- net labels added: ADV_CECCLK
- no-connect marks 32 -> 31
Changed lines of the file:
@@
 NoConn ~ 1850 3450
 NoConn ~ 1850 3350
-NoConn ~ 1850 3250
 NoConn ~ 1850 5050
 NoConn ~ 1850 5150
@@
 NoConn ~ 3450 5050
 NoConn ~ 3450 5150
+Text GLabel 1850 3250 0    50   Input ~ 0
+ADV_CECCLK
 $EndSCHEMATC

Commit message: Add an oscillator for the CEC functionality.
Connections:
- net labels removed: ADV_CECCLK
- no-connect marks 31 -> 32
Changed lines of the file:
@@
 NoConn ~ 3450 5050
 NoConn ~ 3450 5150
-Text GLabel 1850 3250 0    50   Input ~ 0
-ADV_CECCLK
+NoConn ~ 1850 3250
 $EndSCHEMATC

Commit message: Changed zener diode footprint for easy soldering. Fixed pins, U861/2 and U761/2 they now connect correctly to ground.
Connections:
- wire segments 34 -> 32
Changed lines of the file:
@@
 EESchema Schematic File Version 4
-LIBS:qmtech-minimig-cache
 EELAYER 30 0
 EELAYER END
@@
 Text GLabel 1700 2350 0    50   Input ~ 0
 3V3
-Text GLabel 1700 5250 0    50   Input ~ 0
-3V3
-Text GLabel 3600 5250 2    50   Input ~ 0
-3V3
-Wire Wire Line
-	3600 5350 3450 5350
-Text GLabel 3600 5350 2    50   Input ~ 0
+Text GLabel 1850 5250 0    50   Input ~ 0
+GND
+Text GLabel 3450 5250 2    50   Input ~ 0
+GND
+Text GLabel 3450 5350 2    50   Input ~ 0
 VIN5V
-Wire Wire Line
-	3450 5250 3600 5250
-Text GLabel 1700 5350 0    50   Input ~ 0
+Text GLabel 1850 5350 0    50   Input ~ 0
 VIN5V
 Wire Wire Line
@@
 GND
 Text GLabel 9950 5250 2    50   Input ~ 0
-3V3
+GND
 Text GLabel 9950 5350 2    50   Input ~ 0
 VIN5V
 Text GLabel 8350 5250 0    50   Input ~ 0
-3V3
+GND
 Text GLabel 8350 5350 0    50   Input ~ 0
 VIN5V

Commit message: Fixed reversed labeling of the QMTECH FPGA board pins.
Parts:
- added D31: 7, LED_SMD:LED_0603_1608Metric, symbol Device:LED
- added D32: 6, LED_SMD:LED_0603_1608Metric, symbol Device:LED
- added R63, R64: 1k, Resistor_SMD:R_0603_1608Metric, symbol Device:R
- D10: value LED0 -> 0
- D5: value LED5 -> 5
- D6: value LED4 -> 4
- D7: value LED3 -> 3
- D8: value LED2 -> 2
- D9: value LED1 -> 1
Connections:
- net labels added: LED6, LED7
- net labels removed: ADV_I2S2, ADV_I2S3
- wire segments 32 -> 40
- no-connect marks 32 -> 26
