File: main_board.sch (KiCad schematic (older format))
At the start: 7 parts, among them U2 QM_XC7A35T_DDR3

Commit message: Wired up the adv7511
Connections:
- net labels removed: MAX_I2S0, MAX_LRCLK, MAX_SCLK
Changed lines of the file:
@@
 Text GLabel 3450 2550 2    50   Input ~ 0
 ADV_R_7
-Text GLabel 9950 5050 2    50   Input ~ 0
+Text GLabel 11025 5050 2    50   Input ~ 0
 PS2_CLK1
-Text GLabel 9950 5150 2    50   Input ~ 0
+Text GLabel 11025 5150 2    50   Input ~ 0
 PS2_DAT1
 $Comp
@@
 Text Label 2700 7100 3    50   ~ 0
 LED0
-Text Label 8350 4450 2    50   ~ 0
-LED0
-Text Label 9950 4750 0    50   ~ 0
-LED1
-Text Label 9950 4850 0    50   ~ 0
+Text Label 11025 4850 0    50   ~ 0
 LED2
-Text Label 9950 4950 0    50   ~ 0
+Text Label 11025 4950 0    50   ~ 0
 LED3
 Text GLabel 3450 3450 2    50   Input ~ 0
@@
 Wire Wire Line
 	2700 6150 2700 5950
-Text GLabel 8350 5150 0    50   Input ~ 0
-MAX_LRCLK
-Text GLabel 8350 5050 0    50   Input ~ 0
-MAX_SCLK
-Text GLabel 8350 4750 0    50   Input ~ 0
-MAX_I2S0
 Text GLabel 1850 3550 0    50   Input ~ 0
 ESP_INT
-Text GLabel 8350 4850 0    50   Input ~ 0
+Text GLabel 7375 5050 0    50   Input ~ 0
 PS2_CLK2
-Text GLabel 8350 4950 0    50   Input ~ 0
+Text GLabel 7375 5150 0    50   Input ~ 0
 PS2_DAT2
 Text GLabel 3450 3650 2    50   Input ~ 0
@@
 Text GLabel 1850 4150 0    50   Input ~ 0
 ADV_DE
-Text GLabel 8350 3450 0    50   Input ~ 0
-SDRAM_A3
-Text GLabel 9950 3450 2    50   Input ~ 0
-SDRAM_A4
-Text GLabel 8350 3550 0    50   Input ~ 0
-SDRAM_A1
-Text GLabel 9950 3550 2    50   Input ~ 0
-SDRAM_A2
-Text GLabel 8350 3650 0    50   Input ~ 0
-SDRAM_A10
-Text GLabel 9950 3650 2    50   Input ~ 0
-SDRAM_A0
-Text GLabel 8350 3750 0    50   Input ~ 0
-SDRAM_BA0
-Text GLabel 9950 3750 2    50   Input ~ 0
-SDRAM_BA1
-Text GLabel 8350 3850 0    50   Input ~ 0
-SDRAM_RAS
-Text GLabel 9950 3850 2    50   Input ~ 0
-SDRAM_CS
-Text GLabel 8350 3950 0    50   Input ~ 0
-SDRAM_WE
 Text GLabel 1850 4250 0    50   Input ~ 0
 ADV_VSYNC
-Text GLabel 8350 4650 0    50   Input ~ 0
+Text GLabel 8350 3850 0    50   Input ~ 0
 JS_INTA
-Text GLabel 8350 4550 0    50   Input ~ 0
+Text GLabel 8350 3650 0    50   Input ~ 0
 JS_MISO
-Text GLabel 9950 4650 2    50   Input ~ 0
-JS_SCK
 Text GLabel 1850 4650 0    50   Input ~ 0
 EXP_SEL0
@@
 Text Notes 3475 6275 0    50   ~ 0
 Decoupling Cap\n
-Text GLabel 8350 4350 0    50   Input ~ 0
-SDRAM_D0
-Text GLabel 8350 4250 0    50   Input ~ 0
-SDRAM_D3
-Text GLabel 8350 4150 0    50   Input ~ 0
-SDRAM_D5
-Text GLabel 8350 4050 0    50   Input ~ 0
-SDRAM_D7
-Text GLabel 9950 4450 2    50   Input ~ 0
-JS_MOSI
-Text GLabel 9950 4550 2    50   Input ~ 0
-JS_CS
-Text GLabel 9950 4350 2    50   Input ~ 0
-SDRAM_D1
-Text GLabel 9950 4250 2    50   Input ~ 0
-SDRAM_D4
-Text GLabel 9950 4150 2    50   Input ~ 0
-SDRAM_D6
-Text GLabel 9950 4050 2    50   Input ~ 0
-SDRAM_DQML
-Text GLabel 9950 3950 2    50   Input ~ 0
-SDRAM_CAS
 $Comp
 L QM_XC7A35T_DDR3:QM_XC7A35T_DDR3_2part U2
@@
 	1    0    0    -1
 $EndComp
-Text GLabel 9950 2550 2    50   Input ~ 0
-SDRAM_D15
-Text GLabel 9950 2650 2    50   Input ~ 0
-SDRAM_D13
-Text GLabel 9950 2750 2    50   Input ~ 0
-SDRAM_D11
-Text GLabel 9950 2850 2    50   Input ~ 0
-SDRAM_D9
-Text GLabel 9950 2950 2    50   Input ~ 0
-SDRAM_DQMH
-Text GLabel 9950 3050 2    50   Input ~ 0
-SDRAM_CKE
-Text GLabel 9950 3150 2    50   Input ~ 0
-SDRAM_A11
-Text GLabel 9950 3250 2    50   Input ~ 0
-SDRAM_A8
-Text GLabel 9950 3350 2    50   Input ~ 0
-SDRAM_A6
-Text GLabel 8350 2550 0    50   Input ~ 0
+Text GLabel 8350 2650 0    50   Input ~ 0
 SDRAM_D14
-Text GLabel 8350 2650 0    50   Input ~ 0
+Text GLabel 8350 2750 0    50   Input ~ 0
 SDRAM_D12
-Text GLabel 8350 2750 0    50   Input ~ 0
+Text GLabel 8350 2850 0    50   Input ~ 0
 SDRAM_D10
-Text GLabel 8350 2850 0    50   Input ~ 0
+Text GLabel 8350 2950 0    50   Input ~ 0
 SDRAM_D8
-Text GLabel 8350 2950 0    50   Input ~ 0
+Text GLabel 8350 3050 0    50   Input ~ 0
 SDRAM_CLK
-Text GLabel 8350 3050 0    50   Input ~ 0
+Text GLabel 8350 3150 0    50   Input ~ 0
 SDRAM_A12
-Text GLabel 8350 3150 0    50   Input ~ 0
+Text GLabel 8350 3250 0    50   Input ~ 0
 SDRAM_A9
-Text GLabel 8350 3250 0    50   Input ~ 0
+Text GLabel 8350 3350 0    50   Input ~ 0
 SDRAM_A7
-Text GLabel 8350 3350 0    50   Input ~ 0
+Text GLabel 8350 3450 0    50   Input ~ 0
 SDRAM_A5
 $Comp
@@
 	1    0    0    -1
 $EndComp
+Text GLabel 9950 3450 2    50   Input ~ 0
+SDRAM_A6
+Text GLabel 9950 3350 2    50   Input ~ 0
+SDRAM_A8
+Text GLabel 9950 3250 2    50   Input ~ 0
+SDRAM_A11
+Text GLabel 9950 3150 2    50   Input ~ 0
+SDRAM_CKE
+Text GLabel 9950 3050 2    50   Input ~ 0
+SDRAM_DQMH
+Text GLabel 9950 2950 2    50   Input ~ 0
+SDRAM_D9
+Text GLabel 9950 2850 2    50   Input ~ 0
+SDRAM_D11
+Text GLabel 9950 2750 2    50   Input ~ 0
+SDRAM_D13
+Text GLabel 9950 2650 2    50   Input ~ 0
+SDRAM_D15
+Text GLabel 9950 4750 2    50   Input ~ 0
+SDRAM_CAS
+Text GLabel 9950 4850 2    50   Input ~ 0
+SDRAM_DQML
+Text GLabel 9950 4950 2    50   Input ~ 0
+SDRAM_D6
+Text GLabel 9950 5050 2    50   Input ~ 0
+SDRAM_D4
+Text GLabel 9950 5150 2    50   Input ~ 0
+SDRAM_D1
+Text GLabel 9950 4650 2    50   Input ~ 0
+SDRAM_CS
+Text GLabel 9950 4550 2    50   Input ~ 0
+SDRAM_BA1
+Text GLabel 9950 4450 2    50   Input ~ 0
+SDRAM_A0
+Text GLabel 9950 3850 2    50   Input ~ 0
+SDRAM_A2
+Text GLabel 9950 3550 2    50   Input ~ 0
+SDRAM_A4
+Text GLabel 9950 3750 2    50   Input ~ 0
+JS_CS
+Text GLabel 9950 3650 2    50   Input ~ 0
+JS_MOSI
+Text GLabel 8350 3750 0    50   Input ~ 0
+JS_SCK
+Text Label 11025 4750 0    50   ~ 0
+LED1
+Text GLabel 8350 3550 0    50   Input ~ 0
+SDRAM_A3
+Text GLabel 8350 4950 0    50   Input ~ 0
+SDRAM_D7
+Text GLabel 8350 5050 0    50   Input ~ 0
+SDRAM_D5
+Text GLabel 8350 5150 0    50   Input ~ 0
+SDRAM_D3
+Text GLabel 7375 4750 0    50   Input ~ 0
+SDRAM_D0
+Text GLabel 8350 4850 0    50   Input ~ 0
+SDRAM_WE
+Text GLabel 8350 4750 0    50   Input ~ 0
+SDRAM_RAS
+Text GLabel 8350 4650 0    50   Input ~ 0
+SDRAM_BA0
+Text GLabel 8350 4550 0    50   Input ~ 0
+SDRAM_A10
+Text GLabel 8350 4450 0    50   Input ~ 0
+SDRAM_A1
+Text Label 7375 4850 2    50   ~ 0
+LED0
 $EndSCHEMATC

Commit message: First rough version of the Open AARS V4
Parts:
- added H1, H2, H3, H4, H5, H6: MountingHole_Pad, MountingHole:MountingHole_3.2mm_M3_DIN965_Pad, symbol Mechanical:MountingHole_Pad
- added J6: Conn_01x03_Male, Connector_PinHeader_2.54mm:PinHeader_1x03_P2.54mm_Vertical, symbol Connector:Conn_01x03_Male
Connections:
- net labels added: ADV_D0, ADV_D1, ADV_D10, ADV_D11, ADV_D2, ADV_D3, ADV_D4, ADV_D5, ADV_D6, ADV_D7, ADV_D8, ADV_D9, ESP_SD_CLK, ESP_SD_CMD, ESP_SD_DATA0, ESP_SD_DATA1, ESP_SD_DATA2, ESP_SD_DATA3, MAX_I2S0, MAX_LRCLK, MAX_SCLK, SDRAM_D2, UART_RX, UART_TX
- net labels removed: ADV_B_0, ADV_B_1, ADV_B_2, ADV_B_3, ADV_B_4, ADV_B_5, ADV_B_6, ADV_B_7, ADV_G_0, ADV_G_1, ADV_G_2, ADV_G_3, ADV_G_4, ADV_G_5, ADV_G_6, ADV_G_7, ADV_R_0, ADV_R_1, ADV_R_2, ADV_R_3, ADV_R_4, ADV_R_5, ADV_R_6, ADV_R_7
- wire segments 26 -> 30
Other:
- note added: "UART RX/TX"

Commit message: Fixed issues with V4 board, length matching, region matching, footprints, symbols.
Parts:
- U2: footprint qmtech-minimig-new:QM_XC7A35T_DDR3_Daughterboard_rev2 -> qmtech-minimig-new:QM_XC7A100T_DDR3_Daughterboard_rev2; symbol QM_XC7A35T_DDR3:QM_XC7A35T_DDR3_2part -> QM_XC7A35T_DDR3:QM_XC7A100T_DDR3_2part
Connections:
- wire segments 30 -> 28
Changed lines of the file:
@@
 	3450 2350 3600 2350
-Wire Wire Line
-	3450 2450 3600 2450
-Text GLabel 3600 2450 2    50   Input ~ 0
-GND
 Wire Wire Line
 	3450 2250 3600 2250
@@
 Text GLabel 1700 2250 0    50   Input ~ 0
 GND
-Text GLabel 1700 2450 0    50   Input ~ 0
-GND
 Wire Wire Line
 	1700 2250 1850 2250
-Wire Wire Line
-	1700 2450 1850 2450
 Wire Wire Line
 	1700 2350 1850 2350
@@
 Text GLabel 1850 2950 0    50   Input ~ 0
 ESP_VSPI_CLK
-Text GLabel 3450 2750 2    50   Input ~ 0
-ESP_VSPI_MISO
-Text GLabel 1850 2850 0    50   Input ~ 0
+Text GLabel 1850 2750 0    50   Input ~ 0
 ESP_VSPI_MOSI
-Text GLabel 3450 2950 2    50   Input ~ 0
-ESP_VSPI_CS
 Wire Wire Line
 	1650 6150 1650 5950
@@
 Wire Wire Line
 	2700 6150 2700 5950
-Text GLabel 1850 3050 0    50   Input ~ 0
+Text GLabel 1850 2850 0    50   Input ~ 0
 ESP_INT
 Text GLabel 1850 5050 0    50   Input ~ 0
@@
 Text GLabel 1850 4950 0    50   Input ~ 0
 PS2_DAT2
-Text GLabel 1850 3650 0    50   Input ~ 0
+Text GLabel 3450 3850 2    50   Input ~ 0
 ADV_CLK
-Text GLabel 3450 3850 2    50   Input ~ 0
-ADV_HSYNC
-Text GLabel 1850 3850 0    50   Input ~ 0
+Text GLabel 3450 4150 2    50   Input ~ 0
+ADV_VSYNC
+Text GLabel 3450 3950 2    50   Input ~ 0
 ADV_DE
 Text GLabel 9950 4850 2    50   Input ~ 0
@@
 Text GLabel 8350 4950 0    50   Input ~ 0
 JS_MISO
-Text GLabel 1850 4150 0    50   Input ~ 0
+Text GLabel 1850 4050 0    50   Input ~ 0
 EXP_SEL0
-Text GLabel 3450 4150 2    50   Input ~ 0
+Text GLabel 3450 4050 2    50   Input ~ 0
 EXP_SEL1
 Text GLabel 1850 4250 0    50   Input ~ 0
@@
 Decoupling Cap\n
 $Comp
-L QM_XC7A35T_DDR3:QM_XC7A35T_DDR3_2part U2
+L QM_XC7A35T_DDR3:QM_XC7A100T_DDR3_2part U2
 U 1 1 5D70654A
 P 9150 3850
@@
 F 0 "U2" H 9119 5705 50  0000 C CNN
 F 1 "QM_XC7A35T_DDR3" H 9119 5614 50  0000 C CNN
-F 2 "qmtech-minimig-new:QM_XC7A35T_DDR3_Daughterboard_rev2" H 9119 5523 50  0000 C CNN
+F 2 "qmtech-minimig-new:QM_XC7A100T_DDR3_Daughterboard_rev2" H 9119 5523 50  0000 C CNN
 F 3 "" H 5850 2400 50  0001 C CNN
 	1    9150 3850
@@
 $EndComp
 $Comp
-L QM_XC7A35T_DDR3:QM_XC7A35T_DDR3_2part U?
+L QM_XC7A35T_DDR3:QM_XC7A100T_DDR3_2part U?
 U 2 1 5F7C0F58
 P 2650 3850
@@
 F 0 "U2" H 2619 5705 50  0000 C CNN
 F 1 "QM_XC7A35T_DDR3" H 2619 5614 50  0000 C CNN
-F 2 "qmtech-minimig-new:QM_XC7A35T_DDR3_Daughterboard_rev2" H 2619 5523 50  0000 C CNN
+F 2 "qmtech-minimig-new:QM_XC7A100T_DDR3_Daughterboard_rev2" H 2619 5523 50  0000 C CNN
 F 3 "" H -650 2400 50  0001 C CNN
 	2    2650 3850
 	-1   0    0    1
 $EndComp
-Text GLabel 8350 4650 0    50   Input ~ 0
+Text GLabel 8350 4750 0    50   Input ~ 0
 SDRAM_D14
 Text GLabel 8350 4450 0    50   Input ~ 0
@@
 Text GLabel 8350 4550 0    50   Input ~ 0
 SDRAM_D13
-Text GLabel 8350 4750 0    50   Input ~ 0
+Text GLabel 8350 4850 0    50   Input ~ 0
 SDRAM_D15
 Text GLabel 9950 3750 2    50   Input ~ 0
@@
 Text GLabel 9950 5050 2    50   Input ~ 0
 JS_MOSI
-Text GLabel 8350 5050 0    50   Input ~ 0
+Text GLabel 8350 4650 0    50   Input ~ 0
 JS_SCK
 Text GLabel 9950 2850 2    50   Input ~ 0
@@
 Wire Wire Line
 	6300 1250 6600 1250
-Text GLabel 3450 2550 2    50   Input ~ 0
-ESP_SD_CMD
+Text GLabel 1850 2450 0    50   Input ~ 0
+ESP_SD_DATA3
 Text GLabel 1850 2550 0    50   Input ~ 0
-ESP_SD_DATA3
+ESP_SD_DATA2
 Text GLabel 1850 2650 0    50   Input ~ 0
-ESP_SD_DATA2
-Text GLabel 1850 2750 0    50   Input ~ 0
 ESP_SD_CLK
-Text GLabel 3450 2850 2    50   Input ~ 0
-ESP_SD_DATA0
-Text GLabel 3450 2650 2    50   Input ~ 0
-ESP_SD_DATA1
 Text GLabel 3450 5350 2    50   Input ~ 0
 GND
@@
 Text GLabel 3450 3050 2    50   Input ~ 0
 ADV_SCL
-Text GLabel 1850 3150 0    50   Input ~ 0
+Text GLabel 1850 3250 0    50   Input ~ 0
 ADV_D11
-Text GLabel 1850 3250 0    50   Input ~ 0
+Text GLabel 1850 3350 0    50   Input ~ 0
 ADV_D10
-Text GLabel 3450 3250 2    50   Input ~ 0
+Text GLabel 3450 3350 2    50   Input ~ 0
 ADV_D9
-Text GLabel 1850 3350 0    50   Input ~ 0
+Text GLabel 1850 3450 0    50   Input ~ 0
 ADV_D8
-Text GLabel 3450 3350 2    50   Input ~ 0
+Text GLabel 3450 3450 2    50   Input ~ 0
 ADV_D7
-Text GLabel 1850 3450 0    50   Input ~ 0
+Text GLabel 1850 3550 0    50   Input ~ 0
 ADV_D6
-Text GLabel 3450 3450 2    50   Input ~ 0
+Text GLabel 3450 3550 2    50   Input ~ 0
 ADV_D5
-Text GLabel 1850 3550 0    50   Input ~ 0
+Text GLabel 1850 3650 0    50   Input ~ 0
 ADV_D4
-Text GLabel 3450 3550 2    50   Input ~ 0
+Text GLabel 3450 3650 2    50   Input ~ 0
 ADV_D3
-Text GLabel 3450 3650 2    50   Input ~ 0
+Text GLabel 1850 3750 0    50   Input ~ 0
 ADV_D2
-Text GLabel 1850 3750 0    50   Input ~ 0
+Text GLabel 3450 3750 2    50   Input ~ 0
 ADV_D1
-Text GLabel 3450 3750 2    50   Input ~ 0
+Text GLabel 1850 3850 0    50   Input ~ 0
 ADV_D0
-Text GLabel 1850 3950 0    50   Input ~ 0
-ADV_VSYNC
 Text GLabel 3450 3150 2    50   Input ~ 0
 ADV_SDA
@@
 Text Notes 5950 6350 0    50   ~ 0
 UART RX/TX
+Text GLabel 1850 4150 0    50   Input ~ 0
+ADV_HSYNC
+Text GLabel 3450 2650 2    50   Input ~ 0
+ESP_SD_DATA1
+Text GLabel 3450 2850 2    50   Input ~ 0
+ESP_SD_DATA0
+Text GLabel 3450 2550 2    50   Input ~ 0
+ESP_SD_CMD
+Text GLabel 3450 2950 2    50   Input ~ 0
+ESP_VSPI_CS
+Text GLabel 3450 2750 2    50   Input ~ 0
+ESP_VSPI_MISO
 $EndSCHEMATC

Commit message: Brought compenents back to the front for easy soldering.
Parts:
- removed J6: Conn_01x03_Male, Connector_PinHeader_2.54mm:PinHeader_1x03_P2.54mm_Vertical, symbol Connector:Conn_01x03_Male
- added H7: MountingHole_Pad, MountingHole:MountingHole_3.2mm_M3_DIN965_Pad, symbol Mechanical:MountingHole_Pad
Connections:
- net labels added: ADV_CECCLK, FGPA_UART0_TX, FPGA_SD_CLK, FPGA_SD_CMD, FPGA_SD_DATA0, FPGA_SD_DATA1, FPGA_SD_DATA2, FPGA_SD_DATA3, FPGA_UART0_RX, OSC_74.25
- net labels removed: ESP_SD_CLK, ESP_SD_CMD, ESP_SD_DATA0, ESP_SD_DATA1, ESP_SD_DATA2, ESP_SD_DATA3, UART_RX, UART_TX
- wire segments 28 -> 25
- no-connect marks 0 -> 1
Other:
- note removed: "UART RX/TX"
Changed lines of the file:
@@
 Comment4 ""
 $EndDescr
-Wire Wire Line
-	3450 2350 3600 2350
-Wire Wire Line
-	3450 2250 3600 2250
-Text GLabel 3600 2250 2    50   Input ~ 0
-GND
-Text GLabel 1700 2250 0    50   Input ~ 0
-GND
-Wire Wire Line
-	1700 2250 1850 2250
-Wire Wire Line
-	1700 2350 1850 2350
-Text GLabel 1700 2350 0    50   Input ~ 0
-3V3
 Text GLabel 1850 5150 0    50   Input ~ 0
 GND
 Text GLabel 3450 5150 2    50   Input ~ 0
 GND
-Text GLabel 3600 2350 2    50   Input ~ 0
-3V3
 Text GLabel 9950 2350 2    50   Input ~ 0
 GND
@@
 Text Label 2000 7100 3    50   ~ 0
 LED2
-Text Label 1650 7100 3    50   ~ 0
-LED3
 Text Notes 1600 5850 0    100  ~ 0
 LED indicators
@@
 Text Label 2700 7100 3    50   ~ 0
 LED0
-Text GLabel 1850 2950 0    50   Input ~ 0
-ESP_VSPI_CLK
-Text GLabel 1850 2750 0    50   Input ~ 0
-ESP_VSPI_MOSI
 Wire Wire Line
 	1650 6150 1650 5950
@@
 Wire Wire Line
 	2700 6150 2700 5950
-Text GLabel 1850 2850 0    50   Input ~ 0
-ESP_INT
 Text GLabel 1850 5050 0    50   Input ~ 0
 PS2_CLK2
@@
 Text GLabel 8350 4650 0    50   Input ~ 0
 JS_SCK
-Text GLabel 9950 2850 2    50   Input ~ 0
+Text GLabel 8350 2850 0    50   Input ~ 0
 SDRAM_A3
 Text GLabel 9950 4050 2    50   Input ~ 0
@@
 Text GLabel 9950 3050 2    50   Input ~ 0
 SDRAM_A1
-Text GLabel 8350 2550 0    50   Input ~ 0
+Text GLabel 9950 2850 2    50   Input ~ 0
 MAX_LRCLK
-Text GLabel 9950 2450 2    50   Input ~ 0
+Text GLabel 8350 2750 0    50   Input ~ 0
 MAX_SCLK
-Text GLabel 8350 2450 0    50   Input ~ 0
+Text GLabel 9950 2750 2    50   Input ~ 0
 MAX_I2S0
 Text GLabel 9950 4550 2    50   Input ~ 0
@@
 Wire Wire Line
 	6300 1250 6600 1250
-Text GLabel 1850 2450 0    50   Input ~ 0
-ESP_SD_DATA3
-Text GLabel 1850 2550 0    50   Input ~ 0
-ESP_SD_DATA2
-Text GLabel 1850 2650 0    50   Input ~ 0
-ESP_SD_CLK
 Text GLabel 3450 5350 2    50   Input ~ 0
 GND
@@
 Text GLabel 3450 5250 2    50   Input ~ 0
 3V3
-Text GLabel 3450 3050 2    50   Input ~ 0
+Text GLabel 3450 3150 2    50   Input ~ 0
 ADV_SCL
 Text GLabel 1850 3250 0    50   Input ~ 0
@@
 Text GLabel 1850 3850 0    50   Input ~ 0
 ADV_D0
-Text GLabel 3450 3150 2    50   Input ~ 0
+Text GLabel 3450 3250 2    50   Input ~ 0
 ADV_SDA
 Text GLabel 3450 5050 2    50   Input ~ 0
@@
 Text GLabel 3450 4850 2    50   Input ~ 0
 LED0
-Text GLabel 1850 4850 0    50   Input ~ 0
-LED1
 Text GLabel 3450 4750 2    50   Input ~ 0
 LED2
-Text GLabel 1850 4750 0    50   Input ~ 0
-LED3
-Text GLabel 9950 2550 2    50   Input ~ 0
-UART_RX
-Text GLabel 8350 2650 0    50   Input ~ 0
-UART_TX
-$Comp
-L Connector:Conn_01x03_Male J6
-U 1 1 5FDF1E05
-P 5900 6700
-F 0 "J6" H 6008 6981 50  0000 C CNN
-F 1 "Conn_01x03_Male" H 6008 6890 50  0000 C CNN
-F 2 "Connector_PinHeader_2.54mm:PinHeader_1x03_P2.54mm_Vertical" H 5900 6700 50  0001 C CNN
-F 3 "~" H 5900 6700 50  0001 C CNN
-	1    5900 6700
-	1    0    0    -1
-$EndComp
-Text GLabel 6100 6600 2    50   Input ~ 0
-UART_RX
-Text GLabel 6100 6700 2    50   Input ~ 0
-UART_TX
-Text GLabel 6100 6800 2    50   Input ~ 0
-GND
-Text Notes 5950 6350 0    50   ~ 0
-UART RX/TX
 Text GLabel 1850 4150 0    50   Input ~ 0
 ADV_HSYNC
 Text GLabel 3450 2650 2    50   Input ~ 0
-ESP_SD_DATA1
-Text GLabel 3450 2850 2    50   Input ~ 0
-ESP_SD_DATA0
+FPGA_SD_DATA1
+Text GLabel 3450 2750 2    50   Input ~ 0
+FPGA_SD_DATA0
 Text GLabel 3450 2550 2    50   Input ~ 0
-ESP_SD_CMD
+FPGA_SD_CMD
 Text GLabel 3450 2950 2    50   Input ~ 0
 ESP_VSPI_CS
-Text GLabel 3450 2750 2    50   Input ~ 0
+Text GLabel 1850 2850 0    50   Input ~ 0
 ESP_VSPI_MISO
+Text GLabel 1850 2750 0    50   Input ~ 0
+FPGA_SD_CLK
+Text GLabel 1850 2650 0    50   Input ~ 0
+FPGA_SD_DATA2
+Text GLabel 1850 2550 0    50   Input ~ 0
+FPGA_SD_DATA3
+Text GLabel 1850 3050 0    50   Input ~ 0
+ESP_INT
+Text GLabel 3450 2850 2    50   Input ~ 0
+ESP_VSPI_MOSI
+Text GLabel 1850 2950 0    50   Input ~ 0
+ESP_VSPI_CLK
+Text GLabel 3450 2450 2    50   Input ~ 0
+FGPA_UART0_TX
+Text GLabel 1850 2450 0    50   Input ~ 0
+FPGA_UART0_RX
+Text GLabel 1850 3150 0    50   Input ~ 0
+OSC_74.25
+$Comp
+L Mechanical:MountingHole_Pad H7
+U 1 1 5FA3C754
+P 6900 1150
+F 0 "H7" H 7000 1199 50  0000 L CNN
+F 1 "MountingHole_Pad" H 7000 1108 50  0000 L CNN
+F 2 "MountingHole:MountingHole_3.2mm_M3_DIN965_Pad" H 6900 1150 50  0001 C CNN
+F 3 "~" H 6900 1150 50  0001 C CNN
+	1    6900 1150
+	1    0    0    -1
+$EndComp
+Wire Wire Line
+	6900 1250 6600 1250
+Connection ~ 6600 1250
+Text GLabel 3450 3050 2    50   Input ~ 0
+ADV_CECCLK
+Text Label 1650 7100 3    50   ~ 0
+LED3
+Text GLabel 1850 4850 0    50   Input ~ 0
+LED1
+Text GLabel 1850 4750 0    50   Input ~ 0
+LED3
+Text GLabel 1850 2350 0    50   Input ~ 0
+GND
+Text GLabel 3450 2350 2    50   Input ~ 0
+GND
+Text GLabel 3450 2250 2    50   Input ~ 0
+VIN5V
+NoConn ~ 1850 2250
 $EndSCHEMATC
