File: joystick.sch (KiCad schematic (older format))
At the start: 18 parts, among them J1 DB9_Male, J2 DB9_Male

Commit message: Added protection diodes to the joystick ports.
Parts:
- added D12, D13, D14, D15, D16, D17, D18, D19, D20, D21, D22, D23, D24, D25, D26, D27: D_Zener 3.6V BZT52C395, Diode_SMD:D_SOD-323, symbol Device:D_Zener
Connections:
- wire segments 84 -> 134

Commit message: Add an oscillator for the CEC functionality.
Parts:
- R1, R10, R11, R12, R13, R14, R15, R16, R2, R3, R4, R5, R6, R7, R8, R9: footprint Resistor_SMD:R_0201_0603Metric -> Resistor_SMD:R_0603_1608Metric
Changed lines of the file:
@@
 F 0 "R15" V 7150 1150 50  0000 L CNN
 F 1 "47K" V 7250 1200 50  0000 L CNN
-F 2 "Resistor_SMD:R_0201_0603Metric" H 7220 1159 50  0001 L CNN
+F 2 "Resistor_SMD:R_0603_1608Metric" H 7220 1159 50  0001 L CNN
 F 3 "~" H 7150 1250 50  0001 C CNN
 	1    7150 1250
@@
 F 0 "R13" V 6950 1150 50  0000 L CNN
 F 1 "47K" V 7050 1200 50  0000 L CNN
-F 2 "Resistor_SMD:R_0201_0603Metric" H 7020 1159 50  0001 L CNN
+F 2 "Resistor_SMD:R_0603_1608Metric" H 7020 1159 50  0001 L CNN
 F 3 "~" H 6950 1250 50  0001 C CNN
 	1    6950 1250
@@
 F 0 "R11" V 6750 1150 50  0000 L CNN
 F 1 "47K" V 6850 1200 50  0000 L CNN
-F 2 "Resistor_SMD:R_0201_0603Metric" H 6820 1159 50  0001 L CNN
+F 2 "Resistor_SMD:R_0603_1608Metric" H 6820 1159 50  0001 L CNN
 F 3 "~" H 6750 1250 50  0001 C CNN
 	1    6750 1250
@@
 F 0 "R9" V 6550 1150 50  0000 L CNN
 F 1 "47K" V 6650 1200 50  0000 L CNN
-F 2 "Resistor_SMD:R_0201_0603Metric" H 6620 1159 50  0001 L CNN
+F 2 "Resistor_SMD:R_0603_1608Metric" H 6620 1159 50  0001 L CNN
 F 3 "~" H 6550 1250 50  0001 C CNN
 	1    6550 1250
@@
 F 0 "R7" V 6350 1150 50  0000 L CNN
 F 1 "47K" V 6450 1200 50  0000 L CNN
-F 2 "Resistor_SMD:R_0201_0603Metric" H 6420 1159 50  0001 L CNN
+F 2 "Resistor_SMD:R_0603_1608Metric" H 6420 1159 50  0001 L CNN
 F 3 "~" H 6350 1250 50  0001 C CNN
 	1    6350 1250
@@
 F 0 "R5" V 6150 1150 50  0000 L CNN
 F 1 "47K" V 6250 1200 50  0000 L CNN
-F 2 "Resistor_SMD:R_0201_0603Metric" H 6220 1159 50  0001 L CNN
+F 2 "Resistor_SMD:R_0603_1608Metric" H 6220 1159 50  0001 L CNN
 F 3 "~" H 6150 1250 50  0001 C CNN
 	1    6150 1250
@@
 F 0 "R1" V 5750 1150 50  0000 L CNN
 F 1 "47K" V 5850 1200 50  0000 L CNN
-F 2 "Resistor_SMD:R_0201_0603Metric" H 5820 1159 50  0001 L CNN
+F 2 "Resistor_SMD:R_0603_1608Metric" H 5820 1159 50  0001 L CNN
 F 3 "~" H 5750 1250 50  0001 C CNN
 	1    5750 1250
@@
 F 0 "R3" V 5950 1150 50  0000 L CNN
 F 1 "47K" V 6050 1200 50  0000 L CNN
-F 2 "Resistor_SMD:R_0201_0603Metric" H 6020 1159 50  0001 L CNN
+F 2 "Resistor_SMD:R_0603_1608Metric" H 6020 1159 50  0001 L CNN
 F 3 "~" H 5950 1250 50  0001 C CNN
 	1    5950 1250
@@
 F 0 "R16" V 7200 4250 50  0000 L CNN
 F 1 "47K" V 7300 4300 50  0000 L CNN
-F 2 "Resistor_SMD:R_0201_0603Metric" H 7270 4259 50  0001 L CNN
+F 2 "Resistor_SMD:R_0603_1608Metric" H 7270 4259 50  0001 L CNN
 F 3 "~" H 7200 4350 50  0001 C CNN
 	1    7200 4350
@@
 F 0 "R14" V 7000 4250 50  0000 L CNN
 F 1 "47K" V 7100 4300 50  0000 L CNN
-F 2 "Resistor_SMD:R_0201_0603Metric" H 7070 4259 50  0001 L CNN
+F 2 "Resistor_SMD:R_0603_1608Metric" H 7070 4259 50  0001 L CNN
 F 3 "~" H 7000 4350 50  0001 C CNN
 	1    7000 4350
@@
 F 0 "R12" V 6800 4250 50  0000 L CNN
 F 1 "47K" V 6900 4300 50  0000 L CNN
-F 2 "Resistor_SMD:R_0201_0603Metric" H 6870 4259 50  0001 L CNN
+F 2 "Resistor_SMD:R_0603_1608Metric" H 6870 4259 50  0001 L CNN
 F 3 "~" H 6800 4350 50  0001 C CNN
 	1    6800 4350
@@
 F 0 "R10" V 6600 4250 50  0000 L CNN
 F 1 "47K" V 6700 4300 50  0000 L CNN
-F 2 "Resistor_SMD:R_0201_0603Metric" H 6670 4259 50  0001 L CNN
+F 2 "Resistor_SMD:R_0603_1608Metric" H 6670 4259 50  0001 L CNN
 F 3 "~" H 6600 4350 50  0001 C CNN
 	1    6600 4350
@@
 F 0 "R8" V 6400 4250 50  0000 L CNN
 F 1 "47K" V 6500 4300 50  0000 L CNN
-F 2 "Resistor_SMD:R_0201_0603Metric" H 6470 4259 50  0001 L CNN
+F 2 "Resistor_SMD:R_0603_1608Metric" H 6470 4259 50  0001 L CNN
 F 3 "~" H 6400 4350 50  0001 C CNN
 	1    6400 4350
@@
 F 0 "R6" V 6200 4250 50  0000 L CNN
 F 1 "47K" V 6300 4300 50  0000 L CNN
-F 2 "Resistor_SMD:R_0201_0603Metric" H 6270 4259 50  0001 L CNN
+F 2 "Resistor_SMD:R_0603_1608Metric" H 6270 4259 50  0001 L CNN
 F 3 "~" H 6200 4350 50  0001 C CNN
 	1    6200 4350
@@
 F 0 "R2" V 5800 4250 50  0000 L CNN
 F 1 "47K" V 5900 4300 50  0000 L CNN
-F 2 "Resistor_SMD:R_0201_0603Metric" H 5870 4259 50  0001 L CNN
+F 2 "Resistor_SMD:R_0603_1608Metric" H 5870 4259 50  0001 L CNN
 F 3 "~" H 5800 4350 50  0001 C CNN
 	1    5800 4350
@@
 F 0 "R4" V 6000 4250 50  0000 L CNN
 F 1 "47K" V 6100 4300 50  0000 L CNN
-F 2 "Resistor_SMD:R_0201_0603Metric" H 6070 4259 50  0001 L CNN
+F 2 "Resistor_SMD:R_0603_1608Metric" H 6070 4259 50  0001 L CNN
 F 3 "~" H 6000 4350 50  0001 C CNN
 	1    6000 4350

Commit message: Changed zener diode footprint for easy soldering. Fixed pins, U861/2 and U761/2 they now connect correctly to ground.
Parts:
- D12, D13, D14, D15, D16, D17, D18, D19, D20, D21, D22, D23, D24, D25, D26, D27: footprint Diode_SMD:D_SOD-323 -> Diode_SMD:D_SOD-323_HandSoldering
Changed lines of the file:
@@
 EESchema Schematic File Version 4
-LIBS:qmtech-minimig-cache
 EELAYER 30 0
 EELAYER END
@@
 U 1 1 5D803038
 P 5750 2800
-F 0 "D12" V 5750 2879 50  0000 L CNN
+F 0 "D12" V 5875 2800 50  0000 L CNN
 F 1 "D_Zener 3.6V BZT52C395" V 5795 2879 50  0001 L CNN
-F 2 "Diode_SMD:D_SOD-323" H 5750 2800 50  0001 C CNN
+F 2 "Diode_SMD:D_SOD-323_HandSoldering" H 5750 2800 50  0001 C CNN
 F 3 "https://www.application-datasheet.com/pdf/diodes/bzt52c4v7s-7-f.pdf" H 5750 2800 50  0001 C CNN
 	1    5750 2800
@@
 U 1 1 5D804405
 P 5950 2800
-F 0 "D14" V 5950 2879 50  0000 L CNN
+F 0 "D14" V 6075 2800 50  0000 L CNN
 F 1 "D_Zener 3.6V BZT52C395" V 5995 2879 50  0001 L CNN
-F 2 "Diode_SMD:D_SOD-323" H 5950 2800 50  0001 C CNN
+F 2 "Diode_SMD:D_SOD-323_HandSoldering" H 5950 2800 50  0001 C CNN
 F 3 "https://www.application-datasheet.com/pdf/diodes/bzt52c4v7s-7-f.pdf" H 5950 2800 50  0001 C CNN
 	1    5950 2800
@@
 U 1 1 5D804621
 P 6150 2800
-F 0 "D16" V 6150 2879 50  0000 L CNN
+F 0 "D16" V 6275 2800 50  0000 L CNN
 F 1 "D_Zener 3.6V BZT52C395" V 6195 2879 50  0001 L CNN
-F 2 "Diode_SMD:D_SOD-323" H 6150 2800 50  0001 C CNN
+F 2 "Diode_SMD:D_SOD-323_HandSoldering" H 6150 2800 50  0001 C CNN
 F 3 "https://www.application-datasheet.com/pdf/diodes/bzt52c4v7s-7-f.pdf" H 6150 2800 50  0001 C CNN
 	1    6150 2800
@@
 U 1 1 5D804F7F
 P 6350 2800
-F 0 "D18" V 6350 2879 50  0000 L CNN
+F 0 "D18" V 6475 2800 50  0000 L CNN
 F 1 "D_Zener 3.6V BZT52C395" V 6395 2879 50  0001 L CNN
-F 2 "Diode_SMD:D_SOD-323" H 6350 2800 50  0001 C CNN
+F 2 "Diode_SMD:D_SOD-323_HandSoldering" H 6350 2800 50  0001 C CNN
 F 3 "https://www.application-datasheet.com/pdf/diodes/bzt52c4v7s-7-f.pdf" H 6350 2800 50  0001 C CNN
 	1    6350 2800
@@
 U 1 1 5D8051B7
 P 6550 2800
-F 0 "D20" V 6550 2879 50  0000 L CNN
+F 0 "D20" V 6675 2800 50  0000 L CNN
 F 1 "D_Zener 3.6V BZT52C395" V 6595 2879 50  0001 L CNN
-F 2 "Diode_SMD:D_SOD-323" H 6550 2800 50  0001 C CNN
+F 2 "Diode_SMD:D_SOD-323_HandSoldering" H 6550 2800 50  0001 C CNN
 F 3 "https://www.application-datasheet.com/pdf/diodes/bzt52c4v7s-7-f.pdf" H 6550 2800 50  0001 C CNN
 	1    6550 2800
@@
 U 1 1 5D8053FF
 P 6750 2800
-F 0 "D22" V 6750 2879 50  0000 L CNN
+F 0 "D22" V 6875 2800 50  0000 L CNN
 F 1 "D_Zener 3.6V BZT52C395" V 6795 2879 50  0001 L CNN
-F 2 "Diode_SMD:D_SOD-323" H 6750 2800 50  0001 C CNN
+F 2 "Diode_SMD:D_SOD-323_HandSoldering" H 6750 2800 50  0001 C CNN
 F 3 "https://www.application-datasheet.com/pdf/diodes/bzt52c4v7s-7-f.pdf" H 6750 2800 50  0001 C CNN
 	1    6750 2800
@@
 U 1 1 5D805657
 P 6950 2800
-F 0 "D24" V 6950 2879 50  0000 L CNN
+F 0 "D24" V 7075 2800 50  0000 L CNN
 F 1 "D_Zener 3.6V BZT52C395" V 6995 2879 50  0001 L CNN
-F 2 "Diode_SMD:D_SOD-323" H 6950 2800 50  0001 C CNN
+F 2 "Diode_SMD:D_SOD-323_HandSoldering" H 6950 2800 50  0001 C CNN
 F 3 "https://www.application-datasheet.com/pdf/diodes/bzt52c4v7s-7-f.pdf" H 6950 2800 50  0001 C CNN
 	1    6950 2800
@@
 U 1 1 5D8058BF
 P 7150 2800
-F 0 "D26" V 7150 2879 50  0000 L CNN
+F 0 "D26" V 7275 2825 50  0000 L CNN
 F 1 "D_Zener 3.6V BZT52C395" V 7195 2879 50  0001 L CNN
-F 2 "Diode_SMD:D_SOD-323" H 7150 2800 50  0001 C CNN
+F 2 "Diode_SMD:D_SOD-323_HandSoldering" H 7150 2800 50  0001 C CNN
 F 3 "https://www.application-datasheet.com/pdf/diodes/bzt52c4v7s-7-f.pdf" H 7150 2800 50  0001 C CNN
 	1    7150 2800
@@
 F 0 "D13" V 5800 5979 50  0000 L CNN
 F 1 "D_Zener 3.6V BZT52C395" V 5845 5979 50  0001 L CNN
-F 2 "Diode_SMD:D_SOD-323" H 5800 5900 50  0001 C CNN
+F 2 "Diode_SMD:D_SOD-323_HandSoldering" H 5800 5900 50  0001 C CNN
 F 3 "https://www.application-datasheet.com/pdf/diodes/bzt52c4v7s-7-f.pdf" H 5800 5900 50  0001 C CNN
 	1    5800 5900
@@
 F 0 "D15" V 6000 5979 50  0000 L CNN
 F 1 "D_Zener 3.6V BZT52C395" V 6045 5979 50  0001 L CNN
-F 2 "Diode_SMD:D_SOD-323" H 6000 5900 50  0001 C CNN
+F 2 "Diode_SMD:D_SOD-323_HandSoldering" H 6000 5900 50  0001 C CNN
 F 3 "https://www.application-datasheet.com/pdf/diodes/bzt52c4v7s-7-f.pdf" H 6000 5900 50  0001 C CNN
 	1    6000 5900
@@
 F 0 "D17" V 6200 5979 50  0000 L CNN
 F 1 "D_Zener 3.6V BZT52C395" V 6245 5979 50  0001 L CNN
-F 2 "Diode_SMD:D_SOD-323" H 6200 5900 50  0001 C CNN
+F 2 "Diode_SMD:D_SOD-323_HandSoldering" H 6200 5900 50  0001 C CNN
 F 3 "https://www.application-datasheet.com/pdf/diodes/bzt52c4v7s-7-f.pdf" H 6200 5900 50  0001 C CNN
 	1    6200 5900
@@
 F 0 "D19" V 6400 5979 50  0000 L CNN
 F 1 "D_Zener 3.6V BZT52C395" V 6445 5979 50  0001 L CNN
-F 2 "Diode_SMD:D_SOD-323" H 6400 5900 50  0001 C CNN
+F 2 "Diode_SMD:D_SOD-323_HandSoldering" H 6400 5900 50  0001 C CNN
 F 3 "https://www.application-datasheet.com/pdf/diodes/bzt52c4v7s-7-f.pdf" H 6400 5900 50  0001 C CNN
 	1    6400 5900
@@
 F 0 "D21" V 6600 5979 50  0000 L CNN
 F 1 "D_Zener 3.6V BZT52C395" V 6645 5979 50  0001 L CNN
-F 2 "Diode_SMD:D_SOD-323" H 6600 5900 50  0001 C CNN
+F 2 "Diode_SMD:D_SOD-323_HandSoldering" H 6600 5900 50  0001 C CNN
 F 3 "https://www.application-datasheet.com/pdf/diodes/bzt52c4v7s-7-f.pdf" H 6600 5900 50  0001 C CNN
 	1    6600 5900
@@
 F 0 "D23" V 6800 5979 50  0000 L CNN
 F 1 "D_Zener 3.6V BZT52C395" V 6845 5979 50  0001 L CNN
-F 2 "Diode_SMD:D_SOD-323" H 6800 5900 50  0001 C CNN
+F 2 "Diode_SMD:D_SOD-323_HandSoldering" H 6800 5900 50  0001 C CNN
 F 3 "https://www.application-datasheet.com/pdf/diodes/bzt52c4v7s-7-f.pdf" H 6800 5900 50  0001 C CNN
 	1    6800 5900
@@
 F 0 "D25" V 7000 5979 50  0000 L CNN
 F 1 "D_Zener 3.6V BZT52C395" V 7045 5979 50  0001 L CNN
-F 2 "Diode_SMD:D_SOD-323" H 7000 5900 50  0001 C CNN
+F 2 "Diode_SMD:D_SOD-323_HandSoldering" H 7000 5900 50  0001 C CNN
 F 3 "https://www.application-datasheet.com/pdf/diodes/bzt52c4v7s-7-f.pdf" H 7000 5900 50  0001 C CNN
 	1    7000 5900
@@
 F 0 "D27" V 7200 5979 50  0000 L CNN
 F 1 "D_Zener 3.6V BZT52C395" V 7245 5979 50  0001 L CNN
-F 2 "Diode_SMD:D_SOD-323" H 7200 5900 50  0001 C CNN
+F 2 "Diode_SMD:D_SOD-323_HandSoldering" H 7200 5900 50  0001 C CNN
 F 3 "https://www.application-datasheet.com/pdf/diodes/bzt52c4v7s-7-f.pdf" H 7200 5900 50  0001 C CNN
 	1    7200 5900

Commit message: Changed Joystick configuration to level shifting IC.
Parts:
- removed D12, D13, D14, D15, D16, D17, D18, D19, D20, D21, D22, D23, D24, D25, D26, D27: D_Zener 3.6V BZT52C395, Diode_SMD:D_SOD-323_HandSoldering, symbol Device:D_Zener
- removed R10, R11, R12, R13, R14, R15, R16, R3, R4, R5, R6, R7, R8, R9: 47K, Resistor_SMD:R_0603_1608Metric, symbol Device:R
- added C5, C50, C51, C52: 100nF, Capacitor_SMD:C_0603_1608Metric, symbol Device:C
- added F1, F2: Polyfuse 100mA, Fuse:Fuse_0805_2012Metric, symbol Device:Polyfuse
- added U8, U9: TXS0108EPWR, Package_SO:TSSOP-20_4.4x6.5mm_P0.65mm, symbol TXS0108EPWR:TXS0108EPWR
- R1, R2: value 47K -> 10K
Connections:
- net labels added: VIN5V
- net labels removed: JS1_7, JS2_7
- wire segments 134 -> 42
- no-connect marks 0 -> 4
