File: joystick.sch (KiCad schematic (older format))
At the start: 12 parts, among them J1 DB9_Male, J2 DB9_Male, U10 TXS0108EPWR, U9 TXS0108EPWR

Commit message: The DB9 connectors now have ground on the outer sleve.
Changed lines of the file:
@@
 Text GLabel 6825 6250 0    50   Input ~ 0
 VIN5V
+Text GLabel 8300 1450 1    50   Input ~ 0
+GND
+Text GLabel 8350 4550 1    50   Input ~ 0
+GND
 $EndSCHEMATC

Commit message: First checkin of SDRAM Open AARS board.
Parts:
- removed C56, C58, C59: 100nF, Capacitor_SMD:C_0603_1608Metric, symbol Device:C
- removed R1: 10k, Resistor_SMD:R_0603_1608Metric, symbol Device:R
- removed U10, U9: TXS0108EPWR, SOP65P640X120-20N, symbol TXS0108EPWR:TXS0108EPWR
- added C20, C24: 100nF, Capacitor_SMD:C_0603_1608Metric, symbol Device:C
- added R7: 10k, Resistor_SMD:R_0603_1608Metric, symbol Device:R
- added U6: TXB0106PWR, SOP65P640X120-16N, symbol TXB0106PWR:TXB0106PWR
- added U9: MCP23S17, Package_SO:SSOP-28_5.3x10.2mm_P0.65mm, symbol microchip:MCP23S17
Connections:
- net labels added: JS_CS, JS_CS_5V, JS_INTA, JS_INTA_5V, JS_INTB, JS_INTB_5V, JS_MISO, JS_MOSI, JS_SCK
- wire segments 46 -> 48
- no-connect marks 4 -> 0
Other:
- note added: "5V SPI\n"

Commit message: Implemented the Floppy interface, fixed 12V power up issue with the board.
Parts:
- added R1, R13, R14, R15, R16, R28, R29, R44, R45, R48, R49, R63, R64, R66, R67, R90: 10k, Resistor_SMD:R_0603_1608Metric, symbol Device:R
Connections:
- wire segments 48 -> 101
- no-connect marks 0 -> 2

Commit message: Version that was sent to JLCPCB 20200716.
Parts:
- removed R13, R14: 10k, Resistor_SMD:R_0603_1608Metric, symbol Device:R
- added R12, R87: 10k, Resistor_SMD:R_0603_1608Metric, symbol Device:R
Connections:
- wire segments 101 -> 92
- no-connect marks 2 -> 0
Other:
- note added: "I/O expander to SPI"
- note added: "Not strictly needed, \ncan poll with the FPGA."
Changed lines of the file:
@@
 Text Notes 3875 3225 0    50   ~ 0
 5V SPI\n
-Wire Bus Line
-	7075 4575 5500 4575
-Wire Bus Line
-	5500 4575 5500 3850
-Wire Bus Line
-	7075 4575 7075 4850
-Wire Bus Line
-	7000 1750 7000 2750
-Wire Bus Line
-	7000 2750 5500 2750
-Wire Bus Line
-	5500 2750 5500 3575
-Text GLabel 3625 3950 0    50   Input ~ 0
+Text GLabel 4500 3950 0    50   Input ~ 0
 JS_INTA_5V
-Text GLabel 3625 4050 0    50   Input ~ 0
+Text GLabel 4500 4050 0    50   Input ~ 0
 JS_INTB_5V
 $Comp
@@
 AR Path="/5D74B9F4/5F3EA536" Ref="R15"  Part="1"
 AR Path="/5DE41876/5F3EA536" Ref="R?"  Part="1"
-F 0 "R15" V 6818 1250 50  0000 C CNN
-F 1 "10k" V 6909 1250 50  0000 C CNN
+F 0 "R15" V 7025 1050 50  0000 C CNN
+F 1 "10k" V 7025 1250 50  0000 C CNN
 F 2 "Resistor_SMD:R_0603_1608Metric" V 6955 1250 50  0001 C CNN
 F 3 "~" H 7025 1250 50  0001 C CNN
@@
 AR Path="/5D74B9F4/5F3EA53C" Ref="R28"  Part="1"
 AR Path="/5DE41876/5F3EA53C" Ref="R?"  Part="1"
-F 0 "R28" V 6943 1250 50  0000 C CNN
-F 1 "10k" V 7034 1250 50  0000 C CNN
+F 0 "R28" V 7150 1050 50  0000 C CNN
+F 1 "10k" V 7150 1250 50  0000 C CNN
 F 2 "Resistor_SMD:R_0603_1608Metric" V 7080 1250 50  0001 C CNN
 F 3 "~" H 7150 1250 50  0001 C CNN
@@
 AR Path="/5D74B9F4/5F3EA542" Ref="R44"  Part="1"
 AR Path="/5DE41876/5F3EA542" Ref="R?"  Part="1"
-F 0 "R44" V 7068 1250 50  0000 C CNN
-F 1 "10k" V 7159 1250 50  0000 C CNN
+F 0 "R44" V 7275 1050 50  0000 C CNN
+F 1 "10k" V 7275 1250 50  0000 C CNN
 F 2 "Resistor_SMD:R_0603_1608Metric" V 7205 1250 50  0001 C CNN
 F 3 "~" H 7275 1250 50  0001 C CNN
@@
 AR Path="/5D74B9F4/5F3EA548" Ref="R48"  Part="1"
 AR Path="/5DE41876/5F3EA548" Ref="R?"  Part="1"
-F 0 "R48" V 7193 1250 50  0000 C CNN
-F 1 "10k" V 7284 1250 50  0000 C CNN
+F 0 "R48" V 7400 1050 50  0000 C CNN
+F 1 "10k" V 7400 1250 50  0000 C CNN
 F 2 "Resistor_SMD:R_0603_1608Metric" V 7330 1250 50  0001 C CNN
 F 3 "~" H 7400 1250 50  0001 C CNN
@@
 AR Path="/5D74B9F4/5F3EA54E" Ref="R63"  Part="1"
 AR Path="/5DE41876/5F3EA54E" Ref="R?"  Part="1"
-F 0 "R63" V 7443 1250 50  0000 C CNN
-F 1 "10k" V 7534 1250 50  0000 C CNN
+F 0 "R63" V 7650 1050 50  0000 C CNN
+F 1 "10k" V 7650 1250 50  0000 C CNN
 F 2 "Resistor_SMD:R_0603_1608Metric" V 7580 1250 50  0001 C CNN
 F 3 "~" H 7650 1250 50  0001 C CNN
@@
 AR Path="/5D74B9F4/5F3EA554" Ref="R66"  Part="1"
 AR Path="/5DE41876/5F3EA554" Ref="R?"  Part="1"
-F 0 "R66" V 7568 1250 50  0000 C CNN
-F 1 "10k" V 7659 1250 50  0000 C CNN
+F 0 "R66" V 7775 1050 50  0000 C CNN
+F 1 "10k" V 7775 1250 50  0000 C CNN
 F 2 "Resistor_SMD:R_0603_1608Metric" V 7705 1250 50  0001 C CNN
 F 3 "~" H 7775 1250 50  0001 C CNN
@@
 Text GLabel 2775 2850 2    50   Input ~ 0
 JS_MISO
-Wire Wire Line
-	4500 3950 4100 3950
-Wire Wire Line
-	4500 4050 4200 4050
 Text GLabel 3950 4675 3    50   Input ~ 0
 VIN5V
-$Comp
-L Device:R R13
-U 1 1 5F4336EA
-P 4100 4400
-AR Path="/5D74B9F4/5F4336EA" Ref="R13"  Part="1"
-AR Path="/5DE41876/5F4336EA" Ref="R?"  Part="1"
-F 0 "R13" V 4100 4525 50  0000 L CNN
-F 1 "10k" V 4100 4325 50  0000 L CNN
-F 2 "Resistor_SMD:R_0603_1608Metric" V 4030 4400 50  0001 C CNN
-F 3 "~" H 4100 4400 50  0001 C CNN
-	1    4100 4400
-	1    0    0    -1
-$EndComp
 Wire Wire Line
 	4500 4450 4425 4450
@@
 	4425 4450 4425 4550
 Wire Wire Line
-	4425 4550 4200 4550
-Wire Wire Line
-	4200 4550 4100 4550
-Connection ~ 4200 4550
-Connection ~ 4100 4550
-Wire Wire Line
 	3950 4675 3950 4550
-Wire Wire Line
-	4200 4250 4200 4050
-Connection ~ 4200 4050
-Wire Wire Line
-	4200 4050 3625 4050
-Wire Wire Line
-	4100 4250 4100 3950
-Connection ~ 4100 3950
-Wire Wire Line
-	4100 3950 3625 3950
 Connection ~ 7025 1750
 Wire Wire Line
@@
 AR Path="/5D74B9F4/5F5E0F02" Ref="R1"  Part="1"
 AR Path="/5DE41876/5F5E0F02" Ref="R?"  Part="1"
-F 0 "R1" V 7318 1250 50  0000 C CNN
-F 1 "10k" V 7409 1250 50  0000 C CNN
+F 0 "R1" V 7525 1075 50  0000 C CNN
+F 1 "10k" V 7525 1250 50  0000 C CNN
 F 2 "Resistor_SMD:R_0603_1608Metric" V 7455 1250 50  0001 C CNN
 F 3 "~" H 7525 1250 50  0001 C CNN
@@
 	7200 4500 7200 4950
 Connection ~ 7075 4850
-Wire Bus Line
-	7075 4850 7075 5450
 Wire Wire Line
 	7075 4850 8150 4850
@@
 Wire Wire Line
 	7525 1100 7650 1100
-Text GLabel 3625 3550 0    50   Input ~ 0
+Text GLabel 4500 3550 0    50   Input ~ 0
 JS_CS_5V
-$Comp
-L Device:R R14
-U 1 1 5F435F60
-P 4200 4400
-AR Path="/5D74B9F4/5F435F60" Ref="R14"  Part="1"
-AR Path="/5DE41876/5F435F60" Ref="R?"  Part="1"
-F 0 "R14" V 4200 4600 50  0000 C CNN
-F 1 "10k" V 4200 4400 50  0000 C CNN
-F 2 "Resistor_SMD:R_0603_1608Metric" V 4130 4400 50  0001 C CNN
-F 3 "~" H 4200 4400 50  0001 C CNN
-	1    4200 4400
-	1    0    0    -1
-$EndComp
+Wire Wire Line
+	2775 3450 4500 3450
+Wire Wire Line
+	2775 3350 4500 3350
+Wire Wire Line
+	2775 3250 4500 3250
+$Comp
+L Device:R R87
+U 1 1 5FC2A341
+P 5650 3750
+AR Path="/5D74B9F4/5FC2A341" Ref="R87"  Part="1"
+AR Path="/5DE41876/5FC2A341" Ref="R?"  Part="1"
+F 0 "R87" V 5725 3750 50  0000 C CNN
+F 1 "10k" V 5650 3750 50  0000 C CNN
+F 2 "Resistor_SMD:R_0603_1608Metric" V 5580 3750 50  0001 C CNN
+F 3 "~" H 5650 3750 50  0001 C CNN
+	1    5650 3750
+	0    -1   -1   0
+$EndComp
+Text GLabel 5800 3750 2    50   Input ~ 0
+GND
+$Comp
+L Device:R R12
+U 1 1 5FC2FC54
+P 5650 2850
+AR Path="/5D74B9F4/5FC2FC54" Ref="R12"  Part="1"
+AR Path="/5DE41876/5FC2FC54" Ref="R?"  Part="1"
+F 0 "R12" V 5725 2850 50  0000 C CNN
+F 1 "10k" V 5650 2850 50  0000 C CNN
+F 2 "Resistor_SMD:R_0603_1608Metric" V 5580 2850 50  0001 C CNN
+F 3 "~" H 5650 2850 50  0001 C CNN
+	1    5650 2850
+	0    -1   -1   0
+$EndComp
+Text GLabel 5800 2850 2    50   Input ~ 0
+GND
+Text Notes 4850 2350 0    50   ~ 0
+I/O expander to SPI
+Text Notes 3675 3875 0    50   ~ 0
+Not strictly needed, \ncan poll with the FPGA.
 $Comp
 L microchip:MCP23S17 U9
@@
 $EndComp
 Wire Wire Line
-	3625 3550 4500 3550
-Wire Wire Line
-	2775 3450 4500 3450
-Wire Wire Line
-	2775 3350 4500 3350
-Wire Wire Line
-	2775 3250 4500 3250
-Wire Wire Line
-	3950 4550 4100 4550
-NoConn ~ 5500 3750
-NoConn ~ 5500 2850
+	3950 4550 4425 4550
 $EndSCHEMATC
