File: joystick.sch (KiCad schematic (older format))
At the start: 27 parts, among them J1 DB9_Male, J2 DB9_Male, U6 TXB0106PWR, U9 MCP23S17

Commit message: Fixed regression from an earlier pin numbering mistake. Changed Joystick pullups for resistor network.
Parts:
- removed R1, R15, R16, R28, R29, R44, R45, R48, R49, R63, R64, R66, R67, R90: 10k, Resistor_SMD:R_0603_1608Metric, symbol Device:R
- added RN1, RN2, RN3, RN4: 10K, Resistor_SMD:R_Array_Convex_4x0603, symbol Device:R_Pack04
Connections:
- wire segments 92 -> 94

Commit message: Did some placement to make the PCB smaller.
Parts:
- U9: symbol microchip:MCP23S17 -> Interface_Expansion:MCP23S17_SO
Connections:
- wire segments 94 -> 92
Changed lines of the file:
@@
 Wire Wire Line
 	7450 5450 7450 5650
-Text GLabel 5000 2650 1    50   Input ~ 0
-GND
-Text GLabel 5000 5025 3    50   Input ~ 0
+Text GLabel 5300 5150 3    50   Input ~ 0
+GND
+Text GLabel 5300 2950 1    50   Input ~ 0
 VIN5V
 Text GLabel 8100 2250 0    50   Input ~ 0
@@
 L Device:C C57
 U 1 1 5E30EED8
-P 4850 4900
-F 0 "C57" V 4598 4900 50  0000 C CNN
-F 1 "100nF" V 4689 4900 50  0000 C CNN
-F 2 "Capacitor_SMD:C_0603_1608Metric" H 4888 4750 50  0001 C CNN
-F 3 "~" H 4850 4900 50  0001 C CNN
-	1    4850 4900
-	0    -1   -1   0
-$EndComp
-Wire Wire Line
-	5000 4650 5000 4900
-Text GLabel 4700 4900 0    50   Input ~ 0
+P 5450 2950
+F 0 "C57" V 5198 2950 50  0000 C CNN
+F 1 "100nF" V 5289 2950 50  0000 C CNN
+F 2 "Capacitor_SMD:C_0603_1608Metric" H 5488 2800 50  0001 C CNN
+F 3 "~" H 5450 2950 50  0001 C CNN
+	1    5450 2950
+	0    1    1    0
+$EndComp
+Text GLabel 5600 2950 2    50   Input ~ 0
 GND
 $Comp
@@
 Text GLabel 8350 4550 1    50   Input ~ 0
 GND
-Text GLabel 5500 4450 2    50   Input ~ 0
+Text GLabel 6000 4850 2    50   Input ~ 0
 JS2_5
-Text GLabel 5500 4350 2    50   Input ~ 0
+Text GLabel 6000 4750 2    50   Input ~ 0
 JS2_9
-Text GLabel 5500 4250 2    50   Input ~ 0
+Text GLabel 6000 4650 2    50   Input ~ 0
 JS2_4
-Text GLabel 5500 4150 2    50   Input ~ 0
+Text GLabel 6000 4550 2    50   Input ~ 0
 JS2_3
-Text GLabel 5500 4050 2    50   Input ~ 0
+Text GLabel 6000 4450 2    50   Input ~ 0
 JS2_2
-Text GLabel 5500 3950 2    50   Input ~ 0
+Text GLabel 6000 4350 2    50   Input ~ 0
 JS2_6
-Text GLabel 5500 3850 2    50   Input ~ 0
+Text GLabel 6000 4250 2    50   Input ~ 0
 JS2_1
-Text GLabel 5500 3550 2    50   Input ~ 0
+Text GLabel 6000 3950 2    50   Input ~ 0
 JS1_1
-Text GLabel 5500 3450 2    50   Input ~ 0
+Text GLabel 6000 3850 2    50   Input ~ 0
 JS1_6
-Text GLabel 5500 3350 2    50   Input ~ 0
+Text GLabel 6000 3750 2    50   Input ~ 0
 JS1_2
-Text GLabel 5500 3250 2    50   Input ~ 0
+Text GLabel 6000 3650 2    50   Input ~ 0
 JS1_3
-Text GLabel 5500 3150 2    50   Input ~ 0
+Text GLabel 6000 3550 2    50   Input ~ 0
 JS1_4
-Text GLabel 5500 3050 2    50   Input ~ 0
+Text GLabel 6000 3450 2    50   Input ~ 0
 JS1_9
-Text GLabel 5500 2950 2    50   Input ~ 0
+Text GLabel 6000 3350 2    50   Input ~ 0
 JS1_5
-Connection ~ 5000 4900
-Wire Wire Line
-	5000 4900 5000 5025
 Text Notes 3875 3225 0    50   ~ 0
 5V SPI\n
-Text GLabel 4500 3950 0    50   Input ~ 0
+Text GLabel 4600 3850 0    50   Input ~ 0
 JS_INTA_5V
-Text GLabel 4500 4050 0    50   Input ~ 0
+Text GLabel 4600 3950 0    50   Input ~ 0
 JS_INTB_5V
 $Comp
@@
 L Device:R R7
 U 1 1 5F3A2FEA
-P 4275 2950
+P 4375 4750
 AR Path="/5D74B9F4/5F3A2FEA" Ref="R7"  Part="1"
 AR Path="/5DE41876/5F3A2FEA" Ref="R?"  Part="1"
-F 0 "R7" V 4068 2950 50  0000 C CNN
-F 1 "10k" V 4159 2950 50  0000 C CNN
-F 2 "Resistor_SMD:R_0603_1608Metric" V 4205 2950 50  0001 C CNN
-F 3 "~" H 4275 2950 50  0001 C CNN
-	1    4275 2950
-	0    1    1    0
-$EndComp
-Text GLabel 4125 2950 0    50   Input ~ 0
-GND
-Wire Wire Line
-	4500 3050 4425 3050
-Wire Wire Line
-	4425 3050 4425 2950
-Wire Wire Line
-	4425 2950 4425 2850
-Wire Wire Line
-	4425 2850 4500 2850
-Connection ~ 4425 2950
-Wire Wire Line
-	4500 2950 4425 2950
+F 0 "R7" V 4168 4750 50  0000 C CNN
+F 1 "10k" V 4259 4750 50  0000 C CNN
+F 2 "Resistor_SMD:R_0603_1608Metric" V 4305 4750 50  0001 C CNN
+F 3 "~" H 4375 4750 50  0001 C CNN
+	1    4375 4750
+	0    1    1    0
+$EndComp
+Wire Wire Line
+	4600 4850 4525 4850
+Wire Wire Line
+	4525 4850 4525 4750
+Wire Wire Line
+	4525 4750 4525 4650
+Wire Wire Line
+	4525 4650 4600 4650
+Connection ~ 4525 4750
+Wire Wire Line
+	4600 4750 4525 4750
 Text GLabel 7400 1100 1    50   Input ~ 0
 J1IN5V
@@
 Text GLabel 2775 2850 2    50   Input ~ 0
 JS_MISO
-Text GLabel 3950 4675 3    50   Input ~ 0
-VIN5V
-Wire Wire Line
-	4500 4450 4425 4450
-Wire Wire Line
-	4425 4450 4425 4550
-Wire Wire Line
-	3950 4675 3950 4550
-Text GLabel 4500 3550 0    50   Input ~ 0
+Text GLabel 4200 3250 0    50   Input ~ 0
 JS_CS_5V
 Wire Wire Line
-	2775 3450 4500 3450
-Wire Wire Line
-	2775 3350 4500 3350
-Wire Wire Line
-	2775 3250 4500 3250
+	2775 3350 3350 3350
+Wire Wire Line
+	2775 3250 3350 3250
 $Comp
 L Device:R R87
 U 1 1 5FC2A341
-P 5650 3750
+P 6150 4150
 AR Path="/5D74B9F4/5FC2A341" Ref="R87"  Part="1"
 AR Path="/5DE41876/5FC2A341" Ref="R?"  Part="1"
-F 0 "R87" V 5725 3750 50  0000 C CNN
-F 1 "10k" V 5650 3750 50  0000 C CNN
-F 2 "Resistor_SMD:R_0603_1608Metric" V 5580 3750 50  0001 C CNN
-F 3 "~" H 5650 3750 50  0001 C CNN
-	1    5650 3750
+F 0 "R87" V 6225 4150 50  0000 C CNN
+F 1 "10k" V 6150 4150 50  0000 C CNN
+F 2 "Resistor_SMD:R_0603_1608Metric" V 6080 4150 50  0001 C CNN
+F 3 "~" H 6150 4150 50  0001 C CNN
+	1    6150 4150
 	0    -1   -1   0
 $EndComp
-Text GLabel 5800 3750 2    50   Input ~ 0
+Text GLabel 6300 4150 2    50   Input ~ 0
 GND
 $Comp
 L Device:R R12
 U 1 1 5FC2FC54
-P 5650 2850
+P 6150 3250
 AR Path="/5D74B9F4/5FC2FC54" Ref="R12"  Part="1"
 AR Path="/5DE41876/5FC2FC54" Ref="R?"  Part="1"
-F 0 "R12" V 5725 2850 50  0000 C CNN
-F 1 "10k" V 5650 2850 50  0000 C CNN
-F 2 "Resistor_SMD:R_0603_1608Metric" V 5580 2850 50  0001 C CNN
-F 3 "~" H 5650 2850 50  0001 C CNN
-	1    5650 2850
+F 0 "R12" V 6225 3250 50  0000 C CNN
+F 1 "10k" V 6150 3250 50  0000 C CNN
+F 2 "Resistor_SMD:R_0603_1608Metric" V 6080 3250 50  0001 C CNN
+F 3 "~" H 6150 3250 50  0001 C CNN
+	1    6150 3250
 	0    -1   -1   0
 $EndComp
-Text GLabel 5800 2850 2    50   Input ~ 0
+Text GLabel 6300 3250 2    50   Input ~ 0
 GND
 Text Notes 4850 2350 0    50   ~ 0
 I/O expander to SPI
-Text Notes 3675 3875 0    50   ~ 0
+Text Notes 3775 3775 0    50   ~ 0
 Not strictly needed, \ncan poll with the FPGA.
-$Comp
-L microchip:MCP23S17 U9
-U 1 1 5F13EE93
-P 5000 3650
-F 0 "U9" H 5000 2469 50  0000 C CNN
-F 1 "MCP23S17" H 5000 2560 50  0000 C CNN
-F 2 "Package_SO:SSOP-28_5.3x10.2mm_P0.65mm" H 5050 2700 50  0001 L CNN
-F 3 "http://ww1.microchip.com/downloads/en/DeviceDoc/20001952C.pdf" H 5250 4650 50  0001 C CNN
-	1    5000 3650
-	-1   0    0    1
-$EndComp
-Wire Wire Line
-	3950 4550 4425 4550
 Text Label 2875 3250 0    50   ~ 0
 JS_MISO_5V
@@
 Wire Wire Line
 	7425 4600 7425 5150
+$Comp
+L Interface_Expansion:MCP23S17_SO U9
+U 1 1 5F13EE93
+P 5300 4050
+F 0 "U9" H 5300 2869 50  0000 C CNN
+F 1 "MCP23S17" H 5300 2960 50  0000 C CNN
+F 2 "Package_SO:SSOP-28_5.3x10.2mm_P0.65mm" H 5350 3100 50  0001 L CNN
+F 3 "http://ww1.microchip.com/downloads/en/DeviceDoc/20001952C.pdf" H 5550 5050 50  0001 C CNN
+	1    5300 4050
+	1    0    0    -1
+$EndComp
+Wire Wire Line
+	2775 3450 3350 3450
+Wire Wire Line
+	4600 3350 4200 3350
+Wire Wire Line
+	4600 3450 4200 3450
+Wire Wire Line
+	4600 3550 4200 3550
+Wire Wire Line
+	4200 3250 4600 3250
+Text Label 4200 3350 0    50   ~ 0
+JS_SCK_5V
+Text Label 4200 3450 0    50   ~ 0
+JS_MOSI_5V
+Text Label 4200 3550 0    50   ~ 0
+JS_MISO_5V
+Text GLabel 4625 4150 0    50   Input ~ 0
+VIN5V
+Text GLabel 4225 4750 0    50   Input ~ 0
+GND
 $EndSCHEMATC

Commit message: Removed ESP32, as it's no longer needed, we have soft cores.
Parts:
- renumbered C20 to C25, C24 to C26, C57 to C27, F2 to F1, F3 to F2, J1 to J3, J2 to J4, R2 to R17, R7 to R18, R12 to R19, R87 to R20, RN1 to RN2, RN2 to RN4, RN4 to RN5, U6 to U5, U9 to U6
Changed lines of the file:
@@
 $EndDescr
 $Comp
-L Connector:DB9_Male J1
+L Connector:DB9_Male J3
 U 1 1 5D74BDB1
 P 8400 2150
-F 0 "J1" H 8580 2196 50  0000 L CNN
+F 0 "J3" H 8580 2196 50  0000 L CNN
 F 1 "DB9_Male" H 8580 2105 50  0000 L CNN
 F 2 "Connector_Dsub:DSUB-9_Male_Horizontal_P2.77x2.84mm_EdgePinOffset7.70mm_Housed_MountingHolesOffset9.12mm" H 8580 2059 50  0001 L CNN
@@
 JS1_1
 $Comp
-L Connector:DB9_Male J2
+L Connector:DB9_Male J4
 U 1 1 5D78EA68
 P 8450 5250
-F 0 "J2" H 8630 5296 50  0000 L CNN
+F 0 "J4" H 8630 5296 50  0000 L CNN
 F 1 "DB9_Male" H 8630 5205 50  0000 L CNN
 F 2 "Connector_Dsub:DSUB-9_Male_Horizontal_P2.77x2.84mm_EdgePinOffset7.70mm_Housed_MountingHolesOffset9.12mm" H 8630 5159 50  0001 L CNN
@@
 	7400 2350 7400 2550
 $Comp
-L Device:C C57
+L Device:C C27
 U 1 1 5E30EED8
 P 5450 2950
-F 0 "C57" V 5198 2950 50  0000 C CNN
+F 0 "C27" V 5198 2950 50  0000 C CNN
 F 1 "100nF" V 5289 2950 50  0000 C CNN
 F 2 "Capacitor_SMD:C_0603_1608Metric" H 5488 2800 50  0001 C CNN
@@
 GND
 $Comp
-L Device:Polyfuse F3
+L Device:Polyfuse F2
 U 1 1 5E31E80F
 P 7250 3000
-F 0 "F3" V 7025 3000 50  0000 C CNN
+F 0 "F2" V 7025 3000 50  0000 C CNN
 F 1 "100mA" V 7116 3000 50  0000 C CNN
 F 2 "Fuse:Fuse_0805_2012Metric" H 7300 2800 50  0001 L CNN
@@
 VIN5V
 $Comp
-L Device:Polyfuse F2
+L Device:Polyfuse F1
 U 1 1 5E320D9B
 P 6975 6250
-F 0 "F2" V 6750 6250 50  0000 C CNN
+F 0 "F1" V 6750 6250 50  0000 C CNN
 F 1 "100mA" V 6841 6250 50  0000 C CNN
 F 2 "Fuse:Fuse_0805_2012Metric" H 7025 6050 50  0001 L CNN
@@
 JS_INTB_5V
 $Comp
-L Device:C C24
+L Device:C C26
 U 1 1 5F31A37C
 P 3325 1850
-F 0 "C24" V 3073 1850 50  0000 C CNN
+F 0 "C26" V 3073 1850 50  0000 C CNN
 F 1 "100nF" V 3164 1850 50  0000 C CNN
 F 2 "Capacitor_SMD:C_0603_1608Metric" H 3363 1700 50  0001 C CNN
@@
 GND
 $Comp
-L Device:R R7
+L Device:R R18
 U 1 1 5F3A2FEA
 P 4375 4750
-AR Path="/5D74B9F4/5F3A2FEA" Ref="R7"  Part="1"
+AR Path="/5D74B9F4/5F3A2FEA" Ref="R18"  Part="1"
 AR Path="/5DE41876/5F3A2FEA" Ref="R?"  Part="1"
-F 0 "R7" V 4168 4750 50  0000 C CNN
+F 0 "R18" V 4168 4750 50  0000 C CNN
 F 1 "10k" V 4259 4750 50  0000 C CNN
 F 2 "Resistor_SMD:R_0603_1608Metric" V 4305 4750 50  0001 C CNN
@@
 GND
 $Comp
-L Device:C C20
+L Device:C C25
 U 1 1 5F319691
 P 2600 1850
-F 0 "C20" V 2348 1850 50  0000 C CNN
+F 0 "C25" V 2348 1850 50  0000 C CNN
 F 1 "100nF" V 2439 1850 50  0000 C CNN
 F 2 "Capacitor_SMD:C_0603_1608Metric" H 2638 1700 50  0001 C CNN
@@
 JS_INTA
 $Comp
-L TXB0106PWR:TXB0106PWR U6
+L TXB0106PWR:TXB0106PWR U5
 U 1 1 5F2E87E4
 P 2075 3050
-F 0 "U6" H 2075 4020 50  0000 C CNN
+F 0 "U5" H 2075 4020 50  0000 C CNN
 F 1 "TXB0106PWR" H 2075 3929 50  0000 C CNN
 F 2 "SOP65P640X120-16N" H 2075 3050 50  0001 L BNN
@@
 3V3
 $Comp
-L Device:R R2
+L Device:R R17
 U 1 1 5F2DF875
 P 1225 2650
-F 0 "R2" V 1018 2650 50  0000 C CNN
+F 0 "R17" V 1018 2650 50  0000 C CNN
 F 1 "10k" V 1109 2650 50  0000 C CNN
 F 2 "Resistor_SMD:R_0603_1608Metric" V 1155 2650 50  0001 C CNN
@@
 	2775 3250 3350 3250
 $Comp
-L Device:R R87
+L Device:R R20
 U 1 1 5FC2A341
 P 6150 4150
-AR Path="/5D74B9F4/5FC2A341" Ref="R87"  Part="1"
+AR Path="/5D74B9F4/5FC2A341" Ref="R20"  Part="1"
 AR Path="/5DE41876/5FC2A341" Ref="R?"  Part="1"
-F 0 "R87" V 6225 4150 50  0000 C CNN
+F 0 "R20" V 6225 4150 50  0000 C CNN
 F 1 "10k" V 6150 4150 50  0000 C CNN
 F 2 "Resistor_SMD:R_0603_1608Metric" V 6080 4150 50  0001 C CNN
@@
 GND
 $Comp
-L Device:R R12
+L Device:R R19
 U 1 1 5FC2FC54
 P 6150 3250
-AR Path="/5D74B9F4/5FC2FC54" Ref="R12"  Part="1"
+AR Path="/5D74B9F4/5FC2FC54" Ref="R19"  Part="1"
 AR Path="/5DE41876/5FC2FC54" Ref="R?"  Part="1"
-F 0 "R12" V 6225 3250 50  0000 C CNN
+F 0 "R19" V 6225 3250 50  0000 C CNN
 F 1 "10k" V 6150 3250 50  0000 C CNN
 F 2 "Resistor_SMD:R_0603_1608Metric" V 6080 3250 50  0001 C CNN
@@
 JS_SCK_5V
 $Comp
-L Device:R_Pack04 RN1
+L Device:R_Pack04 RN2
 U 1 1 5F73821B
 P 7225 1300
-F 0 "RN1" H 7413 1346 50  0000 L CNN
+F 0 "RN2" H 7413 1346 50  0000 L CNN
 F 1 "10K" H 7413 1255 50  0000 L CNN
 F 2 "Resistor_SMD:R_Array_Convex_4x0603" V 7500 1300 50  0001 C CNN
@@
 	7225 1100 7325 1100
 $Comp
-L Device:R_Pack04 RN2
+L Device:R_Pack04 RN4
 U 1 1 5F76013F
 P 7825 1300
-F 0 "RN2" H 8013 1346 50  0000 L CNN
+F 0 "RN4" H 8013 1346 50  0000 L CNN
 F 1 "10K" H 8013 1255 50  0000 L CNN
 F 2 "Resistor_SMD:R_Array_Convex_4x0603" V 8100 1300 50  0001 C CNN
@@
 	7325 4200 7425 4200
 $Comp
-L Device:R_Pack04 RN4
+L Device:R_Pack04 RN5
 U 1 1 5F831CB4
 P 7925 4400
-F 0 "RN4" H 8113 4446 50  0000 L CNN
+F 0 "RN5" H 8113 4446 50  0000 L CNN
 F 1 "10K" H 8113 4355 50  0000 L CNN
 F 2 "Resistor_SMD:R_Array_Convex_4x0603" V 8200 4400 50  0001 C CNN
@@
 	7425 4600 7425 5150
 $Comp
-L Interface_Expansion:MCP23S17_SO U9
+L Interface_Expansion:MCP23S17_SO U6
 U 1 1 5F13EE93
 P 5300 4050
-F 0 "U9" H 5300 2869 50  0000 C CNN
+F 0 "U6" H 5300 2869 50  0000 C CNN
 F 1 "MCP23S17" H 5300 2960 50  0000 C CNN
 F 2 "Package_SO:SSOP-28_5.3x10.2mm_P0.65mm" H 5350 3100 50  0001 L CNN

Commit message: Fixed decoupling of VDD SDRAM, fixed pinout error in V4 board pinout sheet.
Changed lines of the file:
@@
 Text GLabel 7050 5450 0    50   Input ~ 0
 JS2_1
-Text GLabel 7050 5750 2    50   Input ~ 0
-GND
 Text GLabel 8150 5350 0    50   Input ~ 0
 J2IN5V
@@
 VIN5V
 Text GLabel 8300 1450 1    50   Input ~ 0
-GND
-Text GLabel 8350 4550 1    50   Input ~ 0
 GND
 Text GLabel 6000 4850 2    50   Input ~ 0
@@
 Text Label 4200 3550 0    50   ~ 0
 JS_MISO_5V
-Text GLabel 4625 4150 0    50   Input ~ 0
+Text GLabel 4600 4150 0    50   Input ~ 0
 VIN5V
 Text GLabel 4225 4750 0    50   Input ~ 0
