File: keyboard.sch (KiCad schematic (older format))
At the start: 1 part, among them J6 Mini-DIN-6

Commit message: Connected adv7511 unused inputs to ground. Added high voltage protection on PS2 port. Added indicators for the rubber glue on feet.
Parts:
- added D28, D29: 3.6V, Diode_SMD:D_SOD-323, symbol Device:D_Zener
Connections:
- wire segments 4 -> 6
Changed lines of the file:
@@
 Title ""
 Date ""
-Rev ""
-Comp ""
+Rev "0.1"
+Comp "deFEEST"
 Comment1 ""
 Comment2 ""
@@
 $EndComp
 Wire Wire Line
-	5150 3150 4800 3150
+	5150 3150 4950 3150
 Wire Wire Line
-	5150 2950 4800 2950
+	5150 2950 4950 2950
 Wire Wire Line
 	5150 3050 4800 3050
@@
 Text GLabel 5150 2950 2    50   Input ~ 0
 PS2_CLK1
+$Comp
+L Device:D_Zener D28
+U 1 1 5D7D382B
+P 4950 2800
+F 0 "D28" V 4996 2721 50  0000 R CNN
+F 1 "3.6V" V 4905 2721 50  0000 R CNN
+F 2 "Diode_SMD:D_SOD-323" H 4950 2800 50  0001 C CNN
+F 3 "~" H 4950 2800 50  0001 C CNN
+	1    4950 2800
+	0    -1   -1   0
+$EndComp
+Connection ~ 4950 2950
+Wire Wire Line
+	4950 2950 4800 2950
+Text GLabel 4950 2650 1    50   Input ~ 0
+GND
+$Comp
+L Device:D_Zener D29
+U 1 1 5D7D3DDC
+P 4950 3300
+F 0 "D29" V 4904 3379 50  0000 L CNN
+F 1 "3.6V" V 4995 3379 50  0000 L CNN
+F 2 "Diode_SMD:D_SOD-323" H 4950 3300 50  0001 C CNN
+F 3 "~" H 4950 3300 50  0001 C CNN
+	1    4950 3300
+	0    1    1    0
+$EndComp
+Connection ~ 4950 3150
+Wire Wire Line
+	4950 3150 4800 3150
+Text GLabel 4950 3450 3    50   Input ~ 0
+GND
 $EndSCHEMATC

Commit message: Fixed some issues with the 50 Ohm impedance of the SPI lines. Added pinout .odt.
Parts:
- added C46: 10uF, Capacitor_SMD:C_0805_2012Metric, symbol Device:C
- added R? (x2): 330, Resistor_SMD:R_0603_1608Metric, symbol Device:R
Connections:
- wire segments 6 -> 9
- no-connect marks 0 -> 3
Changed lines of the file:
@@
 $EndComp
 Wire Wire Line
-	5150 3150 4950 3150
-Wire Wire Line
-	5150 2950 4950 2950
-Wire Wire Line
-	5150 3050 4800 3050
-Wire Wire Line
-	3900 3050 4200 3050
-Text GLabel 3900 3050 0    50   Input ~ 0
+	3750 3050 3850 3050
+Text GLabel 3750 3050 0    50   Input ~ 0
 VIN5V
-Text GLabel 5150 3050 2    50   Input ~ 0
+Text GLabel 5525 3050 2    50   Input ~ 0
 GND
-Text GLabel 5150 3150 2    50   Input ~ 0
+Text GLabel 5525 3150 2    50   Input ~ 0
 PS2_DAT1
-Text GLabel 5150 2950 2    50   Input ~ 0
+Text GLabel 5525 2950 2    50   Input ~ 0
 PS2_CLK1
 $Comp
 L Device:D_Zener D28
 U 1 1 5D7D382B
-P 4950 2800
-F 0 "D28" V 4996 2721 50  0000 R CNN
-F 1 "3.6V" V 4905 2721 50  0000 R CNN
-F 2 "Diode_SMD:D_SOD-323" H 4950 2800 50  0001 C CNN
-F 3 "~" H 4950 2800 50  0001 C CNN
-	1    4950 2800
+P 5375 2800
+F 0 "D28" V 5421 2721 50  0000 R CNN
+F 1 "3.6V" V 5330 2721 50  0000 R CNN
+F 2 "Diode_SMD:D_SOD-323" H 5375 2800 50  0001 C CNN
+F 3 "~" H 5375 2800 50  0001 C CNN
+	1    5375 2800
 	0    -1   -1   0
 $EndComp
-Connection ~ 4950 2950
 Wire Wire Line
 	4950 2950 4800 2950
-Text GLabel 4950 2650 1    50   Input ~ 0
+Text GLabel 5375 2650 1    50   Input ~ 0
 GND
 $Comp
 L Device:D_Zener D29
 U 1 1 5D7D3DDC
-P 4950 3300
-F 0 "D29" V 4904 3379 50  0000 L CNN
-F 1 "3.6V" V 4995 3379 50  0000 L CNN
-F 2 "Diode_SMD:D_SOD-323" H 4950 3300 50  0001 C CNN
-F 3 "~" H 4950 3300 50  0001 C CNN
-	1    4950 3300
+P 5375 3300
+F 0 "D29" V 5329 3379 50  0000 L CNN
+F 1 "3.6V" V 5420 3379 50  0000 L CNN
+F 2 "Diode_SMD:D_SOD-323" H 5375 3300 50  0001 C CNN
+F 3 "~" H 5375 3300 50  0001 C CNN
+	1    5375 3300
 	0    1    1    0
 $EndComp
-Connection ~ 4950 3150
+Text GLabel 5375 3450 3    50   Input ~ 0
+GND
+$Comp
+L Device:C C46
+U 1 1 5DB2AAC3
+P 3850 3200
+F 0 "C46" H 3965 3246 50  0000 L CNN
+F 1 "10uF" H 3965 3155 50  0000 L CNN
+F 2 "Capacitor_SMD:C_0805_2012Metric" H 3888 3050 50  0001 C CNN
+F 3 "~" H 3850 3200 50  0001 C CNN
+	1    3850 3200
+	1    0    0    -1
+$EndComp
+Text GLabel 3850 3350 3    50   Input ~ 0
+GND
+Connection ~ 3850 3050
 Wire Wire Line
-	4950 3150 4800 3150
-Text GLabel 4950 3450 3    50   Input ~ 0
-GND
+	3850 3050 4200 3050
+NoConn ~ 4200 2950
+NoConn ~ 4200 3150
+NoConn ~ 4750 3300
+$Comp
+L Device:R R?
+U 1 1 5DB2DE3D
+P 5100 2950
+F 0 "R?" V 5025 2950 50  0000 C CNN
+F 1 "330" V 5100 2950 50  0000 C CNN
+F 2 "Resistor_SMD:R_0603_1608Metric" V 5030 2950 50  0001 C CNN
+F 3 "~" H 5100 2950 50  0001 C CNN
+	1    5100 2950
+	0    1    1    0
+$EndComp
+Wire Wire Line
+	5250 2950 5375 2950
+Connection ~ 5375 2950
+Wire Wire Line
+	5375 2950 5525 2950
+$Comp
+L Device:R R?
+U 1 1 5DB31CC1
+P 5100 3150
+F 0 "R?" V 5025 3150 50  0000 C CNN
+F 1 "330" V 5100 3150 50  0000 C CNN
+F 2 "Resistor_SMD:R_0603_1608Metric" V 5030 3150 50  0001 C CNN
+F 3 "~" H 5100 3150 50  0001 C CNN
+	1    5100 3150
+	0    1    1    0
+$EndComp
+Wire Wire Line
+	5525 3050 4800 3050
+Wire Wire Line
+	4800 3150 4950 3150
+Wire Wire Line
+	5250 3150 5375 3150
+Connection ~ 5375 3150
+Wire Wire Line
+	5375 3150 5525 3150
 $EndSCHEMATC

Commit message: Removed an extra esp32 footprint that was outside of the design.
Parts:
- gave numbers to parts that had none: 2
Changed lines of the file:
@@
 NoConn ~ 4750 3300
 $Comp
-L Device:R R?
+L Device:R R46
 U 1 1 5DB2DE3D
 P 5100 2950
-F 0 "R?" V 5025 2950 50  0000 C CNN
+F 0 "R46" V 5025 2950 50  0000 C CNN
 F 1 "330" V 5100 2950 50  0000 C CNN
 F 2 "Resistor_SMD:R_0603_1608Metric" V 5030 2950 50  0001 C CNN
@@
 	5375 2950 5525 2950
 $Comp
-L Device:R R?
+L Device:R R47
 U 1 1 5DB31CC1
 P 5100 3150
-F 0 "R?" V 5025 3150 50  0000 C CNN
+F 0 "R47" V 5025 3150 50  0000 C CNN
 F 1 "330" V 5100 3150 50  0000 C CNN
 F 2 "Resistor_SMD:R_0603_1608Metric" V 5030 3150 50  0001 C CNN

Commit message: Changed zener diode footprint for easy soldering. Fixed pins, U861/2 and U761/2 they now connect correctly to ground.
Parts:
- D28, D29: footprint Diode_SMD:D_SOD-323 -> Diode_SMD:D_SOD-323_HandSoldering
Changed lines of the file:
@@
 EESchema Schematic File Version 4
-LIBS:qmtech-minimig-cache
 EELAYER 30 0
 EELAYER END
@@
 F 0 "D28" V 5421 2721 50  0000 R CNN
 F 1 "3.6V" V 5330 2721 50  0000 R CNN
-F 2 "Diode_SMD:D_SOD-323" H 5375 2800 50  0001 C CNN
+F 2 "Diode_SMD:D_SOD-323_HandSoldering" H 5375 2800 50  0001 C CNN
 F 3 "~" H 5375 2800 50  0001 C CNN
 	1    5375 2800
@@
 F 0 "D29" V 5329 3379 50  0000 L CNN
 F 1 "3.6V" V 5420 3379 50  0000 L CNN
-F 2 "Diode_SMD:D_SOD-323" H 5375 3300 50  0001 C CNN
+F 2 "Diode_SMD:D_SOD-323_HandSoldering" H 5375 3300 50  0001 C CNN
 F 3 "~" H 5375 3300 50  0001 C CNN
 	1    5375 3300

Commit message: Changed Joystick configuration to level shifting IC.
Parts:
- added F3: Polyfuse 100mA, Fuse:Fuse_0805_2012Metric, symbol Device:Polyfuse
Connections:
- wire segments 9 -> 10
- no-connect marks 3 -> 2
Changed lines of the file:
@@
 Wire Wire Line
 	3750 3050 3850 3050
-Text GLabel 3750 3050 0    50   Input ~ 0
+Text GLabel 3300 3050 0    50   Input ~ 0
 VIN5V
 Text GLabel 5525 3050 2    50   Input ~ 0
@@
 NoConn ~ 4200 2950
 NoConn ~ 4200 3150
-NoConn ~ 4750 3300
 $Comp
 L Device:R R46
@@
 Wire Wire Line
 	5375 3150 5525 3150
+$Comp
+L Device:Polyfuse F?
+U 1 1 5E09EDF9
+P 3600 3050
+AR Path="/5D74B9F4/5E09EDF9" Ref="F?"  Part="1"
+AR Path="/5DC624E5/5E09EDF9" Ref="F3"  Part="1"
+F 0 "F3" V 3375 3050 50  0000 C CNN
+F 1 "Polyfuse 100mA" V 3466 3050 50  0000 C CNN
+F 2 "Fuse:Fuse_0805_2012Metric" H 3650 2850 50  0001 L CNN
+F 3 "~" H 3600 3050 50  0001 C CNN
+	1    3600 3050
+	0    1    1    0
+$EndComp
+Wire Wire Line
+	3450 3050 3300 3050
 $EndSCHEMATC
