File: keyboard.sch (KiCad schematic (older format))
At the start: 14 parts, among them P1 Mini-DIN_6pins_ver3, P2 Mini-DIN_6pins_ver3

Commit message: Revert "Fixed some external dependencies."
This reverts commit ddca1efdf68af69ddd54947bcdaa3cfa1d913e0d.
Parts:
- C43, C46: symbol qmtech-minimig-rescue:C-Device -> Device:C
- D12, D13, D28, D29: symbol qmtech-minimig-rescue:D_Zener-Device -> Device:D_Zener
- F4, F5: symbol qmtech-minimig-rescue:Polyfuse-Device -> Device:Polyfuse
- R4, R46, R47, R5: symbol qmtech-minimig-rescue:R-Device -> Device:R
Changed lines of the file:
@@
 GND
 $Comp
-L qmtech-minimig-rescue:C-Device C46
+L Device:C C46
 U 1 1 5DB2AAC3
 P 3850 3200
@@
 	5525 3050 4800 3050
 $Comp
-L qmtech-minimig-rescue:Polyfuse-Device F4
+L Device:Polyfuse F4
 U 1 1 5E3388F3
 P 3600 3050
@@
 PS2_DAT1
 $Comp
-L qmtech-minimig-rescue:D_Zener-Device D29
+L Device:D_Zener D29
 U 1 1 5D7D3DDC
 P 5375 3400
@@
 GND
 $Comp
-L qmtech-minimig-rescue:R-Device R47
+L Device:R R47
 U 1 1 5DB31CC1
 P 5100 3250
@@
 PS2_CLK1
 $Comp
-L qmtech-minimig-rescue:D_Zener-Device D28
+L Device:D_Zener D28
 U 1 1 5D7D382B
 P 5375 2700
@@
 GND
 $Comp
-L qmtech-minimig-rescue:R-Device R46
+L Device:R R46
 U 1 1 5DB2DE3D
 P 5100 2850
@@
 GND
 $Comp
-L qmtech-minimig-rescue:C-Device C43
+L Device:C C43
 U 1 1 5E56B0B8
 P 3850 5375
@@
 	5525 5225 4800 5225
 $Comp
-L qmtech-minimig-rescue:Polyfuse-Device F5
+L Device:Polyfuse F5
 U 1 1 5E56B0C4
 P 3600 5225
@@
 PS2_DAT2
 $Comp
-L qmtech-minimig-rescue:D_Zener-Device D13
+L Device:D_Zener D13
 U 1 1 5E56B0D1
 P 5375 5575
@@
 GND
 $Comp
-L qmtech-minimig-rescue:R-Device R5
+L Device:R R5
 U 1 1 5E56B0D8
 P 5100 5425
@@
 PS2_CLK2
 $Comp
-L qmtech-minimig-rescue:D_Zener-Device D12
+L Device:D_Zener D12
 U 1 1 5E56B0E3
 P 5375 4875
@@
 GND
 $Comp
-L qmtech-minimig-rescue:R-Device R4
+L Device:R R4
 U 1 1 5E56B0EB
 P 5100 5025

Commit message: Fixed some external dependencies.
Parts:
- C43, C46: symbol Device:C -> qmtech-minimig-rescue:C-Device
- D12, D13, D28, D29: symbol Device:D_Zener -> qmtech-minimig-rescue:D_Zener-Device
- F4, F5: symbol Device:Polyfuse -> qmtech-minimig-rescue:Polyfuse-Device
- R4, R46, R47, R5: symbol Device:R -> qmtech-minimig-rescue:R-Device
Changed lines of the file:
@@
 GND
 $Comp
-L Device:C C46
+L qmtech-minimig-rescue:C-Device C46
 U 1 1 5DB2AAC3
 P 3850 3200
@@
 	5525 3050 4800 3050
 $Comp
-L Device:Polyfuse F4
+L qmtech-minimig-rescue:Polyfuse-Device F4
 U 1 1 5E3388F3
 P 3600 3050
@@
 PS2_DAT1
 $Comp
-L Device:D_Zener D29
+L qmtech-minimig-rescue:D_Zener-Device D29
 U 1 1 5D7D3DDC
 P 5375 3400
@@
 GND
 $Comp
-L Device:R R47
+L qmtech-minimig-rescue:R-Device R47
 U 1 1 5DB31CC1
 P 5100 3250
@@
 PS2_CLK1
 $Comp
-L Device:D_Zener D28
+L qmtech-minimig-rescue:D_Zener-Device D28
 U 1 1 5D7D382B
 P 5375 2700
@@
 GND
 $Comp
-L Device:R R46
+L qmtech-minimig-rescue:R-Device R46
 U 1 1 5DB2DE3D
 P 5100 2850
@@
 GND
 $Comp
-L Device:C C43
+L qmtech-minimig-rescue:C-Device C43
 U 1 1 5E56B0B8
 P 3850 5375
@@
 	5525 5225 4800 5225
 $Comp
-L Device:Polyfuse F5
+L qmtech-minimig-rescue:Polyfuse-Device F5
 U 1 1 5E56B0C4
 P 3600 5225
@@
 PS2_DAT2
 $Comp
-L Device:D_Zener D13
+L qmtech-minimig-rescue:D_Zener-Device D13
 U 1 1 5E56B0D1
 P 5375 5575
@@
 GND
 $Comp
-L Device:R R5
+L qmtech-minimig-rescue:R-Device R5
 U 1 1 5E56B0D8
 P 5100 5425
@@
 PS2_CLK2
 $Comp
-L Device:D_Zener D12
+L qmtech-minimig-rescue:D_Zener-Device D12
 U 1 1 5E56B0E3
 P 5375 4875
@@
 GND
 $Comp
-L Device:R R4
+L qmtech-minimig-rescue:R-Device R4
 U 1 1 5E56B0EB
 P 5100 5025
