File: keyboard.sch (KiCad schematic (older format))
At the start: 14 parts, among them P1 Mini-DIN_6pins_ver3, P2 Mini-DIN_6pins_ver3

Commit message: Removed ESP32, as it's no longer needed, we have soft cores.
Parts:
- renumbered C46 to C42, D12 to D10, D13 to D11, D28 to D8, D29 to D9, F4 to F3, F5 to F4, R46 to R27, R47 to R28, R4 to R29, R5 to R30
Changed lines of the file:
@@
 GND
 $Comp
-L Device:C C46
+L Device:C C42
 U 1 1 5DB2AAC3
 P 3850 3200
-F 0 "C46" H 3965 3246 50  0000 L CNN
+F 0 "C42" H 3965 3246 50  0000 L CNN
 F 1 "10uF" H 3965 3155 50  0000 L CNN
 F 2 "Capacitor_SMD:C_0805_2012Metric" H 3888 3050 50  0001 C CNN
@@
 	5525 3050 4800 3050
 $Comp
-L Device:Polyfuse F4
+L Device:Polyfuse F3
 U 1 1 5E3388F3
 P 3600 3050
-F 0 "F4" V 3375 3050 50  0000 C CNN
+F 0 "F3" V 3375 3050 50  0000 C CNN
 F 1 "0.35A" V 3466 3050 50  0000 C CNN
 F 2 "Fuse:Fuse_0805_2012Metric" H 3650 2850 50  0001 L CNN
@@
 PS2_DAT1
 $Comp
-L Device:D_Zener D29
+L Device:D_Zener D9
 U 1 1 5D7D3DDC
 P 5375 3400
-F 0 "D29" V 5329 3479 50  0000 L CNN
+F 0 "D9" V 5329 3479 50  0000 L CNN
 F 1 "3.6V" V 5420 3479 50  0000 L CNN
 F 2 "Diode_SMD:D_SOD-323_HandSoldering" H 5375 3400 50  0001 C CNN
@@
 GND
 $Comp
-L Device:R R47
+L Device:R R28
 U 1 1 5DB31CC1
 P 5100 3250
-F 0 "R47" V 5025 3250 50  0000 C CNN
+F 0 "R28" V 5025 3250 50  0000 C CNN
 F 1 "330" V 5100 3250 50  0000 C CNN
 F 2 "Resistor_SMD:R_0603_1608Metric" V 5030 3250 50  0001 C CNN
@@
 PS2_CLK1
 $Comp
-L Device:D_Zener D28
+L Device:D_Zener D8
 U 1 1 5D7D382B
 P 5375 2700
-F 0 "D28" V 5421 2621 50  0000 R CNN
+F 0 "D8" V 5421 2621 50  0000 R CNN
 F 1 "3.6V" V 5330 2621 50  0000 R CNN
 F 2 "Diode_SMD:D_SOD-323_HandSoldering" H 5375 2700 50  0001 C CNN
@@
 GND
 $Comp
-L Device:R R46
+L Device:R R27
 U 1 1 5DB2DE3D
 P 5100 2850
-F 0 "R46" V 5025 2850 50  0000 C CNN
+F 0 "R27" V 5025 2850 50  0000 C CNN
 F 1 "330" V 5100 2850 50  0000 C CNN
 F 2 "Resistor_SMD:R_0603_1608Metric" V 5030 2850 50  0001 C CNN
@@
 	5525 5225 4800 5225
 $Comp
-L Device:Polyfuse F5
+L Device:Polyfuse F4
 U 1 1 5E56B0C4
 P 3600 5225
-F 0 "F5" V 3375 5225 50  0000 C CNN
+F 0 "F4" V 3375 5225 50  0000 C CNN
 F 1 "0.35A" V 3466 5225 50  0000 C CNN
 F 2 "Fuse:Fuse_0805_2012Metric" H 3650 5025 50  0001 L CNN
@@
 PS2_DAT2
 $Comp
-L Device:D_Zener D13
+L Device:D_Zener D11
 U 1 1 5E56B0D1
 P 5375 5575
-F 0 "D13" V 5329 5654 50  0000 L CNN
+F 0 "D11" V 5329 5654 50  0000 L CNN
 F 1 "3.6V" V 5420 5654 50  0000 L CNN
 F 2 "Diode_SMD:D_SOD-323_HandSoldering" H 5375 5575 50  0001 C CNN
@@
 GND
 $Comp
-L Device:R R5
+L Device:R R30
 U 1 1 5E56B0D8
 P 5100 5425
-F 0 "R5" V 5025 5425 50  0000 C CNN
+F 0 "R30" V 5025 5425 50  0000 C CNN
 F 1 "330" V 5100 5425 50  0000 C CNN
 F 2 "Resistor_SMD:R_0603_1608Metric" V 5030 5425 50  0001 C CNN
@@
 PS2_CLK2
 $Comp
-L Device:D_Zener D12
+L Device:D_Zener D10
 U 1 1 5E56B0E3
 P 5375 4875
-F 0 "D12" V 5421 4796 50  0000 R CNN
+F 0 "D10" V 5421 4796 50  0000 R CNN
 F 1 "3.6V" V 5330 4796 50  0000 R CNN
 F 2 "Diode_SMD:D_SOD-323_HandSoldering" H 5375 4875 50  0001 C CNN
@@
 GND
 $Comp
-L Device:R R4
+L Device:R R29
 U 1 1 5E56B0EB
 P 5100 5025
-F 0 "R4" V 5025 5025 50  0000 C CNN
+F 0 "R29" V 5025 5025 50  0000 C CNN
 F 1 "330" V 5100 5025 50  0000 C CNN
 F 2 "Resistor_SMD:R_0603_1608Metric" V 5030 5025 50  0001 C CNN

Commit message: Fixed issue with missing PS2 pullups, add line to adv interrupt.
Parts:
- added R60, R61, R62, R63: 2k7, Resistor_SMD:R_0603_1608Metric, symbol Device:R
Connections:
- net labels added: 3V3
- wire segments 18 -> 22
Changed lines of the file:
@@
 $EndComp
 Wire Wire Line
-	4800 3250 4950 3250
+	4800 3250 4925 3250
 Wire Wire Line
 	5250 3250 5375 3250
@@
 P 4500 5225
 F 0 "P2" H 4500 5696 50  0000 C CNN
-F 1 "Mini-DIN_6pins_ver3" H 4500 5605 50  0000 C CNN
+F 1 "Mini-DIN_6pins_ver3" H 4500 5600 50  0000 C CNN
 F 2 "Custom_Footprints:Connector_Mini-DIN_Female_6Pin_2rows" H 4500 5514 50  0000 C CNN
 F 3 "" H 4500 5245 50  0000 C CNN
@@
 	0    1    1    0
 $EndComp
-Wire Wire Line
-	4800 5425 4950 5425
 Wire Wire Line
 	5250 5425 5375 5425
@@
 	0    -1   -1   0
 $EndComp
-Wire Wire Line
-	4950 5025 4800 5025
 Text GLabel 5375 4725 1    50   Input ~ 0
 GND
@@
 Text Notes 4500 2250 0    50   ~ 0
 Keyboard PS/2
-Text Notes 4500 4500 0    50   ~ 0
+Text Notes 4575 4500 0    50   ~ 0
 Mouse PS/2
+$Comp
+L Device:R R61
+U 1 1 60495A98
+P 4925 5575
+F 0 "R61" V 4850 5575 50  0000 C CNN
+F 1 "2k7" V 4925 5575 50  0000 C CNN
+F 2 "Resistor_SMD:R_0603_1608Metric" V 4855 5575 50  0001 C CNN
+F 3 "~" H 4925 5575 50  0001 C CNN
+	1    4925 5575
+	1    0    0    -1
+$EndComp
+Text GLabel 4925 5725 3    50   Input ~ 0
+3V3
+$Comp
+L Device:R R63
+U 1 1 60499475
+P 4950 4725
+F 0 "R63" V 4875 4725 50  0000 C CNN
+F 1 "2k7" V 4950 4725 50  0000 C CNN
+F 2 "Resistor_SMD:R_0603_1608Metric" V 4880 4725 50  0001 C CNN
+F 3 "~" H 4950 4725 50  0001 C CNN
+	1    4950 4725
+	-1   0    0    1
+$EndComp
+Text GLabel 4950 4575 1    50   Input ~ 0
+3V3
+Wire Wire Line
+	4950 4875 4950 5025
+Text Notes 4575 2325 0    50   ~ 0
+Mouse PS/2
+$Comp
+L Device:R R62
+U 1 1 6049DC6A
+P 4950 2550
+F 0 "R62" V 4875 2550 50  0000 C CNN
+F 1 "2k7" V 4950 2550 50  0000 C CNN
+F 2 "Resistor_SMD:R_0603_1608Metric" V 4880 2550 50  0001 C CNN
+F 3 "~" H 4950 2550 50  0001 C CNN
+	1    4950 2550
+	-1   0    0    1
+$EndComp
+Text GLabel 4950 2400 1    50   Input ~ 0
+3V3
+Wire Wire Line
+	4950 2700 4950 2850
+Connection ~ 4950 5025
+Wire Wire Line
+	4800 5025 4950 5025
+Connection ~ 4925 5425
+Wire Wire Line
+	4925 5425 4950 5425
+Wire Wire Line
+	4800 5425 4925 5425
+$Comp
+L Device:R R60
+U 1 1 604A3ADC
+P 4925 3400
+F 0 "R60" V 4850 3400 50  0000 C CNN
+F 1 "2k7" V 4925 3400 50  0000 C CNN
+F 2 "Resistor_SMD:R_0603_1608Metric" V 4855 3400 50  0001 C CNN
+F 3 "~" H 4925 3400 50  0001 C CNN
+	1    4925 3400
+	1    0    0    -1
+$EndComp
+Text GLabel 4925 3550 3    50   Input ~ 0
+3V3
+Connection ~ 4925 3250
+Wire Wire Line
+	4925 3250 4950 3250
+Connection ~ 4950 2850
 $EndSCHEMATC
