File: audio.sch (KiCad schematic (older format))
At the start: 5 parts, among them J5 AUDIO-CONNECTOR-6P-SMD-344003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

Commit message: Add the External floppy interface. Routed the HDMI tracks + match impendence.
Parts:
- C27, C28: footprint Capacitor_SMD:C_0603_1608Metric -> Capacitor_SMD:C_0805_2012Metric
Changed lines of the file:
@@
 F 0 "C27" V 3398 3000 50  0000 C CNN
 F 1 "4700pF" V 3489 3000 50  0000 C CNN
-F 2 "Capacitor_SMD:C_0603_1608Metric" H 3688 2850 50  0001 C CNN
+F 2 "Capacitor_SMD:C_0805_2012Metric" H 3688 2850 50  0001 C CNN
 F 3 "~" H 3650 3000 50  0001 C CNN
 	1    3650 3000
@@
 F 0 "C28" V 5948 3150 50  0000 C CNN
 F 1 "4700pF" V 6039 3150 50  0000 C CNN
-F 2 "Capacitor_SMD:C_0603_1608Metric" H 6238 3000 50  0001 C CNN
+F 2 "Capacitor_SMD:C_0805_2012Metric" H 6238 3000 50  0001 C CNN
 F 3 "~" H 6200 3150 50  0001 C CNN
 	1    6200 3150

Commit message: Add Max9850 to handle audio.
Parts:
- removed R28, R29: 3.3K, Resistor_SMD:R_0603_1608Metric, symbol Device:R
- added C5: 10nF, Capacitor_SMD:C_0603_1608Metric, symbol Device:C
- added C50: 0.47uF, Capacitor_SMD:C_0603_1608Metric, symbol Device:C
- added C51, C53, C54, C55: 1uF, Capacitor_SMD:C_0603_1608Metric, symbol Device:C
- added C52: 2.2uF, Capacitor_SMD:C_0805_2012Metric, symbol Device:C
- added U8: INTERFACE-MAX9850ETI+-(QFN28), Package_DFN_QFN:QFN-28-1EP_5x5mm_P0.5mm_EP3.35x3.35mm, symbol max98089:INTERFACE-MAX9850ETI+-(QFN28)
- added X2: SG-210STF, Oscillator:Oscillator_SMD_SeikoEpson_SG210-4Pin_2.5x2.0mm, symbol Oscillator:SG-210STF
- C27, C28: value 4700pF -> 1uF; footprint Capacitor_SMD:C_0805_2012Metric -> Capacitor_SMD:C_0603_1608Metric
Connections:
- net labels added: 3V3, ADV_SCL, ADV_SDA, HPL, HPR, HPS, MAX_I2S0, MAX_LRCLK, MAX_SCLK
- net labels removed: AUDIO_LEFT, AUDIO_RIGHT
- wire segments 9 -> 23
- no-connect marks 0 -> 5

Commit message: Joystick port 7 is not powered at 5V, polyfuses have been added, txs0108 are used for the joystick ports.
Parts:
- X2: value SG-210STF -> 11.2896MHz
Changed lines of the file:
@@
 P 2775 3650
 F 0 "X2" H 3119 3696 50  0000 L CNN
-F 1 "SG-210STF" H 3119 3605 50  0000 L CNN
+F 1 "11.2896MHz" H 3119 3605 50  0000 L CNN
 F 2 "Oscillator:Oscillator_SMD_SeikoEpson_SG210-4Pin_2.5x2.0mm" H 3225 3300 50  0001 C CNN
 F 3 "https://support.epson.biz/td/api/doc_check.php?mode=dl&lang=en&Parts=SG-210STF" H 2675 3650 50  0001 C CNN

Commit message: Change order of the VSPI to FPGA to make sure the clock pin connects to an FPGA clock capable pin.
Changed lines of the file:
@@
 Text GLabel 5775 4925 3    50   Input ~ 0
 GND
-Wire Wire Line
-	5475 2750 5475 1875
-Text GLabel 5475 1725 1    50   Input ~ 0
+Text GLabel 5475 1625 1    50   Input ~ 0
 3V3
 $Comp
 L Device:C C28
 U 1 1 5E238986
-P 5625 1875
-F 0 "C28" H 5740 1921 50  0000 L CNN
-F 1 "1uF" H 5740 1830 50  0000 L CNN
-F 2 "Capacitor_SMD:C_0603_1608Metric" H 5663 1725 50  0001 C CNN
-F 3 "~" H 5625 1875 50  0001 C CNN
-	1    5625 1875
+P 5625 1675
+F 0 "C28" H 5740 1721 50  0000 L CNN
+F 1 "1uF" H 5740 1630 50  0000 L CNN
+F 2 "Capacitor_SMD:C_0603_1608Metric" H 5663 1525 50  0001 C CNN
+F 3 "~" H 5625 1675 50  0001 C CNN
+	1    5625 1675
 	0    1    1    0
 $EndComp
-Text GLabel 5775 1875 2    50   Input ~ 0
+Text GLabel 5775 1675 2    50   Input ~ 0
 GND
-Connection ~ 5475 1875
 Wire Wire Line
-	5475 1875 5475 1725
-Wire Wire Line
-	6375 3650 7825 3650
+	6375 3650 7875 3650
 Text GLabel 7975 3650 2    50   Input ~ 0
 3V3
@@
 L Device:C C55
 U 1 1 5E23909A
-P 7825 3800
-F 0 "C55" H 7940 3846 50  0000 L CNN
-F 1 "1uF" H 7940 3755 50  0000 L CNN
-F 2 "Capacitor_SMD:C_0603_1608Metric" H 7863 3650 50  0001 C CNN
-F 3 "~" H 7825 3800 50  0001 C CNN
-	1    7825 3800
+P 7875 3800
+F 0 "C55" H 7990 3846 50  0000 L CNN
+F 1 "1uF" H 7990 3755 50  0000 L CNN
+F 2 "Capacitor_SMD:C_0603_1608Metric" H 7913 3650 50  0001 C CNN
+F 3 "~" H 7875 3800 50  0001 C CNN
+	1    7875 3800
 	-1   0    0    1
 $EndComp
-Text GLabel 7825 3950 3    50   Input ~ 0
+Text GLabel 7875 3950 3    50   Input ~ 0
 GND
-Connection ~ 7825 3650
+Connection ~ 7875 3650
 Wire Wire Line
-	7825 3650 7975 3650
+	7875 3650 7975 3650
 Wire Wire Line
 	6375 3750 7250 3750
@@
 	-1   0    0    1
 $EndComp
+Wire Wire Line
+	5475 1625 5475 1675
+Connection ~ 5475 1675
+Wire Wire Line
+	5475 1675 5475 2750
 $EndSCHEMATC
