File: audio.sch (KiCad schematic (older format))
At the start: 15 parts, among them J5 AUDIO-CONNECTOR-6P-SMD-344003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, U8 INTERFACE-MAX9850ETI+-(QFN28), X2 11.2896MHz

Commit message: Removed all libraries that depend on absolute paths.
Parts:
- J5: symbol BPS6001_Classic_Computing_Shield-eagle-import:AUDIO-CONNECTOR-6P-SMD-3440030P1 -> qmtech-minimig-rescue:AUDIO-CONNECTOR-6P-SMD-3440030P1-BPS6001_Classic_Computing_Shield-eagle-import
- U8: symbol max98089:INTERFACE-MAX9850ETI+-(QFN28) -> qmtech-minimig-rescue:INTERFACE-MAX9850ETI+-(QFN28)-max98089
Changed lines of the file:
@@
 $EndDescr
 $Comp
-L BPS6001_Classic_Computing_Shield-eagle-import:AUDIO-CONNECTOR-6P-SMD-3440030P1 J5
+L qmtech-minimig-rescue:AUDIO-CONNECTOR-6P-SMD-3440030P1-BPS6001_Classic_Computing_Shield-eagle-import J5
 U 1 1 5DC6A556
 P 9900 3500
@@
 GND
 $Comp
-L max98089:INTERFACE-MAX9850ETI+-(QFN28) U8
+L qmtech-minimig-rescue:INTERFACE-MAX9850ETI+-(QFN28)-max98089 U8
 U 1 1 5E228931
 P 5575 3550
