File: audio.sch (KiCad schematic (older format))
At the start: 12 parts, among them J5 AUDIO-CONNECTOR-6P-SMD-344003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, U8 INTERFACE-MAX9850ETI+-(QFN28), X2 11.2896MHz

Commit message: Add 3d models to most components, Add decoupling of the Line ins of the max9850. Add new defeest Logos.
Parts:
- added C45, C60: 100nF, Capacitor_SMD:C_0603_1608Metric, symbol Device:C
Connections:
- wire segments 23 -> 26
- no-connect marks 5 -> 3
Other:
- note added: "Decouple Line ins"
- note added: "I2S to FPGA"
- note added: "Negative voltage pump"
Changed lines of the file:
@@
 Text GLabel 5875 4350 3    50   Input ~ 0
 GND
-NoConn ~ 5375 4350
-NoConn ~ 5475 4350
+NoConn ~ 5675 4350
 NoConn ~ 5575 4350
-NoConn ~ 5675 4350
 Text GLabel 5175 2750 1    50   Input ~ 0
 GND
@@
 Wire Wire Line
 	5775 4350 5775 4625
+Wire Wire Line
+	5475 1625 5475 1675
+Connection ~ 5475 1675
+Wire Wire Line
+	5475 1675 5475 2750
+$Comp
+L Device:C C45
+U 1 1 5E664493
+P 5375 5175
+F 0 "C45" H 5490 5221 50  0000 L CNN
+F 1 "100nF" H 5490 5130 50  0000 L CNN
+F 2 "Capacitor_SMD:C_0603_1608Metric" H 5413 5025 50  0001 C CNN
+F 3 "~" H 5375 5175 50  0001 C CNN
+	1    5375 5175
+	-1   0    0    1
+$EndComp
+$Comp
+L Device:C C60
+U 1 1 5E664499
+P 5475 4925
+F 0 "C60" H 5590 4971 50  0000 L CNN
+F 1 "100nF" H 5590 4880 50  0000 L CNN
+F 2 "Capacitor_SMD:C_0603_1608Metric" H 5513 4775 50  0001 C CNN
+F 3 "~" H 5475 4925 50  0001 C CNN
+	1    5475 4925
+	-1   0    0    1
+$EndComp
+Text GLabel 5475 5325 3    50   Input ~ 0
+GND
+Text GLabel 5375 5325 3    50   Input ~ 0
+GND
+Wire Wire Line
+	5475 5075 5475 5325
 $Comp
 L Device:C C51
@@
 $EndComp
 Wire Wire Line
-	5475 1625 5475 1675
-Connection ~ 5475 1675
+	5375 4350 5375 5025
 Wire Wire Line
-	5475 1675 5475 2750
+	5475 4350 5475 4775
+Text Notes 5125 5625 0    50   ~ 0
+Decouple Line ins
+Text Notes 5900 2775 0    50   ~ 0
+Negative voltage pump
+Text Notes 4300 3175 0    50   ~ 0
+I2S to FPGA
 $EndSCHEMATC

Commit message: Implemented the Floppy interface, fixed 12V power up issue with the board.
Parts:
- added R9: 10k, Resistor_SMD:R_0603_1608Metric, symbol Device:R
Changed lines of the file:
@@
 Text GLabel 3075 3175 2    50   Input ~ 0
 GND
-Text GLabel 2475 3650 0    50   Input ~ 0
+Text GLabel 2175 3650 0    50   Input ~ 0
 3V3
 Text GLabel 5275 2750 1    50   Input ~ 0
@@
 Text Notes 4300 3175 0    50   ~ 0
 I2S to FPGA
+$Comp
+L Device:R R9
+U 1 1 5FBC48A3
+P 2325 3650
+F 0 "R9" V 2118 3650 50  0000 C CNN
+F 1 "10k" V 2209 3650 50  0000 C CNN
+F 2 "Resistor_SMD:R_0603_1608Metric" V 2255 3650 50  0001 C CNN
+F 3 "~" H 2325 3650 50  0001 C CNN
+	1    2325 3650
+	0    1    1    0
+$EndComp
 $EndSCHEMATC

Commit message: Fixed some external dependencies.
Parts:
- C27, C28, C45, C5, C50, C51, C52, C53, C54, C55, C60: symbol Device:C -> qmtech-minimig-rescue:C-Device
- R9: symbol Device:R -> qmtech-minimig-rescue:R-Device
- X2: symbol Oscillator:SG-210STF -> qmtech-minimig-rescue:SG-210STF-Oscillator
Changed lines of the file:
@@
 HPS
 $Comp
-L Device:C C53
+L qmtech-minimig-rescue:C-Device C53
 U 1 1 5E230840
 P 6625 4000
@@
 3V3
 $Comp
-L Device:C C27
+L qmtech-minimig-rescue:C-Device C27
 U 1 1 5E23398A
 P 3900 3400
@@
 3V3
 $Comp
-L Device:C C28
+L qmtech-minimig-rescue:C-Device C28
 U 1 1 5E238986
 P 5625 1675
@@
 3V3
 $Comp
-L Device:C C55
+L qmtech-minimig-rescue:C-Device C55
 U 1 1 5E23909A
 P 7875 3800
@@
 3V3
 $Comp
-L Device:C C54
+L qmtech-minimig-rescue:C-Device C54
 U 1 1 5E23F5E7
 P 7250 3900
@@
 	7250 3750 7400 3750
 $Comp
-L Device:C C50
+L qmtech-minimig-rescue:C-Device C50
 U 1 1 5E249C1F
 P 5750 2250
@@
 	5875 2650 5875 2750
 $Comp
-L Device:C C52
+L qmtech-minimig-rescue:C-Device C52
 U 1 1 5E24C1DB
 P 6500 2500
@@
 GND
 $Comp
-L Oscillator:SG-210STF X2
+L qmtech-minimig-rescue:SG-210STF-Oscillator X2
 U 1 1 5E2537D2
 P 2775 3650
@@
 3V3
 $Comp
-L Device:C C5
+L qmtech-minimig-rescue:C-Device C5
 U 1 1 5E2567D0
 P 2925 3175
@@
 	5475 1675 5475 2750
 $Comp
-L Device:C C45
+L qmtech-minimig-rescue:C-Device C45
 U 1 1 5E664493
 P 5375 5175
@@
 $EndComp
 $Comp
-L Device:C C60
+L qmtech-minimig-rescue:C-Device C60
 U 1 1 5E664499
 P 5475 4925
@@
 	5475 5075 5475 5325
 $Comp
-L Device:C C51
+L qmtech-minimig-rescue:C-Device C51
 U 1 1 5E23572F
 P 5775 4775
@@
 I2S to FPGA
 $Comp
-L Device:R R9
+L qmtech-minimig-rescue:R-Device R9
 U 1 1 5FBC48A3
 P 2325 3650

Commit message: Revert "Fixed some external dependencies."
This reverts commit ddca1efdf68af69ddd54947bcdaa3cfa1d913e0d.
Parts:
- C27, C28, C45, C5, C50, C51, C52, C53, C54, C55, C60: symbol qmtech-minimig-rescue:C-Device -> Device:C
- R9: symbol qmtech-minimig-rescue:R-Device -> Device:R
- X2: symbol qmtech-minimig-rescue:SG-210STF-Oscillator -> Oscillator:SG-210STF
Changed lines of the file:
@@
 HPS
 $Comp
-L qmtech-minimig-rescue:C-Device C53
+L Device:C C53
 U 1 1 5E230840
 P 6625 4000
@@
 3V3
 $Comp
-L qmtech-minimig-rescue:C-Device C27
+L Device:C C27
 U 1 1 5E23398A
 P 3900 3400
@@
 3V3
 $Comp
-L qmtech-minimig-rescue:C-Device C28
+L Device:C C28
 U 1 1 5E238986
 P 5625 1675
@@
 3V3
 $Comp
-L qmtech-minimig-rescue:C-Device C55
+L Device:C C55
 U 1 1 5E23909A
 P 7875 3800
@@
 3V3
 $Comp
-L qmtech-minimig-rescue:C-Device C54
+L Device:C C54
 U 1 1 5E23F5E7
 P 7250 3900
@@
 	7250 3750 7400 3750
 $Comp
-L qmtech-minimig-rescue:C-Device C50
+L Device:C C50
 U 1 1 5E249C1F
 P 5750 2250
@@
 	5875 2650 5875 2750
 $Comp
-L qmtech-minimig-rescue:C-Device C52
+L Device:C C52
 U 1 1 5E24C1DB
 P 6500 2500
@@
 GND
 $Comp
-L qmtech-minimig-rescue:SG-210STF-Oscillator X2
+L Oscillator:SG-210STF X2
 U 1 1 5E2537D2
 P 2775 3650
@@
 3V3
 $Comp
-L qmtech-minimig-rescue:C-Device C5
+L Device:C C5
 U 1 1 5E2567D0
 P 2925 3175
@@
 	5475 1675 5475 2750
 $Comp
-L qmtech-minimig-rescue:C-Device C45
+L Device:C C45
 U 1 1 5E664493
 P 5375 5175
@@
 $EndComp
 $Comp
-L qmtech-minimig-rescue:C-Device C60
+L Device:C C60
 U 1 1 5E664499
 P 5475 4925
@@
 	5475 5075 5475 5325
 $Comp
-L qmtech-minimig-rescue:C-Device C51
+L Device:C C51
 U 1 1 5E23572F
 P 5775 4775
@@
 I2S to FPGA
 $Comp
-L qmtech-minimig-rescue:R-Device R9
+L Device:R R9
 U 1 1 5FBC48A3
 P 2325 3650

Commit message: First rough version of the Open AARS V4
Changed lines of the file:
@@
 L BPS6001_Classic_Computing_Shield-eagle-import:AUDIO-CONNECTOR-6P-SMD-3440030P1 J5
 U 1 1 5DC6A556
-P 9900 3500
-F 0 "J5" V 9203 3500 42  0000 C CNN
-F 1 "AUDIO-CONNECTOR-6P-SMD-3440030P1" V 9282 3500 42  0000 C CNN
-F 2 "c64-wing-kicad:6P-SMD-3.5" H 9900 3500 50  0001 C CNN
-F 3 "" H 9900 3500 50  0001 C CNN
-	1    9900 3500
-	-1   0    0    1
+P 9600 3100
+F 0 "J5" V 8903 3100 42  0000 C CNN
+F 1 "AUDIO-CONNECTOR-6P-SMD-3440030P1" V 8982 3100 42  0000 C CNN
+F 2 "c64-wing-kicad:6P-SMD-3.5" H 9600 3100 50  0001 C CNN
+F 3 "" H 9600 3100 50  0001 C CNN
+	1    9600 3100
+	1    0    0    -1
 $EndComp
-Text GLabel 9450 3100 1    50   Input ~ 0
+Text GLabel 10050 3500 3    50   Input ~ 0
 GND
-Text GLabel 9550 3900 3    50   Input ~ 0
+Text GLabel 9950 2700 1    50   Input ~ 0
 GND
 $Comp
@@
 	1    0    0    -1
 $EndComp
-Text GLabel 9750 3900 3    50   Input ~ 0
+Text GLabel 9750 2700 1    50   Input ~ 0
 HPR
-Text GLabel 10150 3100 1    50   Input ~ 0
+Text GLabel 9350 3500 3    50   Input ~ 0
 HPL
 Text GLabel 6375 3550 2    50   Input ~ 0
@@
 Text GLabel 6375 3250 2    50   Input ~ 0
 HPS
-Text GLabel 10350 3100 1    50   Input ~ 0
+Text GLabel 9150 3500 3    50   Input ~ 0
 HPS
 $Comp

Commit message: Brought compenents back to the front for easy soldering.
Connections:
- net labels added: MAX_OSC
Changed lines of the file:
@@
 	0    1    1    0
 $EndComp
+Text Label 4175 3650 2    50   ~ 0
+MAX_OSC
 $EndSCHEMATC

Commit message: Removed ESP32, as it's no longer needed, we have soft cores.
Parts:
- renumbered C5 to C31, C27 to C32, C45 to C33, C60 to C34, C28 to C35, C50 to C36, C51 to C37, C52 to C38, C53 to C39, C54 to C40, C55 to C41, J5 to J6, R9 to R26, U8 to U7, X2 to X1
Changed lines of the file:
@@
 $EndDescr
 $Comp
-L BPS6001_Classic_Computing_Shield-eagle-import:AUDIO-CONNECTOR-6P-SMD-3440030P1 J5
+L BPS6001_Classic_Computing_Shield-eagle-import:AUDIO-CONNECTOR-6P-SMD-3440030P1 J6
 U 1 1 5DC6A556
 P 9600 3100
-F 0 "J5" V 8903 3100 42  0000 C CNN
+F 0 "J6" V 8903 3100 42  0000 C CNN
 F 1 "AUDIO-CONNECTOR-6P-SMD-3440030P1" V 8982 3100 42  0000 C CNN
 F 2 "c64-wing-kicad:6P-SMD-3.5" H 9600 3100 50  0001 C CNN
@@
 GND
 $Comp
-L max98089:INTERFACE-MAX9850ETI+-(QFN28) U8
+L max98089:INTERFACE-MAX9850ETI+-(QFN28) U7
 U 1 1 5E228931
 P 5575 3550
-F 0 "U8" H 6419 3596 50  0000 L CNN
+F 0 "U7" H 6419 3596 50  0000 L CNN
 F 1 "INTERFACE-MAX9850ETI+-(QFN28)" H 4900 3975 50  0000 L CNN
 F 2 "Package_DFN_QFN:QFN-28-1EP_5x5mm_P0.5mm_EP3.35x3.35mm" H 5175 3550 50  0001 L BNN
@@
 HPS
 $Comp
-L Device:C C53
+L Device:C C39
 U 1 1 5E230840
 P 6625 4000
-F 0 "C53" H 6740 4046 50  0000 L CNN
+F 0 "C39" H 6740 4046 50  0000 L CNN
 F 1 "1uF" H 6740 3955 50  0000 L CNN
 F 2 "Capacitor_SMD:C_0603_1608Metric" H 6663 3850 50  0001 C CNN
@@
 3V3
 $Comp
-L Device:C C27
+L Device:C C32
 U 1 1 5E23398A
 P 3900 3400
-F 0 "C27" H 4015 3446 50  0000 L CNN
+F 0 "C32" H 4015 3446 50  0000 L CNN
 F 1 "1uF" H 4015 3355 50  0000 L CNN
 F 2 "Capacitor_SMD:C_0603_1608Metric" H 3938 3250 50  0001 C CNN
@@
 3V3
 $Comp
-L Device:C C28
+L Device:C C35
 U 1 1 5E238986
 P 5625 1675
-F 0 "C28" H 5740 1721 50  0000 L CNN
+F 0 "C35" H 5740 1721 50  0000 L CNN
 F 1 "1uF" H 5740 1630 50  0000 L CNN
 F 2 "Capacitor_SMD:C_0603_1608Metric" H 5663 1525 50  0001 C CNN
@@
 3V3
 $Comp
-L Device:C C55
+L Device:C C41
 U 1 1 5E23909A
 P 7875 3800
-F 0 "C55" H 7990 3846 50  0000 L CNN
+F 0 "C41" H 7990 3846 50  0000 L CNN
 F 1 "1uF" H 7990 3755 50  0000 L CNN
 F 2 "Capacitor_SMD:C_0603_1608Metric" H 7913 3650 50  0001 C CNN
@@
 3V3
 $Comp
-L Device:C C54
+L Device:C C40
 U 1 1 5E23F5E7
 P 7250 3900
-F 0 "C54" H 7365 3946 50  0000 L CNN
+F 0 "C40" H 7365 3946 50  0000 L CNN
 F 1 "1uF" H 7365 3855 50  0000 L CNN
 F 2 "Capacitor_SMD:C_0603_1608Metric" H 7288 3750 50  0001 C CNN
@@
 	7250 3750 7400 3750
 $Comp
-L Device:C C50
+L Device:C C36
 U 1 1 5E249C1F
 P 5750 2250
-F 0 "C50" V 5498 2250 50  0000 C CNN
+F 0 "C36" V 5498 2250 50  0000 C CNN
 F 1 "0.47uF" V 5589 2250 50  0000 C CNN
 F 2 "Capacitor_SMD:C_0603_1608Metric" H 5788 2100 50  0001 C CNN
@@
 	5875 2650 5875 2750
 $Comp
-L Device:C C52
+L Device:C C38
 U 1 1 5E24C1DB
 P 6500 2500
-F 0 "C52" H 6615 2546 50  0000 L CNN
+F 0 "C38" H 6615 2546 50  0000 L CNN
 F 1 "2.2uF" H 6615 2455 50  0000 L CNN
 F 2 "Capacitor_SMD:C_0805_2012Metric" H 6538 2350 50  0001 C CNN
@@
 GND
 $Comp
-L Oscillator:SG-210STF X2
+L Oscillator:SG-210STF X1
 U 1 1 5E2537D2
 P 2775 3650
-F 0 "X2" H 3119 3696 50  0000 L CNN
+F 0 "X1" H 3119 3696 50  0000 L CNN
 F 1 "11.2896MHz" H 3119 3605 50  0000 L CNN
 F 2 "Oscillator:Oscillator_SMD_SeikoEpson_SG210-4Pin_2.5x2.0mm" H 3225 3300 50  0001 C CNN
@@
 3V3
 $Comp
-L Device:C C5
+L Device:C C31
 U 1 1 5E2567D0
 P 2925 3175
-F 0 "C5" V 3177 3175 50  0000 C CNN
+F 0 "C31" V 3177 3175 50  0000 C CNN
 F 1 "10nF" V 3086 3175 50  0000 C CNN
 F 2 "Capacitor_SMD:C_0603_1608Metric" H 2963 3025 50  0001 C CNN
@@
 	5475 1675 5475 2750
 $Comp
-L Device:C C45
+L Device:C C33
 U 1 1 5E664493
 P 5375 5175
-F 0 "C45" H 5490 5221 50  0000 L CNN
+F 0 "C33" H 5490 5221 50  0000 L CNN
 F 1 "100nF" H 5490 5130 50  0000 L CNN
 F 2 "Capacitor_SMD:C_0603_1608Metric" H 5413 5025 50  0001 C CNN
@@
 $EndComp
 $Comp
-L Device:C C60
+L Device:C C34
 U 1 1 5E664499
 P 5475 4925
-F 0 "C60" H 5590 4971 50  0000 L CNN
+F 0 "C34" H 5590 4971 50  0000 L CNN
 F 1 "100nF" H 5590 4880 50  0000 L CNN
 F 2 "Capacitor_SMD:C_0603_1608Metric" H 5513 4775 50  0001 C CNN
@@
 	5475 5075 5475 5325
 $Comp
-L Device:C C51
+L Device:C C37
 U 1 1 5E23572F
 P 5775 4775
-F 0 "C51" H 5890 4821 50  0000 L CNN
+F 0 "C37" H 5890 4821 50  0000 L CNN
 F 1 "1uF" H 5890 4730 50  0000 L CNN
 F 2 "Capacitor_SMD:C_0603_1608Metric" H 5813 4625 50  0001 C CNN
@@
 I2S to FPGA
 $Comp
-L Device:R R9
+L Device:R R26
 U 1 1 5FBC48A3
 P 2325 3650
-F 0 "R9" V 2118 3650 50  0000 C CNN
+F 0 "R26" V 2118 3650 50  0000 C CNN
 F 1 "10k" V 2209 3650 50  0000 C CNN
 F 2 "Resistor_SMD:R_0603_1608Metric" V 2255 3650 50  0001 C CNN
