File: floppy.sch (KiCad schematic (older format))
At the start: 1 part, among them J7 Conn_02x13_Odd_Even

Commit message: Integrated the Rover V2 into the board, added level shifters for the floppy interface.
Parts:
- added C13, C16, C18, C20, C24, C25, C26: 100nF, Capacitor_SMD:C_0603_1608Metric, symbol Device:C
- added C14, C15, C17, C19: 22uF, Capacitor_SMD:C_0805_2012Metric, symbol Device:C
- added D3: SS34_Zener, Diode_SMD:D_SMC, symbol Device:D_Zener
- added J8: Conn_01x04, Connectors:JST-4-PTH-VERT, symbol Connector_Generic:Conn_01x04
- added L5: 22uH, CDRH104RNP-220NC:INDPM102100X400N, symbol Device:L
- added R35: 63k, Resistor_SMD:R_0603_1608Metric, symbol Device:R
- added R36: 3.3k, Resistor_SMD:R_0603_1608Metric, symbol Device:R
- added R37: 10k, Resistor_SMD:R_0603_1608Metric, symbol Device:R
- added U5: MT3608, Package_TO_SOT_SMD:SOT-23-6, symbol MT3608:MT3608
- added U6, U7: TXS0108EPWR, SOP65P640X120-20N, symbol TXS0108EPWR:TXS0108EPWR
Connections:
- net labels added: 3V3, H_EXP_02, H_EXP_04, H_EXP_06, H_EXP_08, H_EXP_10, H_EXP_12, H_EXP_14, H_EXP_16, H_EXP_18, H_EXP_20, H_EXP_22, H_EXP_24, H_EXP_26, H_EXP_28, H_EXP_30, H_EXP_32, H_EXP_34, VIN12V, VIN5V
- net labels removed: EXP_06, EXP_14
- wire segments 0 -> 57

Commit message: Add the External floppy interface. Routed the HDMI tracks + match impendence.
Parts:
- added J10: DB23_Female_MountingHoles, c64-wing-kicad:DSUB-23_Female_Horizontal_P2.77x2.84mm_EdgePinOffset7.70mm_Housed_MountingHolesOffset9.12mm, symbol qmtech-minimig-rescue:DB23_Female_MountingHoles
- added J11: Conn_01x03_Male, Connector_PinHeader_2.54mm:PinHeader_1x03_P2.54mm_Vertical, symbol Connector:Conn_01x03_Male
Connections:
- net labels added: EXP_35, H_EXP_35, VIOSEL
Other:
- note added: "Voltage selector\ndisk I/O 3V3 / 5V"
Changed lines of the file:
@@
 Text GLabel 8050 1550 2    50   Input ~ 0
 3V3
-Text GLabel 8050 1650 2    50   Input ~ 0
-VIN5V
 Text GLabel 6400 1850 0    50   Input ~ 0
 3V3
@@
 Text GLabel 7950 1000 1    50   Input ~ 0
 GND
-Text GLabel 7400 2050 2    50   Input ~ 0
+Text GLabel 7400 2750 2    50   Input ~ 0
 H_EXP_02
-Text GLabel 7400 2150 2    50   Input ~ 0
+Text GLabel 7400 2650 2    50   Input ~ 0
 H_EXP_04
+Text GLabel 7400 2350 2    50   Input ~ 0
+H_EXP_12
 Text GLabel 7400 2250 2    50   Input ~ 0
-H_EXP_08
-Text GLabel 7400 2350 2    50   Input ~ 0
-H_EXP_10
-Text GLabel 7400 2450 2    50   Input ~ 0
-H_EXP_12
-Text GLabel 7400 2550 2    50   Input ~ 0
 H_EXP_16
-Text GLabel 6400 2050 0    50   Input ~ 0
+Text GLabel 6400 2750 0    50   Input ~ 0
 EXP_02
-Text GLabel 6400 2150 0    50   Input ~ 0
+Text GLabel 6400 2650 0    50   Input ~ 0
 EXP_04
+Text GLabel 6400 2550 0    50   Input ~ 0
+EXP_08
+Text GLabel 6400 2450 0    50   Input ~ 0
+EXP_10
+Text GLabel 6400 2350 0    50   Input ~ 0
+EXP_12
 Text GLabel 6400 2250 0    50   Input ~ 0
-EXP_08
-Text GLabel 6400 2350 0    50   Input ~ 0
-EXP_10
-Text GLabel 6400 2450 0    50   Input ~ 0
-EXP_12
-Text GLabel 6400 2550 0    50   Input ~ 0
 EXP_16
 Text GLabel 8100 4250 2    50   Input ~ 0
 3V3
-Text GLabel 8100 4350 2    50   Input ~ 0
-VIN5V
 Text GLabel 6450 4550 0    50   Input ~ 0
 3V3
@@
 Text GLabel 8000 3700 1    50   Input ~ 0
 GND
+Text GLabel 7450 4950 2    50   Input ~ 0
+H_EXP_32
+Text GLabel 7450 5050 2    50   Input ~ 0
+H_EXP_30
+Text GLabel 7450 5150 2    50   Input ~ 0
+H_EXP_28
 Text GLabel 7450 5250 2    50   Input ~ 0
+H_EXP_26
+Text GLabel 7450 5350 2    50   Input ~ 0
+H_EXP_24
+Text GLabel 7450 5450 2    50   Input ~ 0
+H_EXP_22
+Text GLabel 7400 2050 2    50   Input ~ 0
+H_EXP_20
+Text GLabel 7400 2150 2    50   Input ~ 0
+H_EXP_18
+Text GLabel 6450 4950 0    50   Input ~ 0
+EXP_32
+Text GLabel 6450 5050 0    50   Input ~ 0
+EXP_30
+Text GLabel 6450 5150 0    50   Input ~ 0
+EXP_28
+Text GLabel 6450 5250 0    50   Input ~ 0
+EXP_26
+Text GLabel 6450 5350 0    50   Input ~ 0
+EXP_24
+Text GLabel 6450 5450 0    50   Input ~ 0
+EXP_22
+Text GLabel 6400 2050 0    50   Input ~ 0
+EXP_20
+Text GLabel 6400 2150 0    50   Input ~ 0
+EXP_18
+Text GLabel 6450 4850 0    50   Input ~ 0
+EXP_34
+Text GLabel 7450 4850 2    50   Input ~ 0
+H_EXP_34
+$Comp
+L qmtech-minimig-rescue:DB23_Female_MountingHoles J10
+U 1 1 5D9CC860
+P 1150 2700
+F 0 "J10" H 1329 2684 50  0000 L CNN
+F 1 "DB23_Female_MountingHoles" H 1329 2775 50  0000 L CNN
+F 2 "c64-wing-kicad:DSUB-23_Female_Horizontal_P2.77x2.84mm_EdgePinOffset7.70mm_Housed_MountingHolesOffset9.12mm" H 1150 2700 50  0001 C CNN
+F 3 " ~" H 1150 2700 50  0001 C CNN
+	1    1150 2700
+	-1   0    0    1
+$EndComp
+Text GLabel 1450 1700 2    50   Input ~ 0
+VIN5V
+Text GLabel 1450 1800 2    50   Input ~ 0
+VIN12V
+Text GLabel 1450 3500 2    50   Input ~ 0
+GND
+Text GLabel 1450 3300 2    50   Input ~ 0
+GND
+Text GLabel 1450 3100 2    50   Input ~ 0
+GND
+Text GLabel 1450 2900 2    50   Input ~ 0
+GND
+Text GLabel 1450 2700 2    50   Input ~ 0
+GND
+Text GLabel 7400 2450 2    50   Input ~ 0
+H_EXP_10
+Text GLabel 7400 2550 2    50   Input ~ 0
+H_EXP_08
+Text Label 8100 4350 0    50   ~ 0
+VIOSEL
+Text Label 8050 1650 0    50   ~ 0
+VIOSEL
+$Comp
+L Connector:Conn_01x03_Male J11
+U 1 1 5DA5CD20
+P 10000 2650
+F 0 "J11" H 9972 2582 50  0000 R CNN
+F 1 "Conn_01x03_Male" H 9972 2673 50  0000 R CNN
+F 2 "Connector_PinHeader_2.54mm:PinHeader_1x03_P2.54mm_Vertical" H 10000 2650 50  0001 C CNN
+F 3 "~" H 10000 2650 50  0001 C CNN
+	1    10000 2650
+	-1   0    0    1
+$EndComp
+Text Label 9800 2650 2    50   ~ 0
+VIOSEL
+Text GLabel 9800 2550 0    50   Input ~ 0
+3V3
+Text GLabel 9800 2750 0    50   Input ~ 0
+VIN5V
+Text Notes 9475 2425 0    50   ~ 0
+Voltage selector\ndisk I/O 3V3 / 5V
+Text GLabel 6450 4750 0    50   Input ~ 0
+EXP_35
+Text GLabel 7450 4750 2    50   Input ~ 0
+H_EXP_35
+Text GLabel 1450 3900 2    50   Input ~ 0
+H_EXP_35
+Text GLabel 1450 3800 2    50   Input ~ 0
+H_EXP_34
+Text GLabel 1450 3700 2    50   Input ~ 0
 H_EXP_32
-Text GLabel 7450 5150 2    50   Input ~ 0
+Text GLabel 1450 3600 2    50   Input ~ 0
 H_EXP_30
-Text GLabel 7450 5050 2    50   Input ~ 0
+Text GLabel 1450 3400 2    50   Input ~ 0
 H_EXP_28
-Text GLabel 7450 4950 2    50   Input ~ 0
+Text GLabel 1450 3200 2    50   Input ~ 0
 H_EXP_26
-Text GLabel 7450 4850 2    50   Input ~ 0
+Text GLabel 1450 3000 2    50   Input ~ 0
 H_EXP_24
-Text GLabel 7450 4750 2    50   Input ~ 0
+Text GLabel 1450 2800 2    50   Input ~ 0
 H_EXP_22
-Text GLabel 7400 2750 2    50   Input ~ 0
+Text GLabel 1450 2600 2    50   Input ~ 0
 H_EXP_20
-Text GLabel 7400 2650 2    50   Input ~ 0
+Text GLabel 1450 2500 2    50   Input ~ 0
 H_EXP_18
-Text GLabel 6450 5250 0    50   Input ~ 0
-EXP_32
-Text GLabel 6450 5150 0    50   Input ~ 0
-EXP_30
-Text GLabel 6450 5050 0    50   Input ~ 0
-EXP_28
-Text GLabel 6450 4950 0    50   Input ~ 0
-EXP_26
-Text GLabel 6450 4850 0    50   Input ~ 0
-EXP_24
-Text GLabel 6450 4750 0    50   Input ~ 0
-EXP_22
-Text GLabel 6400 2750 0    50   Input ~ 0
-EXP_20
-Text GLabel 6400 2650 0    50   Input ~ 0
-EXP_18
-Text GLabel 6450 5350 0    50   Input ~ 0
-EXP_34
-Text GLabel 7450 5350 2    50   Input ~ 0
-H_EXP_34
+Text GLabel 1450 2400 2    50   Input ~ 0
+H_EXP_16
+Text GLabel 1450 2300 2    50   Input ~ 0
+H_EXP_12
+Text GLabel 1450 2200 2    50   Input ~ 0
+H_EXP_10
+Text GLabel 1450 1900 2    50   Input ~ 0
+H_EXP_02
+Text GLabel 1450 2000 2    50   Input ~ 0
+H_EXP_04
+Text GLabel 1450 2100 2    50   Input ~ 0
+H_EXP_08
+Text GLabel 1150 1450 1    50   Input ~ 0
+GND
 $EndSCHEMATC

Commit message: Fixed HDMI Impedance to 50Ohm, 100Ohm differential, for 0.1mm bord. Add pullups to HDMI I2C, connected DE pin to FPGA.
Parts:
- added JP1: Jumper, Connector_PinHeader_2.54mm:PinHeader_1x02_P2.54mm_Vertical, symbol Device:Jumper
- added R40: 1M, Resistor_SMD:R_0603_1608Metric, symbol Device:R
- added TP3, TP4: TestPoint, TestPoint:TestPoint_Keystone_5019_Minature, symbol Connector:TestPoint
Connections:
- wire segments 57 -> 63
Other:
- note added: "12V power supply for the floppy drive"
- note added: "Alternative pereferal connector"
- note added: "Floppy power connector"
- note added: "Levershifter floppy IO"
Changed lines of the file:
@@
 $EndComp
 Wire Wire Line
-	1500 6300 1700 6300
-Text GLabel 5000 6300 2    50   Input ~ 0
-GND
-Text GLabel 5000 5400 2    50   Input ~ 0
+	1100 6300 1200 6300
+Text GLabel 5625 6300 2    50   Input ~ 0
+GND
+Text GLabel 5600 5400 2    50   Input ~ 0
 VIN5V
 Wire Wire Line
@@
 Wire Wire Line
 	1700 5700 1700 5400
-Connection ~ 1700 5400
-Wire Wire Line
-	1700 5400 1500 5400
-Text GLabel 1500 5400 0    50   Input ~ 0
+Wire Wire Line
+	1700 5400 1400 5400
+Text GLabel 1075 5400 0    50   Input ~ 0
 VIN12V
-Text GLabel 1500 6300 0    50   Input ~ 0
+Text GLabel 1100 6300 0    50   Input ~ 0
 GND
 $Comp
@@
 Connection ~ 4750 6300
 Wire Wire Line
-	4750 6300 5000 6300
+	4750 6300 5625 6300
 Wire Wire Line
 	4350 6000 4350 6300
@@
 	2400 5400 2350 5400
 Connection ~ 2350 5400
-Connection ~ 1700 6300
 $Comp
 L Connector_Generic:Conn_01x04 J8
@@
 P 1150 2700
 F 0 "J10" H 1329 2684 50  0000 L CNN
-F 1 "DB23_Female_MountingHoles" H 1329 2775 50  0000 L CNN
+F 1 "DB23_Female_MountingHoles" V 1400 2825 50  0000 L CNN
 F 2 "c64-wing-kicad:DSUB-23_Female_Horizontal_P2.77x2.84mm_EdgePinOffset7.70mm_Housed_MountingHolesOffset9.12mm" H 1150 2700 50  0001 C CNN
 F 3 " ~" H 1150 2700 50  0001 C CNN
@@
 Text GLabel 1150 1450 1    50   Input ~ 0
 GND
+$Comp
+L Device:Jumper JP1
+U 1 1 5D9FBDE3
+P 5300 5400
+F 0 "JP1" H 5300 5664 50  0000 C CNN
+F 1 "Jumper" H 5300 5573 50  0000 C CNN
+F 2 "Connector_PinHeader_2.54mm:PinHeader_1x02_P2.54mm_Vertical" H 5300 5400 50  0001 C CNN
+F 3 "~" H 5300 5400 50  0001 C CNN
+	1    5300 5400
+	1    0    0    -1
+$EndComp
+$Comp
+L Connector:TestPoint TP3
+U 1 1 5DA056F9
+P 1175 5400
+F 0 "TP3" H 1233 5518 50  0000 L CNN
+F 1 "TestPoint" H 1233 5427 50  0000 L CNN
+F 2 "TestPoint:TestPoint_Keystone_5019_Minature" H 1375 5400 50  0001 C CNN
+F 3 "~" H 1375 5400 50  0001 C CNN
+	1    1175 5400
+	1    0    0    -1
+$EndComp
+Connection ~ 1175 5400
+Wire Wire Line
+	1175 5400 1075 5400
+$Comp
+L Connector:TestPoint TP4
+U 1 1 5DA05BA0
+P 1200 6300
+F 0 "TP4" H 1258 6418 50  0000 L CNN
+F 1 "TestPoint" H 1258 6327 50  0000 L CNN
+F 2 "TestPoint:TestPoint_Keystone_5019_Minature" H 1400 6300 50  0001 C CNN
+F 3 "~" H 1400 6300 50  0001 C CNN
+	1    1200 6300
+	1    0    0    -1
+$EndComp
+Connection ~ 1200 6300
+Wire Wire Line
+	1200 6300 1400 6300
+Text Notes 3250 5000 0    50   ~ 0
+12V power supply for the floppy drive
+Text Notes 6525 725  0    50   ~ 0
+Levershifter floppy IO
+Text Notes 8850 4700 0    50   ~ 0
+Floppy power connector
+Text Notes 2850 2000 0    50   ~ 0
+Alternative pereferal connector
+Connection ~ 1700 5400
+Connection ~ 1700 6300
+$Comp
+L Device:R R40
+U 1 1 5DA350F1
+P 1400 5850
+F 0 "R40" H 1470 5896 50  0000 L CNN
+F 1 "1M" H 1470 5805 50  0000 L CNN
+F 2 "Resistor_SMD:R_0603_1608Metric" V 1330 5850 50  0001 C CNN
+F 3 "~" H 1400 5850 50  0001 C CNN
+	1    1400 5850
+	1    0    0    1
+$EndComp
+Wire Wire Line
+	1400 5700 1400 5400
+Connection ~ 1400 5400
+Wire Wire Line
+	1400 5400 1175 5400
+Wire Wire Line
+	1400 6000 1400 6300
+Connection ~ 1400 6300
+Wire Wire Line
+	1400 6300 1700 6300
 $EndSCHEMATC

Commit message: Added ESD protection, and removed the curved lines around the adv7511.
Parts:
- L5: footprint CDRH104RNP-220NC:INDPM102100X400N -> Inductor_SMD:L_10.4x10.4_H4.8
- U6, U7: footprint SOP65P640X120-20N -> Package_SO:TSSOP-20_4.4x6.5mm_P0.65mm
Changed lines of the file:
@@
 F 0 "L5" V 3340 5400 50  0000 C CNN
 F 1 "22uH" V 3249 5400 50  0000 C CNN
-F 2 "CDRH104RNP-220NC:INDPM102100X400N" H 3150 5400 50  0001 C CNN
+F 2 "Inductor_SMD:L_10.4x10.4_H4.8" H 3150 5400 50  0001 C CNN
 F 3 "~" H 3150 5400 50  0001 C CNN
 	1    3150 5400
@@
 F 0 "U6" H 6900 3217 50  0000 C CNN
 F 1 "TXS0108EPWR" H 6900 3126 50  0000 C CNN
-F 2 "SOP65P640X120-20N" H 6900 2250 50  0001 L BNN
+F 2 "Package_SO:TSSOP-20_4.4x6.5mm_P0.65mm" H 6900 2250 50  0001 L BNN
 F 3 "TSSOP-20 Texas Instruments" H 6900 2250 50  0001 L BNN
 F 4 "Voltage Level Translator 20-Pin TSSOP T/R" H 6900 2250 50  0001 L BNN "Field4"
@@
 F 0 "U7" H 6950 5917 50  0000 C CNN
 F 1 "TXS0108EPWR" H 6950 5826 50  0000 C CNN
-F 2 "SOP65P640X120-20N" H 6950 4950 50  0001 L BNN
+F 2 "Package_SO:TSSOP-20_4.4x6.5mm_P0.65mm" H 6950 4950 50  0001 L BNN
 F 3 "TSSOP-20 Texas Instruments" H 6950 4950 50  0001 L BNN
 F 4 "Voltage Level Translator 20-Pin TSSOP T/R" H 6950 4950 50  0001 L BNN "Field4"

Commit message: Add Max9850 to handle audio.
Parts:
- added D33: LED, LED_SMD:LED_0603_1608Metric, symbol Device:LED
- added F1: 2A, Fuse:Fuse_0805_2012Metric, symbol Device:Polyfuse
- added R65: 1k, Resistor_SMD:R_0603_1608Metric, symbol Device:R
- JP1: value Jumper -> 12V Enable
- TP3: value TestPoint -> +12V
- TP4: value TestPoint -> GND
Connections:
- wire segments 63 -> 70

Commit message: Change order of the VSPI to FPGA to make sure the clock pin connects to an FPGA clock capable pin.
Parts:
- +12V1: renamed from TP3; footprint TestPoint:TestPoint_Keystone_5019_Minature -> TestPoint:TestPoint_THTPad_1.0x1.0mm_Drill0.5mm
- GND1: renamed from TP4; footprint TestPoint:TestPoint_Keystone_5019_Minature -> TestPoint:TestPoint_THTPad_1.0x1.0mm_Drill0.5mm
- U6, U7: footprint Package_SO:TSSOP-20_4.4x6.5mm_P0.65mm -> TXS0108EPWR:SOP65P640X120-20N
Changed lines of the file:
@@
 F 0 "U6" H 7750 3317 50  0000 C CNN
 F 1 "TXS0108EPWR" H 7750 3226 50  0000 C CNN
-F 2 "Package_SO:TSSOP-20_4.4x6.5mm_P0.65mm" H 7750 2350 50  0001 L BNN
+F 2 "TXS0108EPWR:SOP65P640X120-20N" H 7750 2350 50  0001 L BNN
 F 3 "TSSOP-20 Texas Instruments" H 7750 2350 50  0001 L BNN
 F 4 "Voltage Level Translator 20-Pin TSSOP T/R" H 7750 2350 50  0001 L BNN "Field4"
@@
 F 0 "U7" H 7800 6017 50  0000 C CNN
 F 1 "TXS0108EPWR" H 7800 5926 50  0000 C CNN
-F 2 "Package_SO:TSSOP-20_4.4x6.5mm_P0.65mm" H 7800 5050 50  0001 L BNN
+F 2 "TXS0108EPWR:SOP65P640X120-20N" H 7800 5050 50  0001 L BNN
 F 3 "TSSOP-20 Texas Instruments" H 7800 5050 50  0001 L BNN
 F 4 "Voltage Level Translator 20-Pin TSSOP T/R" H 7800 5050 50  0001 L BNN "Field4"
@@
 $EndComp
 $Comp
-L Connector:TestPoint TP3
+L Connector:TestPoint +12V1
 U 1 1 5DA056F9
 P 925 5400
-F 0 "TP3" H 983 5518 50  0000 L CNN
+F 0 "+12V1" H 983 5518 50  0000 L CNN
 F 1 "+12V" H 983 5427 50  0000 L CNN
-F 2 "TestPoint:TestPoint_Keystone_5019_Minature" H 1125 5400 50  0001 C CNN
+F 2 "TestPoint:TestPoint_THTPad_1.0x1.0mm_Drill0.5mm" H 1125 5400 50  0001 C CNN
 F 3 "~" H 1125 5400 50  0001 C CNN
 	1    925  5400
@@
 	925  5400 825  5400
 $Comp
-L Connector:TestPoint TP4
+L Connector:TestPoint GND1
 U 1 1 5DA05BA0
 P 950 6300
-F 0 "TP4" H 1008 6418 50  0000 L CNN
+F 0 "GND1" H 1008 6418 50  0000 L CNN
 F 1 "GND" H 1008 6327 50  0000 L CNN
-F 2 "TestPoint:TestPoint_Keystone_5019_Minature" H 1150 6300 50  0001 C CNN
+F 2 "TestPoint:TestPoint_THTPad_1.0x1.0mm_Drill0.5mm" H 1150 6300 50  0001 C CNN
 F 3 "~" H 1150 6300 50  0001 C CNN
 	1    950  6300

Commit message: First checkin of SDRAM Open AARS board.
Parts:
- removed C20, C24: 100nF, Capacitor_SMD:C_0603_1608Metric, symbol Device:C
- removed J11: Conn_01x03_Male, Connector_PinHeader_2.54mm:PinHeader_1x03_P2.54mm_Vertical, symbol Connector:Conn_01x03_Male
- removed U6, U7: TXS0108EPWR, TXS0108EPWR:SOP65P640X120-20N, symbol TXS0108EPWR:TXS0108EPWR
- added C66: 100nF, Capacitor_SMD:C_0603_1608Metric, symbol Device:C
- added R6, R8: 10k, Resistor_SMD:R_0603_1608Metric, symbol Device:R
- added U10: MCP23S17, Package_SO:SSOP-28_5.3x10.2mm_P0.65mm, symbol microchip:MCP23S17
- added U7: TXB0106PWR, SOP65P640X120-16N, symbol TXB0106PWR:TXB0106PWR
Connections:
- net labels added: CS_5V, FLP_SPI_CS, FLP_SPI_INTA, FLP_SPI_INTB, FLP_SPI_MISO, FLP_SPI_MOSI, FLP_SPI_SCK, INTA_5V, INTB_5V, SCK_5V, SI_5V, SO_5V
- net labels removed: EXP_02, EXP_04, EXP_08, EXP_10, EXP_12, EXP_16, EXP_18, EXP_20, EXP_22, EXP_24, EXP_26, EXP_28, EXP_30, EXP_32, EXP_34, EXP_35, VIOSEL
- wire segments 70 -> 73
Other:
- note added: "5V SPI\n"
- note added: "Left pin 20 out, 'select drive 3'"
- note removed: "Voltage selector\ndisk I/O 3V3 / 5V"
