File: floppy.sch (KiCad schematic (older format))
At the start: 50 parts, among them J10 DB23_Female_MountingHoles, J7 Conn_02x13_Odd_Even, J8 Conn_01x04, U5 MT3608, U7 SN74LS06NSR

Commit message: Revert "Fixed some external dependencies."
This reverts commit ddca1efdf68af69ddd54947bcdaa3cfa1d913e0d.
Parts:
- +12V1, GND1: symbol qmtech-minimig-rescue:TestPoint-Connector -> Connector:TestPoint
- C13, C14, C15, C16, C17, C18, C19, C25: symbol qmtech-minimig-rescue:C-Device -> Device:C
- C26: symbol qmtech-minimig-rescue:CP-Device -> Device:CP
- D3: symbol qmtech-minimig-rescue:D_Zener-Device -> Device:D_Zener
- D33: symbol qmtech-minimig-rescue:LED-Device -> Device:LED
- D5, D6: symbol qmtech-minimig-rescue:D_Schottky-Device -> Device:D_Schottky
- F1: symbol qmtech-minimig-rescue:Polyfuse-Device -> Device:Polyfuse
- J7: symbol qmtech-minimig-rescue:Conn_02x17_Odd_Even-Connector_Generic -> Connector_Generic:Conn_02x17_Odd_Even
- J8: symbol qmtech-minimig-rescue:Conn_01x04-Connector_Generic -> Connector_Generic:Conn_01x04
- JP1: symbol qmtech-minimig-rescue:Jumper-Device -> Device:Jumper
- L5: symbol qmtech-minimig-rescue:L-Device -> Device:L
- R10, R35, R36, R37, R40, R6, R65, R68, R69, R70, R71, R72, R73, R74, R75, R76, R77, R78, R79, R8, R80, R81, R82, R83, R84, R85, R86: symbol qmtech-minimig-rescue:R-Device -> Device:R
- U7: symbol qmtech-minimig-rescue:SN74LS06NSR-SN74LS06NSR -> SN74LS06NSR:SN74LS06NSR
Changed lines of the file:
@@
 $EndDescr
 $Comp
-L qmtech-minimig-rescue:Conn_02x17_Odd_Even-Connector_Generic J7
+L Connector_Generic:Conn_02x17_Odd_Even J7
 U 1 1 5DA33CAD
 P 3275 3125
@@
 	5150 5400 5000 5400
 $Comp
-L qmtech-minimig-rescue:L-Device L5
+L Device:L L5
 U 1 1 5D800064
 P 2900 5400
@@
 	2750 5400 2450 5400
 $Comp
-L qmtech-minimig-rescue:C-Device C14
+L Device:C C14
 U 1 1 5D80045A
 P 1850 5850
@@
 $EndComp
 $Comp
-L qmtech-minimig-rescue:C-Device C13
+L Device:C C13
 U 1 1 5D80075E
 P 1450 5850
@@
 	3550 5400 3050 5400
 $Comp
-L qmtech-minimig-rescue:R-Device R37
+L Device:R R37
 U 1 1 5D80165B
 P 3750 5650
@@
 	2450 5800 2450 5400
 $Comp
-L qmtech-minimig-rescue:R-Device R35
+L Device:R R35
 U 1 1 5D801FCC
 P 2100 5650
@@
 $EndComp
 $Comp
-L qmtech-minimig-rescue:R-Device R36
+L Device:R R36
 U 1 1 5D802173
 P 2100 6100
@@
 GND
 $Comp
-L qmtech-minimig-rescue:C-Device C15
+L Device:C C15
 U 1 1 5D805ACA
 P 4075 5825
@@
 $EndComp
 $Comp
-L qmtech-minimig-rescue:C-Device C16
+L Device:C C16
 U 1 1 5D806142
 P 4500 5850
@@
 	1450 5400 1850 5400
 $Comp
-L qmtech-minimig-rescue:D_Zener-Device D3
+L Device:D_Zener D3
 U 1 1 5D811ECA
 P 2300 5400
@@
 Connection ~ 2100 5400
 $Comp
-L qmtech-minimig-rescue:Conn_01x04-Connector_Generic J8
+L Connector_Generic:Conn_01x04 J8
 U 1 1 5D870819
 P 10525 5525
@@
 	9325 5425 9525 5425
 $Comp
-L qmtech-minimig-rescue:C-Device C17
+L Device:C C17
 U 1 1 5D874600
 P 9525 5275
@@
 GND
 $Comp
-L qmtech-minimig-rescue:C-Device C18
+L Device:C C18
 U 1 1 5D88AB92
 P 9925 5275
@@
 	9725 5725 9925 5725
 $Comp
-L qmtech-minimig-rescue:C-Device C19
+L Device:C C19
 U 1 1 5D88C77B
 P 9925 6025
@@
 GND
 $Comp
-L qmtech-minimig-rescue:Jumper-Device JP1
+L Device:Jumper JP1
 U 1 1 5D9FBDE3
 P 5450 5400
@@
 $EndComp
 $Comp
-L qmtech-minimig-rescue:TestPoint-Connector +12V1
+L Connector:TestPoint +12V1
 U 1 1 5DA056F9
 P 925 5400
@@
 	925  5400 825  5400
 $Comp
-L qmtech-minimig-rescue:TestPoint-Connector GND1
+L Connector:TestPoint GND1
 U 1 1 5DA05BA0
 P 950 6300
@@
 Connection ~ 1450 6300
 $Comp
-L qmtech-minimig-rescue:R-Device R40
+L Device:R R40
 U 1 1 5DA350F1
 P 1150 5850
@@
 Connection ~ 4500 6300
 $Comp
-L qmtech-minimig-rescue:R-Device R65
+L Device:R R65
 U 1 1 5E193A2D
 P 5000 5625
@@
 	5000 5400 4500 5400
 $Comp
-L qmtech-minimig-rescue:LED-Device D33
+L Device:LED D33
 U 1 1 5E19F0D4
 P 5000 6075
@@
 $EndComp
 $Comp
-L qmtech-minimig-rescue:Polyfuse-Device F1
+L Device:Polyfuse F1
 U 1 1 5E1DBC83
 P 6025 5400
@@
 H_EXP_02
 $Comp
-L qmtech-minimig-rescue:SN74LS06NSR-SN74LS06NSR U7
+L SN74LS06NSR:SN74LS06NSR U7
 U 1 1 5F71E393
 P 6500 4175
@@
 EXP_TRK0
 $Comp
-L qmtech-minimig-rescue:R-Device R6
+L Device:R R6
 U 1 1 5F77216C
 P 5225 1150
@@
 $EndComp
 $Comp
-L qmtech-minimig-rescue:R-Device R8
+L Device:R R8
 U 1 1 5F797809
 P 5525 1150
@@
 $EndComp
 $Comp
-L qmtech-minimig-rescue:R-Device R68
+L Device:R R68
 U 1 1 5F79883B
 P 5675 1150
@@
 $EndComp
 $Comp
-L qmtech-minimig-rescue:R-Device R69
+L Device:R R69
 U 1 1 5F79986D
 P 5825 1150
@@
 $EndComp
 $Comp
-L qmtech-minimig-rescue:R-Device R70
+L Device:R R70
 U 1 1 5F79A90B
 P 5975 1150
@@
 $EndComp
 $Comp
-L qmtech-minimig-rescue:R-Device R71
+L Device:R R71
 U 1 1 5F79B911
 P 6125 1150
@@
 	5125 1550 5225 1550
 $Comp
-L qmtech-minimig-rescue:R-Device R73
+L Device:R R73
 U 1 1 5F79EDB5
 P 7200 1550
@@
 $EndComp
 $Comp
-L qmtech-minimig-rescue:R-Device R74
+L Device:R R74
 U 1 1 5F7BDC23
 P 7200 1900
@@
 $EndComp
 $Comp
-L qmtech-minimig-rescue:R-Device R75
+L Device:R R75
 U 1 1 5F7BEF0B
 P 7200 2075
@@
 $EndComp
 $Comp
-L qmtech-minimig-rescue:R-Device R78
+L Device:R R78
 U 1 1 5F7C0A47
 P 7200 2250
@@
 $EndComp
 $Comp
-L qmtech-minimig-rescue:R-Device R76
+L Device:R R76
 U 1 1 5F7C1D3F
 P 7200 2425
@@
 VFLP5V
 $Comp
-L qmtech-minimig-rescue:R-Device R84
+L Device:R R84
 U 1 1 5F7F2B33
 P 8525 2875
@@
 $EndComp
 $Comp
-L qmtech-minimig-rescue:R-Device R83
+L Device:R R83
 U 1 1 5F7F2B39
 P 8375 2875
@@
 $EndComp
 $Comp
-L qmtech-minimig-rescue:R-Device R82
+L Device:R R82
 U 1 1 5F7F2B3F
 P 8225 2875
@@
 $EndComp
 $Comp
-L qmtech-minimig-rescue:R-Device R81
+L Device:R R81
 U 1 1 5F7F2B45
 P 8075 2875
@@
 $EndComp
 $Comp
-L qmtech-minimig-rescue:R-Device R80
+L Device:R R80
 U 1 1 5F7F2B4B
 P 7775 2875
@@
 	6125 1300 6125 2600
 $Comp
-L qmtech-minimig-rescue:R-Device R77
+L Device:R R77
 U 1 1 5F877496
 P 7200 2600
@@
 	5125 2600 6125 2600
 $Comp
-L qmtech-minimig-rescue:R-Device R86
+L Device:R R86
 U 1 1 5F88D6F1
 P 8675 2875
@@
 EXP_SEL0
 $Comp
-L qmtech-minimig-rescue:R-Device R72
+L Device:R R72
 U 1 1 5F9F68F6
 P 5375 1150
@@
 	5375 1000 5225 1000
 $Comp
-L qmtech-minimig-rescue:R-Device R79
+L Device:R R79
 U 1 1 5F9FA7F0
 P 7200 1725
@@
 	5375 1725 6500 1725
 $Comp
-L qmtech-minimig-rescue:R-Device R85
+L Device:R R85
 U 1 1 5FA136D8
 P 7925 2875
@@
 H_EXP_24
 $Comp
-L qmtech-minimig-rescue:C-Device C25
+L Device:C C25
 U 1 1 5FAA021B
 P 5600 3725
@@
 	5600 3875 5800 3875
 $Comp
-L qmtech-minimig-rescue:D_Schottky-Device D5
+L Device:D_Schottky D5
 U 1 1 5FACC1D5
 P 6500 1150
@@
 $EndComp
 $Comp
-L qmtech-minimig-rescue:D_Schottky-Device D6
+L Device:D_Schottky D6
 U 1 1 5FACE80C
 P 6750 1150
@@
 H_EXP_34
 $Comp
-L qmtech-minimig-rescue:R-Device R10
+L Device:R R10
 U 1 1 5FC81D81
 P 2075 2100
@@
 	5750 5400 5850 5400
 $Comp
-L qmtech-minimig-rescue:CP-Device C26
+L Device:CP C26
 U 1 1 5FCF3E95
 P 5850 5850

Commit message: Fixed some external dependencies.
Parts:
- +12V1, GND1: symbol Connector:TestPoint -> qmtech-minimig-rescue:TestPoint-Connector
- C13, C14, C15, C16, C17, C18, C19, C25: symbol Device:C -> qmtech-minimig-rescue:C-Device
- C26: symbol Device:CP -> qmtech-minimig-rescue:CP-Device
- D3: symbol Device:D_Zener -> qmtech-minimig-rescue:D_Zener-Device
- D33: symbol Device:LED -> qmtech-minimig-rescue:LED-Device
- D5, D6: symbol Device:D_Schottky -> qmtech-minimig-rescue:D_Schottky-Device
- F1: symbol Device:Polyfuse -> qmtech-minimig-rescue:Polyfuse-Device
- J7: symbol Connector_Generic:Conn_02x17_Odd_Even -> qmtech-minimig-rescue:Conn_02x17_Odd_Even-Connector_Generic
- J8: symbol Connector_Generic:Conn_01x04 -> qmtech-minimig-rescue:Conn_01x04-Connector_Generic
- JP1: symbol Device:Jumper -> qmtech-minimig-rescue:Jumper-Device
- L5: symbol Device:L -> qmtech-minimig-rescue:L-Device
- R10, R35, R36, R37, R40, R6, R65, R68, R69, R70, R71, R72, R73, R74, R75, R76, R77, R78, R79, R8, R80, R81, R82, R83, R84, R85, R86: symbol Device:R -> qmtech-minimig-rescue:R-Device
- U7: symbol SN74LS06NSR:SN74LS06NSR -> qmtech-minimig-rescue:SN74LS06NSR-SN74LS06NSR
Changed lines of the file:
@@
 $EndDescr
 $Comp
-L Connector_Generic:Conn_02x17_Odd_Even J7
+L qmtech-minimig-rescue:Conn_02x17_Odd_Even-Connector_Generic J7
 U 1 1 5DA33CAD
 P 3275 3125
@@
 	5150 5400 5000 5400
 $Comp
-L Device:L L5
+L qmtech-minimig-rescue:L-Device L5
 U 1 1 5D800064
 P 2900 5400
@@
 	2750 5400 2450 5400
 $Comp
-L Device:C C14
+L qmtech-minimig-rescue:C-Device C14
 U 1 1 5D80045A
 P 1850 5850
@@
 $EndComp
 $Comp
-L Device:C C13
+L qmtech-minimig-rescue:C-Device C13
 U 1 1 5D80075E
 P 1450 5850
@@
 	3550 5400 3050 5400
 $Comp
-L Device:R R37
+L qmtech-minimig-rescue:R-Device R37
 U 1 1 5D80165B
 P 3750 5650
@@
 	2450 5800 2450 5400
 $Comp
-L Device:R R35
+L qmtech-minimig-rescue:R-Device R35
 U 1 1 5D801FCC
 P 2100 5650
@@
 $EndComp
 $Comp
-L Device:R R36
+L qmtech-minimig-rescue:R-Device R36
 U 1 1 5D802173
 P 2100 6100
@@
 GND
 $Comp
-L Device:C C15
+L qmtech-minimig-rescue:C-Device C15
 U 1 1 5D805ACA
 P 4075 5825
@@
 $EndComp
 $Comp
-L Device:C C16
+L qmtech-minimig-rescue:C-Device C16
 U 1 1 5D806142
 P 4500 5850
@@
 	1450 5400 1850 5400
 $Comp
-L Device:D_Zener D3
+L qmtech-minimig-rescue:D_Zener-Device D3
 U 1 1 5D811ECA
 P 2300 5400
@@
 Connection ~ 2100 5400
 $Comp
-L Connector_Generic:Conn_01x04 J8
+L qmtech-minimig-rescue:Conn_01x04-Connector_Generic J8
 U 1 1 5D870819
 P 10525 5525
@@
 	9325 5425 9525 5425
 $Comp
-L Device:C C17
+L qmtech-minimig-rescue:C-Device C17
 U 1 1 5D874600
 P 9525 5275
@@
 GND
 $Comp
-L Device:C C18
+L qmtech-minimig-rescue:C-Device C18
 U 1 1 5D88AB92
 P 9925 5275
@@
 	9725 5725 9925 5725
 $Comp
-L Device:C C19
+L qmtech-minimig-rescue:C-Device C19
 U 1 1 5D88C77B
 P 9925 6025
@@
 GND
 $Comp
-L Device:Jumper JP1
+L qmtech-minimig-rescue:Jumper-Device JP1
 U 1 1 5D9FBDE3
 P 5450 5400
@@
 $EndComp
 $Comp
-L Connector:TestPoint +12V1
+L qmtech-minimig-rescue:TestPoint-Connector +12V1
 U 1 1 5DA056F9
 P 925 5400
@@
 	925  5400 825  5400
 $Comp
-L Connector:TestPoint GND1
+L qmtech-minimig-rescue:TestPoint-Connector GND1
 U 1 1 5DA05BA0
 P 950 6300
@@
 Connection ~ 1450 6300
 $Comp
-L Device:R R40
+L qmtech-minimig-rescue:R-Device R40
 U 1 1 5DA350F1
 P 1150 5850
@@
 Connection ~ 4500 6300
 $Comp
-L Device:R R65
+L qmtech-minimig-rescue:R-Device R65
 U 1 1 5E193A2D
 P 5000 5625
@@
 	5000 5400 4500 5400
 $Comp
-L Device:LED D33
+L qmtech-minimig-rescue:LED-Device D33
 U 1 1 5E19F0D4
 P 5000 6075
@@
 $EndComp
 $Comp
-L Device:Polyfuse F1
+L qmtech-minimig-rescue:Polyfuse-Device F1
 U 1 1 5E1DBC83
 P 6025 5400
@@
 H_EXP_02
 $Comp
-L SN74LS06NSR:SN74LS06NSR U7
+L qmtech-minimig-rescue:SN74LS06NSR-SN74LS06NSR U7
 U 1 1 5F71E393
 P 6500 4175
@@
 EXP_TRK0
 $Comp
-L Device:R R6
+L qmtech-minimig-rescue:R-Device R6
 U 1 1 5F77216C
 P 5225 1150
@@
 $EndComp
 $Comp
-L Device:R R8
+L qmtech-minimig-rescue:R-Device R8
 U 1 1 5F797809
 P 5525 1150
@@
 $EndComp
 $Comp
-L Device:R R68
+L qmtech-minimig-rescue:R-Device R68
 U 1 1 5F79883B
 P 5675 1150
@@
 $EndComp
 $Comp
-L Device:R R69
+L qmtech-minimig-rescue:R-Device R69
 U 1 1 5F79986D
 P 5825 1150
@@
 $EndComp
 $Comp
-L Device:R R70
+L qmtech-minimig-rescue:R-Device R70
 U 1 1 5F79A90B
 P 5975 1150
@@
 $EndComp
 $Comp
-L Device:R R71
+L qmtech-minimig-rescue:R-Device R71
 U 1 1 5F79B911
 P 6125 1150
@@
 	5125 1550 5225 1550
 $Comp
-L Device:R R73
+L qmtech-minimig-rescue:R-Device R73
 U 1 1 5F79EDB5
 P 7200 1550
@@
 $EndComp
 $Comp
-L Device:R R74
+L qmtech-minimig-rescue:R-Device R74
 U 1 1 5F7BDC23
 P 7200 1900
@@
 $EndComp
 $Comp
-L Device:R R75
+L qmtech-minimig-rescue:R-Device R75
 U 1 1 5F7BEF0B
 P 7200 2075
@@
 $EndComp
 $Comp
-L Device:R R78
+L qmtech-minimig-rescue:R-Device R78
 U 1 1 5F7C0A47
 P 7200 2250
@@
 $EndComp
 $Comp
-L Device:R R76
+L qmtech-minimig-rescue:R-Device R76
 U 1 1 5F7C1D3F
 P 7200 2425
@@
 VFLP5V
 $Comp
-L Device:R R84
+L qmtech-minimig-rescue:R-Device R84
 U 1 1 5F7F2B33
 P 8525 2875
@@
 $EndComp
 $Comp
-L Device:R R83
+L qmtech-minimig-rescue:R-Device R83
 U 1 1 5F7F2B39
 P 8375 2875
@@
 $EndComp
 $Comp
-L Device:R R82
+L qmtech-minimig-rescue:R-Device R82
 U 1 1 5F7F2B3F
 P 8225 2875
@@
 $EndComp
 $Comp
-L Device:R R81
+L qmtech-minimig-rescue:R-Device R81
 U 1 1 5F7F2B45
 P 8075 2875
@@
 $EndComp
 $Comp
-L Device:R R80
+L qmtech-minimig-rescue:R-Device R80
 U 1 1 5F7F2B4B
 P 7775 2875
@@
 	6125 1300 6125 2600
 $Comp
-L Device:R R77
+L qmtech-minimig-rescue:R-Device R77
 U 1 1 5F877496
 P 7200 2600
@@
 	5125 2600 6125 2600
 $Comp
-L Device:R R86
+L qmtech-minimig-rescue:R-Device R86
 U 1 1 5F88D6F1
 P 8675 2875
@@
 EXP_SEL0
 $Comp
-L Device:R R72
+L qmtech-minimig-rescue:R-Device R72
 U 1 1 5F9F68F6
 P 5375 1150
@@
 	5375 1000 5225 1000
 $Comp
-L Device:R R79
+L qmtech-minimig-rescue:R-Device R79
 U 1 1 5F9FA7F0
 P 7200 1725
@@
 	5375 1725 6500 1725
 $Comp
-L Device:R R85
+L qmtech-minimig-rescue:R-Device R85
 U 1 1 5FA136D8
 P 7925 2875
@@
 H_EXP_24
 $Comp
-L Device:C C25
+L qmtech-minimig-rescue:C-Device C25
 U 1 1 5FAA021B
 P 5600 3725
@@
 	5600 3875 5800 3875
 $Comp
-L Device:D_Schottky D5
+L qmtech-minimig-rescue:D_Schottky-Device D5
 U 1 1 5FACC1D5
 P 6500 1150
@@
 $EndComp
 $Comp
-L Device:D_Schottky D6
+L qmtech-minimig-rescue:D_Schottky-Device D6
 U 1 1 5FACE80C
 P 6750 1150
@@
 H_EXP_34
 $Comp
-L Device:R R10
+L qmtech-minimig-rescue:R-Device R10
 U 1 1 5FC81D81
 P 2075 2100
@@
 	5750 5400 5850 5400
 $Comp
-L Device:CP C26
+L qmtech-minimig-rescue:CP-Device C26
 U 1 1 5FCF3E95
 P 5850 5850
