File: floppy.sch (KiCad schematic (older format))
At the start: 30 parts, among them J10 DB23_Female_MountingHoles, J7 Conn_02x13_Odd_Even, J8 Conn_01x04, U10 MCP23S17, U5 MT3608, U7 TXB0106PWR

Commit message: Implemented the Floppy interface, fixed 12V power up issue with the board.
Parts:
- removed C26, C66: 100nF, Capacitor_SMD:C_0603_1608Metric, symbol Device:C
- removed U10: MCP23S17, Package_SO:SSOP-28_5.3x10.2mm_P0.65mm, symbol microchip:MCP23S17
- removed U7: TXB0106PWR, SOP65P640X120-16N, symbol TXB0106PWR:TXB0106PWR
- added D5, D6: D_Schottky, Diode_SMD:D_0603_1608Metric, symbol Device:D_Schottky
- added R68, R69, R70, R71, R72: 1k, Resistor_SMD:R_0603_1608Metric, symbol Device:R
- added R73, R74, R75, R76, R77, R78, R79: 2.7k, Resistor_SMD:R_0603_1608Metric, symbol Device:R
- added R80, R81, R82, R83, R84, R85, R86: 6k8, Resistor_SMD:R_0603_1608Metric, symbol Device:R
- added U7: SN74LS06NSR, Package_SO:SO-14_5.3x10.2mm_P1.27mm, symbol SN74LS06NSR:SN74LS06NSR
- R6, R8: value 10k -> 1k
Connections:
- net labels added: EXP_CHNG, EXP_DIR, EXP_DKRD, EXP_DKWDB, EXP_DKWEB, EXP_INDEX, EXP_RDY, EXP_SEL0, EXP_SEL1, EXP_SIDE, EXP_STEP, EXP_TRK0
- net labels removed: 3V3, CS_5V, FLP_SPI_CS, FLP_SPI_INTA, FLP_SPI_INTB, FLP_SPI_MISO, FLP_SPI_MOSI, FLP_SPI_SCK, H_EXP_06, H_EXP_14, INTA_5V, INTB_5V, SCK_5V, SI_5V, SO_5V
- wire segments 73 -> 124
Other:
- note added: "Input lines with voltage devider"
- note added: "Output lines, using invertor"
- note removed: "5V SPI\n"
- note removed: "Left pin 20 out, 'select drive 3'"
- note removed: "Levershifter floppy IO"

Commit message: Version that was sent to JLCPCB 20200716.
Parts:
- added C26: 22uF, Capacitor_SMD:CP_Elec_5x5.4, symbol Device:CP
- added R10: 1k, Resistor_SMD:R_0603_1608Metric, symbol Device:R
Connections:
- net labels added: EXP_MTRON, VFLP5V
- net labels removed: H_EXP_16, H_EXP_35
- wire segments 124 -> 129
Other:
- note added: "Motor on, second pin"
- note added: "Schema based on http://amigadrive.blogspot.com/"
Changed lines of the file:
@@
 L Device:C C15
 U 1 1 5D805ACA
-P 5775 5825
-F 0 "C15" H 5890 5871 50  0000 L CNN
-F 1 "22uF" H 5890 5780 50  0000 L CNN
-F 2 "Capacitor_SMD:C_0805_2012Metric" H 5813 5675 50  0001 C CNN
-F 3 "~" H 5775 5825 50  0001 C CNN
-	1    5775 5825
+P 4075 5825
+F 0 "C15" H 4190 5871 50  0000 L CNN
+F 1 "22uF" H 4190 5780 50  0000 L CNN
+F 2 "Capacitor_SMD:C_0805_2012Metric" H 4113 5675 50  0001 C CNN
+F 3 "~" H 4075 5825 50  0001 C CNN
+	1    4075 5825
 	1    0    0    -1
 $EndComp
@@
 Wire Wire Line
 	9325 5425 9525 5425
-Text GLabel 9325 5425 0    50   Input ~ 0
-VIN5V
 $Comp
 L Device:C C17
@@
 	-1   0    0    1
 $EndComp
-Text GLabel 1450 1700 2    50   Input ~ 0
-VIN5V
 Text GLabel 1450 1800 2    50   Input ~ 0
 VIN12V
@@
 Text GLabel 1450 2700 2    50   Input ~ 0
 GND
-Text GLabel 1450 3900 2    50   Input ~ 0
-H_EXP_35
-Text GLabel 1450 3800 2    50   Input ~ 0
-H_EXP_34
-Text GLabel 1450 3700 2    50   Input ~ 0
-H_EXP_32
-Text GLabel 1450 3600 2    50   Input ~ 0
-H_EXP_30
-Text GLabel 1450 3400 2    50   Input ~ 0
-H_EXP_28
-Text GLabel 1450 3200 2    50   Input ~ 0
-H_EXP_26
-Text GLabel 1450 3000 2    50   Input ~ 0
-H_EXP_24
-Text GLabel 1450 2800 2    50   Input ~ 0
-H_EXP_22
-Text GLabel 1450 2600 2    50   Input ~ 0
-H_EXP_20
-Text GLabel 1450 2500 2    50   Input ~ 0
-H_EXP_18
-Text GLabel 1450 2400 2    50   Input ~ 0
-H_EXP_16
-Text GLabel 1450 2300 2    50   Input ~ 0
-H_EXP_12
-Text GLabel 1450 2200 2    50   Input ~ 0
-H_EXP_10
-Text GLabel 1450 1900 2    50   Input ~ 0
-H_EXP_02
-Text GLabel 1450 2000 2    50   Input ~ 0
-H_EXP_04
-Text GLabel 1450 2100 2    50   Input ~ 0
-H_EXP_08
 Text GLabel 1150 1450 1    50   Input ~ 0
 GND
@@
 Connection ~ 5000 6300
 Wire Wire Line
-	5000 6300 5775 6300
-Wire Wire Line
 	5000 5775 5000 5925
 Wire Wire Line
@@
 	0    1    1    0
 $EndComp
-Wire Wire Line
-	5875 5400 5775 5400
 Wire Wire Line
 	6250 5400 6175 5400
@@
 H_EXP_30
 Text GLabel 5500 3875 0    50   Input ~ 0
-VIN5V
+VFLP5V
 Text GLabel 5800 4775 0    50   Input ~ 0
 GND
@@
 Connection ~ 5225 1000
 Text GLabel 5075 950  1    50   Input ~ 0
-VIN5V
+VFLP5V
 $Comp
 L Device:R R84
@@
 	6750 1900 7050 1900
 Wire Wire Line
-	3750 5400 4500 5400
-Wire Wire Line
-	2450 6300 4500 6300
-Wire Wire Line
-	5775 5675 5775 5400
-Connection ~ 5775 5400
-Wire Wire Line
-	5775 5400 5750 5400
-Wire Wire Line
-	5775 5975 5775 6300
-Connection ~ 5775 6300
-Wire Wire Line
-	5775 6300 6250 6300
+	3750 5400 4075 5400
+Wire Wire Line
+	2450 6300 4075 6300
+Wire Wire Line
+	4075 5675 4075 5400
+Wire Wire Line
+	4075 5975 4075 6300
+Text Notes 7525 1250 0    50   ~ 0
+Schema based on http://amigadrive.blogspot.com/
+Text GLabel 1450 1900 2    50   Input ~ 0
+H_EXP_02
+Text GLabel 1450 2500 2    50   Input ~ 0
+H_EXP_04
+Text GLabel 1450 2000 2    50   Input ~ 0
+H_EXP_08
+Text GLabel 1450 2200 2    50   Input ~ 0
+H_EXP_12
+Text GLabel 1450 2600 2    50   Input ~ 0
+H_EXP_18
+Text GLabel 1450 2800 2    50   Input ~ 0
+H_EXP_20
+Text GLabel 1450 3000 2    50   Input ~ 0
+H_EXP_22
+Text GLabel 1450 3200 2    50   Input ~ 0
+H_EXP_24
+Text GLabel 1450 3400 2    50   Input ~ 0
+H_EXP_26
+Text GLabel 1450 3600 2    50   Input ~ 0
+H_EXP_28
+Text GLabel 1450 3700 2    50   Input ~ 0
+H_EXP_30
+Text GLabel 1450 3800 2    50   Input ~ 0
+H_EXP_32
+Text GLabel 1450 3900 2    50   Input ~ 0
+H_EXP_34
+$Comp
+L Device:R R10
+U 1 1 5FC81D81
+P 2075 2100
+F 0 "R10" V 2000 2050 50  0000 L CNN
+F 1 "1k" V 2075 2050 50  0000 L CNN
+F 2 "Resistor_SMD:R_0603_1608Metric" V 2005 2100 50  0001 C CNN
+F 3 "~" H 2075 2100 50  0001 C CNN
+	1    2075 2100
+	0    1    1    0
+$EndComp
+Wire Wire Line
+	1925 2100 1450 2100
+Text GLabel 2225 2100 2    50   Input ~ 0
+VFLP5V
+Text GLabel 7200 4375 2    50   Input ~ 0
+EXP_MTRON
+Text GLabel 5800 4575 0    50   Input ~ 0
+H_EXP_04
+Text GLabel 3575 2425 2    50   Input ~ 0
+H_EXP_04
+Text GLabel 3575 3025 2    50   Input ~ 0
+H_EXP_04
+Text Notes 4000 3050 0    50   ~ 0
+Motor on, second pin
+Connection ~ 4075 5400
+Wire Wire Line
+	4075 5400 4500 5400
+Connection ~ 4075 6300
+Wire Wire Line
+	4075 6300 4500 6300
+Wire Wire Line
+	5000 6300 5850 6300
+Wire Wire Line
+	5750 5400 5850 5400
+$Comp
+L Device:CP C26
+U 1 1 5FCF3E95
+P 5850 5850
+F 0 "C26" H 5968 5896 50  0000 L CNN
+F 1 "22uF" H 5968 5805 50  0000 L CNN
+F 2 "Capacitor_SMD:CP_Elec_5x5.4" H 5888 5700 50  0001 C CNN
+F 3 "~" H 5850 5850 50  0001 C CNN
+	1    5850 5850
+	1    0    0    -1
+$EndComp
+Wire Wire Line
+	5850 5700 5850 5400
+Connection ~ 5850 5400
+Wire Wire Line
+	5850 5400 5875 5400
+Wire Wire Line
+	5850 6000 5850 6300
+Connection ~ 5850 6300
+Wire Wire Line
+	5850 6300 6250 6300
+Text GLabel 5850 5400 1    50   Input ~ 0
+VFLP5V
+Text GLabel 1450 1700 2    50   Input ~ 0
+VFLP5V
+Text GLabel 9325 5425 0    50   Input ~ 0
+VFLP5V
 $EndSCHEMATC

Commit message: Did some placement to make the PCB smaller.
Parts:
- removed +12V1: +12V, TestPoint:TestPoint_THTPad_1.0x1.0mm_Drill0.5mm, symbol Connector:TestPoint
- removed GND1: GND, TestPoint:TestPoint_THTPad_1.0x1.0mm_Drill0.5mm, symbol Connector:TestPoint
Connections:
- wire segments 129 -> 127
Changed lines of the file:
@@
 	1    0    0    -1
 $EndComp
-Wire Wire Line
-	850  6300 950  6300
 Text GLabel 6250 5400 2    50   Input ~ 0
 VIN5V
@@
 	1    0    0    -1
 $EndComp
-$Comp
-L Connector:TestPoint +12V1
-U 1 1 5DA056F9
-P 925 5400
-F 0 "+12V1" H 983 5518 50  0000 L CNN
-F 1 "+12V" H 983 5427 50  0000 L CNN
-F 2 "TestPoint:TestPoint_THTPad_1.0x1.0mm_Drill0.5mm" H 1125 5400 50  0001 C CNN
-F 3 "~" H 1125 5400 50  0001 C CNN
-	1    925  5400
-	1    0    0    -1
-$EndComp
-Connection ~ 925  5400
-Wire Wire Line
-	925  5400 825  5400
-$Comp
-L Connector:TestPoint GND1
-U 1 1 5DA05BA0
-P 950 6300
-F 0 "GND1" H 1008 6418 50  0000 L CNN
-F 1 "GND" H 1008 6327 50  0000 L CNN
-F 2 "TestPoint:TestPoint_THTPad_1.0x1.0mm_Drill0.5mm" H 1150 6300 50  0001 C CNN
-F 3 "~" H 1150 6300 50  0001 C CNN
-	1    950  6300
-	1    0    0    -1
-$EndComp
-Connection ~ 950  6300
-Wire Wire Line
-	950  6300 1150 6300
 Text Notes 3000 5000 0    50   ~ 0
 12V power supply for the floppy drive
@@
 	1150 5700 1150 5400
 Connection ~ 1150 5400
-Wire Wire Line
-	1150 5400 925  5400
 Wire Wire Line
 	1150 6000 1150 6300
@@
 Text GLabel 9325 5425 0    50   Input ~ 0
 VFLP5V
+Wire Wire Line
+	825  5400 1150 5400
+Wire Wire Line
+	850  6300 1150 6300
 $EndSCHEMATC

Commit message: Removed ESP32, as it's no longer needed, we have soft cores.
Parts:
- renumbered C13 to C44, C14 to C45, C15 to C46, C16 to C47, C25 to C48, C26 to C49, C17 to C50, C18 to C51, C19 to C52, D3 to D12, D33 to D13, D5 to D14, D6 to D15, F1 to F5, J10 to J7, J7 to J8, J8 to J9, R40 to R31, R10 to R32, R35 to R33, R36 to R34, R37 to R35, R65 to R36, R6 to R37, R72 to R38, R8 to R39, R68 to R40, R69 to R41, R70 to R42, R71 to R43, R73 to R44, R79 to R45, R74 to R46, R75 to R47, R78 to R48, R76 to R49, R77 to R50, R80 to R51, R85 to R52, R81 to R53, R82 to R54, R83 to R55, R84 to R56, R86 to R57, U5 to U8, U7 to U9
