File: sd_card.sch (KiCad schematic (older format))
At the start: 1 part, among them J3 SCHA5B0200

Commit message: First step to implement floppy interface. ESP32 check wireing in.
Parts:
- added C11: C, Capacitor_SMD:C_0603_1608Metric, symbol Device:C
- added C12: 100n, Capacitor_SMD:C_0603_1608Metric, symbol Device:C
- added C5, C6: 100nF, Capacitor_SMD:C_0603_1608Metric, symbol Device:C
- added Q3: BSS84, Package_TO_SOT_SMD:SOT-23, symbol Transistor_FET:BSS84
- added R20, R21, R22, R23: 10k, Resistor_SMD:R_0603_1608Metric, symbol Device:R
- added R32: 100k, Resistor_SMD:R_0603_1608Metric, symbol Device:R
- added R33: 10K, Resistor_SMD:R_0603_1608Metric, symbol Device:R
Connections:
- net labels added: ESP_SD_CLK, ESP_SD_CMD, ESP_SD_DATA0, ESP_SD_DATA1, ESP_SD_DATA2, ESP_SD_DATA3, ESP_SD_SW, ESP_SD_VCC_EN
- net labels removed: SD_SPI2_CS, SD_SPI2_MISO, SD_SPI2_MOSI, SD_SPI2_SCK, SD_SW
- wire segments 0 -> 37

Commit message: Changed zener diode footprint for easy soldering. Fixed pins, U861/2 and U761/2 they now connect correctly to ground.
Parts:
- C11: value C -> 100nF
- C12: value 100n -> 100nF
- J3: footprint ALPS_SCHA5B0200 -> SHA5B0200:ALPS_SCHA5B0200
Changed lines of the file:
@@
 EESchema Schematic File Version 4
-LIBS:qmtech-minimig-cache
 EELAYER 30 0
 EELAYER END
@@
 F 0 "J3" H 4600 5117 50  0000 C CNN
 F 1 "SCHA5B0200" H 4600 5026 50  0000 C CNN
-F 2 "ALPS_SCHA5B0200" H 4600 4550 50  0001 L BNN
+F 2 "SHA5B0200:ALPS_SCHA5B0200" H 4600 4550 50  0001 L BNN
 F 3 "Unavailable" H 4600 4550 50  0001 L BNN
 F 4 "None" H 4600 4550 50  0001 L BNN "Field4"
@@
 P 5650 4000
 F 0 "C11" V 5398 4000 50  0000 C CNN
-F 1 "C" V 5489 4000 50  0000 C CNN
+F 1 "100nF" V 5489 4000 50  0000 C CNN
 F 2 "Capacitor_SMD:C_0603_1608Metric" H 5688 3850 50  0001 C CNN
 F 3 "~" H 5650 4000 50  0001 C CNN
@@
 P 5950 4700
 F 0 "C12" H 6065 4746 50  0000 L CNN
-F 1 "100n" H 6065 4655 50  0000 L CNN
+F 1 "100nF" H 6065 4655 50  0000 L CNN
 F 2 "Capacitor_SMD:C_0603_1608Metric" H 5988 4550 50  0001 C CNN
 F 3 "~" H 5950 4700 50  0001 C CNN

Commit message: Fixed reversed labeling of the QMTECH FPGA board pins.
Parts:
- removed C5: 100nF, Capacitor_SMD:C_0603_1608Metric, symbol Device:C
Connections:
- wire segments 37 -> 36
Changed lines of the file:
@@
 Text GLabel 2550 4650 0    50   Input ~ 0
 ESP_SD_CMD
-Text GLabel 5500 2850 1    50   Input ~ 0
+Text GLabel 5500 2225 1    50   Input ~ 0
 3V3
 Text GLabel 2550 4250 0    50   Input ~ 0
@@
 	3650 3750 3650 3300
 Connection ~ 3650 3300
-Wire Wire Line
-	3650 3300 3950 3300
-$Comp
-L Device:C C5
-U 1 1 5D7BDF8A
-P 3950 3500
-F 0 "C5" H 4065 3546 50  0000 L CNN
-F 1 "100nF" H 4065 3455 50  0000 L CNN
-F 2 "Capacitor_SMD:C_0603_1608Metric" H 3988 3350 50  0001 C CNN
-F 3 "~" H 3950 3500 50  0001 C CNN
-	1    3950 3500
-	1    0    0    -1
-$EndComp
 $Comp
 L Device:C C6
@@
 Wire Wire Line
 	4400 3300 4400 3350
-Wire Wire Line
-	3950 3300 3950 3350
-Connection ~ 3950 3300
-Wire Wire Line
-	3950 3300 4400 3300
-Text GLabel 3950 3650 3    50   Input ~ 0
-GND
 Text GLabel 4400 3650 3    50   Input ~ 0
 GND
-Text GLabel 3350 3100 1    50   Input ~ 0
-3V3
 Wire Wire Line
 	3900 4350 2550 4350
@@
 L Transistor_FET:BSS84 Q3
 U 1 1 5D7D8B8E
-P 5600 3450
-F 0 "Q3" H 5806 3404 50  0000 L CNN
-F 1 "BSS84" H 5806 3495 50  0000 L CNN
-F 2 "Package_TO_SOT_SMD:SOT-23" H 5800 3375 50  0001 L CIN
-F 3 "http://assets.nexperia.com/documents/data-sheet/BSS84.pdf" H 5600 3450 50  0001 L CNN
-	1    5600 3450
+P 5600 2825
+F 0 "Q3" H 5806 2779 50  0000 L CNN
+F 1 "BSS84" H 5806 2870 50  0000 L CNN
+F 2 "Package_TO_SOT_SMD:SOT-23" H 5800 2750 50  0001 L CIN
+F 3 "http://assets.nexperia.com/documents/data-sheet/BSS84.pdf" H 5600 2825 50  0001 L CNN
+	1    5600 2825
 	-1   0    0    1
 $EndComp
-Text GLabel 6150 3450 2    50   Input ~ 0
+Text GLabel 6150 2825 2    50   Input ~ 0
 ESP_SD_VCC_EN
 Wire Wire Line
-	5500 2850 5500 2900
+	5500 2225 5500 2275
 $Comp
 L Device:R R32
 U 1 1 5D7EDDF8
-P 5800 3150
-F 0 "R32" H 5870 3196 50  0000 L CNN
-F 1 "100k" H 5870 3105 50  0000 L CNN
-F 2 "Resistor_SMD:R_0603_1608Metric" V 5730 3150 50  0001 C CNN
-F 3 "~" H 5800 3150 50  0001 C CNN
-	1    5800 3150
-	1    0    0    -1
-$EndComp
-Wire Wire Line
-	5800 3300 5800 3450
-Connection ~ 5800 3450
-Wire Wire Line
-	5800 3450 6150 3450
-Wire Wire Line
-	5800 3000 5800 2900
-Wire Wire Line
-	5800 2900 5500 2900
-Connection ~ 5500 2900
-Wire Wire Line
-	5500 2900 5500 3250
-Wire Wire Line
-	3350 3300 3350 3100
+P 5800 2525
+F 0 "R32" H 5870 2571 50  0000 L CNN
+F 1 "100k" H 5870 2480 50  0000 L CNN
+F 2 "Resistor_SMD:R_0603_1608Metric" V 5730 2525 50  0001 C CNN
+F 3 "~" H 5800 2525 50  0001 C CNN
+	1    5800 2525
+	1    0    0    -1
+$EndComp
+Wire Wire Line
+	5800 2675 5800 2825
+Connection ~ 5800 2825
+Wire Wire Line
+	5800 2825 6150 2825
+Wire Wire Line
+	5800 2375 5800 2275
+Wire Wire Line
+	5800 2275 5500 2275
+Connection ~ 5500 2275
+Wire Wire Line
+	5500 2275 5500 2625
 Wire Wire Line
 	5300 4250 5500 4250
 Wire Wire Line
-	5500 3650 5500 4000
+	5500 3025 5500 3300
 $Comp
 L Device:C C11
@@
 	0    1    1    0
 $EndComp
-Connection ~ 5500 4000
 Wire Wire Line
 	5500 4000 5500 4250
@@
 Text GLabel 5300 4650 2    50   Input ~ 0
 GND
+Connection ~ 5500 4000
+Wire Wire Line
+	4400 3300 5500 3300
+Connection ~ 4400 3300
+Connection ~ 5500 3300
+Wire Wire Line
+	5500 3300 5500 4000
+Wire Wire Line
+	3650 3300 4400 3300
 $EndSCHEMATC

Commit message: Fixed some external dependencies.
Parts:
- C11, C12, C6: symbol Device:C -> qmtech-minimig-rescue:C-Device
- J3: symbol SHA5B0200:SCHA5B0200 -> qmtech-minimig-rescue:SCHA5B0200-SHA5B0200
- Q3: symbol Transistor_FET:BSS84 -> qmtech-minimig-rescue:BSS84-Transistor_FET
- R20, R21, R22, R23, R32, R33: symbol Device:R -> qmtech-minimig-rescue:R-Device
Changed lines of the file:
@@
 $EndDescr
 $Comp
-L SHA5B0200:SCHA5B0200 J3
+L qmtech-minimig-rescue:SCHA5B0200-SHA5B0200 J3
 U 1 1 5D7BAABF
 P 4600 4550
@@
 	2550 4850 2750 4850
 $Comp
-L Device:R R20
+L qmtech-minimig-rescue:R-Device R20
 U 1 1 5D7B8F06
 P 2750 3900
@@
 $EndComp
 $Comp
-L Device:R R21
+L qmtech-minimig-rescue:R-Device R21
 U 1 1 5D7B9145
 P 3050 3900
@@
 $EndComp
 $Comp
-L Device:R R22
+L qmtech-minimig-rescue:R-Device R22
 U 1 1 5D7B92B5
 P 3350 3900
@@
 $EndComp
 $Comp
-L Device:R R23
+L qmtech-minimig-rescue:R-Device R23
 U 1 1 5D7B9431
 P 3650 3900
@@
 Connection ~ 3650 3300
 $Comp
-L Device:C C6
+L qmtech-minimig-rescue:C-Device C6
 U 1 1 5D7BEF06
 P 4400 3500
@@
 ESP_SD_DATA2
 $Comp
-L Transistor_FET:BSS84 Q3
+L qmtech-minimig-rescue:BSS84-Transistor_FET Q3
 U 1 1 5D7D8B8E
 P 5600 2825
@@
 	5500 2225 5500 2275
 $Comp
-L Device:R R32
+L qmtech-minimig-rescue:R-Device R32
 U 1 1 5D7EDDF8
 P 5800 2525
@@
 	5500 3025 5500 3300
 $Comp
-L Device:C C11
+L qmtech-minimig-rescue:C-Device C11
 U 1 1 5D80369D
 P 5650 4000
@@
 ESP_SD_SW
 $Comp
-L Device:R R33
+L qmtech-minimig-rescue:R-Device R33
 U 1 1 5D9F486E
 P 5950 4400
@@
 3V3
 $Comp
-L Device:C C12
+L qmtech-minimig-rescue:C-Device C12
 U 1 1 5D9F4F23
 P 5950 4700
