File: sd_card.sch (KiCad schematic (older format))
At the start: 11 parts, among them J3 SCHA5B0200, Q3 BSS84

Commit message: Removed all libraries that depend on absolute paths.
Parts:
- J3: symbol SHA5B0200:SCHA5B0200 -> qmtech-minimig-rescue:SCHA5B0200-SHA5B0200
Changed lines of the file:
@@
 $EndDescr
 $Comp
-L SHA5B0200:SCHA5B0200 J3
+L qmtech-minimig-rescue:SCHA5B0200-SHA5B0200 J3
 U 1 1 5D7BAABF
 P 4600 4550
