File: sd_card.sch (KiCad schematic (older format))
At the start: 11 parts, among them J3 SCHA5B0200, Q3 BSS84

Commit message: Revert "Fixed some external dependencies."
This reverts commit ddca1efdf68af69ddd54947bcdaa3cfa1d913e0d.
Parts:
- C11, C12, C6: symbol qmtech-minimig-rescue:C-Device -> Device:C
- J3: symbol qmtech-minimig-rescue:SCHA5B0200-SHA5B0200 -> SHA5B0200:SCHA5B0200
- Q3: symbol qmtech-minimig-rescue:BSS84-Transistor_FET -> Transistor_FET:BSS84
- R20, R21, R22, R23, R32, R33: symbol qmtech-minimig-rescue:R-Device -> Device:R
Changed lines of the file:
@@
 $EndDescr
 $Comp
-L qmtech-minimig-rescue:SCHA5B0200-SHA5B0200 J3
+L SHA5B0200:SCHA5B0200 J3
 U 1 1 5D7BAABF
 P 4600 4550
@@
 	2550 4850 2750 4850
 $Comp
-L qmtech-minimig-rescue:R-Device R20
+L Device:R R20
 U 1 1 5D7B8F06
 P 2750 3900
@@
 $EndComp
 $Comp
-L qmtech-minimig-rescue:R-Device R21
+L Device:R R21
 U 1 1 5D7B9145
 P 3050 3900
@@
 $EndComp
 $Comp
-L qmtech-minimig-rescue:R-Device R22
+L Device:R R22
 U 1 1 5D7B92B5
 P 3350 3900
@@
 $EndComp
 $Comp
-L qmtech-minimig-rescue:R-Device R23
+L Device:R R23
 U 1 1 5D7B9431
 P 3650 3900
@@
 Connection ~ 3650 3300
 $Comp
-L qmtech-minimig-rescue:C-Device C6
+L Device:C C6
 U 1 1 5D7BEF06
 P 4400 3500
@@
 ESP_SD_DATA2
 $Comp
-L qmtech-minimig-rescue:BSS84-Transistor_FET Q3
+L Transistor_FET:BSS84 Q3
 U 1 1 5D7D8B8E
 P 5600 2825
@@
 	5500 2225 5500 2275
 $Comp
-L qmtech-minimig-rescue:R-Device R32
+L Device:R R32
 U 1 1 5D7EDDF8
 P 5800 2525
@@
 	5500 3025 5500 3300
 $Comp
-L qmtech-minimig-rescue:C-Device C11
+L Device:C C11
 U 1 1 5D80369D
 P 5650 4000
@@
 ESP_SD_SW
 $Comp
-L qmtech-minimig-rescue:R-Device R33
+L Device:R R33
 U 1 1 5D9F486E
 P 5950 4400
@@
 3V3
 $Comp
-L qmtech-minimig-rescue:C-Device C12
+L Device:C C12
 U 1 1 5D9F4F23
 P 5950 4700

Commit message: Did some placement to make the PCB smaller.
Parts:
- J3: symbol SHA5B0200:SCHA5B0200 -> SCHA5B0200:SCHA5B0200
Changed lines of the file:
@@
 $EndDescr
 $Comp
-L SHA5B0200:SCHA5B0200 J3
+L SCHA5B0200:SCHA5B0200 J3
 U 1 1 5D7BAABF
 P 4600 4550

Commit message: Brought compenents back to the front for easy soldering.
Parts:
- added C71: 100nF, Capacitor_SMD:C_0603_1608Metric, symbol Device:C
- added J6: Micro_SD_Card, qmtech-minimig-new:MicroSD-SOFNG-TF-002-H18, symbol Connector:Micro_SD_Card
- added R13, R14, R15, R16: 10k, Resistor_SMD:R_0603_1608Metric, symbol Device:R
Connections:
- net labels added: FPGA_SD_CLK, FPGA_SD_CMD, FPGA_SD_DATA0, FPGA_SD_DATA1, FPGA_SD_DATA2, FPGA_SD_DATA3, FPGA_SD_SW, SD_VDD
- net labels removed: ESP_SD_SW
- wire segments 36 -> 61
Other:
- note added: "ESP32 sd-card"
- note added: "FPGA SD-CARD"

Commit message: Removed ESP32, as it's no longer needed, we have soft cores.
Parts:
- removed C71: 100nF, Capacitor_SMD:C_0603_1608Metric, symbol Device:C
- removed J6: Micro_SD_Card, qmtech-minimig-new:MicroSD-SOFNG-TF-002-H18, symbol Connector:Micro_SD_Card
- removed Q3: BSS84, Package_TO_SOT_SMD:SOT-23, symbol Transistor_FET:BSS84
- removed R13, R14, R15, R16: 10k, Resistor_SMD:R_0603_1608Metric, symbol Device:R
- removed R32: 100k, Resistor_SMD:R_0603_1608Metric, symbol Device:R
- renumbered C6 to C28, C11 to C29, C12 to C30, J3 to J5, R20 to R21, R21 to R22, R22 to R23, R23 to R24, R33 to R25
Connections:
- net labels removed: ESP_SD_CLK, ESP_SD_CMD, ESP_SD_DATA0, ESP_SD_DATA1, ESP_SD_DATA2, ESP_SD_DATA3, ESP_SD_VCC_EN, SD_VDD
- wire segments 61 -> 29
Other:
- note removed: "ESP32 sd-card"
Changed lines of the file:
@@
 $EndDescr
 $Comp
-L SCHA5B0200:SCHA5B0200 J3
+L SCHA5B0200:SCHA5B0200 J5
 U 1 1 5D7BAABF
 P 3700 3175
-F 0 "J3" H 3700 3742 50  0000 C CNN
+F 0 "J5" H 3700 3742 50  0000 C CNN
 F 1 "SCHA5B0200" H 3700 3651 50  0000 C CNN
 F 2 "SHA5B0200:ALPS_SCHA5B0200" H 3700 3175 50  0001 L BNN
@@
 Text GLabel 1650 3275 0    50   Input ~ 0
 FPGA_SD_CMD
-Text GLabel 3150 4700 1    50   Input ~ 0
-3V3
 Text GLabel 1650 2875 0    50   Input ~ 0
 FPGA_SD_DATA0
@@
 	1650 3475 1850 3475
 $Comp
-L Device:R R20
+L Device:R R21
 U 1 1 5D7B8F06
 P 1850 2525
-F 0 "R20" H 1920 2571 50  0000 L CNN
+F 0 "R21" H 1920 2571 50  0000 L CNN
 F 1 "10k" H 1920 2480 50  0000 L CNN
 F 2 "Resistor_SMD:R_0603_1608Metric" V 1780 2525 50  0001 C CNN
@@
 $EndComp
 $Comp
-L Device:R R21
+L Device:R R22
 U 1 1 5D7B9145
 P 2150 2525
-F 0 "R21" H 2220 2571 50  0000 L CNN
+F 0 "R22" H 2220 2571 50  0000 L CNN
 F 1 "10k" H 2220 2480 50  0000 L CNN
 F 2 "Resistor_SMD:R_0603_1608Metric" V 2080 2525 50  0001 C CNN
@@
 $EndComp
 $Comp
-L Device:R R22
+L Device:R R23
 U 1 1 5D7B92B5
 P 2450 2525
-F 0 "R22" H 2520 2571 50  0000 L CNN
+F 0 "R23" H 2520 2571 50  0000 L CNN
 F 1 "10k" H 2520 2480 50  0000 L CNN
 F 2 "Resistor_SMD:R_0603_1608Metric" V 2380 2525 50  0001 C CNN
@@
 $EndComp
 $Comp
-L Device:R R23
+L Device:R R24
 U 1 1 5D7B9431
 P 2750 2525
-F 0 "R23" H 2820 2571 50  0000 L CNN
+F 0 "R24" H 2820 2571 50  0000 L CNN
 F 1 "10k" H 2820 2480 50  0000 L CNN
 F 2 "Resistor_SMD:R_0603_1608Metric" V 2680 2525 50  0001 C CNN
@@
 Connection ~ 2750 1925
 $Comp
-L Device:C C6
+L Device:C C28
 U 1 1 5D7BEF06
 P 3500 2125
-F 0 "C6" H 3615 2171 50  0000 L CNN
+F 0 "C28" H 3615 2171 50  0000 L CNN
 F 1 "100nF" H 3615 2080 50  0000 L CNN
 F 2 "Capacitor_SMD:C_0603_1608Metric" H 3538 1975 50  0001 C CNN
@@
 Text GLabel 1650 3075 0    50   Input ~ 0
 FPGA_SD_DATA2
-$Comp
-L Transistor_FET:BSS84 Q3
-U 1 1 5D7D8B8E
-P 3250 5125
-F 0 "Q3" H 3456 5079 50  0000 L CNN
-F 1 "BSS84" H 3456 5170 50  0000 L CNN
-F 2 "Package_TO_SOT_SMD:SOT-23" H 3450 5050 50  0001 L CIN
-F 3 "http://assets.nexperia.com/documents/data-sheet/BSS84.pdf" H 3250 5125 50  0001 L CNN
-	1    3250 5125
-	-1   0    0    1
-$EndComp
-Text GLabel 3500 5125 2    50   Input ~ 0
-ESP_SD_VCC_EN
-Wire Wire Line
-	3150 4700 3150 4750
-$Comp
-L Device:R R32
-U 1 1 5D7EDDF8
-P 3450 4925
-F 0 "R32" H 3520 4971 50  0000 L CNN
-F 1 "100k" H 3520 4880 50  0000 L CNN
-F 2 "Resistor_SMD:R_0603_1608Metric" V 3380 4925 50  0001 C CNN
-F 3 "~" H 3450 4925 50  0001 C CNN
-	1    3450 4925
-	1    0    0    -1
-$EndComp
-Wire Wire Line
-	3450 5075 3450 5125
-Connection ~ 3450 5125
-Wire Wire Line
-	3450 5125 3500 5125
-Wire Wire Line
-	3450 4775 3450 4750
-Wire Wire Line
-	3450 4750 3150 4750
-Connection ~ 3150 4750
-Wire Wire Line
-	3150 4750 3150 4925
 Wire Wire Line
 	4400 2875 4600 2875
-Wire Wire Line
-	3150 5325 3150 5375
-$Comp
-L Device:C C11
+$Comp
+L Device:C C29
 U 1 1 5D80369D
 P 4750 2625
-F 0 "C11" V 4498 2625 50  0000 C CNN
+F 0 "C29" V 4498 2625 50  0000 C CNN
 F 1 "100nF" V 4589 2625 50  0000 C CNN
 F 2 "Capacitor_SMD:C_0603_1608Metric" H 4788 2475 50  0001 C CNN
@@
 FPGA_SD_SW
 $Comp
-L Device:R R33
+L Device:R R25
 U 1 1 5D9F486E
 P 5050 3025
-F 0 "R33" H 5120 3071 50  0000 L CNN
+F 0 "R25" H 5120 3071 50  0000 L CNN
 F 1 "10K" H 5120 2980 50  0000 L CNN
 F 2 "Resistor_SMD:R_0603_1608Metric" V 4980 3025 50  0001 C CNN
@@
 3V3
 $Comp
-L Device:C C12
+L Device:C C30
 U 1 1 5D9F4F23
 P 5050 3325
-F 0 "C12" H 5165 3371 50  0000 L CNN
+F 0 "C30" H 5165 3371 50  0000 L CNN
 F 1 "100nF" H 5165 3280 50  0000 L CNN
 F 2 "Capacitor_SMD:C_0603_1608Metric" H 5088 3175 50  0001 C CNN
@@
 Wire Notes Line
 	475  475  6025 475
-Wire Notes Line
-	6025 3750 475  3750
 Text Notes 675  625  0    50   ~ 0
 FPGA SD-CARD
-$Comp
-L Connector:Micro_SD_Card J6
-U 1 1 5F9C5FBC
-P 4150 6700
-F 0 "J6" H 4100 7417 50  0000 C CNN
-F 1 "Micro_SD_Card" H 4100 7326 50  0000 C CNN
-F 2 "qmtech-minimig-new:MicroSD-SOFNG-TF-002-H18" H 5300 7000 50  0001 C CNN
-F 3 "http://katalog.we-online.de/em/datasheet/693072010801.pdf" H 4150 6700 50  0001 C CNN
-	1    4150 6700
-	1    0    0    -1
-$EndComp
-$Comp
-L Device:R R13
-U 1 1 5F9CD895
-P 1800 5975
-F 0 "R13" H 1870 6021 50  0000 L CNN
-F 1 "10k" H 1870 5930 50  0000 L CNN
-F 2 "Resistor_SMD:R_0603_1608Metric" V 1730 5975 50  0001 C CNN
-F 3 "~" H 1800 5975 50  0001 C CNN
-	1    1800 5975
-	1    0    0    -1
-$EndComp
-$Comp
-L Device:R R14
-U 1 1 5F9CD89B
-P 2100 5975
-F 0 "R14" H 2170 6021 50  0000 L CNN
-F 1 "10k" H 2170 5930 50  0000 L CNN
-F 2 "Resistor_SMD:R_0603_1608Metric" V 2030 5975 50  0001 C CNN
-F 3 "~" H 2100 5975 50  0001 C CNN
-	1    2100 5975
-	1    0    0    -1
-$EndComp
-$Comp
-L Device:R R15
-U 1 1 5F9CD8A1
-P 2400 5975
-F 0 "R15" H 2470 6021 50  0000 L CNN
-F 1 "10k" H 2470 5930 50  0000 L CNN
-F 2 "Resistor_SMD:R_0603_1608Metric" V 2330 5975 50  0001 C CNN
-F 3 "~" H 2400 5975 50  0001 C CNN
-	1    2400 5975
-	1    0    0    -1
-$EndComp
-$Comp
-L Device:R R16
-U 1 1 5F9CD8A7
-P 2700 5975
-F 0 "R16" H 2770 6021 50  0000 L CNN
-F 1 "10k" H 2770 5930 50  0000 L CNN
-F 2 "Resistor_SMD:R_0603_1608Metric" V 2630 5975 50  0001 C CNN
-F 3 "~" H 2700 5975 50  0001 C CNN
-	1    2700 5975
-	1    0    0    -1
-$EndComp
-Wire Wire Line
-	1800 6125 1800 7000
-Wire Wire Line
-	2100 6125 2100 6800
-Wire Wire Line
-	2400 6125 2400 6600
-Wire Wire Line
-	2700 6125 2700 6500
-Wire Wire Line
-	1800 5825 1800 5375
-Wire Wire Line
-	1800 5375 2100 5375
-Wire Wire Line
-	2100 5825 2100 5375
-Connection ~ 2100 5375
-Wire Wire Line
-	2100 5375 2400 5375
-Wire Wire Line
-	2400 5375 2400 5825
-Connection ~ 2400 5375
-Wire Wire Line
-	2400 5375 2700 5375
-Wire Wire Line
-	2700 5825 2700 5375
-Connection ~ 2700 5375
-Wire Wire Line
-	2700 5375 3150 5375
-Wire Wire Line
-	3250 7000 1800 7000
-Wire Wire Line
-	3250 7100 1625 7100
-Wire Wire Line
-	3250 6400 1625 6400
-Wire Wire Line
-	3250 6500 2700 6500
-Wire Wire Line
-	3250 6600 2400 6600
-Wire Wire Line
-	3250 6800 2100 6800
-Text GLabel 3250 6900 0    50   Input ~ 0
-GND
-Wire Wire Line
-	3250 6700 3150 6700
-Wire Wire Line
-	3150 6700 3150 5950
-Connection ~ 2700 6500
-Wire Wire Line
-	2700 6500 1625 6500
-Connection ~ 1800 7000
-Wire Wire Line
-	1800 7000 1625 7000
-Connection ~ 2400 6600
-Wire Wire Line
-	2400 6600 1625 6600
-Connection ~ 2100 6800
-Wire Wire Line
-	2100 6800 1625 6800
-$Comp
-L Device:C C71
-U 1 1 5F9E87BB
-P 3300 5950
-F 0 "C71" V 3048 5950 50  0000 C CNN
-F 1 "100nF" V 3139 5950 50  0000 C CNN
-F 2 "Capacitor_SMD:C_0603_1608Metric" H 3338 5800 50  0001 C CNN
-F 3 "~" H 3300 5950 50  0001 C CNN
-	1    3300 5950
-	0    1    1    0
-$EndComp
-Text GLabel 3450 5950 2    50   Input ~ 0
-GND
-Connection ~ 3150 5950
-Wire Wire Line
-	3150 5950 3150 5375
-Text GLabel 4950 7300 2    50   Input ~ 0
-GND
-Text GLabel 1625 6500 0    50   Input ~ 0
-ESP_SD_DATA3
-Text GLabel 1625 6600 0    50   Input ~ 0
-ESP_SD_CMD
-Text GLabel 1625 7000 0    50   Input ~ 0
-ESP_SD_DATA0
-Text GLabel 1625 6800 0    50   Input ~ 0
-ESP_SD_CLK
-Text GLabel 1625 7100 0    50   Input ~ 0
-ESP_SD_DATA1
-Text GLabel 1625 6400 0    50   Input ~ 0
-ESP_SD_DATA2
-Connection ~ 3150 5375
-Text Notes 700  3975 0    50   ~ 0
-ESP32 sd-card
 Wire Notes Line
 	6025 7800 475  7800
 Wire Notes Line
-	6025 475  6025 7800
-Wire Notes Line
 	475  475  475  7800
-Text Label 2600 5375 0    50   ~ 0
-SD_VDD
 Text GLabel 3775 1925 1    50   Input ~ 0
 3V3

Commit message: Fixed decoupling of VDD SDRAM, fixed pinout error in V4 board pinout sheet.
Parts:
- added R? (x2): 10k, Resistor_SMD:R_0603_1608Metric, symbol Device:R
Connections:
- wire segments 29 -> 37
Changed lines of the file:
@@
 Text GLabel 4400 3475 2    50   Input ~ 0
 GND
-Text GLabel 1650 3175 0    50   Input ~ 0
+Text GLabel 1500 3175 0    50   Input ~ 0
 FPGA_SD_DATA3
-Text GLabel 1650 3275 0    50   Input ~ 0
+Text GLabel 1500 3275 0    50   Input ~ 0
 FPGA_SD_CMD
-Text GLabel 1650 2875 0    50   Input ~ 0
+Text GLabel 1500 2875 0    50   Input ~ 0
 FPGA_SD_DATA0
-Text GLabel 1650 3475 0    50   Input ~ 0
+Text GLabel 1500 3475 0    50   Input ~ 0
 FPGA_SD_CLK
 Text GLabel 4400 3375 2    50   Input ~ 0
 GND
 Wire Wire Line
-	1650 2875 2750 2875
-Wire Wire Line
-	1650 3175 2450 3175
-Wire Wire Line
-	1650 3275 2150 3275
-Wire Wire Line
-	1650 3475 1850 3475
+	1500 3175 2125 3175
+Wire Wire Line
+	1500 3275 1850 3275
+Wire Wire Line
+	1500 3475 1575 3475
 $Comp
 L Device:R R21
 U 1 1 5D7B8F06
+P 1575 2525
+F 0 "R21" H 1645 2571 50  0000 L CNN
+F 1 "10k" H 1645 2480 50  0000 L CNN
+F 2 "Resistor_SMD:R_0603_1608Metric" V 1505 2525 50  0001 C CNN
+F 3 "~" H 1575 2525 50  0001 C CNN
+	1    1575 2525
+	1    0    0    -1
+$EndComp
+$Comp
+L Device:R R22
+U 1 1 5D7B9145
 P 1850 2525
-F 0 "R21" H 1920 2571 50  0000 L CNN
+F 0 "R22" H 1920 2571 50  0000 L CNN
 F 1 "10k" H 1920 2480 50  0000 L CNN
 F 2 "Resistor_SMD:R_0603_1608Metric" V 1780 2525 50  0001 C CNN
@@
 $EndComp
 $Comp
-L Device:R R22
-U 1 1 5D7B9145
-P 2150 2525
-F 0 "R22" H 2220 2571 50  0000 L CNN
-F 1 "10k" H 2220 2480 50  0000 L CNN
-F 2 "Resistor_SMD:R_0603_1608Metric" V 2080 2525 50  0001 C CNN
-F 3 "~" H 2150 2525 50  0001 C CNN
-	1    2150 2525
-	1    0    0    -1
-$EndComp
-$Comp
 L Device:R R23
 U 1 1 5D7B92B5
-P 2450 2525
-F 0 "R23" H 2520 2571 50  0000 L CNN
-F 1 "10k" H 2520 2480 50  0000 L CNN
-F 2 "Resistor_SMD:R_0603_1608Metric" V 2380 2525 50  0001 C CNN
-F 3 "~" H 2450 2525 50  0001 C CNN
-	1    2450 2525
+P 2125 2525
+F 0 "R23" H 2195 2571 50  0000 L CNN
+F 1 "10k" H 2195 2480 50  0000 L CNN
+F 2 "Resistor_SMD:R_0603_1608Metric" V 2055 2525 50  0001 C CNN
+F 3 "~" H 2125 2525 50  0001 C CNN
+	1    2125 2525
 	1    0    0    -1
 $EndComp
@@
 L Device:R R24
 U 1 1 5D7B9431
-P 2750 2525
-F 0 "R24" H 2820 2571 50  0000 L CNN
-F 1 "10k" H 2820 2480 50  0000 L CNN
-F 2 "Resistor_SMD:R_0603_1608Metric" V 2680 2525 50  0001 C CNN
-F 3 "~" H 2750 2525 50  0001 C CNN
-	1    2750 2525
-	1    0    0    -1
-$EndComp
-Wire Wire Line
-	1850 2675 1850 3475
-Connection ~ 1850 3475
-Wire Wire Line
-	1850 3475 3000 3475
-Wire Wire Line
-	2150 2675 2150 3275
-Connection ~ 2150 3275
-Wire Wire Line
-	2150 3275 3000 3275
-Wire Wire Line
-	2450 2675 2450 3175
-Connection ~ 2450 3175
-Wire Wire Line
-	2450 3175 3000 3175
-Wire Wire Line
-	2750 2675 2750 2875
-Connection ~ 2750 2875
-Wire Wire Line
-	2750 2875 3000 2875
+P 2975 2525
+F 0 "R24" H 3045 2571 50  0000 L CNN
+F 1 "10k" H 3045 2480 50  0000 L CNN
+F 2 "Resistor_SMD:R_0603_1608Metric" V 2905 2525 50  0001 C CNN
+F 3 "~" H 2975 2525 50  0001 C CNN
+	1    2975 2525
+	1    0    0    -1
+$EndComp
+Wire Wire Line
+	1575 2675 1575 3475
+Wire Wire Line
+	1850 2675 1850 3275
+Wire Wire Line
+	2125 2675 2125 3175
+Wire Wire Line
+	2975 2675 2975 2875
+Wire Wire Line
+	1575 2375 1575 1925
+Wire Wire Line
+	1575 1925 1850 1925
 Wire Wire Line
 	1850 2375 1850 1925
 Wire Wire Line
-	1850 1925 2150 1925
-Wire Wire Line
-	2150 2375 2150 1925
-Connection ~ 2150 1925
-Wire Wire Line
-	2150 1925 2450 1925
-Wire Wire Line
-	2450 1925 2450 2375
-Connection ~ 2450 1925
-Wire Wire Line
-	2450 1925 2750 1925
-Wire Wire Line
-	2750 2375 2750 1925
-Connection ~ 2750 1925
+	2125 1925 2125 2375
+Wire Wire Line
+	2975 2375 2975 1925
 $Comp
 L Device:C C28
@@
 Text GLabel 3500 2275 3    50   Input ~ 0
 GND
-Wire Wire Line
-	3000 2975 1650 2975
-Wire Wire Line
-	3000 3075 1650 3075
-Text GLabel 1650 2975 0    50   Input ~ 0
+Text GLabel 1500 2975 0    50   Input ~ 0
 FPGA_SD_DATA1
-Text GLabel 1650 3075 0    50   Input ~ 0
+Text GLabel 1500 3075 0    50   Input ~ 0
 FPGA_SD_DATA2
 Wire Wire Line
@@
 Wire Wire Line
 	4600 1925 4600 2625
-Wire Wire Line
-	2750 1925 3500 1925
 Wire Notes Line
 	475  475  6025 475
@@
 Text GLabel 3775 1925 1    50   Input ~ 0
 3V3
+$Comp
+L Device:R R?
+U 1 1 5FC58804
+P 2675 2525
+F 0 "R?" H 2745 2571 50  0000 L CNN
+F 1 "10k" H 2745 2480 50  0000 L CNN
+F 2 "Resistor_SMD:R_0603_1608Metric" V 2605 2525 50  0001 C CNN
+F 3 "~" H 2675 2525 50  0001 C CNN
+	1    2675 2525
+	1    0    0    -1
+$EndComp
+Wire Wire Line
+	2675 2375 2675 1925
+Wire Wire Line
+	2675 2675 2675 2975
+$Comp
+L Device:R R?
+U 1 1 5FC5A596
+P 2400 2525
+F 0 "R?" H 2470 2571 50  0000 L CNN
+F 1 "10k" H 2470 2480 50  0000 L CNN
+F 2 "Resistor_SMD:R_0603_1608Metric" V 2330 2525 50  0001 C CNN
+F 3 "~" H 2400 2525 50  0001 C CNN
+	1    2400 2525
+	1    0    0    -1
+$EndComp
+Wire Wire Line
+	2400 2375 2400 1925
+Wire Wire Line
+	2400 2675 2400 3075
+Connection ~ 2975 1925
+Wire Wire Line
+	2975 1925 3500 1925
+Connection ~ 2975 2875
+Wire Wire Line
+	2975 2875 3000 2875
+Wire Wire Line
+	1500 2875 2975 2875
+Wire Wire Line
+	1500 2975 2675 2975
+Wire Wire Line
+	1500 3075 2400 3075
+Connection ~ 1575 3475
+Wire Wire Line
+	1575 3475 3000 3475
+Connection ~ 1850 1925
+Connection ~ 1850 3275
+Wire Wire Line
+	1850 3275 3000 3275
+Wire Wire Line
+	1850 1925 2125 1925
+Connection ~ 2125 1925
+Connection ~ 2125 3175
+Wire Wire Line
+	2125 3175 3000 3175
+Wire Wire Line
+	2125 1925 2400 1925
+Connection ~ 2400 1925
+Connection ~ 2400 3075
+Wire Wire Line
+	2400 3075 3000 3075
+Wire Wire Line
+	2400 1925 2675 1925
+Connection ~ 2675 1925
+Connection ~ 2675 2975
+Wire Wire Line
+	2675 2975 3000 2975
+Wire Wire Line
+	2675 1925 2975 1925
 $EndSCHEMATC

Commit message: Fixed issue with missing PS2 pullups, add line to adv interrupt.
Parts:
- gave numbers to parts that had none: 2
Changed lines of the file:
@@
 3V3
 $Comp
-L Device:R R?
+L Device:R R59
 U 1 1 5FC58804
 P 2675 2525
-F 0 "R?" H 2745 2571 50  0000 L CNN
+F 0 "R59" H 2745 2571 50  0000 L CNN
 F 1 "10k" H 2745 2480 50  0000 L CNN
 F 2 "Resistor_SMD:R_0603_1608Metric" V 2605 2525 50  0001 C CNN
@@
 	2675 2675 2675 2975
 $Comp
-L Device:R R?
+L Device:R R58
 U 1 1 5FC5A596
 P 2400 2525
-F 0 "R?" H 2470 2571 50  0000 L CNN
+F 0 "R58" H 2470 2571 50  0000 L CNN
 F 1 "10k" H 2470 2480 50  0000 L CNN
 F 2 "Resistor_SMD:R_0603_1608Metric" V 2330 2525 50  0001 C CNN
