File: sdram.sch (KiCad schematic (older format))
At the start: 10 parts, among them IC2 AS4C16M16SA-6TCN

Commit message: Implemented the Floppy interface, fixed 12V power up issue with the board.
Parts:
- removed R1: 10k, Resistor_SMD:R_0603_1608Metric, symbol Device:R
- C56, C58, C59, C61, C62, C63: value 100n -> 100nF
- C64, C65: value 10u -> 10uF
Connections:
- wire segments 41 -> 38
Changed lines of the file:
@@
 Text GLabel 6600 5100 2    50   Input ~ 0
 SDRAM_A4
-$Comp
-L Device:R R1
-U 1 1 5F1B5BCA
-P 8000 4150
-F 0 "R1" V 7793 4150 50  0000 C CNN
-F 1 "10k" V 7884 4150 50  0000 C CNN
-F 2 "Resistor_SMD:R_0603_1608Metric" V 7930 4150 50  0001 C CNN
-F 3 "~" H 8000 4150 50  0001 C CNN
-	1    8000 4150
-	1    0    0    -1
-$EndComp
 Text GLabel 8000 2250 1    50   Input ~ 0
 3V3
-Wire Wire Line
-	6600 4300 8000 4300
 Text GLabel 6600 4400 2    50   Input ~ 0
 SDRAM_A12
@@
 P 1250 2900
 F 0 "C56" H 1365 2946 50  0000 L CNN
-F 1 "100n" H 1365 2855 50  0000 L CNN
+F 1 "100nF" H 1365 2855 50  0000 L CNN
 F 2 "Capacitor_SMD:C_0603_1608Metric" H 1288 2750 50  0001 C CNN
 F 3 "~" H 1250 2900 50  0001 C CNN
@@
 P 1750 2900
 F 0 "C59" H 1865 2946 50  0000 L CNN
-F 1 "100n" H 1865 2855 50  0000 L CNN
+F 1 "100nF" H 1865 2855 50  0000 L CNN
 F 2 "Capacitor_SMD:C_0603_1608Metric" H 1788 2750 50  0001 C CNN
 F 3 "~" H 1750 2900 50  0001 C CNN
@@
 P 2250 2900
 F 0 "C62" H 2365 2946 50  0000 L CNN
-F 1 "100n" H 2365 2855 50  0000 L CNN
+F 1 "100nF" H 2365 2855 50  0000 L CNN
 F 2 "Capacitor_SMD:C_0603_1608Metric" H 2288 2750 50  0001 C CNN
 F 3 "~" H 2250 2900 50  0001 C CNN
@@
 P 2750 2900
 F 0 "C64" H 2865 2946 50  0000 L CNN
-F 1 "10u" H 2865 2855 50  0000 L CNN
+F 1 "10uF" H 2865 2855 50  0000 L CNN
 F 2 "Capacitor_SMD:C_0805_2012Metric" H 2788 2750 50  0001 C CNN
 F 3 "~" H 2750 2900 50  0001 C CNN
@@
 P 1250 4150
 F 0 "C58" H 1365 4196 50  0000 L CNN
-F 1 "100n" H 1365 4105 50  0000 L CNN
+F 1 "100nF" H 1365 4105 50  0000 L CNN
 F 2 "Capacitor_SMD:C_0603_1608Metric" H 1288 4000 50  0001 C CNN
 F 3 "~" H 1250 4150 50  0001 C CNN
@@
 P 1750 4150
 F 0 "C61" H 1865 4196 50  0000 L CNN
-F 1 "100n" H 1865 4105 50  0000 L CNN
+F 1 "100nF" H 1865 4105 50  0000 L CNN
 F 2 "Capacitor_SMD:C_0603_1608Metric" H 1788 4000 50  0001 C CNN
 F 3 "~" H 1750 4150 50  0001 C CNN
@@
 P 2250 4150
 F 0 "C63" H 2365 4196 50  0000 L CNN
-F 1 "100n" H 2365 4105 50  0000 L CNN
+F 1 "100nF" H 2365 4105 50  0000 L CNN
 F 2 "Capacitor_SMD:C_0603_1608Metric" H 2288 4000 50  0001 C CNN
 F 3 "~" H 2250 4150 50  0001 C CNN
@@
 P 2750 4150
 F 0 "C65" H 2865 4196 50  0000 L CNN
-F 1 "10u" H 2865 4105 50  0000 L CNN
+F 1 "10uF" H 2865 4105 50  0000 L CNN
 F 2 "Capacitor_SMD:C_0805_2012Metric" H 2788 4000 50  0001 C CNN
 F 3 "~" H 2750 4150 50  0001 C CNN
@@
 Text GLabel 1250 2750 1    50   Input ~ 0
 3V3
-Text GLabel 8100 4300 2    50   Input ~ 0
+Text GLabel 6600 4300 2    50   Input ~ 0
 SDRAM_CKE
-Wire Wire Line
-	8000 4300 8100 4300
-Connection ~ 8000 4300
-Wire Wire Line
-	8000 4000 8000 3700
-Connection ~ 8000 3700
 $EndSCHEMATC

Commit message: Version that was sent to JLCPCB 20200716.
Connections:
- no-connect marks 0 -> 1
Changed lines of the file:
@@
 Text GLabel 6600 4300 2    50   Input ~ 0
 SDRAM_CKE
+NoConn ~ 6600 4000
 $EndSCHEMATC

Commit message: Fixed SDRAM_A12 missing route, disconnected JS_INT_B.
Connections:
- net labels added: SDRAM_D10, SDRAM_D11, SDRAM_D12, SDRAM_D13, SDRAM_D14, SDRAM_D15, SDRAM_D8, SDRAM_D9
- net labels removed: SDRAM_DQ10, SDRAM_DQ11, SDRAM_DQ12, SDRAM_DQ13, SDRAM_DQ14, SDRAM_DQ15, SDRAM_DQ8, SDRAM_DQ9
Changed lines of the file:
@@
 SDRAM_A3
 Text GLabel 6600 2700 2    50   Input ~ 0
-SDRAM_DQ15
+SDRAM_D15
 Text GLabel 6600 2900 2    50   Input ~ 0
-SDRAM_DQ14
+SDRAM_D14
 Text GLabel 6600 3000 2    50   Input ~ 0
-SDRAM_DQ13
+SDRAM_D13
 Text GLabel 6600 3200 2    50   Input ~ 0
-SDRAM_DQ12
+SDRAM_D12
 Text GLabel 6600 3300 2    50   Input ~ 0
-SDRAM_DQ11
+SDRAM_D11
 Text GLabel 6600 3500 2    50   Input ~ 0
-SDRAM_DQ10
+SDRAM_D10
 Text GLabel 6600 3600 2    50   Input ~ 0
-SDRAM_DQ9
+SDRAM_D9
 Text GLabel 6600 3800 2    50   Input ~ 0
-SDRAM_DQ8
+SDRAM_D8
 Text GLabel 6600 4100 2    50   Input ~ 0
 SDRAM_DQMH

Commit message: Removed all libraries that depend on absolute paths.
Parts:
- IC2: symbol AS4C16M16SA-6TCN:AS4C16M16SA-6TCN -> qmtech-minimig-rescue:AS4C16M16SA-6TCN-AS4C16M16SA-6TCN
Changed lines of the file:
@@
 $EndDescr
 $Comp
-L AS4C16M16SA-6TCN:AS4C16M16SA-6TCN IC2
+L qmtech-minimig-rescue:AS4C16M16SA-6TCN-AS4C16M16SA-6TCN IC2
 U 1 1 5F1B044E
 P 5300 2600
