File: sdram.sch (KiCad schematic (older format))
At the start: 9 parts, among them IC2 AS4C16M16SA-6TCN

Commit message: Fixed some external dependencies.
Parts:
- C56, C58, C59, C61, C62, C63, C64, C65: symbol Device:C -> qmtech-minimig-rescue:C-Device
- IC2: footprint SOP80P1176X120-54N -> qmtech-minimig-new:SOP80P1176X120-54N; symbol AS4C16M16SA-6TCN:AS4C16M16SA-6TCN -> qmtech-minimig-rescue:AS4C16M16SA-6TCN-AS4C16M16SA-6TCN
Changed lines of the file:
@@
 $EndDescr
 $Comp
-L AS4C16M16SA-6TCN:AS4C16M16SA-6TCN IC2
+L qmtech-minimig-rescue:AS4C16M16SA-6TCN-AS4C16M16SA-6TCN IC2
 U 1 1 5F1B044E
 P 5300 2600
 F 0 "IC2" H 5950 2865 50  0000 C CNN
 F 1 "AS4C16M16SA-6TCN" H 5950 2774 50  0000 C CNN
-F 2 "SOP80P1176X120-54N" H 6450 2700 50  0001 L CNN
+F 2 "qmtech-minimig-new:SOP80P1176X120-54N" H 6450 2700 50  0001 L CNN
 F 3 "https://www.alliancememory.com/wp-content/uploads/pdf/dram/256Mb-AS4C16M16SA-C&I_V3.0_March%202015.pdf" H 6450 2600 50  0001 L CNN
 F 4 "256M  (16Mx16bit) Synchronous DRAM (SDRAM)" H 6450 2500 50  0001 L CNN "Description"
@@
 Connection ~ 4500 3700
 $Comp
-L Device:C C56
+L qmtech-minimig-rescue:C-Device C56
 U 1 1 5F1C855A
 P 1250 2900
@@
 $EndComp
 $Comp
-L Device:C C59
+L qmtech-minimig-rescue:C-Device C59
 U 1 1 5F1C918D
 P 1750 2900
@@
 $EndComp
 $Comp
-L Device:C C62
+L qmtech-minimig-rescue:C-Device C62
 U 1 1 5F1C98DC
 P 2250 2900
@@
 $EndComp
 $Comp
-L Device:C C64
+L qmtech-minimig-rescue:C-Device C64
 U 1 1 5F1C9F11
 P 2750 2900
@@
 $EndComp
 $Comp
-L Device:C C58
+L qmtech-minimig-rescue:C-Device C58
 U 1 1 5F1CA689
 P 1250 4150
@@
 $EndComp
 $Comp
-L Device:C C61
+L qmtech-minimig-rescue:C-Device C61
 U 1 1 5F1CADBB
 P 1750 4150
@@
 $EndComp
 $Comp
-L Device:C C63
+L qmtech-minimig-rescue:C-Device C63
 U 1 1 5F1CB5BD
 P 2250 4150
@@
 $EndComp
 $Comp
-L Device:C C65
+L qmtech-minimig-rescue:C-Device C65
 U 1 1 5F1CC080
 P 2750 4150

Commit message: Revert "Fixed some external dependencies."
This reverts commit ddca1efdf68af69ddd54947bcdaa3cfa1d913e0d.
Parts:
- C56, C58, C59, C61, C62, C63, C64, C65: symbol qmtech-minimig-rescue:C-Device -> Device:C
- IC2: footprint qmtech-minimig-new:SOP80P1176X120-54N -> SOP80P1176X120-54N; symbol qmtech-minimig-rescue:AS4C16M16SA-6TCN-AS4C16M16SA-6TCN -> AS4C16M16SA-6TCN:AS4C16M16SA-6TCN
Changed lines of the file:
@@
 $EndDescr
 $Comp
-L qmtech-minimig-rescue:AS4C16M16SA-6TCN-AS4C16M16SA-6TCN IC2
+L AS4C16M16SA-6TCN:AS4C16M16SA-6TCN IC2
 U 1 1 5F1B044E
 P 5300 2600
 F 0 "IC2" H 5950 2865 50  0000 C CNN
 F 1 "AS4C16M16SA-6TCN" H 5950 2774 50  0000 C CNN
-F 2 "qmtech-minimig-new:SOP80P1176X120-54N" H 6450 2700 50  0001 L CNN
+F 2 "SOP80P1176X120-54N" H 6450 2700 50  0001 L CNN
 F 3 "https://www.alliancememory.com/wp-content/uploads/pdf/dram/256Mb-AS4C16M16SA-C&I_V3.0_March%202015.pdf" H 6450 2600 50  0001 L CNN
 F 4 "256M  (16Mx16bit) Synchronous DRAM (SDRAM)" H 6450 2500 50  0001 L CNN "Description"
@@
 Connection ~ 4500 3700
 $Comp
-L qmtech-minimig-rescue:C-Device C56
+L Device:C C56
 U 1 1 5F1C855A
 P 1250 2900
@@
 $EndComp
 $Comp
-L qmtech-minimig-rescue:C-Device C59
+L Device:C C59
 U 1 1 5F1C918D
 P 1750 2900
@@
 $EndComp
 $Comp
-L qmtech-minimig-rescue:C-Device C62
+L Device:C C62
 U 1 1 5F1C98DC
 P 2250 2900
@@
 $EndComp
 $Comp
-L qmtech-minimig-rescue:C-Device C64
+L Device:C C64
 U 1 1 5F1C9F11
 P 2750 2900
@@
 $EndComp
 $Comp
-L qmtech-minimig-rescue:C-Device C58
+L Device:C C58
 U 1 1 5F1CA689
 P 1250 4150
@@
 $EndComp
 $Comp
-L qmtech-minimig-rescue:C-Device C61
+L Device:C C61
 U 1 1 5F1CADBB
 P 1750 4150
@@
 $EndComp
 $Comp
-L qmtech-minimig-rescue:C-Device C63
+L Device:C C63
 U 1 1 5F1CB5BD
 P 2250 4150
@@
 $EndComp
 $Comp
-L qmtech-minimig-rescue:C-Device C65
+L Device:C C65
 U 1 1 5F1CC080
 P 2750 4150

Commit message: Brought compenents back to the front for easy soldering.
Parts:
- added C66, C68, C69: 10nF, Capacitor_SMD:C_0603_1608Metric, symbol Device:C
Connections:
- wire segments 38 -> 44
Other:
- note added: "Return path decoupling"
Changed lines of the file:
@@
 SDRAM_CKE
 NoConn ~ 6600 4000
+Text Notes 1575 6150 0    50   ~ 0
+Return path decoupling
+$Comp
+L Device:C C66
+U 1 1 5F8FCA63
+P 1575 6525
+F 0 "C66" H 1690 6571 50  0000 L CNN
+F 1 "10nF" H 1690 6480 50  0000 L CNN
+F 2 "Capacitor_SMD:C_0603_1608Metric" H 1613 6375 50  0001 C CNN
+F 3 "~" H 1575 6525 50  0001 C CNN
+	1    1575 6525
+	1    0    0    -1
+$EndComp
+$Comp
+L Device:C C68
+U 1 1 5F8FD1C4
+P 2000 6525
+F 0 "C68" H 2115 6571 50  0000 L CNN
+F 1 "10nF" H 2115 6480 50  0000 L CNN
+F 2 "Capacitor_SMD:C_0603_1608Metric" H 2038 6375 50  0001 C CNN
+F 3 "~" H 2000 6525 50  0001 C CNN
+	1    2000 6525
+	1    0    0    -1
+$EndComp
+$Comp
+L Device:C C69
+U 1 1 5F8FD3F9
+P 2425 6525
+F 0 "C69" H 2540 6571 50  0000 L CNN
+F 1 "10nF" H 2540 6480 50  0000 L CNN
+F 2 "Capacitor_SMD:C_0603_1608Metric" H 2463 6375 50  0001 C CNN
+F 3 "~" H 2425 6525 50  0001 C CNN
+	1    2425 6525
+	1    0    0    -1
+$EndComp
+Wire Wire Line
+	2425 6375 2000 6375
+Connection ~ 1575 6375
+Wire Wire Line
+	1575 6375 1325 6375
+Connection ~ 2000 6375
+Wire Wire Line
+	2000 6375 1575 6375
+Wire Wire Line
+	2425 6675 2000 6675
+Connection ~ 1575 6675
+Wire Wire Line
+	1575 6675 1325 6675
+Connection ~ 2000 6675
+Wire Wire Line
+	2000 6675 1575 6675
+Text GLabel 1325 6375 0    50   Input ~ 0
+3V3
+Text GLabel 1325 6675 0    50   Input ~ 0
+GND
 $EndSCHEMATC

Commit message: Removed ESP32, as it's no longer needed, we have soft cores.
Parts:
- renumbered C56 to C53, C58 to C54, C66 to C55, C59 to C56, C61 to C57, C68 to C58, C62 to C59, C63 to C60, C69 to C61, C64 to C62, C65 to C63, IC2 to IC1
Changed lines of the file:
@@
 $EndDescr
 $Comp
-L AS4C16M16SA-6TCN:AS4C16M16SA-6TCN IC2
+L AS4C16M16SA-6TCN:AS4C16M16SA-6TCN IC1
 U 1 1 5F1B044E
 P 5300 2600
-F 0 "IC2" H 5950 2865 50  0000 C CNN
+F 0 "IC1" H 5950 2865 50  0000 C CNN
 F 1 "AS4C16M16SA-6TCN" H 5950 2774 50  0000 C CNN
 F 2 "SOP80P1176X120-54N" H 6450 2700 50  0001 L CNN
@@
 Connection ~ 4500 3700
 $Comp
-L Device:C C56
+L Device:C C53
 U 1 1 5F1C855A
 P 1250 2900
-F 0 "C56" H 1365 2946 50  0000 L CNN
+F 0 "C53" H 1365 2946 50  0000 L CNN
 F 1 "100nF" H 1365 2855 50  0000 L CNN
 F 2 "Capacitor_SMD:C_0603_1608Metric" H 1288 2750 50  0001 C CNN
@@
 $EndComp
 $Comp
-L Device:C C59
+L Device:C C56
 U 1 1 5F1C918D
 P 1750 2900
-F 0 "C59" H 1865 2946 50  0000 L CNN
+F 0 "C56" H 1865 2946 50  0000 L CNN
 F 1 "100nF" H 1865 2855 50  0000 L CNN
 F 2 "Capacitor_SMD:C_0603_1608Metric" H 1788 2750 50  0001 C CNN
@@
 $EndComp
 $Comp
-L Device:C C62
+L Device:C C59
 U 1 1 5F1C98DC
 P 2250 2900
-F 0 "C62" H 2365 2946 50  0000 L CNN
+F 0 "C59" H 2365 2946 50  0000 L CNN
 F 1 "100nF" H 2365 2855 50  0000 L CNN
 F 2 "Capacitor_SMD:C_0603_1608Metric" H 2288 2750 50  0001 C CNN
@@
 $EndComp
 $Comp
-L Device:C C64
+L Device:C C62
 U 1 1 5F1C9F11
 P 2750 2900
-F 0 "C64" H 2865 2946 50  0000 L CNN
+F 0 "C62" H 2865 2946 50  0000 L CNN
 F 1 "10uF" H 2865 2855 50  0000 L CNN
 F 2 "Capacitor_SMD:C_0805_2012Metric" H 2788 2750 50  0001 C CNN
@@
 $EndComp
 $Comp
-L Device:C C58
+L Device:C C54
 U 1 1 5F1CA689
 P 1250 4150
-F 0 "C58" H 1365 4196 50  0000 L CNN
+F 0 "C54" H 1365 4196 50  0000 L CNN
 F 1 "100nF" H 1365 4105 50  0000 L CNN
 F 2 "Capacitor_SMD:C_0603_1608Metric" H 1288 4000 50  0001 C CNN
@@
 $EndComp
 $Comp
-L Device:C C61
+L Device:C C57
 U 1 1 5F1CADBB
 P 1750 4150
-F 0 "C61" H 1865 4196 50  0000 L CNN
+F 0 "C57" H 1865 4196 50  0000 L CNN
 F 1 "100nF" H 1865 4105 50  0000 L CNN
 F 2 "Capacitor_SMD:C_0603_1608Metric" H 1788 4000 50  0001 C CNN
@@
 $EndComp
 $Comp
-L Device:C C63
+L Device:C C60
 U 1 1 5F1CB5BD
 P 2250 4150
-F 0 "C63" H 2365 4196 50  0000 L CNN
+F 0 "C60" H 2365 4196 50  0000 L CNN
 F 1 "100nF" H 2365 4105 50  0000 L CNN
 F 2 "Capacitor_SMD:C_0603_1608Metric" H 2288 4000 50  0001 C CNN
@@
 $EndComp
 $Comp
-L Device:C C65
+L Device:C C63
 U 1 1 5F1CC080
 P 2750 4150
-F 0 "C65" H 2865 4196 50  0000 L CNN
+F 0 "C63" H 2865 4196 50  0000 L CNN
 F 1 "10uF" H 2865 4105 50  0000 L CNN
 F 2 "Capacitor_SMD:C_0805_2012Metric" H 2788 4000 50  0001 C CNN
@@
 Return path decoupling
 $Comp
-L Device:C C66
+L Device:C C55
 U 1 1 5F8FCA63
 P 1575 6525
-F 0 "C66" H 1690 6571 50  0000 L CNN
+F 0 "C55" H 1690 6571 50  0000 L CNN
 F 1 "10nF" H 1690 6480 50  0000 L CNN
 F 2 "Capacitor_SMD:C_0603_1608Metric" H 1613 6375 50  0001 C CNN
@@
 $EndComp
 $Comp
-L Device:C C68
+L Device:C C58
 U 1 1 5F8FD1C4
 P 2000 6525
-F 0 "C68" H 2115 6571 50  0000 L CNN
+F 0 "C58" H 2115 6571 50  0000 L CNN
 F 1 "10nF" H 2115 6480 50  0000 L CNN
 F 2 "Capacitor_SMD:C_0603_1608Metric" H 2038 6375 50  0001 C CNN
@@
 $EndComp
 $Comp
-L Device:C C69
+L Device:C C61
 U 1 1 5F8FD3F9
 P 2425 6525
-F 0 "C69" H 2540 6571 50  0000 L CNN
+F 0 "C61" H 2540 6571 50  0000 L CNN
 F 1 "10nF" H 2540 6480 50  0000 L CNN
 F 2 "Capacitor_SMD:C_0603_1608Metric" H 2463 6375 50  0001 C CNN
