File: audio.kicad_sch (KiCad schematic)
At the start: 15 parts, among them J6 AUDIO-CONNECTOR-6P-SMD-344003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, U7 INTERFACE-MAX9850ETI+-(QFN28), X1 11.2896MHz

Commit message: Fixed board for Kicad 6, replaced some missing footprints.
Parts:
- U7: footprint QFN28G_0.5-5X5MM -> Package_DFN_QFN:QFN-28-1EP_5x5mm_P0.5mm_EP3.35x3.35mm
Changed lines of the file:
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@@
       (effects (font (size 1.27 1.27)) (justify left))
     )
-    (property "Footprint" "QFN28G_0.5-5X5MM" (id 2) (at 131.445 90.17 0)
+    (property "Footprint" "Package_DFN_QFN:QFN-28-1EP_5x5mm_P0.5mm_EP3.35x3.35mm" (id 2) (at 131.445 90.17 0)
       (effects (font (size 1.27 1.27)) (justify left bottom) hide)
     )
