File: file60C4BE23.kicad_sch (KiCad schematic)
At the start: 6 parts, among them U10 PCF2123TS_1,118, Y1 32.768kHz

Commit message: Fixed board for Kicad 6, replaced some missing footprints.
Parts:
- U10: footprint NXP_Semiconductors-SOT402-1-02_2016-0-* -> Package_SO:TSSOP-14_4.4x5mm_P0.65mm
Changed lines of the file:
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@@
     (property "Reference" "U10" (id 0) (at 151.13 85.979 0))
     (property "Value" "PCF2123TS_1,118" (id 1) (at 151.13 88.2904 0))
-    (property "Footprint" "NXP_Semiconductors-SOT402-1-02_2016-0-*" (id 2) (at 133.35 82.55 0)
+    (property "Footprint" "Package_SO:TSSOP-14_4.4x5mm_P0.65mm" (id 2) (at 133.35 82.55 0)
       (effects (font (size 1.27 1.27)) (justify left) hide)
     )
