File: joystick.kicad_sch (KiCad schematic)
At the start: 17 parts, among them J3 DB9_Male, J4 DB9_Male, U5 TXB0106PWR, U6 MCP23S17

Commit message: Fixed board for Kicad 6, replaced some missing footprints.
Parts:
- U5: footprint SOP65P640X120-16N -> Package_SO:TSSOP-16_4.4x5mm_P0.65mm
Changed lines of the file:
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@@
     (property "Reference" "U5" (id 0) (at 52.705 52.832 0))
     (property "Value" "TXB0106PWR" (id 1) (at 52.705 55.1434 0))
-    (property "Footprint" "SOP65P640X120-16N" (id 2) (at 52.705 77.47 0)
+    (property "Footprint" "Package_SO:TSSOP-16_4.4x5mm_P0.65mm" (id 2) (at 52.705 77.47 0)
       (effects (font (size 1.27 1.27)) (justify left bottom) hide)
     )
