File: main_board.kicad_sch (KiCad schematic)
At the start: 19 parts, among them SW1 SW_Push, SW2 SW_Push, SW3 SW_Push, U4 QM_XC7A35T_DDR3

Commit message: Fixed board for Kicad 6, replaced some missing footprints.
Parts:
- U4: footprint QM_XC7A35T_DDR3:QM_XC7A35T_DDR3_Daughterboard_v2 -> qmtech-minimig-new:QM_XC7A100T_DDR3_Daughterboard_rev2
Changed lines of the file:
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@@
     (property "Reference" "U4" (id 0) (at 147.4724 109.347 0))
     (property "Value" "QM_XC7A35T_DDR3" (id 1) (at 147.4724 107.0356 0))
-    (property "Footprint" "QM_XC7A35T_DDR3:QM_XC7A35T_DDR3_Daughterboard_v2" (id 2) (at 147.4724 104.7242 0))
+    (property "Footprint" "qmtech-minimig-new:QM_XC7A100T_DDR3_Daughterboard_rev2" (id 2) (at 147.4724 104.7242 0))
     (property "Datasheet" "" (id 3) (at 230.505 25.4 0)
       (effects (font (size 1.27 1.27)) hide)
@@
     (property "Reference" "U4" (id 0) (at 68.0974 109.347 0))
     (property "Value" "QM_XC7A35T_DDR3" (id 1) (at 68.0974 107.0356 0))
-    (property "Footprint" "QM_XC7A35T_DDR3:QM_XC7A35T_DDR3_Daughterboard_v2" (id 2) (at 68.0974 104.7242 0))
+    (property "Footprint" "qmtech-minimig-new:QM_XC7A100T_DDR3_Daughterboard_rev2" (id 2) (at 68.0974 104.7242 0))
     (property "Datasheet" "" (id 3) (at 151.13 25.4 0)
       (effects (font (size 1.27 1.27)) hide)
